Commit message: refactored URDF to follow REP-120

File: wolfgang_description/urdf/wolfgang.urdf (robot description, URDF)
Before this commit: robot wolves, 23 links, 22 joints
Links:
- removed link gaze
- removed link l_hip_roll
- removed link l_hip_yaw
- removed link l_shank
- removed link l_shoulder_pitch
- removed link l_thigh
- removed link r_hip_roll
- removed link r_hip_yaw
- removed link r_shank
- removed link r_shoulder_pitch
- removed link r_thigh
- added link head, mass 0.40746
- added link l_hip_1, mass 0.073374; collision mesh filename=package://wolfgang_description/mesh/left_hip_yaw_link.dae; visual mesh filename=package://wolfgang_description/mesh/left_hip_yaw_link.STL
- added link l_hip_2, mass 0.35844; collision mesh filename=package://wolfgang_description/mesh/left_hip_roll_link.dae; visual mesh filename=package://wolfgang_description/mesh/left_hip_roll_link.STL
- added link l_lower_leg, mass 0.20549; collision mesh filename=package://wolfgang_description/mesh/left_shank_link.dae; visual mesh filename=package://wolfgang_description/mesh/left_shank_link.STL
- added link l_shoulder, mass 0.025434; collision mesh filename=package://wolfgang_description/mesh/left_shoulder_pitch_lin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; visual mesh filename=package://wolfgang_description/mesh/left_shoulder_pitch_lin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
- added link l_sole, mass 0.01
- added link l_toe, mass 0.01
- added link l_upper_leg, mass 0.38276; collision mesh filename=package://wolfgang_description/mesh/left_thigh_link.dae; visual mesh filename=package://wolfgang_description/mesh/left_thigh_link.STL
- added link l_wrist
- added link r_hip_1, mass 0.073374; collision mesh filename=package://wolfgang_description/mesh/right_hip_yaw_link.dae; visual mesh filename=package://wolfgang_description/mesh/right_hip_yaw_link.STL
- added link r_hip_2, mass 0.35903; collision mesh filename=package://wolfgang_description/mesh/right_hip_roll_link.dae; visual mesh filename=package://wolfgang_description/mesh/right_hip_roll_link.STL
- added link r_lower_leg, mass 0.20549; collision mesh filename=package://wolfgang_description/mesh/right_shank_link.dae; visual mesh filename=package://wolfgang_description/mesh/right_shank_link.STL
- added link r_shoulder, mass 0.025434; collision mesh filename=package://wolfgang_description/mesh/right_shoulder_pitch_li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; visual mesh filename=package://wolfgang_description/mesh/right_shoulder_pitch_li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
- added link r_sole, mass 0.01
- added link r_toe, mass 0.01
- added link r_upper_leg, mass 0.38276; collision mesh filename=package://wolfgang_description/mesh/left_thigh_link.dae; visual mesh filename=package://wolfgang_description/mesh/left_thigh_link.STL
- added link r_wrist
Joints:
- removed joint camera_joint
- added joint head_to_camera: type fixed, parent head, child camera, origin xyz=0.03 0 0.05 rpy=0 0 0, axis 0 0 0
- added joint l_elbow_to_wrist: type fixed, parent l_lower_arm, child l_wrist, origin xyz=0.17 0 0 rpy=0 0 0
- added joint left_foot_to_sole: type fixed, parent l_foot, child l_sole, origin xyz=0 0 -0.04 rpy=0 0 0, axis 0 0 0
- added joint left_foot_to_toe: type fixed, parent l_sole, child l_toe, origin xyz=0 0 0 rpy=0 0 0, axis 0 0 0
- added joint r_elbow_to_wrist: type fixed, parent r_lower_arm, child r_wrist, origin xyz=0.17 0 0 rpy=0 0 0
- added joint r_foot_to_sole: type fixed, parent r_foot, child r_sole, origin xyz=0 0 -0.04 rpy=0 0 0, axis 0 0 0
- added joint r_foot_to_toe: type fixed, parent r_sole, child r_toe, origin xyz=0 0 0 rpy=0 0 0, axis 0 0 0
- joint HeadTilt: child gaze -> head
- joint LAnklePitch: parent l_shank -> l_lower_leg
- joint LHipPitch: child l_thigh -> l_upper_leg; parent l_hip_roll -> l_hip_2
- joint LHipRoll: child l_hip_roll -> l_hip_2; parent l_hip_yaw -> l_hip_1
- joint LHipYaw: child l_hip_yaw -> l_hip_1
- joint LKnee: child l_shank -> l_lower_leg; parent l_thigh -> l_upper_leg
- joint LShoulderPitch: child l_shoulder_pitch -> l_shoulder
- joint LShoulderRoll: parent l_shoulder_pitch -> l_shoulder
- joint RAnklePitch: parent r_shank -> r_lower_leg
- joint RHipPitch: child r_thigh -> r_upper_leg; parent r_hip_roll -> r_hip_2
- joint RHipRoll: child r_hip_roll -> r_hip_2; parent r_hip_yaw -> r_hip_1
- joint RHipYaw: child r_hip_yaw -> r_hip_1
- joint RKnee: child r_shank -> r_lower_leg; parent r_thigh -> r_upper_leg
- joint RShoulderPitch: child r_shoulder_pitch -> r_shoulder
- joint RShoulderRoll: parent r_shoulder_pitch -> r_shoulder

File: wolfgang_description/urdf/wolfgang.urdf.xacro (robot description, xacro)
@@ -35,5 +35,5 @@
         </collision>
     </link>
-    <link name="r_hip_yaw">
+    <link name="r_hip_1">
         <inertial>
             <origin xyz="4.7878E-16 2.8449E-16 -0.013803" rpy="0 0 0" />
@@ -55,5 +55,5 @@
         </collision>
     </link>
-    <link name="r_hip_roll">
+    <link name="r_hip_2">
         <inertial>
             <origin xyz="0.010896 0.00023756 -0.014538" rpy="0 0 0" />
@@ -75,5 +75,5 @@
         </collision>
     </link>
-    <link name="r_thigh">
+    <link name="r_upper_leg">
         <inertial>
             <origin xyz="0.0038549 0.00023828 -0.1495" rpy="0 0 0" />
@@ -95,5 +95,5 @@
         </collision>
     </link>
-    <link name="r_shank">
+    <link name="r_lower_leg">
         <inertial>
             <origin xyz="-0.0033779 6.578E-10 -0.10469" rpy="0 0 3.14159265359" />
@@ -155,5 +155,19 @@
         </collision>
     </link>
-    <link name="l_hip_yaw">
+    <link name="r_sole">
+        <inertial>
+          <origin xyz="0 0 0" rpy="0 0 0" />
+          <mass value="0.01" />
+          <inertia ixx="0" ixy="0" ixz="0" iyy="0" iyz="0" izz="0" />
+        </inertial>
+    </link>
+    <link name="r_toe">
+        <inertial>
+          <origin xyz="0 0 0" rpy="0 0 0" />
+          <mass value="0.01" />
+          <inertia ixx="0" ixy="0" ixz="0" iyy="0" iyz="0" izz="0" />
+        </inertial>
+    </link>
+    <link name="l_hip_1">
         <inertial>
             <origin xyz="4.996E-16 2.5674E-16 -0.013803" rpy="0 0 0" />
@@ -175,5 +189,5 @@
         </collision>
     </link>
-    <link name="l_hip_roll">
+    <link name="l_hip_2">
         <inertial>
             <origin xyz="-0.019434 -0.0014499 -0.014536" rpy="0 0 0" />
@@ -195,5 +209,5 @@
         </collision>
     </link>
-    <link name="l_thigh">
+    <link name="l_upper_leg">
         <inertial>
             <origin xyz="0.0038576 -0.0014383 -0.1495" rpy="0 0 0" />
@@ -215,5 +229,5 @@
         </collision>
     </link>
-    <link name="l_shank">
+    <link name="l_lower_leg">
         <inertial>
             <origin xyz="-0.0033779 -0.0012 -0.10469" rpy="0 0 0" />
@@ -275,5 +289,19 @@
         </collision>
     </link>
-    <link name="r_shoulder_pitch">
+    <link name="l_sole">
+        <inertial>
+          <origin xyz="0 0 0" rpy="0 0 0" />
+          <mass value="0.01" />
+          <inertia ixx="0" ixy="0" ixz="0" iyy="0" iyz="0" izz="0" />
+        </inertial>
+    </link>
+    <link name="l_toe">
+        <inertial>
+          <origin xyz="0 0 0" rpy="0 0 0" />
+          <mass value="0.01" />
+          <inertia ixx="0" ixy="0" ixz="0" iyy="0" iyz="0" izz="0" />
+        </inertial>
+    </link>
+    <link name="r_shoulder">
         <inertial>
             <origin xyz="0 -0.014621 0" rpy="0 0 0" />
@@ -335,5 +363,6 @@
         </collision>
     </link>
-    <link name="l_shoulder_pitch">
+    <link name="r_wrist"> </link>
+    <link name="l_shoulder">
         <inertial>
             <origin xyz="0 0.014621 0" rpy="0 0 0" />
@@ -395,4 +424,5 @@
         </collision>
     </link>
+    <link name="l_wrist"> </link>
     <link name="neck">
         <inertial>
@@ -416,5 +446,5 @@
     </link>
     <link name="camera" />
-    <link name="gaze">
+    <link name="head">
         <inertial>
             <origin xyz="0.014358 0.0005519 0.069919" rpy="0 0 0" />
@@ -441,5 +471,5 @@
         <origin xyz="-0.019 -0.055 0" rpy="0 0 0" />
         <parent link="base_link" />
-        <child link="r_hip_yaw" />
+        <child link="r_hip_1" />
         <axis xyz="0 0 1" />
         <limit effort="${tofa*2.5}" velocity="5.6548668" lower="-0.9250245035547" upper="0.9250245035547" />
@@ -448,6 +478,6 @@
     <joint name="RHipRoll" type="revolute">
         <origin xyz="-0.0072 0 -0.0438" rpy="0 0 0" />
-        <parent link="r_hip_yaw" />
-        <child link="r_hip_roll" />
+        <parent link="r_hip_1" />
+        <child link="r_hip_2" />
         <axis xyz="1 0 0" />
         <limit effort="${tofa*6.0}" velocity="6.597344565" lower="-1.0122909661542001" upper="0.7853981633955001" />
@@ -456,6 +486,6 @@
     <joint name="RHipPitch" type="revolute">
         <origin xyz="0.0303 0 0" rpy="0 0 0" />
-        <parent link="r_hip_roll" />
-        <child link="r_thigh" />
+        <parent link="r_hip_2" />
+        <child link="r_upper_leg" />
         <axis xyz="0 1 0" />
         <limit effort="${tofa*8.4}" velocity="4.712388975" lower="-1.919862177189" upper="0.48869219055720003" />
@@ -464,6 +494,6 @@
     <joint name="RKnee" type="revolute">
         <origin xyz="0 0 -0.22" rpy="0 0 0" />
-        <parent link="r_thigh" />
-        <child link="r_shank" />
+        <parent link="r_upper_leg" />
+        <child link="r_lower_leg" />
         <axis xyz="0 1 0" />
         <limit effort="${tofa*8.4}" velocity="4.712388975" lower="0" upper="2.268928027587" />
@@ -472,5 +502,5 @@
     <joint name="RAnklePitch" type="revolute">
         <origin xyz="-0.00186 0 -0.22" rpy="0 0 0" />
-        <parent link="r_shank" />
+        <parent link="r_lower_leg" />
         <child link="r_ankle" />
         <axis xyz="0 1 0" />
@@ -486,8 +516,20 @@
         <dynamics damping="${d}" friction="0.0" />
     </joint>
+    <joint name="r_foot_to_sole" type="fixed">
+        <origin xyz="0 0 -0.04" rpy="0 0 0" />
+        <parent link="r_foot" />
+        <child link="r_sole" />
+        <axis xyz="0 0 0" />
+    </joint>
+    <joint name="r_foot_to_toe" type="fixed">
+        <origin xyz="0 0 0" rpy="0 0 0" />
+        <parent link="r_sole" />
+        <child link="r_toe" />
+        <axis xyz="0 0 0" />
+    </joint>
     <joint name="LHipYaw" type="revolute">
         <origin xyz="-0.019 0.055 0" rpy="0 0 0" />
         <parent link="base_link" />
-        <child link="l_hip_yaw" />
+        <child link="l_hip_1" />
         <axis xyz="0 0 1" />
         <limit effort="${tofa*2.5}" velocity="5.6548668" lower="-0.9250245035547" upper="0.9250245035547" />
@@ -496,6 +538,6 @@
     <joint name="LHipRoll" type="revolute">
         <origin xyz="-0.0072 0.0012 -0.0438" rpy="0 0 0" />
-        <parent link="l_hip_yaw" />
-        <child link="l_hip_roll" />
+        <parent link="l_hip_1" />
+        <child link="l_hip_2" />
         <axis xyz="1 0 0" />
         <limit effort="${tofa*6.0}" velocity="6.597344565" lower="-1.0122909661542001" upper="0.7853981633955001" />
@@ -504,6 +546,6 @@
     <joint name="LHipPitch" type="revolute">
         <origin xyz="0.0303 0 0" rpy="0 0 0" />
-        <parent link="l_hip_roll" />
-        <child link="l_thigh" />
+        <parent link="l_hip_2" />
+        <child link="l_upper_leg" />
         <axis xyz="0 1 0" />
         <limit effort="${tofa*8.4}" velocity="4.712388975" lower="-0.48869219055720003" upper="1.919862177189" />
@@ -512,6 +554,6 @@
     <joint name="LKnee" type="revolute">
         <origin xyz="0 0 -0.22" rpy="0 0 0" />
-        <parent link="l_thigh" />
-        <child link="l_shank" />
+        <parent link="l_upper_leg" />
+        <child link="l_lower_leg" />
         <axis xyz="0 1 0" />
         <limit effort="${tofa*8.4}" velocity="4.712388975" lower="-2.268928027587" upper="0" />
@@ -520,5 +562,5 @@
     <joint name="LAnklePitch" type="revolute">
         <origin xyz="-0.00186 0 -0.22" rpy="0 0 0" />
-        <parent link="l_shank" />
+        <parent link="l_lower_leg" />
         <child link="l_ankle" />
         <axis xyz="0 1 0" />
@@ -534,4 +576,16 @@
         <dynamics damping="${d}" friction="0.0" />
     </joint>
+    <joint name="left_foot_to_sole" type="fixed">
+        <origin xyz="0 0 -0.04" rpy="0 0 0" />
+        <parent link="l_foot" />
+        <child link="l_sole" />
+        <axis xyz="0 0 0" />
+    </joint>
+    <joint name="left_foot_to_toe" type="fixed">
+        <origin xyz="0 0 0" rpy="0 0 0" />
+        <parent link="l_sole" />
+        <child link="l_toe" />
+        <axis xyz="0 0 0" />
+    </joint>
     <joint name="base_link_to_torso" type="fixed">
         <parent link="base_link" />
@@ -542,5 +596,5 @@
         <origin xyz="-0.0205 -0.0745 0.1075" rpy="0 0 0" />
         <parent link="torso" />
-        <child link="r_shoulder_pitch" />
+        <child link="r_shoulder" />
         <axis xyz="0 1 0" />
         <limit effort="${tofa*6.0}" velocity="6.597344565" lower="-3.1415926535820002" upper="3.1415926535820002" />
@@ -549,5 +603,5 @@
     <joint name="RShoulderRoll" type="revolute">
         <origin xyz="0 -0.038 0" rpy="0 0 0" />
-        <parent link="r_shoulder_pitch" />
+        <parent link="r_shoulder" />
         <child link="r_upper_arm" />
         <axis xyz="1 0 0" />
@@ -563,8 +617,13 @@
         <dynamics damping="${d}" friction="0.0" />
     </joint>
+    <joint name="r_elbow_to_wrist" type="fixed">
+        <parent link="r_lower_arm" />
+        <child link="r_wrist" />
+        <origin xyz="0.17 0 0" rpy="0 0 0"/> <!--todo-->
+    </joint>
     <joint name="LShoulderPitch" type="revolute">
         <origin xyz="-0.0205 0.0745 0.1075" rpy="0 0 0" />
         <parent link="torso" />
-        <child link="l_shoulder_pitch" />
+        <child link="l_shoulder" />
         <axis xyz="0 -1 0" />
         <limit effort="${tofa*6.0}" velocity="6.597344565" lower="-3.1415926535820002" upper="3.1415926535820002" />
@@ -573,5 +632,5 @@
     <joint name="LShoulderRoll" type="revolute">
         <origin xyz="0 0.038 0" rpy="0 0 0" />
-        <parent link="l_shoulder_pitch" />
+        <parent link="l_shoulder" />
         <child link="l_upper_arm" />
         <axis xyz="1 0 0" />
@@ -587,4 +646,9 @@
         <dynamics damping="${d}" friction="0.0" />
     </joint>
+    <joint name="l_elbow_to_wrist" type="fixed">
+        <parent link="l_lower_arm" />
+        <child link="l_wrist" />
+        <origin xyz="0.17 0 0" rpy="0 0 0"/> <!--todo-->
+    </joint>
     <joint name="HeadPan" type="revolute">
         <origin xyz="-0.0285 0 0.1365" rpy="0 0 0" />
@@ -598,12 +662,12 @@
         <origin xyz="0 0 0.0505" rpy="0 0 0" />
         <parent link="neck" />
-        <child link="gaze" />
+        <child link="head" />
         <axis xyz="0 1 0" />
         <limit effort="${tofa*2.5}" velocity="5.6548668" lower="-1.5707963267910001" upper="0" />
         <dynamics damping="${d}" friction="0.0" />
     </joint>
-    <joint name="camera_joint" type="fixed">
+    <joint name="head_to_camera" type="fixed">
         <origin xyz="0.03 0 0.05" rpy="0 0 0" />
-        <parent link="gaze" />
+        <parent link="head" />
         <child link="camera" />
         <axis xyz="0 0 0" />
@@ -810,6 +874,6 @@
         </actuator>
     </transmission>
-    <gazebo reference="r_foot">
-        <material>Gazebo/Grey</material>
+    <headbo reference="r_foot">
+        <material>headbo/Grey</material>
         <kp>1000000.0</kp>
         <kd>100.0</kd>
@@ -819,7 +883,7 @@
         <maxVel>1.0</maxVel>
         <minDepth>0.00</minDepth>
-    </gazebo>
-    <gazebo reference="l_foot">
-        <material>Gazebo/Grey</material>
+    </headbo>
+    <headbo reference="l_foot">
+        <material>headbo/Grey</material>
         <kp>1000000.0</kp>
         <kd>100.0</kd>
@@ -829,13 +893,13 @@
         <maxVel>1.0</maxVel>
         <minDepth>0.00</minDepth>
-    </gazebo>
+    </headbo>
   <!-- joint controller -->
-    <gazebo>
-        <plugin filename="libgazebo_ros_control.so" name="gazebo_ros_control">
+    <headbo>
+        <plugin filename="libheadbo_ros_control.so" name="headbo_ros_control">
             <robotNamespace>wolves</robotNamespace>
         </plugin>
-    </gazebo>
+    </headbo>
   <!-- camera sensor -->
-  <gazebo reference="camera">
+  <headbo reference="camera">
         <sensor name='camera' type='camera'>
           <pose>-0.050000 -0.010000 0.000000 -1.5708 0.000000 -3.141592</pose>
@@ -854,5 +918,5 @@
           <update_rate>30.000000</update_rate>
           <visualize>1</visualize>
-          <plugin name="camera_controller" filename="libgazebo_ros_camera.so">
+          <plugin name="camera_controller" filename="libheadbo_ros_camera.so">
             <alwaysOn>true</alwaysOn>
             <updateRate>30</updateRate>
@@ -869,7 +933,7 @@
           </plugin>
       </sensor>
-  </gazebo>
+  </headbo>
    <!-- IMU sensor -->
-   <gazebo reference="L_IMU">
+   <headbo reference="L_IMU">
     <gravity>true</gravity>
     <sensor name="imu_sensor" type="imu">
@@ -878,5 +942,5 @@
       <visualize>true</visualize>
       <topic>__default_topic__</topic>
-      <plugin filename="libgazebo_ros_imu_sensor.so" name="imu_plugin">
+      <plugin filename="libheadbo_ros_imu_sensor.so" name="imu_plugin">
         <topicName>imu</topicName>
         <bodyName>torso</bodyName>
@@ -889,9 +953,9 @@
       <pose>0 0 0 0 0 0</pose>
     </sensor>
-  </gazebo>
+  </headbo>
    <!-- fake controller that allows us to move the robot and to get its oposition -->
    <!-- rostopic pub /minibot/cmd_vel geometry_msgs/Twist "{ linear: [ 0.1, 0, 0], angular: [0.2, 0, 0.1] }" -->
-   <!--<gazebo>
-    <plugin name="object_controller" filename="libgazebo_ros_planar_move.so">
+   <!--<headbo>
+    <plugin name="object_controller" filename="libheadbo_ros_planar_move.so">
       <robotNamespace>wolves</robotNamespace>
       <commandTopic>cmd_vel</commandTopic>
@@ -901,4 +965,4 @@
       <robotBaseFrame>base_link</robotBaseFrame>
     </plugin>
-  </gazebo> -->
+  </headbo> -->
 </robot>
