Commit message: fixes

File: wolfgang_description/urdf/wolfgang.urdf.xacro (robot description, xacro)
@@ -874,6 +874,6 @@
         </actuator>
     </transmission>
-    <headbo reference="r_foot">
-        <material>headbo/Grey</material>
+    <gazebo reference="r_foot">
+        <material>gazebo/Grey</material>
         <kp>1000000.0</kp>
         <kd>100.0</kd>
@@ -883,7 +883,7 @@
         <maxVel>1.0</maxVel>
         <minDepth>0.00</minDepth>
-    </headbo>
-    <headbo reference="l_foot">
-        <material>headbo/Grey</material>
+    </gazebo>
+    <gazebo reference="l_foot">
+        <material>gazebo/Grey</material>
         <kp>1000000.0</kp>
         <kd>100.0</kd>
@@ -893,13 +893,13 @@
         <maxVel>1.0</maxVel>
         <minDepth>0.00</minDepth>
-    </headbo>
+    </gazebo>
   <!-- joint controller -->
-    <headbo>
-        <plugin filename="libheadbo_ros_control.so" name="headbo_ros_control">
-            <robotNamespace>wolves</robotNamespace>
+    <gazebo>
+        <plugin filename="libgazebo_ros_control.so" name="gazebo_ros_control">
+            <robotNamespace>wolfgang</robotNamespace>
         </plugin>
-    </headbo>
+    </gazebo>
   <!-- camera sensor -->
-  <headbo reference="camera">
+  <gazebo reference="camera">
         <sensor name='camera' type='camera'>
           <pose>-0.050000 -0.010000 0.000000 -1.5708 0.000000 -3.141592</pose>
@@ -918,5 +918,5 @@
           <update_rate>30.000000</update_rate>
           <visualize>1</visualize>
-          <plugin name="camera_controller" filename="libheadbo_ros_camera.so">
+          <plugin name="camera_controller" filename="libgazebo_ros_camera.so">
             <alwaysOn>true</alwaysOn>
             <updateRate>30</updateRate>
@@ -933,7 +933,7 @@
           </plugin>
       </sensor>
-  </headbo>
+  </gazebo>
    <!-- IMU sensor -->
-   <headbo reference="L_IMU">
+   <gazebo reference="L_IMU">
     <gravity>true</gravity>
     <sensor name="imu_sensor" type="imu">
@@ -942,5 +942,5 @@
       <visualize>true</visualize>
       <topic>__default_topic__</topic>
-      <plugin filename="libheadbo_ros_imu_sensor.so" name="imu_plugin">
+      <plugin filename="libgazebo_ros_imu_sensor.so" name="imu_plugin">
         <topicName>imu</topicName>
         <bodyName>torso</bodyName>
@@ -953,9 +953,9 @@
       <pose>0 0 0 0 0 0</pose>
     </sensor>
-  </headbo>
+  </gazebo>
    <!-- fake controller that allows us to move the robot and to get its oposition -->
    <!-- rostopic pub /minibot/cmd_vel geometry_msgs/Twist "{ linear: [ 0.1, 0, 0], angular: [0.2, 0, 0.1] }" -->
-   <!--<headbo>
-    <plugin name="object_controller" filename="libheadbo_ros_planar_move.so">
+   <!--<gazebo>
+    <plugin name="object_controller" filename="libgazebo_ros_planar_move.so">
       <robotNamespace>wolves</robotNamespace>
       <commandTopic>cmd_vel</commandTopic>
@@ -965,4 +965,4 @@
       <robotBaseFrame>base_link</robotBaseFrame>
     </plugin>
-  </headbo> -->
+  </gazebo> -->
 </robot>

Commit message: removed urdf, we only use the xacro now.

File: wolfgang_description/urdf/wolfgang.urdf.xacro (robot description, xacro)
@@ -1,14 +1,10 @@
 <?xml version="1.0" encoding="UTF-8"?>
 <robot xmlns:xacro="http://www.ros.org/wiki/xacro" name="wolves">
-    <xacro:property name="tofa" value="1" />
-    <!--Torque factor-->
-    <xacro:property name="infa" value="1" />
-    <!--inertia factor-->
-    <xacro:property name="insu" value="0" />
-    <!--inertia summand-->
-    <xacro:property name="d" value="0" />
-    <!-- damping -->
-    <xacro:property name="f" value="0" />
-    <!-- friction -->
+    <xacro:arg name="sim_ns" default="/" />
+    <xacro:property name="tofa" value="1" /> <!--Torque factor-->
+    <xacro:property name="infa" value="1" /> <!--inertia factor-->
+    <xacro:property name="insu" value="0" /> <!--inertia summand-->
+    <xacro:property name="d" value="0" /> <!-- damping -->
+    <xacro:property name="f" value="0" /> <!-- friction -->
     <material name="black">
         <color rgba="0.1 0.1 0.1 1" />
@@ -897,5 +893,5 @@
     <gazebo>
         <plugin filename="libgazebo_ros_control.so" name="gazebo_ros_control">
-            <robotNamespace>wolfgang</robotNamespace>
+            <robotNamespace>$(arg sim_ns)</robotNamespace>
         </plugin>
     </gazebo>

Commit message: fixed robot model, some joints were in the wrong direction

File: wolfgang_description/urdf/wolfgang.urdf.xacro (robot description, xacro)
@@ -465,8 +465,8 @@
     </link>
     <joint name="RHipYaw" type="revolute">
-        <origin xyz="-0.019 -0.055 0" rpy="0 0 0" />
+        <origin xyz="0 -0.055 0" rpy="0 0 0" />
         <parent link="base_link" />
         <child link="r_hip_1" />
-        <axis xyz="0 0 1" />
+        <axis xyz="0 0 -1" />
         <limit effort="${tofa*2.5}" velocity="5.6548668" lower="-0.9250245035547" upper="0.9250245035547" />
         <dynamics damping="${d}" friction="0.0" />
@@ -477,5 +477,5 @@
         <child link="r_hip_2" />
         <axis xyz="1 0 0" />
-        <limit effort="${tofa*6.0}" velocity="6.597344565" lower="-1.0122909661542001" upper="0.7853981633955001" />
+        <limit effort="${tofa*6.0}" velocity="6.597344565" lower="-1.57" upper="0.7853981633955001" />
         <dynamics damping="${d}" friction="0.0" />
     </joint>
@@ -500,5 +500,5 @@
         <parent link="r_lower_leg" />
         <child link="r_ankle" />
-        <axis xyz="0 1 0" />
+        <axis xyz="0 -1 0" />
         <limit effort="${tofa*8.4}" velocity="4.712388975" lower="-1.2391837689129" upper="1.6406094968706" />
         <dynamics damping="${d}" friction="0.0" />
@@ -508,5 +508,5 @@
         <parent link="r_ankle" />
         <child link="r_foot" />
-        <axis xyz="1 0 0" />
+        <axis xyz="-1 0 0" />
         <limit effort="${tofa*6.0}" velocity="6.597344565" lower="-1.4660765716716" upper="1.4660765716716" />
         <dynamics damping="${d}" friction="0.0" />
@@ -525,8 +525,8 @@
     </joint>
     <joint name="LHipYaw" type="revolute">
-        <origin xyz="-0.019 0.055 0" rpy="0 0 0" />
+        <origin xyz="0 0.055 0" rpy="0 0 0" />
         <parent link="base_link" />
         <child link="l_hip_1" />
-        <axis xyz="0 0 1" />
+        <axis xyz="0 0 -1" />
         <limit effort="${tofa*2.5}" velocity="5.6548668" lower="-0.9250245035547" upper="0.9250245035547" />
         <dynamics damping="${d}" friction="0.0" />
@@ -537,5 +537,5 @@
         <child link="l_hip_2" />
         <axis xyz="1 0 0" />
-        <limit effort="${tofa*6.0}" velocity="6.597344565" lower="-1.0122909661542001" upper="0.7853981633955001" />
+        <limit effort="${tofa*6.0}" velocity="6.597344565" lower="-0.7853981633955001" upper="1.57" />
         <dynamics damping="${d}" friction="0.0" />
     </joint>
@@ -544,6 +544,6 @@
         <parent link="l_hip_2" />
         <child link="l_upper_leg" />
-        <axis xyz="0 1 0" />
-        <limit effort="${tofa*8.4}" velocity="4.712388975" lower="-0.48869219055720003" upper="1.919862177189" />
+        <axis xyz="0 -1 0" />
+        <limit effort="${tofa*8.4}" velocity="4.712388975" lower="-1.919862177189" upper="0.48869219055720003" />
         <dynamics damping="${d}" friction="0.0" />
     </joint>
@@ -552,5 +552,5 @@
         <parent link="l_upper_leg" />
         <child link="l_lower_leg" />
-        <axis xyz="0 1 0" />
+        <axis xyz="0 -1 0" />
         <limit effort="${tofa*8.4}" velocity="4.712388975" lower="-2.268928027587" upper="0" />
         <dynamics damping="${d}" friction="0.0" />
@@ -568,5 +568,5 @@
         <parent link="l_ankle" />
         <child link="l_foot" />
-        <axis xyz="1 0 0" />
+        <axis xyz="-1 0 0" />
         <limit effort="${tofa*6.0}" velocity="6.597344565" lower="-1.4660765716716" upper="1.4660765716716" />
         <dynamics damping="${d}" friction="0.0" />
@@ -587,5 +587,5 @@
         <parent link="base_link" />
         <child link="torso" />
-        <origin rpy="0 0 0" xyz="0 0 0.0936" />
+        <origin rpy="0.019 0 0" xyz="0 0 0.0936" />
     </joint>
     <joint name="RShoulderPitch" type="revolute">

Commit message: changed urdf to make it more similar to reality

File: wolfgang_description/urdf/wolfgang.urdf.xacro (robot description, xacro)
@@ -84,10 +84,10 @@
             <material name="black" />
         </visual>
-        <collision>
+        <!--<collision>
             <origin xyz="0 0 0" rpy="0 0 0" />
             <geometry>
                 <mesh filename="package://wolfgang_description/mesh/left_thigh_link.dae" />
             </geometry>
-        </collision>
+        </collision>-->
     </link>
     <link name="r_lower_leg">
@@ -104,10 +104,10 @@
             <material name="black" />
         </visual>
-        <collision>
+        <!--<collision>
             <origin xyz="0 0 0" rpy="0 0 0" />
             <geometry>
                 <mesh filename="package://wolfgang_description/mesh/right_shank_link.dae" />
             </geometry>
-        </collision>
+        </collision>-->
     </link>
     <link name="r_ankle">
@@ -117,5 +117,5 @@
             <inertia ixx="0.00015501" ixy="1.7299E-06" ixz="-8.5156E-06" iyy="0.00032958" iyz="-2.4435E-07" izz="0.00027786" />
         </inertial>
-        <visual>
+        <!--<visual>
             <origin xyz="0 0 0" rpy="0 0 0" />
             <geometry>
@@ -129,5 +129,5 @@
                 <mesh filename="package://wolfgang_description/mesh/right_ankle_link.dae" />
             </geometry>
-        </collision>
+        </collision>-->
     </link>
     <link name="r_foot">
@@ -138,5 +138,5 @@
         </inertial>
         <visual>
-            <origin xyz="0 0 0" rpy="0 0 0" />
+            <origin xyz="0 0 -0.012" rpy="0 0 0" />
             <geometry>
                 <mesh filename="package://wolfgang_description/mesh/right_foot_link.STL" />
@@ -145,5 +145,5 @@
         </visual>
         <collision>
-            <origin xyz="0 0 0" rpy="0 0 0" />
+            <origin xyz="0 0 -0.012" rpy="0 0 0" />
             <geometry>
                 <mesh filename="package://wolfgang_description/mesh/right_foot_link.dae" />
@@ -218,10 +218,10 @@
             <material name="black" />
         </visual>
-        <collision>
+        <!--<collision>
             <origin xyz="0 0 0" rpy="0 0 0" />
             <geometry>
                 <mesh filename="package://wolfgang_description/mesh/left_thigh_link.dae" />
             </geometry>
-        </collision>
+        </collision>-->
     </link>
     <link name="l_lower_leg">
@@ -238,10 +238,10 @@
             <material name="black" />
         </visual>
-        <collision>
+        <!--<collision>
             <origin xyz="0 0 0" rpy="0 0 0" />
             <geometry>
                 <mesh filename="package://wolfgang_description/mesh/left_shank_link.dae" />
             </geometry>
-        </collision>
+        </collision>-->
     </link>
     <link name="l_ankle">
@@ -251,5 +251,5 @@
             <inertia ixx="0.00015503" ixy="-1.738E-06" ixz="-8.5148E-06" iyy="0.0003299" iyz="2.4403E-07" izz="0.0002782" />
         </inertial>
-        <visual>
+        <!--<visual>
             <origin xyz="0 0 0" rpy="0 0 0" />
             <geometry>
@@ -263,5 +263,5 @@
                 <mesh filename="package://wolfgang_description/mesh/left_ankle_link.dae" />
             </geometry>
-        </collision>
+        </collision>-->
     </link>
     <link name="l_foot">
@@ -272,5 +272,5 @@
         </inertial>
         <visual>
-            <origin xyz="0 0 0" rpy="0 0 0" />
+            <origin xyz="0 0 -0.012" rpy="0 0 0" />
             <geometry>
                 <mesh filename="package://wolfgang_description/mesh/left_foot_link.STL" />
@@ -279,5 +279,5 @@
         </visual>
         <collision>
-            <origin xyz="0 0 0" rpy="0 0 0" />
+            <origin xyz="0 0 -0.012" rpy="0 0 0" />
             <geometry>
                 <mesh filename="package://wolfgang_description/mesh/left_foot_link.dae" />
@@ -489,5 +489,5 @@
     </joint>
     <joint name="RKnee" type="revolute">
-        <origin xyz="0 0 -0.22" rpy="0 0 0" />
+        <origin xyz="-0.015 0 -0.17" rpy="0 0 0" />
         <parent link="r_upper_leg" />
         <child link="r_lower_leg" />
@@ -497,5 +497,5 @@
     </joint>
     <joint name="RAnklePitch" type="revolute">
-        <origin xyz="-0.00186 0 -0.22" rpy="0 0 0" />
+        <origin xyz="0.015 0 -0.17" rpy="0 0 0" />
         <parent link="r_lower_leg" />
         <child link="r_ankle" />
@@ -513,5 +513,5 @@
     </joint>
     <joint name="r_foot_to_sole" type="fixed">
-        <origin xyz="0 0 -0.04" rpy="0 0 0" />
+        <origin xyz="0 0 -0.052" rpy="0 0 0" />
         <parent link="r_foot" />
         <child link="r_sole" />
@@ -519,5 +519,5 @@
     </joint>
     <joint name="r_foot_to_toe" type="fixed">
-        <origin xyz="0 0 0" rpy="0 0 0" />
+        <origin xyz="0.105 0 0" rpy="0 0 0" />
         <parent link="r_sole" />
         <child link="r_toe" />
@@ -533,5 +533,5 @@
     </joint>
     <joint name="LHipRoll" type="revolute">
-        <origin xyz="-0.0072 0.0012 -0.0438" rpy="0 0 0" />
+        <origin xyz="-0.0072 0 -0.0438" rpy="0 0 0" />
         <parent link="l_hip_1" />
         <child link="l_hip_2" />
@@ -549,5 +549,5 @@
     </joint>
     <joint name="LKnee" type="revolute">
-        <origin xyz="0 0 -0.22" rpy="0 0 0" />
+        <origin xyz="-0.015 0 -0.17" rpy="0 0 0" />
         <parent link="l_upper_leg" />
         <child link="l_lower_leg" />
@@ -557,5 +557,5 @@
     </joint>
     <joint name="LAnklePitch" type="revolute">
-        <origin xyz="-0.00186 0 -0.22" rpy="0 0 0" />
+        <origin xyz="0.015 0 -0.17" rpy="0 0 0" />
         <parent link="l_lower_leg" />
         <child link="l_ankle" />
@@ -573,5 +573,5 @@
     </joint>
     <joint name="left_foot_to_sole" type="fixed">
-        <origin xyz="0 0 -0.04" rpy="0 0 0" />
+        <origin xyz="0 0 -0.052" rpy="0 0 0" />
         <parent link="l_foot" />
         <child link="l_sole" />
@@ -579,5 +579,5 @@
     </joint>
     <joint name="left_foot_to_toe" type="fixed">
-        <origin xyz="0 0 0" rpy="0 0 0" />
+        <origin xyz="0.105 0 0" rpy="0 0 0" />
         <parent link="l_sole" />
         <child link="l_toe" />
@@ -587,8 +587,8 @@
         <parent link="base_link" />
         <child link="torso" />
-        <origin rpy="0.019 0 0" xyz="0 0 0.0936" />
+        <origin rpy="0.0 0 0" xyz="0 0 0.09" />
     </joint>
     <joint name="RShoulderPitch" type="revolute">
-        <origin xyz="-0.0205 -0.0745 0.1075" rpy="0 0 0" />
+        <origin xyz="0.0 -0.075 0.11" rpy="0 0 0" />
         <parent link="torso" />
         <child link="r_shoulder" />
@@ -598,5 +598,5 @@
     </joint>
     <joint name="RShoulderRoll" type="revolute">
-        <origin xyz="0 -0.038 0" rpy="0 0 0" />
+        <origin xyz="0 -0.04 0" rpy="0 0 0" />
         <parent link="r_shoulder" />
         <child link="r_upper_arm" />
@@ -606,5 +606,5 @@
     </joint>
     <joint name="RElbow" type="revolute">
-        <origin xyz="0.0265 0 -0.1735" rpy="0 0 0" />
+        <origin xyz="-0.0075 0 -0.145" rpy="0 0 0" />
         <parent link="r_upper_arm" />
         <child link="r_lower_arm" />
@@ -616,8 +616,8 @@
         <parent link="r_lower_arm" />
         <child link="r_wrist" />
-        <origin xyz="0.17 0 0" rpy="0 0 0"/> <!--todo-->
+        <origin xyz="0.225 0 0" rpy="0 0 0"/>
     </joint>
     <joint name="LShoulderPitch" type="revolute">
-        <origin xyz="-0.0205 0.0745 0.1075" rpy="0 0 0" />
+        <origin xyz="0.0 0.075 0.11" rpy="0 0 0" />
         <parent link="torso" />
         <child link="l_shoulder" />
@@ -627,5 +627,5 @@
     </joint>
     <joint name="LShoulderRoll" type="revolute">
-        <origin xyz="0 0.038 0" rpy="0 0 0" />
+        <origin xyz="0 0.04 0" rpy="0 0 0" />
         <parent link="l_shoulder" />
         <child link="l_upper_arm" />
@@ -635,5 +635,5 @@
     </joint>
     <joint name="LElbow" type="revolute">
-        <origin xyz="0.0265 0 -0.1735" rpy="0 0 0" />
+        <origin xyz="-0.0075 0 -0.145" rpy="0 0 0" />
         <parent link="l_upper_arm" />
         <child link="l_lower_arm" />
@@ -645,5 +645,5 @@
         <parent link="l_lower_arm" />
         <child link="l_wrist" />
-        <origin xyz="0.17 0 0" rpy="0 0 0"/> <!--todo-->
+        <origin xyz="0.225 0 0" rpy="0 0 0"/>
     </joint>
     <joint name="HeadPan" type="revolute">
