Commit message: updated model

File: wolfgang_description/urdf/wolfgang.urdf.xacro (robot description, xacro)
@@ -1,10 +1,10 @@
 <?xml version="1.0" encoding="UTF-8"?>
-<robot xmlns:xacro="http://www.ros.org/wiki/xacro" name="wolves">
+<robot xmlns:xacro="http://www.ros.org/wiki/xacro" name="wolfgang">
     <xacro:arg name="sim_ns" default="/" />
     <xacro:property name="tofa" value="1" /> <!--Torque factor-->
     <xacro:property name="infa" value="1" /> <!--inertia factor-->
     <xacro:property name="insu" value="0" /> <!--inertia summand-->
-    <xacro:property name="d" value="0" /> <!-- damping -->
-    <xacro:property name="f" value="0" /> <!-- friction -->
+    <xacro:property name="d" value="1" /> <!-- damping -->
+    <xacro:property name="f" value="1" /> <!-- friction -->
     <material name="black">
         <color rgba="0.1 0.1 0.1 1" />
@@ -470,5 +470,5 @@
         <axis xyz="0 0 -1" />
         <limit effort="${tofa*2.5}" velocity="5.6548668" lower="-0.9250245035547" upper="0.9250245035547" />
-        <dynamics damping="${d}" friction="0.0" />
+        <dynamics damping="${d}" friction="${f}" />
     </joint>
     <joint name="RHipRoll" type="revolute">
@@ -478,5 +478,5 @@
         <axis xyz="1 0 0" />
         <limit effort="${tofa*6.0}" velocity="6.597344565" lower="-1.57" upper="0.7853981633955001" />
-        <dynamics damping="${d}" friction="0.0" />
+        <dynamics damping="${d}" friction="${f}" />
     </joint>
     <joint name="RHipPitch" type="revolute">
@@ -486,5 +486,5 @@
         <axis xyz="0 1 0" />
         <limit effort="${tofa*8.4}" velocity="4.712388975" lower="-1.919862177189" upper="0.48869219055720003" />
-        <dynamics damping="${d}" friction="0.0" />
+        <dynamics damping="${d}" friction="${f}" />
     </joint>
     <joint name="RKnee" type="revolute">
@@ -494,5 +494,5 @@
         <axis xyz="0 1 0" />
         <limit effort="${tofa*8.4}" velocity="4.712388975" lower="0" upper="2.268928027587" />
-        <dynamics damping="${d}" friction="0.0" />
+        <dynamics damping="${d}" friction="${f}" />
     </joint>
     <joint name="RAnklePitch" type="revolute">
@@ -502,5 +502,5 @@
         <axis xyz="0 -1 0" />
         <limit effort="${tofa*8.4}" velocity="4.712388975" lower="-1.2391837689129" upper="1.6406094968706" />
-        <dynamics damping="${d}" friction="0.0" />
+        <dynamics damping="${d}" friction="${f}" />
     </joint>
     <joint name="RAnkleRoll" type="revolute">
@@ -510,5 +510,5 @@
         <axis xyz="-1 0 0" />
         <limit effort="${tofa*6.0}" velocity="6.597344565" lower="-1.4660765716716" upper="1.4660765716716" />
-        <dynamics damping="${d}" friction="0.0" />
+        <dynamics damping="${d}" friction="${f}" />
     </joint>
     <joint name="r_foot_to_sole" type="fixed">
@@ -530,5 +530,5 @@
         <axis xyz="0 0 -1" />
         <limit effort="${tofa*2.5}" velocity="5.6548668" lower="-0.9250245035547" upper="0.9250245035547" />
-        <dynamics damping="${d}" friction="0.0" />
+        <dynamics damping="${d}" friction="${f}" />
     </joint>
     <joint name="LHipRoll" type="revolute">
@@ -538,5 +538,5 @@
         <axis xyz="1 0 0" />
         <limit effort="${tofa*6.0}" velocity="6.597344565" lower="-0.7853981633955001" upper="1.57" />
-        <dynamics damping="${d}" friction="0.0" />
+        <dynamics damping="${d}" friction="${f}" />
     </joint>
     <joint name="LHipPitch" type="revolute">
@@ -546,5 +546,5 @@
         <axis xyz="0 -1 0" />
         <limit effort="${tofa*8.4}" velocity="4.712388975" lower="-1.919862177189" upper="0.48869219055720003" />
-        <dynamics damping="${d}" friction="0.0" />
+        <dynamics damping="${d}" friction="${f}" />
     </joint>
     <joint name="LKnee" type="revolute">
@@ -554,5 +554,5 @@
         <axis xyz="0 -1 0" />
         <limit effort="${tofa*8.4}" velocity="4.712388975" lower="-2.268928027587" upper="0" />
-        <dynamics damping="${d}" friction="0.0" />
+        <dynamics damping="${d}" friction="${f}" />
     </joint>
     <joint name="LAnklePitch" type="revolute">
@@ -562,5 +562,5 @@
         <axis xyz="0 1 0" />
         <limit effort="${tofa*8.4}" velocity="4.712388975" lower="-1.6406094968706" upper="1.2391837689129" />
-        <dynamics damping="${d}" friction="0.0" />
+        <dynamics damping="${d}" friction="${f}" />
     </joint>
     <joint name="LAnkleRoll" type="revolute">
@@ -570,5 +570,5 @@
         <axis xyz="-1 0 0" />
         <limit effort="${tofa*6.0}" velocity="6.597344565" lower="-1.4660765716716" upper="1.4660765716716" />
-        <dynamics damping="${d}" friction="0.0" />
+        <dynamics damping="${d}" friction="${f}" />
     </joint>
     <joint name="left_foot_to_sole" type="fixed">
@@ -595,5 +595,5 @@
         <axis xyz="0 1 0" />
         <limit effort="${tofa*6.0}" velocity="6.597344565" lower="-3.1415926535820002" upper="3.1415926535820002" />
-        <dynamics damping="${d}" friction="0.0" />
+        <dynamics damping="${d}" friction="${f}" />
     </joint>
     <joint name="RShoulderRoll" type="revolute">
@@ -603,5 +603,5 @@
         <axis xyz="1 0 0" />
         <limit effort="${tofa*2.5}" velocity="5.648668" lower="-0.7853981633955001" upper="2.3561944901865" />
-        <dynamics damping="${d}" friction="0.0" />
+        <dynamics damping="${d}" friction="${f}" />
     </joint>
     <joint name="RElbow" type="revolute">
@@ -611,5 +611,5 @@
         <axis xyz="0 1 0" />
         <limit effort="${tofa*2.5}" velocity="5.6548668" lower="-1.635" upper="1.5707963267910001" />
-        <dynamics damping="${d}" friction="0.0" />
+        <dynamics damping="${d}" friction="${f}" />
     </joint>
     <joint name="r_elbow_to_wrist" type="fixed">
@@ -624,5 +624,5 @@
         <axis xyz="0 -1 0" />
         <limit effort="${tofa*6.0}" velocity="6.597344565" lower="-3.1415926535820002" upper="3.1415926535820002" />
-        <dynamics damping="${d}" friction="0.0" />
+        <dynamics damping="${d}" friction="${f}" />
     </joint>
     <joint name="LShoulderRoll" type="revolute">
@@ -632,5 +632,5 @@
         <axis xyz="1 0 0" />
         <limit effort="${tofa*2.5}" velocity="5.648668" lower="-2.3561944901865" upper="0.7853981633955001" />
-        <dynamics damping="${d}" friction="0.0" />
+        <dynamics damping="${d}" friction="${f}" />
     </joint>
     <joint name="LElbow" type="revolute">
@@ -640,5 +640,5 @@
         <axis xyz="0 1 0" />
         <limit effort="${tofa*2.5}" velocity="5.6548668" lower="-1.1344640137935" upper="1.5707963267910001" />
-        <dynamics damping="${d}" friction="0.0" />
+        <dynamics damping="${d}" friction="${f}" />
     </joint>
     <joint name="l_elbow_to_wrist" type="fixed">
@@ -653,5 +653,5 @@
         <axis xyz="0 0 1" />
         <limit effort="${tofa*2.5}" velocity="5.6548668" lower="-2.1816615649875" upper="2.1816615649875" />
-        <dynamics damping="${d}" friction="0.0" />
+        <dynamics damping="${d}" friction="${f}" />
     </joint>
     <joint name="HeadTilt" type="revolute">
@@ -661,5 +661,5 @@
         <axis xyz="0 1 0" />
         <limit effort="${tofa*2.5}" velocity="5.6548668" lower="-1.5707963267910001" upper="0" />
-        <dynamics damping="${d}" friction="0.0" />
+        <dynamics damping="${d}" friction="${f}" />
     </joint>
     <joint name="head_to_camera" type="fixed">
@@ -668,5 +668,5 @@
         <child link="camera" />
         <axis xyz="0 0 0" />
-        <dynamics damping="${d}" friction="0.0" />
+        <dynamics damping="${d}" friction="${f}" />
     </joint>
     <transmission name="HeadPanTransmission">

Commit message: small fix for joint limits

File: wolfgang_description/urdf/wolfgang.urdf.xacro (robot description, xacro)
@@ -545,5 +545,5 @@
         <child link="l_upper_leg" />
         <axis xyz="0 -1 0" />
-        <limit effort="${tofa*8.4}" velocity="4.712388975" lower="-1.919862177189" upper="0.48869219055720003" />
+        <limit effort="${tofa*8.4}" velocity="4.712388975" lower="-0.48869219055720003" upper="1.919862177189" />
         <dynamics damping="${d}" friction="${f}" />
     </joint>

Commit message: changes on urdf, wrong arm move direction

File: wolfgang_description/urdf/wolfgang.urdf.xacro (robot description, xacro)
@@ -593,5 +593,5 @@
         <parent link="torso" />
         <child link="r_shoulder" />
-        <axis xyz="0 1 0" />
+        <axis xyz="0 -1 0" />
         <limit effort="${tofa*6.0}" velocity="6.597344565" lower="-3.1415926535820002" upper="3.1415926535820002" />
         <dynamics damping="${d}" friction="${f}" />
@@ -601,5 +601,5 @@
         <parent link="r_shoulder" />
         <child link="r_upper_arm" />
-        <axis xyz="1 0 0" />
+        <axis xyz="-1 0 0" />
         <limit effort="${tofa*2.5}" velocity="5.648668" lower="-0.7853981633955001" upper="2.3561944901865" />
         <dynamics damping="${d}" friction="${f}" />
@@ -622,5 +622,5 @@
         <parent link="torso" />
         <child link="l_shoulder" />
-        <axis xyz="0 -1 0" />
+        <axis xyz="0 1 0" />
         <limit effort="${tofa*6.0}" velocity="6.597344565" lower="-3.1415926535820002" upper="3.1415926535820002" />
         <dynamics damping="${d}" friction="${f}" />
@@ -630,5 +630,5 @@
         <parent link="l_shoulder" />
         <child link="l_upper_arm" />
-        <axis xyz="1 0 0" />
+        <axis xyz="-1 0 0" />
         <limit effort="${tofa*2.5}" velocity="5.648668" lower="-2.3561944901865" upper="0.7853981633955001" />
         <dynamics damping="${d}" friction="${f}" />
@@ -638,5 +638,5 @@
         <parent link="l_upper_arm" />
         <child link="l_lower_arm" />
-        <axis xyz="0 1 0" />
+        <axis xyz="0 -1 0" />
         <limit effort="${tofa*2.5}" velocity="5.6548668" lower="-1.1344640137935" upper="1.5707963267910001" />
         <dynamics damping="${d}" friction="${f}" />

Commit message: corrected urdf, added imu frame

File: wolfgang_description/urdf/wolfgang.urdf.xacro (robot description, xacro)
@@ -442,4 +442,5 @@
     </link>
     <link name="camera" />
+    <link name="imu" />
     <link name="head">
         <inertial>
@@ -489,5 +490,5 @@
     </joint>
     <joint name="RKnee" type="revolute">
-        <origin xyz="-0.015 0 -0.17" rpy="0 0 0" />
+        <origin xyz="-0.03 0 -0.17" rpy="0 0 0" />
         <parent link="r_upper_leg" />
         <child link="r_lower_leg" />
@@ -497,5 +498,5 @@
     </joint>
     <joint name="RAnklePitch" type="revolute">
-        <origin xyz="0.015 0 -0.17" rpy="0 0 0" />
+        <origin xyz="0.02 0 -0.17" rpy="0 0 0" />
         <parent link="r_lower_leg" />
         <child link="r_ankle" />
@@ -513,5 +514,5 @@
     </joint>
     <joint name="r_foot_to_sole" type="fixed">
-        <origin xyz="0 0 -0.052" rpy="0 0 0" />
+        <origin xyz="0 0 -0.06" rpy="0 0 0" /> <!-- -0.04 - stollen-->
         <parent link="r_foot" />
         <child link="r_sole" />
@@ -549,5 +550,5 @@
     </joint>
     <joint name="LKnee" type="revolute">
-        <origin xyz="-0.015 0 -0.17" rpy="0 0 0" />
+        <origin xyz="-0.030 0 -0.17" rpy="0 0 0" />
         <parent link="l_upper_leg" />
         <child link="l_lower_leg" />
@@ -557,5 +558,5 @@
     </joint>
     <joint name="LAnklePitch" type="revolute">
-        <origin xyz="0.015 0 -0.17" rpy="0 0 0" />
+        <origin xyz="0.020 0 -0.17" rpy="0 0 0" />
         <parent link="l_lower_leg" />
         <child link="l_ankle" />
@@ -573,5 +574,5 @@
     </joint>
     <joint name="left_foot_to_sole" type="fixed">
-        <origin xyz="0 0 -0.052" rpy="0 0 0" />
+        <origin xyz="0 0 -0.06" rpy="0 0 0" />
         <parent link="l_foot" />
         <child link="l_sole" />
@@ -588,4 +589,9 @@
         <child link="torso" />
         <origin rpy="0.0 0 0" xyz="0 0 0.09" />
+    </joint>
+    <joint name="torso_to_imu" type="fixed">
+        <parent link="torso" />
+        <child link="imu" />
+        <origin rpy="0.0 0 0" xyz="-0.045 0.025 0.023" />
     </joint>
     <joint name="RShoulderPitch" type="revolute">
@@ -945,5 +951,5 @@
         <xyzOffset>0 0 0</xyzOffset>
         <rpyOffset>0 0 0</rpyOffset>
-        <frameName>L_IMU</frameName>
+        <frameName>imu</frameName>
       </plugin>
       <pose>0 0 0 0 0 0</pose>

Commit message: small fix for toe link in urdf

File: wolfgang_description/urdf/wolfgang.urdf.xacro (robot description, xacro)
@@ -520,5 +520,5 @@
     </joint>
     <joint name="r_foot_to_toe" type="fixed">
-        <origin xyz="0.105 0 0" rpy="0 0 0" />
+        <origin xyz="0.11 -0.01 0" rpy="0 0 0" />
         <parent link="r_sole" />
         <child link="r_toe" />
@@ -574,5 +574,5 @@
     </joint>
     <joint name="left_foot_to_sole" type="fixed">
-        <origin xyz="0 0 -0.06" rpy="0 0 0" />
+        <origin xyz="0 0 -0.06" rpy="0 0 0" /> <!-- -0.04 - stollen-->
         <parent link="l_foot" />
         <child link="l_sole" />
@@ -580,5 +580,5 @@
     </joint>
     <joint name="left_foot_to_toe" type="fixed">
-        <origin xyz="0.105 0 0" rpy="0 0 0" />
+        <origin xyz="0.11 -0.01 0" rpy="0 0 0" />
         <parent link="l_sole" />
         <child link="l_toe" />

Commit message: added camera_fixed frame for look_at in behavior

File: wolfgang_description/urdf/wolfgang.urdf.xacro (robot description, xacro)
@@ -443,4 +443,6 @@
     <link name="camera" />
     <link name="imu" />
+    <link name="camera_fixed">
+    </link>
     <link name="head">
         <inertial>
@@ -594,4 +596,9 @@
         <child link="imu" />
         <origin rpy="0.0 0 0" xyz="-0.045 0.025 0.023" />
+    </joint>
+    <joint name="torso_to_camera_fixed" type="fixed">
+        <parent link="torso" />
+        <child link="camera_fixed" />
+        <origin rpy="0.0 0 0" xyz="0 0 0.237" />
     </joint>
     <joint name="RShoulderPitch" type="revolute">

Commit message: updated moveit conf

File: wolfgang_description/urdf/wolfgang.urdf.xacro (robot description, xacro)
@@ -442,5 +442,5 @@
     </link>
     <link name="camera" />
-    <link name="imu" />
+    <link name="imu_frame" />
     <link name="camera_fixed">
     </link>
@@ -594,5 +594,5 @@
     <joint name="torso_to_imu" type="fixed">
         <parent link="torso" />
-        <child link="imu" />
+        <child link="imu_frame" />
         <origin rpy="0.0 0 0" xyz="-0.045 0.025 0.023" />
     </joint>

Commit message: added optical frame for camera

File: wolfgang_description/urdf/wolfgang.urdf.xacro (robot description, xacro)
@@ -442,4 +442,5 @@
     </link>
     <link name="camera" />
+    <link name="camera_optical_frame"/>
     <link name="imu_frame" />
     <link name="camera_fixed">
@@ -682,4 +683,9 @@
         <axis xyz="0 0 0" />
         <dynamics damping="${d}" friction="${f}" />
+    </joint>
+    <joint name="camera__optical_joint" type="fixed">
+      <origin xyz="0 0 0" rpy="${-pi/2} 0 ${-pi/2}" />
+      <parent link="camera" />
+      <child link="camera_optical_frame" />
     </joint>
     <transmission name="HeadPanTransmission">

Commit message: torso test

File: wolfgang_description/urdf/wolfgang.urdf.xacro (robot description, xacro)
@@ -20,5 +20,5 @@
             <origin xyz="0 0 0" rpy="0 0 0" />
             <geometry>
-                <mesh filename="package://wolfgang_description/mesh/trunk_link.STL" />
+                <mesh filename="package://wolfgang_description/mesh_new/torso_link.stl" />
             </geometry>
             <material name="black" />

Commit message: moved to mesh instead of mesh_new, branches are nice, stl should be rightside up now ...

File: wolfgang_description/urdf/wolfgang.urdf.xacro (robot description, xacro)
@@ -20,5 +20,5 @@
             <origin xyz="0 0 0" rpy="0 0 0" />
             <geometry>
-                <mesh filename="package://wolfgang_description/mesh_new/torso_link.stl" />
+                <mesh filename="package://wolfgang_description/mesh/torso_link.stl" />
             </geometry>
             <material name="black" />

Commit message: dae test

File: wolfgang_description/urdf/wolfgang.urdf.xacro (robot description, xacro)
@@ -40,5 +40,5 @@
             <origin xyz="0 0 0" rpy="0 0 0" />
             <geometry>
-                <mesh filename="package://wolfgang_description/mesh/right_hip_yaw_link.STL" />
+                <mesh filename="package://wolfgang_description/mesh/right_hip_yaw_link.dae" />
             </geometry>
             <material name="black" />

Commit message: scale and rotation of hip yaw

File: wolfgang_description/urdf/wolfgang.urdf.xacro (robot description, xacro)
@@ -20,5 +20,5 @@
             <origin xyz="0 0 0" rpy="0 0 0" />
             <geometry>
-                <mesh filename="package://wolfgang_description/mesh/torso_link.stl" />
+                <mesh filename="package://wolfgang_description/mesh/torso_link.stl"  />
             </geometry>
             <material name="black" />
@@ -40,5 +40,5 @@
             <origin xyz="0 0 0" rpy="0 0 0" />
             <geometry>
-                <mesh filename="package://wolfgang_description/mesh/right_hip_yaw_link.dae" />
+                <mesh filename="package://wolfgang_description/mesh/right_hip_yaw_link.dae" scale="0.001 0.001 0.001"/>
             </geometry>
             <material name="black" />
