Commit message: updated legs and urdf

File: wolfgang_description/urdf/wolfgang.urdf.xacro (robot description, xacro)
@@ -10,4 +10,10 @@
         <color rgba="0.1 0.1 0.1 1" />
     </material>
+    <material name="metal">
+        <color rgba="0.85 0.85 0.85 1" />
+    </material>
+    <material name="carbon">
+        <color rgba="0.5 0.5 0.5 1" />
+    </material>
     <link name="base_link" />
     <link name="torso">
@@ -21,13 +27,20 @@
             <geometry>
                 <mesh filename="package://wolfgang_description/mesh/torso_link.stl"  />
-            </geometry>
-            <material name="black" />
-        </visual>
-        <collision>
+		<material name="metal" />
+            </geometry>
+        </visual>
+	<visual>
+            <origin xyz="0 0 0" rpy="0 0 0" />
+            <geometry>
+                <mesh filename="package://wolfgang_description/mesh/torso_link_motors.stl"/>
+        	<material name="black" />
+	    </geometry>
+        </visual>
+        <!--<collision>
             <origin xyz="0 0 0" rpy="0 0 0" />
             <geometry>
                 <mesh filename="package://wolfgang_description/mesh/trunk_link.dae" />
             </geometry>
-        </collision>
+        </collision>-->
     </link>
     <link name="r_hip_1">
@@ -40,14 +53,14 @@
             <origin xyz="0 0 0" rpy="0 0 0" />
             <geometry>
-                <mesh filename="package://wolfgang_description/mesh/right_hip_yaw_link.dae" scale="0.001 0.001 0.001"/>
-            </geometry>
-            <material name="black" />
-        </visual>
-        <collision>
-            <origin xyz="0 0 0" rpy="0 0 0" />
-            <geometry>
-                <mesh filename="package://wolfgang_description/mesh/right_hip_yaw_link.dae" />
-            </geometry>
-        </collision>
+                <mesh filename="package://wolfgang_description/mesh/hip_connector.stl"/>
+        	<material name="metal" />
+	    </geometry>
+        </visual>
+        <!--<collision>
+            <origin xyz="0 0 0" rpy="0 0 0" />
+            <geometry>
+                <mesh filename="package://wolfgang_description/mesh/right_hip_yaw_link_collision.dae" />
+            </geometry>
+        </collision>-->
     </link>
     <link name="r_hip_2">
@@ -60,14 +73,14 @@
             <origin xyz="0 0 0" rpy="0 0 0" />
             <geometry>
-                <mesh filename="package://wolfgang_description/mesh/right_hip_roll_link.STL" />
-            </geometry>
-            <material name="black" />
-        </visual>
-        <collision>
+                <mesh filename="package://wolfgang_description/mesh/hip_link2.stl" />
+            </geometry>
+            <material name="black" />
+        </visual>
+        <!--<collision>
             <origin xyz="0 0 0" rpy="0 0 0" />
             <geometry>
                 <mesh filename="package://wolfgang_description/mesh/right_hip_roll_link.dae" />
-            </geometry>
-        </collision>
+            </geometry>-->
+        </collision>-->
     </link>
     <link name="r_upper_leg">
@@ -80,7 +93,21 @@
             <origin xyz="0 0 0" rpy="0 0 0" />
             <geometry>
-                <mesh filename="package://wolfgang_description/mesh/left_thigh_link.STL" />
-            </geometry>
-            <material name="black" />
+                <mesh filename="package://wolfgang_description/mesh/upper_leg_motors.stl" />
+            </geometry>
+            <material name="black" />
+        </visual>
+        <visual>
+            <origin xyz="0 0 0" rpy="0 0 0" />
+            <geometry>
+                <mesh filename="package://wolfgang_description/mesh/upper_leg_metal.stl" />
+            </geometry>
+            <material name="metal" />
+        </visual>
+        <visual>
+            <origin xyz="0 0 0" rpy="0 0 0" />
+            <geometry>
+                <mesh filename="package://wolfgang_description/mesh/upper_leg_carbon.stl" />
+            </geometry>
+            <material name="carbon" />
         </visual>
         <!--<collision>
@@ -100,7 +127,7 @@
             <origin xyz="0 0 0" rpy="0 0 0" />
             <geometry>
-                <mesh filename="package://wolfgang_description/mesh/right_shank_link.STL" />
-            </geometry>
-            <material name="black" />
+                <mesh filename="package://wolfgang_description/mesh/lower_leg.stl" />
+            </geometry>
+            <material name="carbon" />
         </visual>
         <!--<collision>
@@ -117,12 +144,12 @@
             <inertia ixx="0.00015501" ixy="1.7299E-06" ixz="-8.5156E-06" iyy="0.00032958" iyz="-2.4435E-07" izz="0.00027786" />
         </inertial>
-        <!--<visual>
-            <origin xyz="0 0 0" rpy="0 0 0" />
-            <geometry>
-                <mesh filename="package://wolfgang_description/mesh/right_ankle_link.STL" />
-            </geometry>
-            <material name="black" />
-        </visual>
-        <collision>
+        <visual>
+            <origin xyz="0 0 0" rpy="0 0 0" />
+            <geometry>
+                <mesh filename="package://wolfgang_description/mesh/ankle.stl" />
+            </geometry>
+            <material name="black" />
+        </visual>
+        <!--<collision>
             <origin xyz="0 0 0" rpy="0 0 0" />
             <geometry>
@@ -140,14 +167,14 @@
             <origin xyz="0 0 -0.012" rpy="0 0 0" />
             <geometry>
-                <mesh filename="package://wolfgang_description/mesh/right_foot_link.STL" />
-            </geometry>
-            <material name="black" />
-        </visual>
-        <collision>
+                <mesh filename="package://wolfgang_description/mesh/right_foot.stl" />
+            </geometry>
+            <material name="metal" />
+        </visual>
+        <!--<collision>
             <origin xyz="0 0 -0.012" rpy="0 0 0" />
             <geometry>
                 <mesh filename="package://wolfgang_description/mesh/right_foot_link.dae" />
             </geometry>
-        </collision>
+        </collision>-->
     </link>
     <link name="r_sole">
@@ -174,14 +201,14 @@
             <origin xyz="0 0 0" rpy="0 0 0" />
             <geometry>
-                <mesh filename="package://wolfgang_description/mesh/left_hip_yaw_link.STL" />
-            </geometry>
-            <material name="black" />
-        </visual>
-        <collision>
+                <mesh filename="package://wolfgang_description/mesh/hip_connector.stl"/>
+        	<material name="metal" />
+	    </geometry>
+        </visual>
+        <!--<collision>
             <origin xyz="0 0 0" rpy="0 0 0" />
             <geometry>
                 <mesh filename="package://wolfgang_description/mesh/left_hip_yaw_link.dae" />
             </geometry>
-        </collision>
+        </collision>-->
     </link>
     <link name="l_hip_2">
@@ -192,16 +219,16 @@
         </inertial>
         <visual>
+            <origin xyz="0 0 0" rpy="0 0 0" />
+            <geometry>
+                <mesh filename="package://wolfgang_description/mesh/hip_link2.stl" />
+            </geometry>
+            <material name="black" />
+        </visual>
+        <!--<collision>
             <origin xyz="0.033 0 0" rpy="0 0 0" />
             <geometry>
-                <mesh filename="package://wolfgang_description/mesh/left_hip_roll_link.STL" />
-            </geometry>
-            <material name="black" />
-        </visual>
-        <collision>
-            <origin xyz="0.033 0 0" rpy="0 0 0" />
-            <geometry>
                 <mesh filename="package://wolfgang_description/mesh/left_hip_roll_link.dae" />
             </geometry>
-        </collision>
+        </collision>-->
     </link>
     <link name="l_upper_leg">
@@ -211,10 +238,24 @@
             <inertia ixx="0.0020952" ixy="-1.9541E-07" ixz="-0.00017822" iyy="0.0020044" iyz="5.4912E-06" izz="0.00027919" />
         </inertial>
-        <visual>
-            <origin xyz="0 0 0" rpy="0 0 0" />
-            <geometry>
-                <mesh filename="package://wolfgang_description/mesh/left_thigh_link.STL" />
-            </geometry>
-            <material name="black" />
+                <visual>
+            <origin xyz="0 0 0" rpy="0 0 0" />
+            <geometry>
+                <mesh filename="package://wolfgang_description/mesh/upper_leg_motors.stl" />
+            </geometry>
+            <material name="black" />
+        </visual>
+        <visual>
+            <origin xyz="0 0 0" rpy="0 0 0" />
+            <geometry>
+                <mesh filename="package://wolfgang_description/mesh/upper_leg_metal.stl" />
+            </geometry>
+            <material name="metal" />
+        </visual>
+        <visual>
+            <origin xyz="0 0 0" rpy="0 0 0" />
+            <geometry>
+                <mesh filename="package://wolfgang_description/mesh/upper_leg_carbon.stl" />
+            </geometry>
+            <material name="carbon" />
         </visual>
         <!--<collision>
@@ -234,7 +275,7 @@
             <origin xyz="0 0 0" rpy="0 0 0" />
             <geometry>
-                <mesh filename="package://wolfgang_description/mesh/left_shank_link.STL" />
-            </geometry>
-            <material name="black" />
+                <mesh filename="package://wolfgang_description/mesh/lower_leg.stl" />
+            </geometry>
+            <material name="carbon" />
         </visual>
         <!--<collision>
@@ -251,12 +292,12 @@
             <inertia ixx="0.00015503" ixy="-1.738E-06" ixz="-8.5148E-06" iyy="0.0003299" iyz="2.4403E-07" izz="0.0002782" />
         </inertial>
-        <!--<visual>
-            <origin xyz="0 0 0" rpy="0 0 0" />
-            <geometry>
-                <mesh filename="package://wolfgang_description/mesh/left_ankle_link.STL" />
-            </geometry>
-            <material name="black" />
-        </visual>
-        <collision>
+        <visual>
+            <origin xyz="0 0 0" rpy="0 0 0" />
+            <geometry>
+                <mesh filename="package://wolfgang_description/mesh/ankle.stl" />
+            </geometry>
+            <material name="black" />
+        </visual>
+        <!--<collision>
             <origin xyz="0 0 0" rpy="0 0 0" />
             <geometry>
@@ -274,14 +315,14 @@
             <origin xyz="0 0 -0.012" rpy="0 0 0" />
             <geometry>
-                <mesh filename="package://wolfgang_description/mesh/left_foot_link.STL" />
-            </geometry>
-            <material name="black" />
-        </visual>
-        <collision>
+                <mesh filename="package://wolfgang_description/mesh/left_foot.stl" />
+            </geometry>
+            <material name="metal" />
+        </visual>
+        <!--<collision>
             <origin xyz="0 0 -0.012" rpy="0 0 0" />
             <geometry>
                 <mesh filename="package://wolfgang_description/mesh/left_foot_link.dae" />
             </geometry>
-        </collision>
+        </collision>-->
     </link>
     <link name="l_sole">
@@ -312,10 +353,10 @@
             <material name="black" />
         </visual>
-        <collision>
+        <!--<collision>
             <origin xyz="0 0 0" rpy="0 0 0" />
             <geometry>
                 <mesh filename="package://wolfgang_description/mesh/right_shoulder_pitch_link.dae" />
             </geometry>
-        </collision>
+        </collision>-->
     </link>
     <link name="r_upper_arm">
@@ -332,10 +373,10 @@
             <material name="black" />
         </visual>
-        <collision>
+        <!--<collision>
             <origin xyz="0 0 0" rpy="0 0 0" />
             <geometry>
                 <mesh filename="package://wolfgang_description/mesh/right_shoulder_arm_link.dae" />
             </geometry>
-        </collision>
+        </collision>-->
     </link>
     <link name="r_lower_arm">
@@ -352,10 +393,10 @@
             <material name="black" />
         </visual>
-        <collision>
+        <!--<collision>
             <origin xyz="0 0 0" rpy="0 -1.57 0" />
             <geometry>
                 <mesh filename="package://wolfgang_description/mesh/right_lower_arm_link.dae" />
             </geometry>
-        </collision>
+        </collision>-->
     </link>
     <link name="r_wrist"> </link>
@@ -373,10 +414,10 @@
             <material name="black" />
         </visual>
-        <collision>
+        <!--<collision>
             <origin xyz="0 0 0" rpy="0 0 0" />
             <geometry>
                 <mesh filename="package://wolfgang_description/mesh/left_shoulder_pitch_link.dae" />
             </geometry>
-        </collision>
+        </collision>-->
     </link>
     <link name="l_upper_arm">
@@ -393,10 +434,10 @@
             <material name="black" />
         </visual>
-        <collision>
+        <!--<collision>
             <origin xyz="0 0 0" rpy="0 0 0" />
             <geometry>
                 <mesh filename="package://wolfgang_description/mesh/left_upper_arm_link.dae" />
             </geometry>
-        </collision>
+        </collision>-->
     </link>
     <link name="l_lower_arm">
@@ -413,10 +454,10 @@
             <material name="black" />
         </visual>
-        <collision>
+        <!--<collision>
             <origin xyz="0 0 0" rpy="0 -1.57 0" />
             <geometry>
                 <mesh filename="package://wolfgang_description/mesh/left_lower_arm_link.dae" />
             </geometry>
-        </collision>
+        </collision>-->
     </link>
     <link name="l_wrist"> </link>
@@ -434,10 +475,10 @@
             <material name="black" />
         </visual>
-        <collision>
+        <!--<collision>
             <origin xyz="0 0 0" rpy="0 0 0" />
             <geometry>
                 <mesh filename="package://wolfgang_description/mesh/neck_link.dae" />
             </geometry>
-        </collision>
+        </collision>-->
     </link>
     <link name="camera" />
@@ -461,5 +502,5 @@
             </material>
         </visual>
-        <collision>
+        <!--<collision>
             <origin xyz="0 0 0" rpy="0 0 0" />
             <geometry>

Commit message: fixed some errors in the urdf

File: wolfgang_description/urdf/wolfgang.urdf.xacro (robot description, xacro)
@@ -73,5 +73,5 @@
             <origin xyz="0 0 0" rpy="0 0 0" />
             <geometry>
-                <mesh filename="package://wolfgang_description/mesh/hip_link2.stl" />
+                <mesh filename="package://wolfgang_description/mesh/hip_link_2.stl" />
             </geometry>
             <material name="black" />
@@ -81,5 +81,5 @@
             <geometry>
                 <mesh filename="package://wolfgang_description/mesh/right_hip_roll_link.dae" />
-            </geometry>-->
+            </geometry>
         </collision>-->
     </link>
@@ -91,12 +91,12 @@
         </inertial>
         <visual>
-            <origin xyz="0 0 0" rpy="0 0 0" />
-            <geometry>
-                <mesh filename="package://wolfgang_description/mesh/upper_leg_motors.stl" />
-            </geometry>
-            <material name="black" />
-        </visual>
-        <visual>
-            <origin xyz="0 0 0" rpy="0 0 0" />
+            <origin xyz="0 0 0" rpy="0 ${pi} 0" />
+            <geometry>
+                <mesh filename="package://wolfgang_description/mesh/upper_leg_motor.stl" />
+            </geometry>
+            <material name="black" />
+        </visual>
+        <visual>
+            <origin xyz="0 0 0" rpy="0 ${pi} 0" />
             <geometry>
                 <mesh filename="package://wolfgang_description/mesh/upper_leg_metal.stl" />
@@ -105,5 +105,5 @@
         </visual>
         <visual>
-            <origin xyz="0 0 0" rpy="0 0 0" />
+            <origin xyz="0 0 0" rpy="0 ${pi} 0" />
             <geometry>
                 <mesh filename="package://wolfgang_description/mesh/upper_leg_carbon.stl" />
@@ -221,5 +221,5 @@
             <origin xyz="0 0 0" rpy="0 0 0" />
             <geometry>
-                <mesh filename="package://wolfgang_description/mesh/hip_link2.stl" />
+                <mesh filename="package://wolfgang_description/mesh/hip_link_2.stl" />
             </geometry>
             <material name="black" />
@@ -239,12 +239,12 @@
         </inertial>
                 <visual>
-            <origin xyz="0 0 0" rpy="0 0 0" />
-            <geometry>
-                <mesh filename="package://wolfgang_description/mesh/upper_leg_motors.stl" />
-            </geometry>
-            <material name="black" />
-        </visual>
-        <visual>
-            <origin xyz="0 0 0" rpy="0 0 0" />
+            <origin xyz="0 0 0" rpy="0 ${pi} 0" />
+            <geometry>
+                <mesh filename="package://wolfgang_description/mesh/upper_leg_motor.stl" />
+            </geometry>
+            <material name="black" />
+        </visual>
+        <visual>
+            <origin xyz="0 0 0" rpy="0 ${pi} 0" />
             <geometry>
                 <mesh filename="package://wolfgang_description/mesh/upper_leg_metal.stl" />
@@ -253,5 +253,5 @@
         </visual>
         <visual>
-            <origin xyz="0 0 0" rpy="0 0 0" />
+            <origin xyz="0 0 0" rpy="0 ${pi} 0" />
             <geometry>
                 <mesh filename="package://wolfgang_description/mesh/upper_leg_carbon.stl" />
@@ -502,5 +502,5 @@
             </material>
         </visual>
-        <!--<collision>
+        <collision>
             <origin xyz="0 0 0" rpy="0 0 0" />
             <geometry>

Commit message: head and neck added

File: wolfgang_description/urdf/wolfgang.urdf.xacro (robot description, xacro)
@@ -471,5 +471,5 @@
             <origin xyz="0 0 0" rpy="0 0 0" />
             <geometry>
-                <mesh filename="package://wolfgang_description/mesh/neck_link.STL" />
+                <mesh filename="package://wolfgang_description/mesh/neck.stl" />
             </geometry>
             <material name="black" />
@@ -493,8 +493,8 @@
             <inertia ixx="0.0014813" ixy="3.1631E-07" ixz="-4.1003E-05" iyy="0.0016361" iyz="6.7483E-07" izz="0.0017353" />
         </inertial>
-        <!--<visual>
-            <origin xyz="0 0 0" rpy="0 0 0" />
-            <geometry>
-                <mesh filename="package://wolfgang_description/mesh/head_link.STL" />
+        <visual>
+            <origin xyz="0 0 0" rpy="0 0 0" />
+            <geometry>
+                <mesh filename="package://wolfgang_description/mesh/head.stl" />
             </geometry>
             <material name="">
@@ -502,5 +502,5 @@
             </material>
         </visual>
-        <collision>
+        <!--<collision>
             <origin xyz="0 0 0" rpy="0 0 0" />
             <geometry>
@@ -703,5 +703,5 @@
     </joint>
     <joint name="HeadPan" type="revolute">
-        <origin xyz="-0.0285 0 0.1365" rpy="0 0 0" />
+        <origin xyz="0.00155 0 0.1471" rpy="0 0 0" />
         <parent link="torso" />
         <child link="neck" />
@@ -711,5 +711,5 @@
     </joint>
     <joint name="HeadTilt" type="revolute">
-        <origin xyz="0 0 0.0505" rpy="0 0 0" />
+        <origin xyz="0.0286 0 0.0205" rpy="0 0 0" />
         <parent link="neck" />
         <child link="head" />
