Commit message: urdf fixes

File: wolfgang_description/urdf/wolfgang.urdf.xacro (robot description, xacro)
@@ -14,5 +14,5 @@
     </material>
     <material name="carbon">
-        <color rgba="0.5 0.5 0.5 1" />
+        <color rgba="0.3 0.3 0.3 1" />
     </material>
     <link name="base_link" />
@@ -27,13 +27,13 @@
             <geometry>
                 <mesh filename="package://wolfgang_description/mesh/torso_link.stl"  />
-		<material name="metal" />
-            </geometry>
-        </visual>
-	<visual>
+            </geometry>
+            <material name="metal" />
+        </visual>
+        <visual>
             <origin xyz="0 0 0" rpy="0 0 0" />
             <geometry>
                 <mesh filename="package://wolfgang_description/mesh/torso_link_motors.stl"/>
-        	<material name="black" />
-	    </geometry>
+            </geometry>
+            <material name="black" />
         </visual>
         <!--<collision>
@@ -54,6 +54,6 @@
             <geometry>
                 <mesh filename="package://wolfgang_description/mesh/hip_connector.stl"/>
-        	<material name="metal" />
-	    </geometry>
+            </geometry>
+            <material name="metal" />
         </visual>
         <!--<collision>
@@ -93,21 +93,21 @@
             <origin xyz="0 0 0" rpy="0 ${pi} 0" />
             <geometry>
+                <mesh filename="package://wolfgang_description/mesh/upper_leg_carbon.stl" />
+            </geometry>
+            <material name="carbon" />
+        </visual>
+        <visual>
+            <origin xyz="0 0 0" rpy="0 ${pi} 0" />
+            <geometry>
+                <mesh filename="package://wolfgang_description/mesh/upper_leg_metal.stl" />
+            </geometry>
+            <material name="metal"/>
+        </visual>
+        <visual>
+            <origin xyz="0 0 0" rpy="0 ${pi} 0" />
+            <geometry>
                 <mesh filename="package://wolfgang_description/mesh/upper_leg_motor.stl" />
             </geometry>
             <material name="black" />
-        </visual>
-        <visual>
-            <origin xyz="0 0 0" rpy="0 ${pi} 0" />
-            <geometry>
-                <mesh filename="package://wolfgang_description/mesh/upper_leg_metal.stl" />
-            </geometry>
-            <material name="metal" />
-        </visual>
-        <visual>
-            <origin xyz="0 0 0" rpy="0 ${pi} 0" />
-            <geometry>
-                <mesh filename="package://wolfgang_description/mesh/upper_leg_carbon.stl" />
-            </geometry>
-            <material name="carbon" />
         </visual>
         <!--<collision>
@@ -165,5 +165,5 @@
         </inertial>
         <visual>
-            <origin xyz="0 0 -0.012" rpy="0 0 0" />
+            <origin xyz="0 0 0" rpy="0 0 0" />
             <geometry>
                 <mesh filename="package://wolfgang_description/mesh/right_foot.stl" />
@@ -202,6 +202,6 @@
             <geometry>
                 <mesh filename="package://wolfgang_description/mesh/hip_connector.stl"/>
-        	<material name="metal" />
-	    </geometry>
+            </geometry>
+            <material name="metal" />
         </visual>
         <!--<collision>
@@ -238,7 +238,14 @@
             <inertia ixx="0.0020952" ixy="-1.9541E-07" ixz="-0.00017822" iyy="0.0020044" iyz="5.4912E-06" izz="0.00027919" />
         </inertial>
-                <visual>
+        <visual>
             <origin xyz="0 0 0" rpy="0 ${pi} 0" />
             <geometry>
+                <mesh filename="package://wolfgang_description/mesh/upper_leg_carbon.stl" />
+            </geometry>
+            <material name="carbon" />
+        </visual>
+        <visual>
+            <origin xyz="0 0 0" rpy="0 ${pi} 0" />
+            <geometry>
                 <mesh filename="package://wolfgang_description/mesh/upper_leg_motor.stl" />
             </geometry>
@@ -251,11 +258,4 @@
             </geometry>
             <material name="metal" />
-        </visual>
-        <visual>
-            <origin xyz="0 0 0" rpy="0 ${pi} 0" />
-            <geometry>
-                <mesh filename="package://wolfgang_description/mesh/upper_leg_carbon.stl" />
-            </geometry>
-            <material name="carbon" />
         </visual>
         <!--<collision>
@@ -313,5 +313,5 @@
         </inertial>
         <visual>
-            <origin xyz="0 0 -0.012" rpy="0 0 0" />
+            <origin xyz="0 0 0" rpy="0 0 0" />
             <geometry>
                 <mesh filename="package://wolfgang_description/mesh/left_foot.stl" />
@@ -518,5 +518,5 @@
     </joint>
     <joint name="RHipRoll" type="revolute">
-        <origin xyz="-0.0072 0 -0.0438" rpy="0 0 0" />
+        <origin xyz="-0.046 0 -0.042" rpy="0 0 0" />
         <parent link="r_hip_1" />
         <child link="r_hip_2" />
@@ -526,5 +526,5 @@
     </joint>
     <joint name="RHipPitch" type="revolute">
-        <origin xyz="0.0303 0 0" rpy="0 0 0" />
+        <origin xyz="0.0692 0 0" rpy="0 0 0" />
         <parent link="r_hip_2" />
         <child link="r_upper_leg" />
@@ -534,5 +534,5 @@
     </joint>
     <joint name="RKnee" type="revolute">
-        <origin xyz="-0.03 0 -0.17" rpy="0 0 0" />
+        <origin xyz="-0.004 0 -0.1692" rpy="0 0 0" />
         <parent link="r_upper_leg" />
         <child link="r_lower_leg" />
@@ -542,5 +542,5 @@
     </joint>
     <joint name="RAnklePitch" type="revolute">
-        <origin xyz="0.02 0 -0.17" rpy="0 0 0" />
+        <origin xyz="0.0 0 -0.17" rpy="0 0 0" />
         <parent link="r_lower_leg" />
         <child link="r_ankle" />
@@ -550,5 +550,5 @@
     </joint>
     <joint name="RAnkleRoll" type="revolute">
-        <origin xyz="0 0 0" rpy="0 0 0" />
+        <origin xyz="-0.0692 0 0" rpy="0 0 0" />
         <parent link="r_ankle" />
         <child link="r_foot" />
@@ -558,5 +558,5 @@
     </joint>
     <joint name="r_foot_to_sole" type="fixed">
-        <origin xyz="0 0 -0.06" rpy="0 0 0" /> <!-- -0.04 - stollen-->
+        <origin xyz="0.082 0 -0.036" rpy="0 0 0" /> <!-- stollen todo-->
         <parent link="r_foot" />
         <child link="r_sole" />
@@ -564,5 +564,5 @@
     </joint>
     <joint name="r_foot_to_toe" type="fixed">
-        <origin xyz="0.11 -0.01 0" rpy="0 0 0" />
+        <origin xyz="0.095 -0.003 0" rpy="0 0 0" />
         <parent link="r_sole" />
         <child link="r_toe" />
@@ -578,5 +578,5 @@
     </joint>
     <joint name="LHipRoll" type="revolute">
-        <origin xyz="-0.0072 0 -0.0438" rpy="0 0 0" />
+        <origin xyz="-0.046 0 -0.042" rpy="0 0 0" />
         <parent link="l_hip_1" />
         <child link="l_hip_2" />
@@ -586,5 +586,5 @@
     </joint>
     <joint name="LHipPitch" type="revolute">
-        <origin xyz="0.0303 0 0" rpy="0 0 0" />
+        <origin xyz="0.0692 0 0" rpy="0 0 0" />
         <parent link="l_hip_2" />
         <child link="l_upper_leg" />
@@ -594,5 +594,5 @@
     </joint>
     <joint name="LKnee" type="revolute">
-        <origin xyz="-0.030 0 -0.17" rpy="0 0 0" />
+        <origin xyz="-0.004 0 -0.1692" rpy="0 0 0" />
         <parent link="l_upper_leg" />
         <child link="l_lower_leg" />
@@ -602,5 +602,5 @@
     </joint>
     <joint name="LAnklePitch" type="revolute">
-        <origin xyz="0.020 0 -0.17" rpy="0 0 0" />
+        <origin xyz="0.0 0 -0.17" rpy="0 0 0" />
         <parent link="l_lower_leg" />
         <child link="l_ankle" />
@@ -610,5 +610,5 @@
     </joint>
     <joint name="LAnkleRoll" type="revolute">
-        <origin xyz="0 0 0" rpy="0 0 0" />
+        <origin xyz="-0.0692 0 0" rpy="0 0 0" />
         <parent link="l_ankle" />
         <child link="l_foot" />
@@ -618,5 +618,5 @@
     </joint>
     <joint name="left_foot_to_sole" type="fixed">
-        <origin xyz="0 0 -0.06" rpy="0 0 0" /> <!-- -0.04 - stollen-->
+        <origin xyz="0.082 0 -0.036" rpy="0 0 0" /> <!-- todo mit stollen!-->
         <parent link="l_foot" />
         <child link="l_sole" />
@@ -624,5 +624,5 @@
     </joint>
     <joint name="left_foot_to_toe" type="fixed">
-        <origin xyz="0.11 -0.01 0" rpy="0 0 0" />
+        <origin xyz="0.095 -0.003 0" rpy="0 0 0" />
         <parent link="l_sole" />
         <child link="l_toe" />
@@ -632,5 +632,5 @@
         <parent link="base_link" />
         <child link="torso" />
-        <origin rpy="0.0 0 0" xyz="0 0 0.09" />
+        <origin rpy="0.0 0 0" xyz="-0.0095 0 0.0905" />
     </joint>
     <joint name="torso_to_imu" type="fixed">

Commit message: arms!

File: wolfgang_description/urdf/wolfgang.urdf.xacro (robot description, xacro)
@@ -349,5 +349,5 @@
             <origin xyz="0 0 0" rpy="0 0 0" />
             <geometry>
-                <mesh filename="package://wolfgang_description/mesh/right_shoulder_pitch_link.STL" />
+                <mesh filename="package://wolfgang_description/mesh/shoulder.stl" />
             </geometry>
             <material name="black" />
@@ -369,5 +369,5 @@
             <origin xyz="0 0 0" rpy="0 0 0" />
             <geometry>
-                <mesh filename="package://wolfgang_description/mesh/right_shoulder_arm_link.STL" />
+                <mesh filename="package://wolfgang_description/mesh/upper_arm.stl" />
             </geometry>
             <material name="black" />
@@ -389,5 +389,5 @@
             <origin xyz="0 0 0" rpy="0 -1.57 0" />
             <geometry>
-                <mesh filename="package://wolfgang_description/mesh/right_lower_arm_link.STL" />
+                <mesh filename="package://wolfgang_description/mesh/lower_arm.stl" />
             </geometry>
             <material name="black" />
@@ -410,5 +410,5 @@
             <origin xyz="0 0 0" rpy="0 0 0" />
             <geometry>
-                <mesh filename="package://wolfgang_description/mesh/left_shoulder_pitch_link.STL" />
+                <mesh filename="package://wolfgang_description/mesh/shoulder.stl" />
             </geometry>
             <material name="black" />
@@ -430,5 +430,5 @@
             <origin xyz="0 0 0" rpy="0 0 0" />
             <geometry>
-                <mesh filename="package://wolfgang_description/mesh/left_upper_arm_link.STL" />
+                <mesh filename="package://wolfgang_description/mesh/upper_arm.stl" />
             </geometry>
             <material name="black" />
@@ -450,5 +450,5 @@
             <origin xyz="0 0 0" rpy="0 -1.57 0" />
             <geometry>
-                <mesh filename="package://wolfgang_description/mesh/left_lower_arm_link.STL" />
+                <mesh filename="package://wolfgang_description/mesh/lower_arm.stl" />
             </geometry>
             <material name="black" />
@@ -653,5 +653,5 @@
     </joint>
     <joint name="RShoulderRoll" type="revolute">
-        <origin xyz="0 -0.04 0" rpy="0 0 0" />
+        <origin xyz="0 -0.042 0" rpy="0 0 0" />
         <parent link="r_shoulder" />
         <child link="r_upper_arm" />
@@ -661,5 +661,5 @@
     </joint>
     <joint name="RElbow" type="revolute">
-        <origin xyz="-0.0075 0 -0.145" rpy="0 0 0" />
+        <origin xyz="0 0 -0.144" rpy="0 0 0" />
         <parent link="r_upper_arm" />
         <child link="r_lower_arm" />
@@ -682,5 +682,5 @@
     </joint>
     <joint name="LShoulderRoll" type="revolute">
-        <origin xyz="0 0.04 0" rpy="0 0 0" />
+        <origin xyz="0 0.042 0" rpy="0 0 0" />
         <parent link="l_shoulder" />
         <child link="l_upper_arm" />
@@ -690,5 +690,5 @@
     </joint>
     <joint name="LElbow" type="revolute">
-        <origin xyz="-0.0075 0 -0.145" rpy="0 0 0" />
+        <origin xyz="0 0 -0.144" rpy="0 0 0" />
         <parent link="l_upper_arm" />
         <child link="l_lower_arm" />
@@ -719,5 +719,5 @@
     </joint>
     <joint name="head_to_camera" type="fixed">
-        <origin xyz="0.03 0 0.05" rpy="0 0 0" />
+        <origin xyz="0.0289 0 0.1115" rpy="0 0 0" />
         <parent link="head" />
         <child link="camera" />
@@ -725,5 +725,5 @@
         <dynamics damping="${d}" friction="${f}" />
     </joint>
-    <joint name="camera__optical_joint" type="fixed">
+	<joint name="camera__optical_joint" type="fixed">
       <origin xyz="0 0 0" rpy="${-pi/2} 0 ${-pi/2}" />
       <parent link="camera" />

Commit message: corrections

File: wolfgang_description/urdf/wolfgang.urdf.xacro (robot description, xacro)
@@ -469,5 +469,5 @@
         </inertial>
         <visual>
-            <origin xyz="0 0 0" rpy="0 0 0" />
+            <origin xyz="0 0 0" rpy="0 0 ${pi}" />
             <geometry>
                 <mesh filename="package://wolfgang_description/mesh/neck.stl" />
@@ -498,7 +498,5 @@
                 <mesh filename="package://wolfgang_description/mesh/head.stl" />
             </geometry>
-            <material name="">
-                <color rgba="0.8 0.8 0.8 1" />
-            </material>
+            <material name="black" />
         </visual>
         <!--<collision>
@@ -642,5 +640,5 @@
         <parent link="torso" />
         <child link="camera_fixed" />
-        <origin rpy="0.0 0 0" xyz="0 0 0.237" />
+        <origin rpy="0.0 0 0" xyz="0.05815 0 0.2791" />
     </joint>
     <joint name="RShoulderPitch" type="revolute">
@@ -719,5 +717,5 @@
     </joint>
     <joint name="head_to_camera" type="fixed">
-        <origin xyz="0.03 0 0.05" rpy="0 0 0" />
+        <origin xyz="0.028 0 0.1115" rpy="0 0 0" />
         <parent link="head" />
         <child link="camera" />

Commit message: urdf from measured assembly

File: wolfgang_description/urdf/wolfgang.urdf.xacro (robot description, xacro)
@@ -342,5 +342,5 @@
     <link name="r_shoulder">
         <inertial>
-            <origin xyz="0 -0.014621 0" rpy="0 0 0" />
+            <origin xyz="0 -0.014621 0" rpy="${pi} 0 0" />
             <mass value="0.025434" />
             <inertia ixx="6.7511E-06" ixy="1.5595E-20" ixz="-5.4198E-21" iyy="1.2425E-05" iyz="-2.4006E-20" izz="1.4317E-05" />
@@ -351,5 +351,5 @@
                 <mesh filename="package://wolfgang_description/mesh/shoulder.stl" />
             </geometry>
-            <material name="black" />
+            <material name="metal" />
         </visual>
         <!--<collision>
@@ -367,5 +367,5 @@
         </inertial>
         <visual>
-            <origin xyz="0 0 0" rpy="0 0 0" />
+            <origin xyz="0 0 0" rpy="0 ${pi} 0" />
             <geometry>
                 <mesh filename="package://wolfgang_description/mesh/upper_arm.stl" />
@@ -387,5 +387,5 @@
         </inertial>
         <visual>
-            <origin xyz="0 0 0" rpy="0 -1.57 0" />
+            <origin xyz="0 0 0" rpy="0 0 0" />
             <geometry>
                 <mesh filename="package://wolfgang_description/mesh/lower_arm.stl" />
@@ -412,5 +412,5 @@
                 <mesh filename="package://wolfgang_description/mesh/shoulder.stl" />
             </geometry>
-            <material name="black" />
+            <material name="metal" />
         </visual>
         <!--<collision>
@@ -428,5 +428,5 @@
         </inertial>
         <visual>
-            <origin xyz="0 0 0" rpy="0 0 0" />
+            <origin xyz="0 0 0" rpy="0 ${pi} 0" />
             <geometry>
                 <mesh filename="package://wolfgang_description/mesh/upper_arm.stl" />
@@ -448,5 +448,5 @@
         </inertial>
         <visual>
-            <origin xyz="0 0 0" rpy="0 -1.57 0" />
+            <origin xyz="0 0 0" rpy="0 0 0" />
             <geometry>
                 <mesh filename="package://wolfgang_description/mesh/lower_arm.stl" />
@@ -717,5 +717,5 @@
     </joint>
     <joint name="head_to_camera" type="fixed">
-        <origin xyz="0.028 0 0.1115" rpy="0 0 0" /> <!--evtl 0.0289-->
+        <origin xyz="0.028 0 0.1115" rpy="0 0 0" />
         <parent link="head" />
         <child link="camera" />

Commit message: visuals for camera removed due to large polygon count

File: wolfgang_description/urdf/wolfgang.urdf.xacro (robot description, xacro)
@@ -493,5 +493,5 @@
             <inertia ixx="0.0014813" ixy="3.1631E-07" ixz="-4.1003E-05" iyy="0.0016361" iyz="6.7483E-07" izz="0.0017353" />
         </inertial>
-        <visual>
+        <!--<visual>
             <origin xyz="0 0 0" rpy="0 0 0" />
             <geometry>
@@ -499,5 +499,5 @@
             </geometry>
             <material name="black" />
-        </visual>
+        </visual>-->
         <!--<collision>
             <origin xyz="0 0 0" rpy="0 0 0" />

Commit message: added cleats with parameter

File: wolfgang_description/urdf/wolfgang.urdf.xacro (robot description, xacro)
@@ -2,4 +2,5 @@
 <robot xmlns:xacro="http://www.ros.org/wiki/xacro" name="wolfgang">
     <xacro:arg name="sim_ns" default="/" />
+    <xacro:arg name="cleats" default="-0.013" />
     <xacro:property name="tofa" value="1" /> <!--Torque factor-->
     <xacro:property name="infa" value="1" /> <!--inertia factor-->
@@ -484,7 +485,14 @@
     <link name="camera" />
     <link name="camera_optical_frame"/>
+    <link name="camera_fixed"/>
     <link name="imu_frame" />
-    <link name="camera_fixed">
-    </link>
+    <link name="l_cleat_l_front"/>
+    <link name="l_cleat_r_front"/>
+    <link name="l_cleat_l_back"/>
+    <link name="l_cleat_r_back"/>
+    <link name="r_cleat_l_front"/>
+    <link name="r_cleat_r_front"/>
+    <link name="r_cleat_l_back"/>
+    <link name="r_cleat_r_back"/>
     <link name="head">
         <inertial>
@@ -507,4 +515,5 @@
         </collision>-->
     </link>
+    <!-- JOINTS JOINTS JOINTS JOINTS JOINTS JOINTS JOINTS JOINTS JOINTS JOINTS -->
     <joint name="RHipYaw" type="revolute">
         <origin xyz="0 -0.055 0" rpy="0 0 0" />
@@ -556,5 +565,5 @@
     </joint>
     <joint name="r_foot_to_sole" type="fixed">
-        <origin xyz="0.082 0 -0.036" rpy="0 0 0" /> <!-- stollen todo-->
+        <origin xyz="0.078 -0.015 -0.039" rpy="0 0 0" />
         <parent link="r_foot" />
         <child link="r_sole" />
@@ -562,5 +571,5 @@
     </joint>
     <joint name="r_foot_to_toe" type="fixed">
-        <origin xyz="0.095 -0.003 0" rpy="0 0 0" />
+        <origin xyz="0.095 0 0" rpy="0 0 0" />
         <parent link="r_sole" />
         <child link="r_toe" />
@@ -616,5 +625,5 @@
     </joint>
     <joint name="left_foot_to_sole" type="fixed">
-        <origin xyz="0.082 0 -0.036" rpy="0 0 0" /> <!-- todo mit stollen!-->
+        <origin xyz="0.078 0.015 -0.039" rpy="0 0 0" /> <!-- todo mit stollen!-->
         <parent link="l_foot" />
         <child link="l_sole" />
@@ -622,5 +631,5 @@
     </joint>
     <joint name="left_foot_to_toe" type="fixed">
-        <origin xyz="0.095 -0.003 0" rpy="0 0 0" />
+        <origin xyz="0.095 0 0" rpy="0 0 0" />
         <parent link="l_sole" />
         <child link="l_toe" />
@@ -728,4 +737,47 @@
       <child link="camera_optical_frame" />
     </joint>
+    <!-- left foot cleats -->
+    <joint name="l_sole_to_l_cleat_l_front" type="fixed">
+      <origin xyz="0.085 0.045 $(arg cleats)" rpy="0 0 0" />
+      <parent link="l_sole" />
+      <child link="l_cleat_l_front" />
+    </joint>
+    <joint name="l_sole_to_l_cleat_r_front" type="fixed">
+      <origin xyz="0.085 -0.045 $(arg cleats)" rpy="0 0 0" />
+      <parent link="l_sole" />
+      <child link="l_cleat_r_front" />
+    </joint>
+    <joint name="l_sole_to_l_cleat_l_back" type="fixed">
+      <origin xyz="-0.085 0.045 $(arg cleats)" rpy="0 0 0" />
+      <parent link="l_sole" />
+      <child link="l_cleat_l_back" />
+    </joint>
+    <joint name="l_sole_to_l_cleat_r_back" type="fixed">
+      <origin xyz="-0.085 -0.045 $(arg cleats)" rpy="0 0 0" />
+      <parent link="l_sole" />
+      <child link="l_cleat_r_back" />
+    </joint>
+    <!-- right foot cleats -->
+    <joint name="r_sole_to_r_cleat_l_front" type="fixed">
+      <origin xyz="0.085 0.045 $(arg cleats)" rpy="0 0 0" />
+      <parent link="r_sole" />
+      <child link="r_cleat_l_front" />
+    </joint>
+    <joint name="r_sole_to_r_cleat_r_front" type="fixed">
+      <origin xyz="0.085 -0.045 $(arg cleats)" rpy="0 0 0" />
+      <parent link="r_sole" />
+      <child link="r_cleat_r_front" />
+    </joint>
+    <joint name="r_sole_to_r_cleat_l_back" type="fixed">
+      <origin xyz="-0.085 0.045 $(arg cleats)" rpy="0 0 0" />
+      <parent link="r_sole" />
+      <child link="r_cleat_l_back" />
+    </joint>
+    <joint name="r_sole_to_r_cleat_r_back" type="fixed">
+      <origin xyz="-0.085 -0.045 $(arg cleats)" rpy="0 0 0" />
+      <parent link="r_sole" />
+      <child link="r_cleat_r_back" />
+    </joint>
+    <!-- TRANSMISSIONS TRANSMISSIONS TRANSMISSIONS TRANSMISSIONS TRANSMISSIONS TRANSMISSIONS TRANSMISSIONS -->
     <transmission name="HeadPanTransmission">
         <type>transmission_interface/SimpleTransmission</type>

Commit message: Fix head motor axis and limits in urdf

File: wolfgang_description/urdf/wolfgang.urdf.xacro (robot description, xacro)
@@ -714,5 +714,5 @@
         <child link="neck" />
         <axis xyz="0 0 1" />
-        <limit effort="${tofa*2.5}" velocity="5.6548668" lower="-2.1816615649875" upper="2.1816615649875" />
+        <limit effort="${tofa*2.5}" velocity="5.6548668" lower="-1" upper="1" />
         <dynamics damping="${d}" friction="${f}" />
     </joint>
@@ -721,6 +721,6 @@
         <parent link="neck" />
         <child link="head" />
-        <axis xyz="0 1 0" />
-        <limit effort="${tofa*2.5}" velocity="5.6548668" lower="-1.5707963267910001" upper="0" />
+        <axis xyz="0 -1 0" />
+        <limit effort="${tofa*2.5}" velocity="5.6548668" lower="-1.2" upper="0" />
         <dynamics damping="${d}" friction="${f}" />
     </joint>

Commit message: Adjust HeadTilt limits

File: wolfgang_description/urdf/wolfgang.urdf.xacro (robot description, xacro)
@@ -722,5 +722,5 @@
         <child link="head" />
         <axis xyz="0 -1 0" />
-        <limit effort="${tofa*2.5}" velocity="5.6548668" lower="-1.2" upper="0" />
+        <limit effort="${tofa*2.5}" velocity="5.6548668" lower="-1.2" upper="0.2" />
         <dynamics damping="${d}" friction="${f}" />
     </joint>

Commit message: Adjust HeadPan limits

File: wolfgang_description/urdf/wolfgang.urdf.xacro (robot description, xacro)
@@ -714,5 +714,5 @@
         <child link="neck" />
         <axis xyz="0 0 1" />
-        <limit effort="${tofa*2.5}" velocity="5.6548668" lower="-1" upper="1" />
+        <limit effort="${tofa*2.5}" velocity="5.6548668" lower="-1.2" upper="1.2" />
         <dynamics damping="${d}" friction="${f}" />
     </joint>
