Commit message: corrected optical center of camera

File: wolfgang_description/urdf/wolfgang.urdf.xacro (robot description, xacro)
@@ -501,5 +501,5 @@
             <inertia ixx="0.0014813" ixy="3.1631E-07" ixz="-4.1003E-05" iyy="0.0016361" iyz="6.7483E-07" izz="0.0017353" />
         </inertial>
-        <!--<visual>
+        <visual>
             <origin xyz="0 0 0" rpy="0 0 0" />
             <geometry>
@@ -507,5 +507,5 @@
             </geometry>
             <material name="black" />
-        </visual>-->
+        </visual>
         <!--<collision>
             <origin xyz="0 0 0" rpy="0 0 0" />
@@ -726,5 +726,5 @@
     </joint>
     <joint name="head_to_camera" type="fixed">
-        <origin xyz="0.028 0 0.1115" rpy="0 0 0" />
+        <origin xyz="0.02 0 0.1115" rpy="0 0 0" />
         <parent link="head" />
         <child link="camera" />

Commit message: removed visuals for camera for performance

File: wolfgang_description/urdf/wolfgang.urdf.xacro (robot description, xacro)
@@ -501,5 +501,5 @@
             <inertia ixx="0.0014813" ixy="3.1631E-07" ixz="-4.1003E-05" iyy="0.0016361" iyz="6.7483E-07" izz="0.0017353" />
         </inertial>
-        <visual>
+        <!--<visual>
             <origin xyz="0 0 0" rpy="0 0 0" />
             <geometry>
@@ -507,5 +507,5 @@
             </geometry>
             <material name="black" />
-        </visual>
+        </visual>-->
         <!--<collision>
             <origin xyz="0 0 0" rpy="0 0 0" />

Commit message: updated the camera fixed frame

File: wolfgang_description/urdf/wolfgang.urdf.xacro (robot description, xacro)
@@ -649,5 +649,5 @@
         <parent link="torso" />
         <child link="camera_fixed" />
-        <origin rpy="0.0 0 0" xyz="0.05815 0 0.2791" />
+        <origin rpy="0.0 0 0" xyz="0.05 0 0.279" />
     </joint>
     <joint name="RShoulderPitch" type="revolute">

Commit message: urdf: added pseudo walk and foot collision

File: wolfgang_description/urdf/wolfgang.urdf.xacro (robot description, xacro)
@@ -172,10 +172,10 @@
             <material name="metal" />
         </visual>
-        <!--<collision>
+        <collision>
             <origin xyz="0 0 -0.012" rpy="0 0 0" />
             <geometry>
-                <mesh filename="package://wolfgang_description/mesh/right_foot_link.dae" />
-            </geometry>
-        </collision>-->
+                <mesh filename="package://wolfgang_description/mesh/right_foot.stl" />
+            </geometry>
+        </collision>
     </link>
     <link name="r_sole">
@@ -320,10 +320,10 @@
             <material name="metal" />
         </visual>
-        <!--<collision>
+        <collision>
             <origin xyz="0 0 -0.012" rpy="0 0 0" />
             <geometry>
-                <mesh filename="package://wolfgang_description/mesh/left_foot_link.dae" />
-            </geometry>
-        </collision>-->
+                <mesh filename="package://wolfgang_description/mesh/left_foot.stl" />
+            </geometry>
+        </collision>
     </link>
     <link name="l_sole">
@@ -1061,14 +1061,14 @@
   </gazebo>
    <!-- fake controller that allows us to move the robot and to get its oposition -->
-   <!-- rostopic pub /minibot/cmd_vel geometry_msgs/Twist "{ linear: [ 0.1, 0, 0], angular: [0.2, 0, 0.1] }" -->
-   <!--<gazebo>
+   <!-- rostopic pub /cmd_vel geometry_msgs/Twist "{ linear: [ 0.1, 0, 0], angular: [0.2, 0, 0.1] }" -->
+   <gazebo>
     <plugin name="object_controller" filename="libgazebo_ros_planar_move.so">
-      <robotNamespace>wolves</robotNamespace>
+      <robotNamespace>/</robotNamespace>
       <commandTopic>cmd_vel</commandTopic>
       <odometryTopic>odom</odometryTopic>
       <odometryFrame>odom</odometryFrame>
       <odometryRate>100.0</odometryRate>
-      <robotBaseFrame>base_link</robotBaseFrame>
+      <robotBaseFrame>base_footprint</robotBaseFrame>
     </plugin>
-  </gazebo> -->
+  </gazebo>
 </robot>

Commit message: Added new functions for simple physic simulation with fake walking

File: wolfgang_description/urdf/wolfgang.urdf.xacro (robot description, xacro)
@@ -3,7 +3,8 @@
     <xacro:arg name="sim_ns" default="/" />
     <xacro:arg name="cleats" default="-0.013" />
-    <xacro:property name="tofa" value="1" /> <!--Torque factor-->
-    <xacro:property name="infa" value="1" /> <!--inertia factor-->
-    <xacro:property name="insu" value="0" /> <!--inertia summand-->
+    <xacro:arg name="use_fake_walk" default="False"/>
+    <xacro:property name="fake_walk" value="$(arg use_fake_walk)" />
+    <xacro:property name="tofa" value="1" />  <!--Torque factor-->
+    <!--<xacro:property name="infa" value="1" /> --> <!--inertia factor-->
     <xacro:property name="d" value="1" /> <!-- damping -->
     <xacro:property name="f" value="1" /> <!-- friction -->
@@ -172,10 +173,13 @@
             <material name="metal" />
         </visual>
-        <collision>
-            <origin xyz="0 0 -0.012" rpy="0 0 0" />
-            <geometry>
-                <mesh filename="package://wolfgang_description/mesh/right_foot.stl" />
-            </geometry>
-        </collision>
+        <xacro:if value="${fake_walk== False}">
+            <!-- only active when fake_walk is off, to prevent collisions with ground -->
+            <collision>
+                <origin xyz="0 0 -0.012" rpy="0 0 0" />
+                <geometry>
+                    <mesh filename="package://wolfgang_description/mesh/right_foot.stl" />
+                </geometry>
+            </collision>
+        </xacro:if>
     </link>
     <link name="r_sole">
@@ -320,10 +324,13 @@
             <material name="metal" />
         </visual>
-        <collision>
-            <origin xyz="0 0 -0.012" rpy="0 0 0" />
-            <geometry>
-                <mesh filename="package://wolfgang_description/mesh/left_foot.stl" />
-            </geometry>
-        </collision>
+        <xacro:if value="${fake_walk== False}">
+        <!-- only active when fake_walk is off, to prevent collisions with ground -->
+            <collision>
+                <origin xyz="0 0 -0.012" rpy="0 0 0" />
+                <geometry>
+                    <mesh filename="package://wolfgang_description/mesh/left_foot.stl" />
+                </geometry>
+            </collision>
+        </xacro:if>
     </link>
     <link name="l_sole">
@@ -348,5 +355,5 @@
         </inertial>
         <visual>
-            <origin xyz="0 0 0" rpy="0 0 0" />
+            <origin xyz="0 0 0" rpy="0 0 ${pi}" />
             <geometry>
                 <mesh filename="package://wolfgang_description/mesh/shoulder.stl" />
@@ -466,5 +473,10 @@
         <inertial>
             <origin xyz="2.1595E-05 0.00064781 0.033208" rpy="0 0 0" />
-            <mass value="0.15587" />
+            <xacro:if value="${fake_walk== True}">
+                <mass value="0.00015587" />
+            </xacro:if>
+            <xacro:if value="${fake_walk== False}">
+                <mass value="0.15587" />
+            </xacro:if>
             <inertia ixx="7.5209E-05" ixy="-1.8422E-06" ixz="-4.9817E-07" iyy="6.2999E-05" iyz="-9.9088E-08" izz="3.826E-05" />
         </inertial>
@@ -498,5 +510,10 @@
         <inertial>
             <origin xyz="0.014358 0.0005519 0.069919" rpy="0 0 0" />
-            <mass value="0.40746" />
+            <xacro:if value="${fake_walk== True}">
+                <mass value="0.00040746" />
+            </xacro:if>
+            <xacro:if value="${fake_walk== False}">
+                <mass value="0.40746" />
+            </xacro:if>
             <inertia ixx="0.0014813" ixy="3.1631E-07" ixz="-4.1003E-05" iyy="0.0016361" iyz="6.7483E-07" izz="0.0017353" />
         </inertial>
@@ -1062,13 +1079,16 @@
    <!-- fake controller that allows us to move the robot and to get its oposition -->
    <!-- rostopic pub /cmd_vel geometry_msgs/Twist "{ linear: [ 0.1, 0, 0], angular: [0.2, 0, 0.1] }" -->
-   <gazebo>
-    <plugin name="object_controller" filename="libgazebo_ros_planar_move.so">
-      <robotNamespace>/</robotNamespace>
-      <commandTopic>cmd_vel</commandTopic>
-      <odometryTopic>odom</odometryTopic>
-      <odometryFrame>odom</odometryFrame>
-      <odometryRate>100.0</odometryRate>
-      <robotBaseFrame>base_footprint</robotBaseFrame>
-    </plugin>
-  </gazebo>
+   <xacro:if value="${fake_walk == True}">
+   <!-- only active when fake_walk param is set to True -->
+    <gazebo>
+        <plugin name="object_controller" filename="libgazebo_ros_planar_move.so">
+        <robotNamespace>/</robotNamespace>
+        <commandTopic>cmd_vel</commandTopic>
+        <odometryTopic>odom</odometryTopic>
+        <odometryFrame>odom</odometryFrame>
+        <odometryRate>100.0</odometryRate>
+        <robotBaseFrame>base_footprint</robotBaseFrame>
+        </plugin>
+    </gazebo>
+    </xacro:if>
 </robot>

Commit message: fixed foot length and added hip z spacer in urdf and mesh

File: wolfgang_description/urdf/wolfgang.urdf.xacro (robot description, xacro)
@@ -582,5 +582,5 @@
     </joint>
     <joint name="r_foot_to_sole" type="fixed">
-        <origin xyz="0.078 -0.015 -0.039" rpy="0 0 0" />
+        <origin xyz="0.083 -0.015 -0.039" rpy="0 0 0" />
         <parent link="r_foot" />
         <child link="r_sole" />
@@ -588,5 +588,5 @@
     </joint>
     <joint name="r_foot_to_toe" type="fixed">
-        <origin xyz="0.095 0 0" rpy="0 0 0" />
+        <origin xyz="0.1 0 0" rpy="0 0 0" />
         <parent link="r_sole" />
         <child link="r_toe" />
@@ -642,5 +642,5 @@
     </joint>
     <joint name="left_foot_to_sole" type="fixed">
-        <origin xyz="0.078 0.015 -0.039" rpy="0 0 0" /> <!-- todo mit stollen!-->
+        <origin xyz="0.083 0.015 -0.039" rpy="0 0 0" />
         <parent link="l_foot" />
         <child link="l_sole" />
@@ -648,5 +648,5 @@
     </joint>
     <joint name="left_foot_to_toe" type="fixed">
-        <origin xyz="0.095 0 0" rpy="0 0 0" />
+        <origin xyz="0.1 0 0" rpy="0 0 0" />
         <parent link="l_sole" />
         <child link="l_toe" />
@@ -656,5 +656,5 @@
         <parent link="base_link" />
         <child link="torso" />
-        <origin rpy="0.0 0 0" xyz="-0.0095 0 0.0905" />
+        <origin rpy="0.0 0 0" xyz="0 0 0.0881" />
     </joint>
     <joint name="torso_to_imu" type="fixed">
@@ -669,5 +669,5 @@
     </joint>
     <joint name="RShoulderPitch" type="revolute">
-        <origin xyz="0.0 -0.075 0.11" rpy="0 0 0" />
+        <origin xyz="-0.0015 -0.076501 0.1155" rpy="0 0 0" />
         <parent link="torso" />
         <child link="r_shoulder" />
@@ -698,5 +698,5 @@
     </joint>
     <joint name="LShoulderPitch" type="revolute">
-        <origin xyz="0.0 0.075 0.11" rpy="0 0 0" />
+        <origin xyz="-0.0015 0.076501 0.1155" rpy="0 0 0" />
         <parent link="torso" />
         <child link="l_shoulder" />
@@ -727,5 +727,5 @@
     </joint>
     <joint name="HeadPan" type="revolute">
-        <origin xyz="0.00155 0 0.1471" rpy="0 0 0" />
+        <origin xyz="0.008 0 0.146501" rpy="0 0 0" />
         <parent link="torso" />
         <child link="neck" />

Commit message: fixed camera fixed

File: wolfgang_description/urdf/wolfgang.urdf.xacro (robot description, xacro)
@@ -666,5 +666,5 @@
         <parent link="torso" />
         <child link="camera_fixed" />
-        <origin rpy="0.0 0 0" xyz="0.05 0 0.279" />
+        <origin rpy="0.0 0 0" xyz="0.057 0 0.278" />
     </joint>
     <joint name="RShoulderPitch" type="revolute">

Commit message: head motor orientation in urdf

File: wolfgang_description/urdf/wolfgang.urdf.xacro (robot description, xacro)
@@ -727,5 +727,5 @@
     </joint>
     <joint name="HeadPan" type="revolute">
-        <origin xyz="0.008 0 0.146501" rpy="0 0 0" />
+        <origin xyz="-0.0095 0 0.146501" rpy="0 0 0" />
         <parent link="torso" />
         <child link="neck" />

Commit message: Fix camera_fixed offset

File: wolfgang_description/urdf/wolfgang.urdf.xacro (robot description, xacro)
@@ -666,5 +666,5 @@
         <parent link="torso" />
         <child link="camera_fixed" />
-        <origin rpy="0.0 0 0" xyz="0.057 0 0.278" />
+        <origin rpy="0.0 0 0" xyz="0.039 0 0.278" />
     </joint>
     <joint name="RShoulderPitch" type="revolute">
