Commit message: added collision model

File: wolfgang_description/urdf/wolfgang.urdf.xacro (robot description, xacro)
@@ -39,10 +39,10 @@
             <material name="black" />
         </visual>
-        <!--<collision>
-            <origin xyz="0 0 0" rpy="0 0 0" />
-            <geometry>
-                <mesh filename="package://wolfgang_description/mesh/trunk_link.dae" />
-            </geometry>
-        </collision>-->
+        <collision>
+            <origin xyz="0 0 0" rpy="0 0 0" />
+            <geometry>
+                <mesh filename="package://wolfgang_description/mesh/collision/torso_link.stl" />
+            </geometry>
+        </collision>
     </link>
     <link name="r_hip_1">
@@ -59,10 +59,10 @@
             <material name="metal" />
         </visual>
-        <!--<collision>
-            <origin xyz="0 0 0" rpy="0 0 0" />
-            <geometry>
-                <mesh filename="package://wolfgang_description/mesh/right_hip_yaw_link_collision.dae" />
-            </geometry>
-        </collision>-->
+        <collision>
+            <origin xyz="0 0 0" rpy="0 0 0" />
+            <geometry>
+                <mesh filename="package://wolfgang_description/mesh/collision/hip_connector.stl" />
+            </geometry>
+        </collision>
     </link>
     <link name="r_hip_2">
@@ -79,10 +79,10 @@
             <material name="black" />
         </visual>
-        <!--<collision>
-            <origin xyz="0 0 0" rpy="0 0 0" />
-            <geometry>
-                <mesh filename="package://wolfgang_description/mesh/right_hip_roll_link.dae" />
-            </geometry>
-        </collision>-->
+        <collision>
+            <origin xyz="0 0 0" rpy="0 0 0" />
+            <geometry>
+                <mesh filename="package://wolfgang_description/mesh/collision/hip_link_2.stl" />
+            </geometry>
+        </collision>
     </link>
     <link name="r_upper_leg">
@@ -113,10 +113,22 @@
             <material name="black" />
         </visual>
-        <!--<collision>
-            <origin xyz="0 0 0" rpy="0 0 0" />
-            <geometry>
-                <mesh filename="package://wolfgang_description/mesh/left_thigh_link.dae" />
-            </geometry>
-        </collision>-->
+        <collision>
+            <origin xyz="0 0 0" rpy="0 ${pi} 0" />
+            <geometry>
+                <mesh filename="package://wolfgang_description/mesh/collision/upper_leg_carbon.stl" />
+            </geometry>
+        </collision>
+        <collision>
+            <origin xyz="0 0 0" rpy="0 ${pi} 0" />
+            <geometry>
+                <mesh filename="package://wolfgang_description/mesh/collision/upper_leg_metal.stl" />
+            </geometry>
+        </collision>
+        <collision>
+            <origin xyz="0 0 0" rpy="0 ${pi} 0" />
+            <geometry>
+                <mesh filename="package://wolfgang_description/mesh/collision/upper_leg_motor.stl" />
+            </geometry>
+        </collision>
     </link>
     <link name="r_lower_leg">
@@ -133,10 +145,10 @@
             <material name="carbon" />
         </visual>
-        <!--<collision>
-            <origin xyz="0 0 0" rpy="0 0 0" />
-            <geometry>
-                <mesh filename="package://wolfgang_description/mesh/right_shank_link.dae" />
-            </geometry>
-        </collision>-->
+        <collision>
+            <origin xyz="0 0 0" rpy="0 0 0" />
+            <geometry>
+                <mesh filename="package://wolfgang_description/mesh/collision/lower_leg.stl" />
+            </geometry>
+        </collision>
     </link>
     <link name="r_ankle">
@@ -153,10 +165,10 @@
             <material name="black" />
         </visual>
-        <!--<collision>
-            <origin xyz="0 0 0" rpy="0 0 0" />
-            <geometry>
-                <mesh filename="package://wolfgang_description/mesh/right_ankle_link.dae" />
-            </geometry>
-        </collision>-->
+        <collision>
+            <origin xyz="0 0 0" rpy="0 0 0" />
+            <geometry>
+                <mesh filename="package://wolfgang_description/mesh/collision/ankle.stl" />
+            </geometry>
+        </collision>
     </link>
     <link name="r_foot">
@@ -178,5 +190,5 @@
                 <origin xyz="0 0 -0.012" rpy="0 0 0" />
                 <geometry>
-                    <mesh filename="package://wolfgang_description/mesh/right_foot.stl" />
+                    <mesh filename="package://wolfgang_description/mesh/collision/right_foot.stl" />
                 </geometry>
             </collision>
@@ -210,10 +222,10 @@
             <material name="metal" />
         </visual>
-        <!--<collision>
-            <origin xyz="0 0 0" rpy="0 0 0" />
-            <geometry>
-                <mesh filename="package://wolfgang_description/mesh/left_hip_yaw_link.dae" />
-            </geometry>
-        </collision>-->
+        <collision>
+            <origin xyz="0 0 0" rpy="0 0 0" />
+            <geometry>
+                <mesh filename="package://wolfgang_description/mesh/collision/hip_connector.stl" />
+            </geometry>
+        </collision>
     </link>
     <link name="l_hip_2">
@@ -230,10 +242,10 @@
             <material name="black" />
         </visual>
-        <!--<collision>
-            <origin xyz="0.033 0 0" rpy="0 0 0" />
-            <geometry>
-                <mesh filename="package://wolfgang_description/mesh/left_hip_roll_link.dae" />
-            </geometry>
-        </collision>-->
+        <collision>
+            <origin xyz="0 0 0" rpy="0 0 0" />
+            <geometry>
+                <mesh filename="package://wolfgang_description/mesh/collision/hip_link_2.stl" />
+            </geometry>
+        </collision>
     </link>
     <link name="l_upper_leg">
@@ -264,10 +276,22 @@
             <material name="metal" />
         </visual>
-        <!--<collision>
-            <origin xyz="0 0 0" rpy="0 0 0" />
-            <geometry>
-                <mesh filename="package://wolfgang_description/mesh/left_thigh_link.dae" />
-            </geometry>
-        </collision>-->
+        <collision>
+            <origin xyz="0 0 0" rpy="0 ${pi} 0" />
+            <geometry>
+                <mesh filename="package://wolfgang_description/mesh/collision/upper_leg_carbon.stl" />
+            </geometry>
+        </collision>
+        <collision>
+            <origin xyz="0 0 0" rpy="0 ${pi} 0" />
+            <geometry>
+                <mesh filename="package://wolfgang_description/mesh/collision/upper_leg_metal.stl" />
+            </geometry>
+        </collision>
+        <collision>
+            <origin xyz="0 0 0" rpy="0 ${pi} 0" />
+            <geometry>
+                <mesh filename="package://wolfgang_description/mesh/collision/upper_leg_motor.stl" />
+            </geometry>
+        </collision>
     </link>
     <link name="l_lower_leg">
@@ -284,10 +308,10 @@
             <material name="carbon" />
         </visual>
-        <!--<collision>
-            <origin xyz="0 0 0" rpy="0 0 0" />
-            <geometry>
-                <mesh filename="package://wolfgang_description/mesh/left_shank_link.dae" />
-            </geometry>
-        </collision>-->
+        <collision>
+            <origin xyz="0 0 0" rpy="0 0 0" />
+            <geometry>
+                <mesh filename="package://wolfgang_description/mesh/collision/lower_leg.stl" />
+            </geometry>
+        </collision>
     </link>
     <link name="l_ankle">
@@ -304,10 +328,11 @@
             <material name="black" />
         </visual>
-        <!--<collision>
-            <origin xyz="0 0 0" rpy="0 0 0" />
-            <geometry>
-                <mesh filename="package://wolfgang_description/mesh/left_ankle_link.dae" />
-            </geometry>
-        </collision>-->
+        <collision>
+            <origin xyz="0 0 0" rpy="0 0 0" />
+            <geometry>
+                <mesh filename="package://wolfgang_description/mesh/collision/ankle.stl" />
+            </geometry>
+            <material name="metal" />
+        </collision>
     </link>
     <link name="l_foot">
@@ -329,5 +354,5 @@
                 <origin xyz="0 0 -0.012" rpy="0 0 0" />
                 <geometry>
-                    <mesh filename="package://wolfgang_description/mesh/left_foot.stl" />
+                    <mesh filename="package://wolfgang_description/mesh/collision/left_foot.stl" />
                 </geometry>
             </collision>
@@ -361,10 +386,10 @@
             <material name="metal" />
         </visual>
-        <!--<collision>
-            <origin xyz="0 0 0" rpy="0 0 0" />
-            <geometry>
-                <mesh filename="package://wolfgang_description/mesh/right_shoulder_pitch_link.dae" />
-            </geometry>
-        </collision>-->
+        <collision>
+            <origin xyz="0 0 0" rpy="0 0 ${pi}" />
+            <geometry>
+                <mesh filename="package://wolfgang_description/mesh/collision/shoulder.stl" />
+            </geometry>
+        </collision>
     </link>
     <link name="r_upper_arm">
@@ -381,10 +406,10 @@
             <material name="black" />
         </visual>
-        <!--<collision>
-            <origin xyz="0 0 0" rpy="0 0 0" />
-            <geometry>
-                <mesh filename="package://wolfgang_description/mesh/right_shoulder_arm_link.dae" />
-            </geometry>
-        </collision>-->
+        <collision>
+            <origin xyz="0 0 0" rpy="0 ${pi} 0" />
+            <geometry>
+                <mesh filename="package://wolfgang_description/mesh/collision/upper_arm.stl" />
+            </geometry>
+        </collision>
     </link>
     <link name="r_lower_arm">
@@ -401,10 +426,10 @@
             <material name="black" />
         </visual>
-        <!--<collision>
-            <origin xyz="0 0 0" rpy="0 -1.57 0" />
-            <geometry>
-                <mesh filename="package://wolfgang_description/mesh/right_lower_arm_link.dae" />
-            </geometry>
-        </collision>-->
+        <collision>
+            <origin xyz="0 0 0" rpy="0 0 0" />
+            <geometry>
+                <mesh filename="package://wolfgang_description/mesh/collision/lower_arm.stl" />
+            </geometry>
+        </collision>
     </link>
     <link name="r_wrist"> </link>
@@ -422,10 +447,10 @@
             <material name="metal" />
         </visual>
-        <!--<collision>
-            <origin xyz="0 0 0" rpy="0 0 0" />
-            <geometry>
-                <mesh filename="package://wolfgang_description/mesh/left_shoulder_pitch_link.dae" />
-            </geometry>
-        </collision>-->
+        <collision>
+            <origin xyz="0 0 0" rpy="0 0 0" />
+            <geometry>
+                <mesh filename="package://wolfgang_description/mesh/collision/shoulder.stl" />
+            </geometry>
+        </collision>
     </link>
     <link name="l_upper_arm">
@@ -442,10 +467,10 @@
             <material name="black" />
         </visual>
-        <!--<collision>
-            <origin xyz="0 0 0" rpy="0 0 0" />
-            <geometry>
-                <mesh filename="package://wolfgang_description/mesh/left_upper_arm_link.dae" />
-            </geometry>
-        </collision>-->
+        <collision>
+            <origin xyz="0 0 0" rpy="0 ${pi} 0" />
+            <geometry>
+                <mesh filename="package://wolfgang_description/mesh/collision/upper_arm.stl" />
+            </geometry>
+        </collision>
     </link>
     <link name="l_lower_arm">
@@ -462,10 +487,10 @@
             <material name="black" />
         </visual>
-        <!--<collision>
-            <origin xyz="0 0 0" rpy="0 -1.57 0" />
-            <geometry>
-                <mesh filename="package://wolfgang_description/mesh/left_lower_arm_link.dae" />
-            </geometry>
-        </collision>-->
+        <collision>
+            <origin xyz="0 0 0" rpy="0 0 0" />
+            <geometry>
+                <mesh filename="package://wolfgang_description/mesh/collision/lower_arm.stl" />
+            </geometry>
+        </collision>
     </link>
     <link name="l_wrist"> </link>
@@ -488,10 +513,10 @@
             <material name="black" />
         </visual>
-        <!--<collision>
-            <origin xyz="0 0 0" rpy="0 0 0" />
-            <geometry>
-                <mesh filename="package://wolfgang_description/mesh/neck_link.dae" />
-            </geometry>
-        </collision>-->
+        <collision>
+            <origin xyz="0 0 0" rpy="0 0 ${pi}" />
+            <geometry>
+                <mesh filename="package://wolfgang_description/mesh/collision/neck.stl" />
+            </geometry>
+        </collision>
     </link>
     <link name="camera" />
@@ -518,5 +543,5 @@
             <inertia ixx="0.0014813" ixy="3.1631E-07" ixz="-4.1003E-05" iyy="0.0016361" iyz="6.7483E-07" izz="0.0017353" />
         </inertial>
-        <!--<visual>
+        <visual>
             <origin xyz="0 0 0" rpy="0 0 0" />
             <geometry>
@@ -524,11 +549,11 @@
             </geometry>
             <material name="black" />
-        </visual>-->
-        <!--<collision>
-            <origin xyz="0 0 0" rpy="0 0 0" />
-            <geometry>
-                <mesh filename="package://wolfgang_description/mesh/head_link.dae" />
-            </geometry>
-        </collision>-->
+        </visual>
+        <collision>
+            <origin xyz="0 0 0" rpy="0 0 0" />
+            <geometry>
+                <mesh filename="package://wolfgang_description/mesh/collision/head.stl" />
+            </geometry>
+        </collision>
     </link>
     <!-- JOINTS JOINTS JOINTS JOINTS JOINTS JOINTS JOINTS JOINTS JOINTS JOINTS -->

Commit message: Remove camera_fixed frame

File: wolfgang_description/urdf/wolfgang.urdf.xacro (robot description, xacro)
@@ -522,5 +522,4 @@
     <link name="camera" />
     <link name="camera_optical_frame"/>
-    <link name="camera_fixed"/>
     <link name="imu_frame" />
     <link name="l_cleat_l_front"/>
@@ -687,9 +686,4 @@
         <child link="imu_frame" />
         <origin rpy="0.0 0 0" xyz="-0.045 0.025 0.023" />
-    </joint>
-    <joint name="torso_to_camera_fixed" type="fixed">
-        <parent link="torso" />
-        <child link="camera_fixed" />
-        <origin rpy="0.0 0 0" xyz="0.039 0 0.278" />
     </joint>
     <joint name="RShoulderPitch" type="revolute">

Commit message: fixed angle induced by upper_leg part

File: wolfgang_description/urdf/wolfgang.urdf.xacro (robot description, xacro)
@@ -139,5 +139,5 @@
         </inertial>
         <visual>
-            <origin xyz="0 0 0" rpy="0 0 0" />
+            <origin xyz="0 0 0" rpy="0 ${-pi/4} 0" />
             <geometry>
                 <mesh filename="package://wolfgang_description/mesh/lower_leg.stl" />
@@ -146,5 +146,5 @@
         </visual>
         <collision>
-            <origin xyz="0 0 0" rpy="0 0 0" />
+            <origin xyz="0 0 0" rpy="0 ${-pi/4} 0" />
             <geometry>
                 <mesh filename="package://wolfgang_description/mesh/collision/lower_leg.stl" />
@@ -302,5 +302,5 @@
         </inertial>
         <visual>
-            <origin xyz="0 0 0" rpy="0 0 0" />
+            <origin xyz="0 0 0" rpy="0 ${-pi/4} 0" />
             <geometry>
                 <mesh filename="package://wolfgang_description/mesh/lower_leg.stl" />
@@ -309,5 +309,5 @@
         </visual>
         <collision>
-            <origin xyz="0 0 0" rpy="0 0 0" />
+            <origin xyz="0 0 0" rpy="0 ${-pi/4} 0" />
             <geometry>
                 <mesh filename="package://wolfgang_description/mesh/collision/lower_leg.stl" />
@@ -582,5 +582,5 @@
     </joint>
     <joint name="RKnee" type="revolute">
-        <origin xyz="-0.004 0 -0.1692" rpy="0 0 0" />
+        <origin xyz="-0.004 0 -0.1692" rpy="0 ${pi/6} 0" />
         <parent link="r_upper_leg" />
         <child link="r_lower_leg" />
@@ -590,5 +590,5 @@
     </joint>
     <joint name="RAnklePitch" type="revolute">
-        <origin xyz="0.0 0 -0.17" rpy="0 0 0" />
+        <origin xyz="0.120208 0 -0.120208" rpy="0 ${-pi/4} 0" />
         <parent link="r_lower_leg" />
         <child link="r_ankle" />
@@ -642,5 +642,5 @@
     </joint>
     <joint name="LKnee" type="revolute">
-        <origin xyz="-0.004 0 -0.1692" rpy="0 0 0" />
+        <origin xyz="-0.004 0 -0.1692" rpy="0 ${pi/6} 0" />
         <parent link="l_upper_leg" />
         <child link="l_lower_leg" />
@@ -650,5 +650,5 @@
     </joint>
     <joint name="LAnklePitch" type="revolute">
-        <origin xyz="0.0 0 -0.17" rpy="0 0 0" />
+        <origin xyz="0.120208 0 -0.120208" rpy="0 ${-pi/4} 0" />
         <parent link="l_lower_leg" />
         <child link="l_ankle" />
@@ -768,5 +768,5 @@
         <dynamics damping="${d}" friction="${f}" />
     </joint>
-	<joint name="camera__optical_joint" type="fixed">
+    <joint name="camera__optical_joint" type="fixed">
       <origin xyz="0 0 0" rpy="${-pi/2} 0 ${-pi/2}" />
       <parent link="camera" />
