Commit message: update effort, velocity

File: wolfgang_description/urdf/wolfgang.urdf.xacro (robot description, xacro)
@@ -586,5 +586,5 @@
         <child link="r_hip_1" />
         <axis xyz="0 0 -1" />
-        <limit effort="${tofa*2.5}" velocity="5.6548668" lower="-0.9250245035547" upper="0.9250245035547" />
+        <limit effort="10.0" velocity="5,759586525" lower="-0.9250245035547" upper="0.9250245035547" />
         <dynamics damping="${d}" friction="${f}" />
     </joint>
@@ -594,5 +594,5 @@
         <child link="r_hip_2" />
         <axis xyz="1 0 0" />
-        <limit effort="${tofa*6.0}" velocity="6.597344565" lower="-1.57" upper="0.7853981633955001" />
+        <limit effort="10.0" velocity="5,759586525" lower="-1.57" upper="0.7853981633955001" />
         <dynamics damping="${d}" friction="${f}" />
     </joint>
@@ -602,5 +602,5 @@
         <child link="r_upper_leg" />
         <axis xyz="0 1 0" />
-        <limit effort="${tofa*8.4}" velocity="4.712388975" lower="-1.919862177189" upper="0.48869219055720003" />
+        <limit effort="10.0" velocity="5,759586525" lower="-1.919862177189" upper="0.48869219055720003" />
         <dynamics damping="${d}" friction="${f}" />
     </joint>
@@ -610,5 +610,5 @@
         <child link="r_lower_leg" />
         <axis xyz="0 1 0" />
-        <limit effort="${tofa*8.4}" velocity="4.712388975" lower="0" upper="2.268928027587" />
+        <limit effort="10.0" velocity="4.712388975" lower="0" upper="2.268928027587" />
         <dynamics damping="${d}" friction="${f}" />
     </joint>
@@ -618,5 +618,5 @@
         <child link="r_ankle" />
         <axis xyz="0 -1 0" />
-        <limit effort="${tofa*8.4}" velocity="4.712388975" lower="-1.2391837689129" upper="1.6406094968706" />
+        <limit effort="10.0" velocity="5,759586525" lower="-1.2391837689129" upper="1.6406094968706" />
         <dynamics damping="${d}" friction="${f}" />
     </joint>
@@ -626,5 +626,5 @@
         <child link="r_foot" />
         <axis xyz="-1 0 0" />
-        <limit effort="${tofa*6.0}" velocity="6.597344565" lower="-1.4660765716716" upper="1.4660765716716" />
+        <limit effort="10.0" velocity="5,759586525" lower="-1.4660765716716" upper="1.4660765716716" />
         <dynamics damping="${d}" friction="${f}" />
     </joint>
@@ -646,5 +646,5 @@
         <child link="l_hip_1" />
         <axis xyz="0 0 -1" />
-        <limit effort="${tofa*2.5}" velocity="5.6548668" lower="-0.9250245035547" upper="0.9250245035547" />
+        <limit effort="10.0" velocity="5,759586525" lower="-0.9250245035547" upper="0.9250245035547" />
         <dynamics damping="${d}" friction="${f}" />
     </joint>
@@ -654,5 +654,5 @@
         <child link="l_hip_2" />
         <axis xyz="1 0 0" />
-        <limit effort="${tofa*6.0}" velocity="6.597344565" lower="-0.7853981633955001" upper="1.57" />
+        <limit effort="10.0" velocity="5,759586525" lower="-0.7853981633955001" upper="1.57" />
         <dynamics damping="${d}" friction="${f}" />
     </joint>
@@ -662,5 +662,5 @@
         <child link="l_upper_leg" />
         <axis xyz="0 -1 0" />
-        <limit effort="${tofa*8.4}" velocity="4.712388975" lower="-0.48869219055720003" upper="1.919862177189" />
+        <limit effort="10.0" velocity="5,759586525" lower="-0.48869219055720003" upper="1.919862177189" />
         <dynamics damping="${d}" friction="${f}" />
     </joint>
@@ -670,5 +670,5 @@
         <child link="l_lower_leg" />
         <axis xyz="0 -1 0" />
-        <limit effort="${tofa*8.4}" velocity="4.712388975" lower="-2.268928027587" upper="0" />
+        <limit effort="10.0" velocity="5,759586525" lower="-2.268928027587" upper="0" />
         <dynamics damping="${d}" friction="${f}" />
     </joint>
@@ -678,5 +678,5 @@
         <child link="l_ankle" />
         <axis xyz="0 1 0" />
-        <limit effort="${tofa*8.4}" velocity="4.712388975" lower="-1.6406094968706" upper="1.2391837689129" />
+        <limit effort="10.0" velocity="5,759586525" lower="-1.6406094968706" upper="1.2391837689129" />
         <dynamics damping="${d}" friction="${f}" />
     </joint>
@@ -686,5 +686,5 @@
         <child link="l_foot" />
         <axis xyz="-1 0 0" />
-        <limit effort="${tofa*6.0}" velocity="6.597344565" lower="-1.4660765716716" upper="1.4660765716716" />
+        <limit effort="10.0" velocity="5,759586525" lower="-1.4660765716716" upper="1.4660765716716" />
         <dynamics damping="${d}" friction="${f}" />
     </joint>
@@ -716,5 +716,5 @@
         <child link="r_shoulder" />
         <axis xyz="0 -1 0" />
-        <limit effort="${tofa*6.0}" velocity="6.597344565" lower="-3.1415926535820002" upper="3.1415926535820002" />
+        <limit effort="7.3" velocity="8,16814089" lower="-3.1415926535820002" upper="3.1415926535820002" />
         <dynamics damping="${d}" friction="${f}" />
     </joint>
@@ -724,5 +724,5 @@
         <child link="r_upper_arm" />
         <axis xyz="-1 0 0" />
-        <limit effort="${tofa*2.5}" velocity="5.648668" lower="-0.7853981633955001" upper="2.3561944901865" />
+        <limit effort="7.3" velocity="8,16814089" lower="-0.7853981633955001" upper="2.3561944901865" />
         <dynamics damping="${d}" friction="${f}" />
     </joint>
@@ -732,5 +732,5 @@
         <child link="r_lower_arm" />
         <axis xyz="0 1 0" />
-        <limit effort="${tofa*2.5}" velocity="5.6548668" lower="-1.635" upper="1.5707963267910001" />
+        <limit effort="7.3" velocity="8,16814089" lower="-1.635" upper="1.5707963267910001" />
         <dynamics damping="${d}" friction="${f}" />
     </joint>
@@ -745,5 +745,5 @@
         <child link="l_shoulder" />
         <axis xyz="0 1 0" />
-        <limit effort="${tofa*6.0}" velocity="6.597344565" lower="-3.1415926535820002" upper="3.1415926535820002" />
+        <limit effort="7.3" velocity="8,16814089" lower="-3.1415926535820002" upper="3.1415926535820002" />
         <dynamics damping="${d}" friction="${f}" />
     </joint>
@@ -753,5 +753,5 @@
         <child link="l_upper_arm" />
         <axis xyz="-1 0 0" />
-        <limit effort="${tofa*2.5}" velocity="5.648668" lower="-2.3561944901865" upper="0.7853981633955001" />
+        <limit effort="7.3" velocity="8,16814089" lower="-2.3561944901865" upper="0.7853981633955001" />
         <dynamics damping="${d}" friction="${f}" />
     </joint>
@@ -761,5 +761,5 @@
         <child link="l_lower_arm" />
         <axis xyz="0 -1 0" />
-        <limit effort="${tofa*2.5}" velocity="5.6548668" lower="-1.1344640137935" upper="1.5707963267910001" />
+        <limit effort="7.3" velocity="8,16814089" lower="-1.1344640137935" upper="1.5707963267910001" />
         <dynamics damping="${d}" friction="${f}" />
     </joint>
@@ -774,5 +774,5 @@
         <child link="neck" />
         <axis xyz="0 0 1" />
-        <limit effort="${tofa*2.5}" velocity="5.6548668" lower="-1.2" upper="1.2" />
+        <limit effort="7.3" velocity="8,16814089" lower="-1.2" upper="1.2" />
         <dynamics damping="${d}" friction="${f}" />
     </joint>
@@ -782,5 +782,5 @@
         <child link="head" />
         <axis xyz="0 -1 0" />
-        <limit effort="${tofa*2.5}" velocity="5.6548668" lower="-1.2" upper="0.2" />
+        <limit effort="7.3" velocity="8,16814089" lower="-1.2" upper="0.2" />
         <dynamics damping="${d}" friction="${f}" />
     </joint>

Commit message: typo fix

File: wolfgang_description/urdf/wolfgang.urdf.xacro (robot description, xacro)
@@ -716,5 +716,5 @@
         <child link="r_shoulder" />
         <axis xyz="0 -1 0" />
-        <limit effort="7.3" velocity="8,16814089" lower="-3.1415926535820002" upper="3.1415926535820002" />
+        <limit effort="7.3" velocity="8.16814089" lower="-3.1415926535820002" upper="3.1415926535820002" />
         <dynamics damping="${d}" friction="${f}" />
     </joint>
@@ -724,5 +724,5 @@
         <child link="r_upper_arm" />
         <axis xyz="-1 0 0" />
-        <limit effort="7.3" velocity="8,16814089" lower="-0.7853981633955001" upper="2.3561944901865" />
+        <limit effort="7.3" velocity="8.16814089" lower="-0.7853981633955001" upper="2.3561944901865" />
         <dynamics damping="${d}" friction="${f}" />
     </joint>
@@ -732,5 +732,5 @@
         <child link="r_lower_arm" />
         <axis xyz="0 1 0" />
-        <limit effort="7.3" velocity="8,16814089" lower="-1.635" upper="1.5707963267910001" />
+        <limit effort="7.3" velocity="8.16814089" lower="-1.635" upper="1.5707963267910001" />
         <dynamics damping="${d}" friction="${f}" />
     </joint>
@@ -745,5 +745,5 @@
         <child link="l_shoulder" />
         <axis xyz="0 1 0" />
-        <limit effort="7.3" velocity="8,16814089" lower="-3.1415926535820002" upper="3.1415926535820002" />
+        <limit effort="7.3" velocity="8.16814089" lower="-3.1415926535820002" upper="3.1415926535820002" />
         <dynamics damping="${d}" friction="${f}" />
     </joint>
@@ -753,5 +753,5 @@
         <child link="l_upper_arm" />
         <axis xyz="-1 0 0" />
-        <limit effort="7.3" velocity="8,16814089" lower="-2.3561944901865" upper="0.7853981633955001" />
+        <limit effort="7.3" velocity="8.16814089" lower="-2.3561944901865" upper="0.7853981633955001" />
         <dynamics damping="${d}" friction="${f}" />
     </joint>
@@ -761,5 +761,5 @@
         <child link="l_lower_arm" />
         <axis xyz="0 -1 0" />
-        <limit effort="7.3" velocity="8,16814089" lower="-1.1344640137935" upper="1.5707963267910001" />
+        <limit effort="7.3" velocity="8.16814089" lower="-1.1344640137935" upper="1.5707963267910001" />
         <dynamics damping="${d}" friction="${f}" />
     </joint>
@@ -774,5 +774,5 @@
         <child link="neck" />
         <axis xyz="0 0 1" />
-        <limit effort="7.3" velocity="8,16814089" lower="-1.2" upper="1.2" />
+        <limit effort="7.3" velocity="8.16814089" lower="-1.2" upper="1.2" />
         <dynamics damping="${d}" friction="${f}" />
     </joint>
@@ -782,5 +782,5 @@
         <child link="head" />
         <axis xyz="0 -1 0" />
-        <limit effort="7.3" velocity="8,16814089" lower="-1.2" upper="0.2" />
+        <limit effort="7.3" velocity="8.16814089" lower="-1.2" upper="0.2" />
         <dynamics damping="${d}" friction="${f}" />
     </joint>

Commit message: Typos fixed

File: wolfgang_description/urdf/wolfgang.urdf.xacro (robot description, xacro)
@@ -586,5 +586,5 @@
         <child link="r_hip_1" />
         <axis xyz="0 0 -1" />
-        <limit effort="10.0" velocity="5,759586525" lower="-0.9250245035547" upper="0.9250245035547" />
+        <limit effort="10.0" velocity="5.759586525" lower="-0.9250245035547" upper="0.9250245035547" />
         <dynamics damping="${d}" friction="${f}" />
     </joint>
@@ -594,5 +594,5 @@
         <child link="r_hip_2" />
         <axis xyz="1 0 0" />
-        <limit effort="10.0" velocity="5,759586525" lower="-1.57" upper="0.7853981633955001" />
+        <limit effort="10.0" velocity="5.759586525" lower="-1.57" upper="0.7853981633955001" />
         <dynamics damping="${d}" friction="${f}" />
     </joint>
@@ -602,5 +602,5 @@
         <child link="r_upper_leg" />
         <axis xyz="0 1 0" />
-        <limit effort="10.0" velocity="5,759586525" lower="-1.919862177189" upper="0.48869219055720003" />
+        <limit effort="10.0" velocity="5.759586525" lower="-1.919862177189" upper="0.48869219055720003" />
         <dynamics damping="${d}" friction="${f}" />
     </joint>
@@ -610,5 +610,5 @@
         <child link="r_lower_leg" />
         <axis xyz="0 1 0" />
-        <limit effort="10.0" velocity="4.712388975" lower="0" upper="2.268928027587" />
+        <limit effort="10.0" velocity="5.759586525" lower="0" upper="2.268928027587" />
         <dynamics damping="${d}" friction="${f}" />
     </joint>
@@ -618,5 +618,5 @@
         <child link="r_ankle" />
         <axis xyz="0 -1 0" />
-        <limit effort="10.0" velocity="5,759586525" lower="-1.2391837689129" upper="1.6406094968706" />
+        <limit effort="10.0" velocity="5.759586525" lower="-1.2391837689129" upper="1.6406094968706" />
         <dynamics damping="${d}" friction="${f}" />
     </joint>
@@ -626,5 +626,5 @@
         <child link="r_foot" />
         <axis xyz="-1 0 0" />
-        <limit effort="10.0" velocity="5,759586525" lower="-1.4660765716716" upper="1.4660765716716" />
+        <limit effort="10.0" velocity="5.759586525" lower="-1.4660765716716" upper="1.4660765716716" />
         <dynamics damping="${d}" friction="${f}" />
     </joint>
@@ -646,5 +646,5 @@
         <child link="l_hip_1" />
         <axis xyz="0 0 -1" />
-        <limit effort="10.0" velocity="5,759586525" lower="-0.9250245035547" upper="0.9250245035547" />
+        <limit effort="10.0" velocity="5.759586525" lower="-0.9250245035547" upper="0.9250245035547" />
         <dynamics damping="${d}" friction="${f}" />
     </joint>
@@ -654,5 +654,5 @@
         <child link="l_hip_2" />
         <axis xyz="1 0 0" />
-        <limit effort="10.0" velocity="5,759586525" lower="-0.7853981633955001" upper="1.57" />
+        <limit effort="10.0" velocity="5.759586525" lower="-0.7853981633955001" upper="1.57" />
         <dynamics damping="${d}" friction="${f}" />
     </joint>
@@ -662,5 +662,5 @@
         <child link="l_upper_leg" />
         <axis xyz="0 -1 0" />
-        <limit effort="10.0" velocity="5,759586525" lower="-0.48869219055720003" upper="1.919862177189" />
+        <limit effort="10.0" velocity="5.759586525" lower="-0.48869219055720003" upper="1.919862177189" />
         <dynamics damping="${d}" friction="${f}" />
     </joint>
@@ -670,5 +670,5 @@
         <child link="l_lower_leg" />
         <axis xyz="0 -1 0" />
-        <limit effort="10.0" velocity="5,759586525" lower="-2.268928027587" upper="0" />
+        <limit effort="10.0" velocity="5.759586525" lower="-2.268928027587" upper="0" />
         <dynamics damping="${d}" friction="${f}" />
     </joint>
@@ -678,5 +678,5 @@
         <child link="l_ankle" />
         <axis xyz="0 1 0" />
-        <limit effort="10.0" velocity="5,759586525" lower="-1.6406094968706" upper="1.2391837689129" />
+        <limit effort="10.0" velocity="5.759586525" lower="-1.6406094968706" upper="1.2391837689129" />
         <dynamics damping="${d}" friction="${f}" />
     </joint>
@@ -686,5 +686,5 @@
         <child link="l_foot" />
         <axis xyz="-1 0 0" />
-        <limit effort="10.0" velocity="5,759586525" lower="-1.4660765716716" upper="1.4660765716716" />
+        <limit effort="10.0" velocity="5.759586525" lower="-1.4660765716716" upper="1.4660765716716" />
         <dynamics damping="${d}" friction="${f}" />
     </joint>

Commit message: Change urdf for basler camera.

File: wolfgang_description/urdf/wolfgang.urdf.xacro (robot description, xacro)
@@ -762,5 +762,5 @@
     </joint>
     <joint name="head_to_camera" type="fixed">
-        <origin xyz="0.02 0 0.1115" rpy="0 0 0" />
+        <origin xyz="-0.00443 0 0.11475" rpy="0 0 0" />
         <parent link="head" />
         <child link="camera" />
@@ -1043,4 +1043,5 @@
     </gazebo>
   <!-- camera sensor -->
+  <!-- TODO basler sensor-->
   <gazebo reference="camera">
         <sensor name='camera' type='camera'>

Commit message: changed robot color in gazebo to black

File: wolfgang_description/urdf/wolfgang.urdf.xacro (robot description, xacro)
@@ -19,4 +19,7 @@
     </material>
     <link name="base_link" />
+    <gazebo reference="torso">
+        <material>Gazebo/FlatBlack</material>
+    </gazebo>
     <link name="torso">
         <inertial>
@@ -46,4 +49,7 @@
         </collision>
     </link>
+    <gazebo reference="r_hip_1">
+        <material>Gazebo/FlatBlack</material>
+    </gazebo>
     <link name="r_hip_1">
         <inertial>
@@ -66,4 +72,7 @@
         </collision>
     </link>
+    <gazebo reference="r_hip_2">
+        <material>Gazebo/FlatBlack</material>
+    </gazebo>
     <link name="r_hip_2">
         <inertial>
@@ -86,4 +95,7 @@
         </collision>
     </link>
+    <gazebo reference="r_upper_leg">
+        <material>Gazebo/FlatBlack</material>
+    </gazebo>
     <link name="r_upper_leg">
         <inertial>
@@ -132,4 +144,7 @@
         </collision>
     </link>
+    <gazebo reference="r_lower_leg">
+        <material>Gazebo/FlatBlack</material>
+    </gazebo>
     <link name="r_lower_leg">
         <inertial>
@@ -152,4 +167,7 @@
         </collision>
     </link>
+    <gazebo reference="r_ankle">
+        <material>Gazebo/FlatBlack</material>
+    </gazebo>
     <link name="r_ankle">
         <inertial>
@@ -172,4 +190,7 @@
         </collision>
     </link>
+    <gazebo reference="r_foot">
+        <material>Gazebo/FlatBlack</material>
+    </gazebo>
     <link name="r_foot">
         <inertial>
@@ -202,4 +223,7 @@
         </inertial>
     </link>
+    <gazebo reference="r_toe">
+        <material>Gazebo/FlatBlack</material>
+    </gazebo>
     <link name="r_toe">
         <inertial>
@@ -209,4 +233,7 @@
         </inertial>
     </link>
+    <gazebo reference="l_hip_1">
+        <material>Gazebo/FlatBlack</material>
+    </gazebo>
     <link name="l_hip_1">
         <inertial>
@@ -229,4 +256,7 @@
         </collision>
     </link>
+    <gazebo reference="l_hip_2">
+        <material>Gazebo/FlatBlack</material>
+    </gazebo>
     <link name="l_hip_2">
         <inertial>
@@ -249,4 +279,7 @@
         </collision>
     </link>
+    <gazebo reference="l_upper_leg">
+        <material>Gazebo/FlatBlack</material>
+    </gazebo>
     <link name="l_upper_leg">
         <inertial>
@@ -295,4 +328,7 @@
         </collision>
     </link>
+    <gazebo reference="l_lower_leg">
+        <material>Gazebo/FlatBlack</material>
+    </gazebo>
     <link name="l_lower_leg">
         <inertial>
@@ -315,4 +351,7 @@
         </collision>
     </link>
+    <gazebo reference="l_ankle">
+        <material>Gazebo/FlatBlack</material>
+    </gazebo>
     <link name="l_ankle">
         <inertial>
@@ -336,4 +375,7 @@
         </collision>
     </link>
+    <gazebo reference="l_foot">
+        <material>Gazebo/FlatBlack</material>
+    </gazebo>
     <link name="l_foot">
         <inertial>
@@ -359,4 +401,7 @@
         </xacro:if>
     </link>
+    <gazebo reference="l_sole">
+        <material>Gazebo/FlatBlack</material>
+    </gazebo>
     <link name="l_sole">
         <inertial>
@@ -366,4 +411,7 @@
         </inertial>
     </link>
+    <gazebo reference="l_toe">
+        <material>Gazebo/FlatBlack</material>
+    </gazebo>
     <link name="l_toe">
         <inertial>
@@ -373,4 +421,7 @@
         </inertial>
     </link>
+    <gazebo reference="r_shoulder">
+        <material>Gazebo/FlatBlack</material>
+    </gazebo>
     <link name="r_shoulder">
         <inertial>
@@ -393,4 +444,7 @@
         </collision>
     </link>
+    <gazebo reference="r_upper_arm">
+        <material>Gazebo/FlatBlack</material>
+    </gazebo>
     <link name="r_upper_arm">
         <inertial>
@@ -413,4 +467,7 @@
         </collision>
     </link>
+    <gazebo reference="r_lower_arm">
+        <material>Gazebo/FlatBlack</material>
+    </gazebo>
     <link name="r_lower_arm">
         <inertial>
@@ -434,4 +491,7 @@
     </link>
     <link name="r_wrist"> </link>
+    <gazebo reference="l_shoulder">
+        <material>Gazebo/FlatBlack</material>
+    </gazebo>
     <link name="l_shoulder">
         <inertial>
@@ -454,4 +514,7 @@
         </collision>
     </link>
+    <gazebo reference="l_upper_arm">
+        <material>Gazebo/FlatBlack</material>
+    </gazebo>
     <link name="l_upper_arm">
         <inertial>
@@ -474,4 +537,7 @@
         </collision>
     </link>
+    <gazebo reference="l_lower_arm">
+        <material>Gazebo/FlatBlack</material>
+    </gazebo>
     <link name="l_lower_arm">
         <inertial>
@@ -495,4 +561,7 @@
     </link>
     <link name="l_wrist"> </link>
+    <gazebo reference="neck">
+        <material>Gazebo/FlatBlack</material>
+    </gazebo>
     <link name="neck">
         <inertial>
@@ -531,4 +600,7 @@
     <link name="r_cleat_l_back"/>
     <link name="r_cleat_r_back"/>
+    <gazebo reference="head">
+        <material>Gazebo/FlatBlack</material>
+    </gazebo>
     <link name="head">
         <inertial>
@@ -1017,5 +1089,5 @@
     </transmission>
     <gazebo reference="r_foot">
-        <material>gazebo/Grey</material>
+        <material>Gazebo/FlatBlack</material>
         <kp>1000000.0</kp>
         <kd>100.0</kd>
@@ -1027,5 +1099,5 @@
     </gazebo>
     <gazebo reference="l_foot">
-        <material>gazebo/Grey</material>
+        <material>Gazebo/FlatBlack</material>
         <kp>1000000.0</kp>
         <kd>100.0</kd>
