Commit message: limits and dynamics tag of joints updated

File: wolfgang_description/urdf/wolfgang.urdf.xacro (robot description, xacro)
@@ -586,6 +586,6 @@
         <child link="r_hip_1" />
         <axis xyz="0 0 -1" />
-        <limit effort="10.0" velocity="5.759586525" lower="-0.9250245035547" upper="0.9250245035547" />
-        <dynamics damping="${d}" friction="${f}" />
+        <limit effort="7.57" velocity="8.22" lower="-0.9250245035547" upper="0.9250245035547" />
+        <dynamics damping="${d}" friction="0.1" />
     </joint>
     <joint name="RHipRoll" type="revolute">
@@ -594,6 +594,6 @@
         <child link="r_hip_2" />
         <axis xyz="1 0 0" />
-        <limit effort="10.0" velocity="5.759586525" lower="-1.57" upper="0.7853981633955001" />
-        <dynamics damping="${d}" friction="${f}" />
+        <limit effort="7.57" velocity="8.22" lower="-1.57" upper="0.7853981633955001" />
+        <dynamics damping="${d}" friction="0.1" />
     </joint>
     <joint name="RHipPitch" type="revolute">
@@ -602,6 +602,6 @@
         <child link="r_upper_leg" />
         <axis xyz="0 1 0" />
-        <limit effort="10.0" velocity="5.759586525" lower="-1.919862177189" upper="0.48869219055720003" />
-        <dynamics damping="${d}" friction="${f}" />
+        <limit effort="7.57" velocity="8.22" lower="-1.919862177189" upper="0.48869219055720003" />
+        <dynamics damping="${d}" friction="0.1" />
     </joint>
     <joint name="RKnee" type="revolute">
@@ -610,6 +610,6 @@
         <child link="r_lower_leg" />
         <axis xyz="0 1 0" />
-        <limit effort="10.0" velocity="5.759586525" lower="0" upper="2.268928027587" />
-        <dynamics damping="${d}" friction="${f}" />
+        <limit effort="7.57" velocity="8.22" lower="0" upper="2.268928027587" />
+        <dynamics damping="${d}" friction="0.1" />
     </joint>
     <joint name="RAnklePitch" type="revolute">
@@ -618,6 +618,6 @@
         <child link="r_ankle" />
         <axis xyz="0 -1 0" />
-        <limit effort="10.0" velocity="5.759586525" lower="-1.2391837689129" upper="1.6406094968706" />
-        <dynamics damping="${d}" friction="${f}" />
+        <limit effort="7.57" velocity="8.22" lower="-1.2391837689129" upper="1.6406094968706" />
+        <dynamics damping="${d}" friction="0.1" />
     </joint>
     <joint name="RAnkleRoll" type="revolute">
@@ -626,6 +626,6 @@
         <child link="r_foot" />
         <axis xyz="-1 0 0" />
-        <limit effort="10.0" velocity="5.759586525" lower="-1.4660765716716" upper="1.4660765716716" />
-        <dynamics damping="${d}" friction="${f}" />
+        <limit effort="7.57" velocity="8.22" lower="-1.4660765716716" upper="1.4660765716716" />
+        <dynamics damping="${d}" friction="0.1" />
     </joint>
     <joint name="r_foot_to_sole" type="fixed">
@@ -646,6 +646,6 @@
         <child link="l_hip_1" />
         <axis xyz="0 0 -1" />
-        <limit effort="10.0" velocity="5.759586525" lower="-0.9250245035547" upper="0.9250245035547" />
-        <dynamics damping="${d}" friction="${f}" />
+        <limit effort="7.57" velocity="8.22" lower="-0.9250245035547" upper="0.9250245035547" />
+        <dynamics damping="${d}" friction="0.1" />
     </joint>
     <joint name="LHipRoll" type="revolute">
@@ -654,6 +654,6 @@
         <child link="l_hip_2" />
         <axis xyz="1 0 0" />
-        <limit effort="10.0" velocity="5.759586525" lower="-0.7853981633955001" upper="1.57" />
-        <dynamics damping="${d}" friction="${f}" />
+        <limit effort="7.57" velocity="8.22" lower="-0.7853981633955001" upper="1.57" />
+        <dynamics damping="${d}" friction="0.1" />
     </joint>
     <joint name="LHipPitch" type="revolute">
@@ -662,6 +662,6 @@
         <child link="l_upper_leg" />
         <axis xyz="0 -1 0" />
-        <limit effort="10.0" velocity="5.759586525" lower="-0.48869219055720003" upper="1.919862177189" />
-        <dynamics damping="${d}" friction="${f}" />
+        <limit effort="7.57" velocity="8.22" lower="-0.48869219055720003" upper="1.919862177189" />
+        <dynamics damping="${d}" friction="0.1" />
     </joint>
     <joint name="LKnee" type="revolute">
@@ -670,6 +670,6 @@
         <child link="l_lower_leg" />
         <axis xyz="0 -1 0" />
-        <limit effort="10.0" velocity="5.759586525" lower="-2.268928027587" upper="0" />
-        <dynamics damping="${d}" friction="${f}" />
+        <limit effort="7.57" velocity="8.22" lower="-2.268928027587" upper="0" />
+        <dynamics damping="${d}" friction="0.1" />
     </joint>
     <joint name="LAnklePitch" type="revolute">
@@ -678,6 +678,6 @@
         <child link="l_ankle" />
         <axis xyz="0 1 0" />
-        <limit effort="10.0" velocity="5.759586525" lower="-1.6406094968706" upper="1.2391837689129" />
-        <dynamics damping="${d}" friction="${f}" />
+        <limit effort="7.57" velocity="8.22" lower="-1.6406094968706" upper="1.2391837689129" />
+        <dynamics damping="${d}" friction="0.1" />
     </joint>
     <joint name="LAnkleRoll" type="revolute">
@@ -686,6 +686,6 @@
         <child link="l_foot" />
         <axis xyz="-1 0 0" />
-        <limit effort="10.0" velocity="5.759586525" lower="-1.4660765716716" upper="1.4660765716716" />
-        <dynamics damping="${d}" friction="${f}" />
+        <limit effort="7.57" velocity="8.22" lower="-1.4660765716716" upper="1.4660765716716" />
+        <dynamics damping="${d}" friction="0.1" />
     </joint>
     <joint name="left_foot_to_sole" type="fixed">
@@ -716,6 +716,6 @@
         <child link="r_shoulder" />
         <axis xyz="0 -1 0" />
-        <limit effort="7.3" velocity="8.16814089" lower="-3.1415926535820002" upper="3.1415926535820002" />
-        <dynamics damping="${d}" friction="${f}" />
+        <limit effort="5.43" velocity="10.33" lower="-3.1415926535820002" upper="3.1415926535820002" />
+        <dynamics damping="${d}" friction="0.09" />
     </joint>
     <joint name="RShoulderRoll" type="revolute">
@@ -724,6 +724,6 @@
         <child link="r_upper_arm" />
         <axis xyz="-1 0 0" />
-        <limit effort="7.3" velocity="8.16814089" lower="-0.7853981633955001" upper="2.3561944901865" />
-        <dynamics damping="${d}" friction="${f}" />
+        <limit effort="5.43" velocity="10.33" lower="-0.7853981633955001" upper="2.3561944901865" />
+        <dynamics damping="${d}" friction="0.09" />
     </joint>
     <joint name="RElbow" type="revolute">
@@ -732,6 +732,6 @@
         <child link="r_lower_arm" />
         <axis xyz="0 1 0" />
-        <limit effort="7.3" velocity="8.16814089" lower="-1.635" upper="1.5707963267910001" />
-        <dynamics damping="${d}" friction="${f}" />
+        <limit effort="5.43" velocity="10.33" lower="-1.635" upper="1.5707963267910001" />
+        <dynamics damping="${d}" friction="0.09" />
     </joint>
     <joint name="r_elbow_to_wrist" type="fixed">
@@ -745,6 +745,6 @@
         <child link="l_shoulder" />
         <axis xyz="0 1 0" />
-        <limit effort="7.3" velocity="8.16814089" lower="-3.1415926535820002" upper="3.1415926535820002" />
-        <dynamics damping="${d}" friction="${f}" />
+        <limit effort="5.43" velocity="10.33" lower="-3.1415926535820002" upper="3.1415926535820002" />
+        <dynamics damping="${d}" friction="0.09" />
     </joint>
     <joint name="LShoulderRoll" type="revolute">
@@ -753,6 +753,6 @@
         <child link="l_upper_arm" />
         <axis xyz="-1 0 0" />
-        <limit effort="7.3" velocity="8.16814089" lower="-2.3561944901865" upper="0.7853981633955001" />
-        <dynamics damping="${d}" friction="${f}" />
+        <limit effort="5.43" velocity="10.33" lower="-2.3561944901865" upper="0.7853981633955001" />
+        <dynamics damping="${d}" friction="0.09" />
     </joint>
     <joint name="LElbow" type="revolute">
@@ -761,6 +761,6 @@
         <child link="l_lower_arm" />
         <axis xyz="0 -1 0" />
-        <limit effort="7.3" velocity="8.16814089" lower="-1.1344640137935" upper="1.5707963267910001" />
-        <dynamics damping="${d}" friction="${f}" />
+        <limit effort="5.43" velocity="10.33" lower="-1.1344640137935" upper="1.5707963267910001" />
+        <dynamics damping="${d}" friction="0.09" />
     </joint>
     <joint name="l_elbow_to_wrist" type="fixed">
@@ -774,6 +774,6 @@
         <child link="neck" />
         <axis xyz="0 0 1" />
-        <limit effort="7.3" velocity="8.16814089" lower="-1.2" upper="1.2" />
-        <dynamics damping="${d}" friction="${f}" />
+        <limit effort="5.43" velocity="10.33" lower="-1.2" upper="1.2" />
+        <dynamics damping="${d}" friction="0.09" />
     </joint>
     <joint name="HeadTilt" type="revolute">
@@ -782,6 +782,6 @@
         <child link="head" />
         <axis xyz="0 -1 0" />
-        <limit effort="7.3" velocity="8.16814089" lower="-1.2" upper="0.2" />
-        <dynamics damping="${d}" friction="${f}" />
+        <limit effort="5.43" velocity="10.33" lower="-1.2" upper="0.2" />
+        <dynamics damping="${d}" friction="0.09" />
     </joint>
     <joint name="head_to_camera" type="fixed">
