Commit message: Add logitech urdf.

File: wolfgang_description/urdf/wolfgang_logitech.urdf.xacro (robot description, xacro)
@@ -762,5 +762,5 @@
     </joint>
     <joint name="head_to_camera" type="fixed">
-        <origin xyz="-0.00443 0 0.11475" rpy="0 0 0" />
+        <origin xyz="0.02 0 0.1115" rpy="0 0 0" />
         <parent link="head" />
         <child link="camera" />
@@ -1043,5 +1043,4 @@
     </gazebo>
   <!-- camera sensor -->
-  <!-- TODO basler sensor-->
   <gazebo reference="camera">
         <sensor name='camera' type='camera'>

Commit message: urdf logitech: update joint limits

File: wolfgang_description/urdf/wolfgang_logitech.urdf.xacro (robot description, xacro)
@@ -682,5 +682,5 @@
         <child link="r_lower_leg" />
         <axis xyz="0 1 0" />
-        <limit effort="7.57" velocity="8.22" lower="0" upper="2.268928027587" />
+        <limit effort="7.57" velocity="8.22" lower="0" upper="2.74016693" />
         <dynamics damping="${d}" friction="0.1" />
     </joint>
@@ -742,5 +742,5 @@
         <child link="l_lower_leg" />
         <axis xyz="0 -1 0" />
-        <limit effort="7.57" velocity="8.22" lower="-2.268928027587" upper="0" />
+        <limit effort="7.57" velocity="8.22" lower="-2.74016693" upper="0" />
         <dynamics damping="${d}" friction="0.1" />
     </joint>
@@ -846,5 +846,5 @@
         <child link="neck" />
         <axis xyz="0 0 1" />
-        <limit effort="5.43" velocity="10.33" lower="-1.2" upper="1.2" />
+        <limit effort="5.43" velocity="10.33" lower="-2.35" upper="2.35" />
         <dynamics damping="${d}" friction="0.09" />
     </joint>
@@ -854,5 +854,5 @@
         <child link="head" />
         <axis xyz="0 -1 0" />
-        <limit effort="5.43" velocity="10.33" lower="-1.2" upper="0.2" />
+        <limit effort="5.43" velocity="10.33" lower="-1.57" upper="0.2" />
         <dynamics damping="${d}" friction="0.09" />
     </joint>
