Commit message: Resolve conflicts

File: wolfgang_description/urdf/wolfgang_basler.urdf.xacro (robot description, xacro)
@@ -19,4 +19,7 @@
     </material>
     <link name="base_link" />
+    <gazebo reference="torso">
+        <material>Gazebo/FlatBlack</material>
+    </gazebo>
     <link name="torso">
         <inertial>
@@ -46,4 +49,7 @@
         </collision>
     </link>
+    <gazebo reference="r_hip_1">
+        <material>Gazebo/FlatBlack</material>
+    </gazebo>
     <link name="r_hip_1">
         <inertial>
@@ -66,4 +72,7 @@
         </collision>
     </link>
+    <gazebo reference="r_hip_2">
+        <material>Gazebo/FlatBlack</material>
+    </gazebo>
     <link name="r_hip_2">
         <inertial>
@@ -86,4 +95,7 @@
         </collision>
     </link>
+    <gazebo reference="r_upper_leg">
+        <material>Gazebo/FlatBlack</material>
+    </gazebo>
     <link name="r_upper_leg">
         <inertial>
@@ -132,4 +144,7 @@
         </collision>
     </link>
+    <gazebo reference="r_lower_leg">
+        <material>Gazebo/FlatBlack</material>
+    </gazebo>
     <link name="r_lower_leg">
         <inertial>
@@ -152,4 +167,7 @@
         </collision>
     </link>
+    <gazebo reference="r_ankle">
+        <material>Gazebo/FlatBlack</material>
+    </gazebo>
     <link name="r_ankle">
         <inertial>
@@ -172,4 +190,7 @@
         </collision>
     </link>
+    <gazebo reference="r_foot">
+        <material>Gazebo/FlatBlack</material>
+    </gazebo>
     <link name="r_foot">
         <inertial>
@@ -202,4 +223,7 @@
         </inertial>
     </link>
+    <gazebo reference="r_toe">
+        <material>Gazebo/FlatBlack</material>
+    </gazebo>
     <link name="r_toe">
         <inertial>
@@ -209,4 +233,7 @@
         </inertial>
     </link>
+    <gazebo reference="l_hip_1">
+        <material>Gazebo/FlatBlack</material>
+    </gazebo>
     <link name="l_hip_1">
         <inertial>
@@ -229,4 +256,7 @@
         </collision>
     </link>
+    <gazebo reference="l_hip_2">
+        <material>Gazebo/FlatBlack</material>
+    </gazebo>
     <link name="l_hip_2">
         <inertial>
@@ -249,4 +279,7 @@
         </collision>
     </link>
+    <gazebo reference="l_upper_leg">
+        <material>Gazebo/FlatBlack</material>
+    </gazebo>
     <link name="l_upper_leg">
         <inertial>
@@ -295,4 +328,7 @@
         </collision>
     </link>
+    <gazebo reference="l_lower_leg">
+        <material>Gazebo/FlatBlack</material>
+    </gazebo>
     <link name="l_lower_leg">
         <inertial>
@@ -315,4 +351,7 @@
         </collision>
     </link>
+    <gazebo reference="l_ankle">
+        <material>Gazebo/FlatBlack</material>
+    </gazebo>
     <link name="l_ankle">
         <inertial>
@@ -336,4 +375,7 @@
         </collision>
     </link>
+    <gazebo reference="l_foot">
+        <material>Gazebo/FlatBlack</material>
+    </gazebo>
     <link name="l_foot">
         <inertial>
@@ -359,4 +401,7 @@
         </xacro:if>
     </link>
+    <gazebo reference="l_sole">
+        <material>Gazebo/FlatBlack</material>
+    </gazebo>
     <link name="l_sole">
         <inertial>
@@ -366,4 +411,7 @@
         </inertial>
     </link>
+    <gazebo reference="l_toe">
+        <material>Gazebo/FlatBlack</material>
+    </gazebo>
     <link name="l_toe">
         <inertial>
@@ -373,4 +421,7 @@
         </inertial>
     </link>
+    <gazebo reference="r_shoulder">
+        <material>Gazebo/FlatBlack</material>
+    </gazebo>
     <link name="r_shoulder">
         <inertial>
@@ -393,4 +444,7 @@
         </collision>
     </link>
+    <gazebo reference="r_upper_arm">
+        <material>Gazebo/FlatBlack</material>
+    </gazebo>
     <link name="r_upper_arm">
         <inertial>
@@ -413,4 +467,7 @@
         </collision>
     </link>
+    <gazebo reference="r_lower_arm">
+        <material>Gazebo/FlatBlack</material>
+    </gazebo>
     <link name="r_lower_arm">
         <inertial>
@@ -434,4 +491,7 @@
     </link>
     <link name="r_wrist"> </link>
+    <gazebo reference="l_shoulder">
+        <material>Gazebo/FlatBlack</material>
+    </gazebo>
     <link name="l_shoulder">
         <inertial>
@@ -454,4 +514,7 @@
         </collision>
     </link>
+    <gazebo reference="l_upper_arm">
+        <material>Gazebo/FlatBlack</material>
+    </gazebo>
     <link name="l_upper_arm">
         <inertial>
@@ -474,4 +537,7 @@
         </collision>
     </link>
+    <gazebo reference="l_lower_arm">
+        <material>Gazebo/FlatBlack</material>
+    </gazebo>
     <link name="l_lower_arm">
         <inertial>
@@ -495,4 +561,7 @@
     </link>
     <link name="l_wrist"> </link>
+    <gazebo reference="neck">
+        <material>Gazebo/FlatBlack</material>
+    </gazebo>
     <link name="neck">
         <inertial>
@@ -531,4 +600,7 @@
     <link name="r_cleat_l_back"/>
     <link name="r_cleat_r_back"/>
+    <gazebo reference="head">
+        <material>Gazebo/FlatBlack</material>
+    </gazebo>
     <link name="head">
         <inertial>
@@ -1017,5 +1089,5 @@
     </transmission>
     <gazebo reference="r_foot">
-        <material>gazebo/Grey</material>
+        <material>Gazebo/FlatBlack</material>
         <kp>1000000.0</kp>
         <kd>100.0</kd>
@@ -1027,5 +1099,5 @@
     </gazebo>
     <gazebo reference="l_foot">
-        <material>gazebo/Grey</material>
+        <material>Gazebo/FlatBlack</material>
         <kp>1000000.0</kp>
         <kd>100.0</kd>
@@ -1043,5 +1115,4 @@
     </gazebo>
   <!-- camera sensor -->
-  <!-- TODO basler sensor-->
   <gazebo reference="camera">
         <sensor name='camera' type='camera'>

File: wolfgang_description/urdf/wolfgang_logitech.urdf.xacro (robot description, xacro)
@@ -19,4 +19,7 @@
     </material>
     <link name="base_link" />
+    <gazebo reference="torso">
+        <material>Gazebo/FlatBlack</material>
+    </gazebo>
     <link name="torso">
         <inertial>
@@ -46,4 +49,7 @@
         </collision>
     </link>
+    <gazebo reference="r_hip_1">
+        <material>Gazebo/FlatBlack</material>
+    </gazebo>
     <link name="r_hip_1">
         <inertial>
@@ -66,4 +72,7 @@
         </collision>
     </link>
+    <gazebo reference="r_hip_2">
+        <material>Gazebo/FlatBlack</material>
+    </gazebo>
     <link name="r_hip_2">
         <inertial>
@@ -86,4 +95,7 @@
         </collision>
     </link>
+    <gazebo reference="r_upper_leg">
+        <material>Gazebo/FlatBlack</material>
+    </gazebo>
     <link name="r_upper_leg">
         <inertial>
@@ -132,4 +144,7 @@
         </collision>
     </link>
+    <gazebo reference="r_lower_leg">
+        <material>Gazebo/FlatBlack</material>
+    </gazebo>
     <link name="r_lower_leg">
         <inertial>
@@ -152,4 +167,7 @@
         </collision>
     </link>
+    <gazebo reference="r_ankle">
+        <material>Gazebo/FlatBlack</material>
+    </gazebo>
     <link name="r_ankle">
         <inertial>
@@ -172,4 +190,7 @@
         </collision>
     </link>
+    <gazebo reference="r_foot">
+        <material>Gazebo/FlatBlack</material>
+    </gazebo>
     <link name="r_foot">
         <inertial>
@@ -202,4 +223,7 @@
         </inertial>
     </link>
+    <gazebo reference="r_toe">
+        <material>Gazebo/FlatBlack</material>
+    </gazebo>
     <link name="r_toe">
         <inertial>
@@ -209,4 +233,7 @@
         </inertial>
     </link>
+    <gazebo reference="l_hip_1">
+        <material>Gazebo/FlatBlack</material>
+    </gazebo>
     <link name="l_hip_1">
         <inertial>
@@ -229,4 +256,7 @@
         </collision>
     </link>
+    <gazebo reference="l_hip_2">
+        <material>Gazebo/FlatBlack</material>
+    </gazebo>
     <link name="l_hip_2">
         <inertial>
@@ -249,4 +279,7 @@
         </collision>
     </link>
+    <gazebo reference="l_upper_leg">
+        <material>Gazebo/FlatBlack</material>
+    </gazebo>
     <link name="l_upper_leg">
         <inertial>
@@ -295,4 +328,7 @@
         </collision>
     </link>
+    <gazebo reference="l_lower_leg">
+        <material>Gazebo/FlatBlack</material>
+    </gazebo>
     <link name="l_lower_leg">
         <inertial>
@@ -315,4 +351,7 @@
         </collision>
     </link>
+    <gazebo reference="l_ankle">
+        <material>Gazebo/FlatBlack</material>
+    </gazebo>
     <link name="l_ankle">
         <inertial>
@@ -336,4 +375,7 @@
         </collision>
     </link>
+    <gazebo reference="l_foot">
+        <material>Gazebo/FlatBlack</material>
+    </gazebo>
     <link name="l_foot">
         <inertial>
@@ -359,4 +401,7 @@
         </xacro:if>
     </link>
+    <gazebo reference="l_sole">
+        <material>Gazebo/FlatBlack</material>
+    </gazebo>
     <link name="l_sole">
         <inertial>
@@ -366,4 +411,7 @@
         </inertial>
     </link>
+    <gazebo reference="l_toe">
+        <material>Gazebo/FlatBlack</material>
+    </gazebo>
     <link name="l_toe">
         <inertial>
@@ -373,4 +421,7 @@
         </inertial>
     </link>
+    <gazebo reference="r_shoulder">
+        <material>Gazebo/FlatBlack</material>
+    </gazebo>
     <link name="r_shoulder">
         <inertial>
@@ -393,4 +444,7 @@
         </collision>
     </link>
+    <gazebo reference="r_upper_arm">
+        <material>Gazebo/FlatBlack</material>
+    </gazebo>
     <link name="r_upper_arm">
         <inertial>
@@ -413,4 +467,7 @@
         </collision>
     </link>
+    <gazebo reference="r_lower_arm">
+        <material>Gazebo/FlatBlack</material>
+    </gazebo>
     <link name="r_lower_arm">
         <inertial>
@@ -434,4 +491,7 @@
     </link>
     <link name="r_wrist"> </link>
+    <gazebo reference="l_shoulder">
+        <material>Gazebo/FlatBlack</material>
+    </gazebo>
     <link name="l_shoulder">
         <inertial>
@@ -454,4 +514,7 @@
         </collision>
     </link>
+    <gazebo reference="l_upper_arm">
+        <material>Gazebo/FlatBlack</material>
+    </gazebo>
     <link name="l_upper_arm">
         <inertial>
@@ -474,4 +537,7 @@
         </collision>
     </link>
+    <gazebo reference="l_lower_arm">
+        <material>Gazebo/FlatBlack</material>
+    </gazebo>
     <link name="l_lower_arm">
         <inertial>
@@ -495,4 +561,7 @@
     </link>
     <link name="l_wrist"> </link>
+    <gazebo reference="neck">
+        <material>Gazebo/FlatBlack</material>
+    </gazebo>
     <link name="neck">
         <inertial>
@@ -531,4 +600,7 @@
     <link name="r_cleat_l_back"/>
     <link name="r_cleat_r_back"/>
+    <gazebo reference="head">
+        <material>Gazebo/FlatBlack</material>
+    </gazebo>
     <link name="head">
         <inertial>
@@ -1017,5 +1089,5 @@
     </transmission>
     <gazebo reference="r_foot">
-        <material>gazebo/Grey</material>
+        <material>Gazebo/FlatBlack</material>
         <kp>1000000.0</kp>
         <kd>100.0</kd>
@@ -1027,5 +1099,5 @@
     </gazebo>
     <gazebo reference="l_foot">
-        <material>gazebo/Grey</material>
+        <material>Gazebo/FlatBlack</material>
         <kp>1000000.0</kp>
         <kd>100.0</kd>

Commit message: fixed knee joint limits

File: wolfgang_description/urdf/wolfgang_basler.urdf.xacro (robot description, xacro)
@@ -658,5 +658,5 @@
         <child link="r_lower_leg" />
         <axis xyz="0 1 0" />
-        <limit effort="${tofa*8.4}" velocity="4.712388975" lower="0" upper="2.268928027587" />
+        <limit effort="${tofa*8.4}" velocity="4.712388975" lower="0" upper="2.74016693" />
         <dynamics damping="${d}" friction="${f}" />
     </joint>
@@ -718,5 +718,5 @@
         <child link="l_lower_leg" />
         <axis xyz="0 -1 0" />
-        <limit effort="${tofa*8.4}" velocity="4.712388975" lower="-2.268928027587" upper="0" />
+        <limit effort="${tofa*8.4}" velocity="4.712388975" lower="-2.74016693" upper="0" />
         <dynamics damping="${d}" friction="${f}" />
     </joint>

Commit message: made head limits wider

File: wolfgang_description/urdf/wolfgang_basler.urdf.xacro (robot description, xacro)
@@ -822,5 +822,5 @@
         <child link="neck" />
         <axis xyz="0 0 1" />
-        <limit effort="${tofa*2.5}" velocity="5.6548668" lower="-1.2" upper="1.2" />
+        <limit effort="${tofa*2.5}" velocity="5.6548668" lower="-2.35" upper="2.35" />
         <dynamics damping="${d}" friction="${f}" />
     </joint>
@@ -830,5 +830,5 @@
         <child link="head" />
         <axis xyz="0 -1 0" />
-        <limit effort="${tofa*2.5}" velocity="5.6548668" lower="-1.2" upper="0.2" />
+        <limit effort="${tofa*2.5}" velocity="5.6548668" lower="-1.57" upper="0.2" />
         <dynamics damping="${d}" friction="${f}" />
     </joint>
