Commit message: urdf basler: update from tanjas measurements

File: wolfgang_description/urdf/wolfgang_basler.urdf.xacro (robot description, xacro)
@@ -24,7 +24,8 @@
     <link name="torso">
         <inertial>
-            <origin xyz="-0.016856 -0.00019822 0.019225" rpy="0 0 0" />
-            <mass value="1.8051" />
-            <inertia ixx="0.016444" ixy="1.4574E-05" ixz="0.00048254" iyy="0.013972" iyz="5.0355E-06" izz="0.0064508" />
+            <!--<origin xyz="0.007 -0.002 0.021" rpy="${-pi/64} ${-pi/32} 0" />-->
+            <origin xyz="0.014563 0.001600 0.016559" rpy="${-pi/64} ${-pi/32} 0" />
+            <mass value="2.889" />
+            <inertia ixx="0.021175651" ixy="0.000145103" ixz="-0.001622146" iyy="0.018733911" iyz="0.000373507" izz="0.009304" />
         </inertial>
         <visual>
@@ -54,7 +55,8 @@
     <link name="r_hip_1">
         <inertial>
-            <origin xyz="4.7878E-16 2.8449E-16 -0.013803" rpy="0 0 0" />
-            <mass value="0.073374" />
-            <inertia ixx="2.6774E-05" ixy="1.5536E-19" ixz="-9.0622E-19" iyy="0.00011478" iyz="-2.2736E-19" izz="0.00010743" />
+            <!--<origin xyz="0 0 -0.011" rpy="0 0 0" />-->
+            <origin xyz="-0.000001 0 -0.014563" rpy="0 0 0" />
+            <mass value="0.098" />
+            <inertia ixx="0.000013709" ixy="-0.000002388" ixz="-0.000000001" iyy="0.000054561" iyz="0" izz="0.000049167" />
         </inertial>
         <visual>
@@ -77,7 +79,8 @@
     <link name="r_hip_2">
         <inertial>
-            <origin xyz="0.010896 0.00023756 -0.014538" rpy="0 0 0" />
-            <mass value="0.35903" />
-            <inertia ixx="0.00015503" ixy="1.738E-06" ixz="8.5148E-06" iyy="0.0003299" iyz="2.4403E-07" izz="0.0002782" />
+            <!--<origin xyz="0.046 -0.002 -0.026" rpy="0 ${pi/64} 0" />-->
+            <origin xyz="0.051391 0.000232 -0.014250" rpy="0 ${pi/64} 0" />
+            <mass value="0.349" />
+            <inertia ixx="0.000156848" ixy="-0.000002134" ixz="-0.000005733" iyy="0.000355019" iyz="-0.000001749" izz="0.000308883" />
         </inertial>
         <visual>
@@ -100,7 +103,8 @@
     <link name="r_upper_leg">
         <inertial>
-            <origin xyz="0.0038549 0.00023828 -0.1495" rpy="0 0 0" />
-            <mass value="0.38276" />
-            <inertia ixx="0.0020951" ixy="1.8755E-07" ixz="-0.00017816" iyy="0.0020043" iyz="-5.4867E-06" izz="0.00027919" />
+            <!--<origin xyz="0.0056 0.004 0.126" rpy="0 0 0" />-->
+            <origin xyz="0.004721 0.000424 -0.132759" rpy="0 0 0" />
+            <mass value="0.248" />
+            <inertia ixx="0.000660963" ixy="0.000000544" ixz="-0.000016736" iyy="0.000606384" iyz="-0.000004189" izz="0.000150136" />
         </inertial>
         <visual>
@@ -149,7 +153,8 @@
     <link name="r_lower_leg">
         <inertial>
-            <origin xyz="-0.0033779 6.578E-10 -0.10469" rpy="0 0 3.14159265359" />
-            <mass value="0.20549" />
-            <inertia ixx="0.0011378" ixy="-2.8771E-12" ixz="9.7123E-05" iyy="0.0010393" iyz="-1.4479E-11" izz="0.00019656" />
+            <!--<origin xyz="0.012 0 -0.076" rpy="0 0 3.14159265359" />-->
+             <origin xyz="0.070129 -0.000102 -0.061824" rpy="0 ${-pi/4} 0" />
+            <mass value="0.085" />
+            <inertia ixx="0.000278504" ixy="0.000000060" ixz="-0.000004917" iyy="0.000241283" iyz="-0.000000066" izz="0.000070447" />
         </inertial>
         <visual>
@@ -172,7 +177,8 @@
     <link name="r_ankle">
         <inertial>
-            <origin xyz="-0.019434 0.00024988 0.014536" rpy="0 0 0" />
-            <mass value="0.35844" />
-            <inertia ixx="0.00015501" ixy="1.7299E-06" ixz="-8.5156E-06" iyy="0.00032958" iyz="-2.4435E-07" izz="0.00027786" />
+            <!--<origin xyz="-0.02 -0.005 0.026" rpy="${-pi/64} ${-pi/32} ${-pi/64}" />-->
+            <origin xyz="-0.017874 0.000190 0.013809" rpy="${-pi/64} ${-pi/32} ${-pi/64}" />
+            <mass value="0.349" />
+            <inertia ixx="0.000159124" ixy="-0.000001620" ixz="0.000011391" iyy="0.000355570" iyz="0.000001710" izz="0.000307157" />
         </inertial>
         <visual>
@@ -195,7 +201,8 @@
     <link name="r_foot">
         <inertial>
-            <origin xyz="0.003669 -0.0081165 -0.030903" rpy="0 0 0" />
-            <mass value="0.1488" />
-            <inertia ixx="0.00018527" ixy="-1.1504E-05" ixz="-7.2667E-06" iyy="0.00060485" iyz="5.8883E-06" izz="0.00075217" />
+            <!--<origin xyz="0.081 0.016 -0.033" rpy="${pi/64} ${-pi/64} 0" />-->
+            <origin xyz="0.075576 -0.013868 -0.035997" rpy="0 ${-pi/64} 0" />
+            <mass value="0.312" />
+            <inertia ixx="0.000320638" ixy="0.000010416" ixz="0.000013477" iyy="0.000978515" iyz="-0.000006347" izz="0.001270766" />
         </inertial>
         <visual>
@@ -238,7 +245,8 @@
     <link name="l_hip_1">
         <inertial>
-            <origin xyz="4.996E-16 2.5674E-16 -0.013803" rpy="0 0 0" />
-            <mass value="0.073374" />
-            <inertia ixx="2.6774E-05" ixy="1.9727E-19" ixz="-8.7961E-19" iyy="0.00011478" iyz="-2.3128E-19" izz="0.00010743" />
+            <!--<origin xyz="0 0 -0.011" rpy="0 0 0" />-->
+            <origin xyz="-0.000001 0 -0.014563" rpy="0 0 0" />
+            <mass value="0.098" />
+            <inertia ixx="0.000013709" ixy="-0.000002388" ixz="-0.000000001" iyy="0.000054561" iyz="0" izz="0.000049167" />
         </inertial>
         <visual>
@@ -260,8 +268,9 @@
     </gazebo>
     <link name="l_hip_2">
-        <inertial>
-            <origin xyz="-0.019434 -0.0014499 -0.014536" rpy="0 0 0" />
-            <mass value="0.35844" />
-            <inertia ixx="0.00015501" ixy="-1.7299E-06" ixz="8.5156E-06" iyy="0.00032958" iyz="-2.4435E-07" izz="0.00027786" />
+         <inertial>
+            <!--<origin xyz="0.046 -0.002 -0.026" rpy="0 ${pi/64} 0" />-->
+            <origin xyz="0.051391 0.000232 -0.014250" rpy="0 ${pi/64} 0" />
+            <mass value="0.349" />
+            <inertia ixx="0.000156848" ixy="-0.000002134" ixz="-0.000005733" iyy="0.000355019" iyz="-0.000001749" izz="0.000308883" />
         </inertial>
         <visual>
@@ -283,8 +292,9 @@
     </gazebo>
     <link name="l_upper_leg">
-        <inertial>
-            <origin xyz="0.0038576 -0.0014383 -0.1495" rpy="0 0 0" />
-            <mass value="0.38276" />
-            <inertia ixx="0.0020952" ixy="-1.9541E-07" ixz="-0.00017822" iyy="0.0020044" iyz="5.4912E-06" izz="0.00027919" />
+         <inertial>
+            <!--<origin xyz="-0.0056 0.004 -0.126" rpy="0 0 0" />-->
+            <origin xyz="0.004721 0.000424 -0.132759" rpy="0 0 0" />
+            <mass value="0.248" />
+            <inertia ixx="0.000660963" ixy="0.000000544" ixz="-0.000016736" iyy="0.000606384" iyz="-0.000004189" izz="0.000150136" />
         </inertial>
         <visual>
@@ -333,7 +343,9 @@
     <link name="l_lower_leg">
         <inertial>
-            <origin xyz="-0.0033779 -0.0012 -0.10469" rpy="0 0 0" />
-            <mass value="0.20549" />
-            <inertia ixx="0.0011378" ixy="-2.8771E-12" ixz="9.7123E-05" iyy="0.0010393" iyz="-1.4479E-11" izz="0.00019656" />
+            <!--<origin xyz="0.062 0 -0.045" rpy="0 ${-pi/4} 0" />-->
+            <!-- gedreht um -45 grad-->
+            <origin xyz="0.070129 -0.000102 -0.061824" rpy="0 ${-pi/4} 0" />
+            <mass value="0.085" />
+            <inertia ixx="0.000278504" ixy="0.000000060" ixz="-0.000004917" iyy="0.000241283" iyz="-0.000000066" izz="0.000070447" />
         </inertial>
         <visual>
@@ -356,7 +368,8 @@
     <link name="l_ankle">
         <inertial>
-            <origin xyz="-0.019418 -0.0014376 0.014538" rpy="0 0 0" />
-            <mass value="0.35903" />
-            <inertia ixx="0.00015503" ixy="-1.738E-06" ixz="-8.5148E-06" iyy="0.0003299" iyz="2.4403E-07" izz="0.0002782" />
+            <!--<origin xyz="-0.02 -0.005 0.026" rpy="${-pi/64} ${-pi/32} ${-pi/64}" />-->
+            <origin xyz="-0.017874 0.000190 0.013809" rpy="${-pi/64} ${-pi/32} ${-pi/64}" />
+            <mass value="0.349" />
+            <inertia ixx="0.000159124" ixy="-0.000001620" ixz="0.000011391" iyy="0.000355570" iyz="0.000001710" izz="0.000307157" />
         </inertial>
         <visual>
@@ -380,7 +393,8 @@
     <link name="l_foot">
         <inertial>
-            <origin xyz="0.0036084 0.0081189 -0.03091" rpy="0 0 0" />
-            <mass value="0.1488" />
-            <inertia ixx="0.0001853" ixy="1.1466E-05" ixz="-8.3793E-06" iyy="0.00060485" iyz="-5.9046E-06" izz="0.00075213" />
+            <!--<origin xyz="0.081 -0.016 -0.033" rpy="${-pi/64} ${-pi/64} 0" />-->
+            <origin xyz="0.075576 0.013868 -0.035997" rpy="0 ${-pi/64} 0" />
+            <mass value="0.312" />
+            <inertia ixx="0.000320638" ixy="0.000010416" ixz="0.000013477" iyy="0.000978515" iyz="-0.000006347" izz="0.001270766" />
         </inertial>
         <visual>
@@ -426,7 +440,9 @@
     <link name="r_shoulder">
         <inertial>
-            <origin xyz="0 -0.014621 0" rpy="${pi} 0 0" />
-            <mass value="0.025434" />
-            <inertia ixx="6.7511E-06" ixy="1.5595E-20" ixz="-5.4198E-21" iyy="1.2425E-05" iyz="-2.4006E-20" izz="1.4317E-05" />
+            <!--<origin xyz="0.012 -0.02 0" rpy="0 ${-pi/8} 0" />-->
+            <origin xyz="0.010164 -0.022268 -0.000376" rpy="0 ${-pi/8} 0" />
+            <mass value="0.097" />
+            <inertia ixx="0.000044153" ixy="-0.000000525" ixz="0.000015185" iyy="0.000086852" iyz="0.000000524" izz="0.000065734" />
+            <!--<inertia ixx="0.000044153" ixy="0.000015185" ixz="-0.000000525" iyy="0.000065734" iyz="0.000000524" izz="0.000086852" />-->
         </inertial>
         <visual>
@@ -449,7 +465,8 @@
     <link name="r_upper_arm">
         <inertial>
-            <origin xyz="0.0013671 0.00022653 -0.049517" rpy="0 0 0" />
-            <mass value="0.2575" />
-            <inertia ixx="0.00081539" ixy="1.1134E-07" ixz="-5.114E-05" iyy="0.0007994" iyz="-2.4756E-06" izz="0.00012883" />
+            <!--<origin xyz="0 0 -0.031" rpy="0 0 0" />-->
+            <origin xyz="0.000158 -0.000012 -0.035495" rpy="0 0 0" />
+            <mass value="0.229" />
+            <inertia ixx="0.000490959" ixy="-0.000000004" ixz="-0.000004117" iyy="0.000461542" iyz="-0.000000191" izz="0.000102122" />
         </inertial>
         <visual>
@@ -472,7 +489,8 @@
     <link name="r_lower_arm">
         <inertial>
-            <origin xyz="0.0018497 -0.00091671 -0.059095" rpy="0 0 0" />
-            <mass value="0.23502" />
-            <inertia ixx="0.0011613" ixy="-5.8221E-07" ixz="-7.4224E-05" iyy="0.0011747" iyz="2.0082E-05" izz="0.00010273" />
+            <!--<origin xyz="0.055 0 0.001" rpy="${pi/8} 0 0" />-->
+            <origin xyz="0.050639 -0.000164 0.000492" rpy="${pi/8} 0 0" />
+            <mass value="0.208" />
+            <inertia ixx="0.000085671" ixy="-0.000002277" ixz="0.000000392" iyy="0.000903139" iyz="0.000001021" izz="0.000904792" />
         </inertial>
         <visual>
@@ -496,7 +514,9 @@
     <link name="l_shoulder">
         <inertial>
-            <origin xyz="0 0.014621 0" rpy="0 0 0" />
-            <mass value="0.025434" />
-            <inertia ixx="6.7511E-06" ixy="6.4644E-21" ixz="-3.365E-21" iyy="1.2425E-05" iyz="-4.6109E-22" izz="1.4317E-05" />
+            <!--<origin xyz="0.012 0.02 0" rpy="0 ${-pi/8} 0" />-->
+            <origin xyz="0.010164 0.022268 -0.000376" rpy="0 ${-pi/8} 0" />
+            <mass value="0.097" />
+            <!--<inertia ixx="0.000044153" ixy="0.000015185" ixz="-0.000000525" iyy="0.000065734" iyz="0.000000524" izz="0.000086852" />-->
+            <inertia ixx="0.000044153" ixy="-0.000000525" ixz="0.000015185" iyy="0.000086852" iyz="0.000000524" izz="0.000065734" />
         </inertial>
         <visual>
@@ -519,7 +539,8 @@
     <link name="l_upper_arm">
         <inertial>
-            <origin xyz="0.0013671 0.00022653 -0.049517" rpy="0 0 0" />
-            <mass value="0.2575" />
-            <inertia ixx="0.00081539" ixy="1.1134E-07" ixz="-5.114E-05" iyy="0.0007994" iyz="-2.4756E-06" izz="0.00012883" />
+            <!--<origin xyz="0 0 -0.031" rpy="0 0 0" />-->
+            <origin xyz="0.000158 -0.000012 -0.035495" rpy="0 0 0" />
+            <mass value="0.229" />
+            <inertia ixx="0.000490959" ixy="-0.000000004" ixz="-0.000004117" iyy="0.000461542" iyz="-0.000000191" izz="0.000102122" />
         </inertial>
         <visual>
@@ -541,8 +562,9 @@
     </gazebo>
     <link name="l_lower_arm">
-        <inertial>
-            <origin xyz="0.001742 -6.4508E-05 -0.059095" rpy="0 0 0" />
-            <mass value="0.23502" />
-            <inertia ixx="0.0011616" ixy="-2.6303E-07" ixz="-7.2367E-05" iyy="0.0011751" iyz="9.5624E-06" izz="0.00010214" />
+       <inertial>
+            <!--<origin xyz="0.055 0 0.001" rpy="${pi/8} 0 0" />-->
+            <origin xyz="0.050639 -0.000164 0.000492" rpy="${pi/8} 0 0" />
+            <mass value="0.208" />
+            <inertia ixx="0.000085671" ixy="-0.000002277" ixz="0.000000392" iyy="0.000903139" iyz="0.000001021" izz="0.000904792" />
         </inertial>
         <visual>
@@ -566,12 +588,13 @@
     <link name="neck">
         <inertial>
-            <origin xyz="2.1595E-05 0.00064781 0.033208" rpy="0 0 0" />
+            <!--<origin xyz="0.0045 0 0.016" rpy="0 0 0" />-->
+            <origin xyz="0.027758 0.000252 0.032356" rpy="0 0 0" />
             <xacro:if value="${fake_walk== True}">
                 <mass value="0.00015587" />
             </xacro:if>
             <xacro:if value="${fake_walk== False}">
-                <mass value="0.15587" />
+                <mass value="0.153" />
             </xacro:if>
-            <inertia ixx="7.5209E-05" ixy="-1.8422E-06" ixz="-4.9817E-07" iyy="6.2999E-05" iyz="-9.9088E-08" izz="3.826E-05" />
+            <inertia ixx="0.000072487" ixy="-0.000000033" ixz="0.000003661" iyy="0.000064592" iyz="0.000001234" izz="0.000044157" />
         </inertial>
         <visual>
@@ -605,12 +628,13 @@
     <link name="head">
         <inertial>
-            <origin xyz="0.014358 0.0005519 0.069919" rpy="0 0 0" />
+            <!--<origin xyz="0.004 0 0.096" rpy="0 0 0" />-->
+            <origin xyz="0.012794 -0.000380 0.100180" rpy="0 0 0" />
             <xacro:if value="${fake_walk== True}">
                 <mass value="0.00040746" />
             </xacro:if>
             <xacro:if value="${fake_walk== False}">
-                <mass value="0.40746" />
+                <mass value="0.110" />
             </xacro:if>
-            <inertia ixx="0.0014813" ixy="3.1631E-07" ixz="-4.1003E-05" iyy="0.0016361" iyz="6.7483E-07" izz="0.0017353" />
+            <inertia ixx="0.000216591" ixy="0.000001444" ixz="-0.000024793" iyy="0.000169162" iyz="0.000000772" izz="0.000081113" />
         </inertial>
         <!-- <visual>
@@ -634,6 +658,6 @@
         <child link="r_hip_1" />
         <axis xyz="0 0 -1" />
-        <limit effort="${tofa*2.5}" velocity="5.6548668" lower="-0.9250245035547" upper="0.9250245035547" />
-        <dynamics damping="${d}" friction="${f}" />
+        <limit effort="7.57" velocity="8.22" lower="-0.9250245035547" upper="0.9250245035547" />
+        <dynamics damping="${d}" friction="0.1" />
     </joint>
     <joint name="RHipRoll" type="revolute">
@@ -642,6 +666,6 @@
         <child link="r_hip_2" />
         <axis xyz="1 0 0" />
-        <limit effort="${tofa*6.0}" velocity="6.597344565" lower="-1.57" upper="0.7853981633955001" />
-        <dynamics damping="${d}" friction="${f}" />
+        <limit effort="7.57" velocity="8.22" lower="-1.57" upper="0.7853981633955001" />
+        <dynamics damping="${d}" friction="0.1" />
     </joint>
     <joint name="RHipPitch" type="revolute">
@@ -650,6 +674,6 @@
         <child link="r_upper_leg" />
         <axis xyz="0 1 0" />
-        <limit effort="${tofa*8.4}" velocity="4.712388975" lower="-1.919862177189" upper="0.48869219055720003" />
-        <dynamics damping="${d}" friction="${f}" />
+        <limit effort="7.57" velocity="8.22" lower="-1.919862177189" upper="0.48869219055720003" />
+        <dynamics damping="${d}" friction="0.1" />
     </joint>
     <joint name="RKnee" type="revolute">
@@ -658,6 +682,6 @@
         <child link="r_lower_leg" />
         <axis xyz="0 1 0" />
-        <limit effort="${tofa*8.4}" velocity="4.712388975" lower="0" upper="2.74016693" />
-        <dynamics damping="${d}" friction="${f}" />
+        <limit effort="7.57" velocity="8.22" lower="0" upper="2.74016693" />
+        <dynamics damping="${d}" friction="0.1" />
     </joint>
     <joint name="RAnklePitch" type="revolute">
@@ -666,6 +690,6 @@
         <child link="r_ankle" />
         <axis xyz="0 -1 0" />
-        <limit effort="${tofa*8.4}" velocity="4.712388975" lower="-1.2391837689129" upper="1.6406094968706" />
-        <dynamics damping="${d}" friction="${f}" />
+        <limit effort="7.57" velocity="8.22" lower="-1.2391837689129" upper="1.6406094968706" />
+        <dynamics damping="${d}" friction="0.1" />
     </joint>
     <joint name="RAnkleRoll" type="revolute">
@@ -674,6 +698,6 @@
         <child link="r_foot" />
         <axis xyz="-1 0 0" />
-        <limit effort="${tofa*6.0}" velocity="6.597344565" lower="-1.4660765716716" upper="1.4660765716716" />
-        <dynamics damping="${d}" friction="${f}" />
+        <limit effort="7.57" velocity="8.22" lower="-1.4660765716716" upper="1.4660765716716" />
+        <dynamics damping="${d}" friction="0.1" />
     </joint>
     <joint name="r_foot_to_sole" type="fixed">
@@ -694,6 +718,6 @@
         <child link="l_hip_1" />
         <axis xyz="0 0 -1" />
-        <limit effort="${tofa*2.5}" velocity="5.6548668" lower="-0.9250245035547" upper="0.9250245035547" />
-        <dynamics damping="${d}" friction="${f}" />
+        <limit effort="7.57" velocity="8.22" lower="-0.9250245035547" upper="0.9250245035547" />
+        <dynamics damping="${d}" friction="0.1" />
     </joint>
     <joint name="LHipRoll" type="revolute">
@@ -702,6 +726,6 @@
         <child link="l_hip_2" />
         <axis xyz="1 0 0" />
-        <limit effort="${tofa*6.0}" velocity="6.597344565" lower="-0.7853981633955001" upper="1.57" />
-        <dynamics damping="${d}" friction="${f}" />
+        <limit effort="7.57" velocity="8.22" lower="-0.7853981633955001" upper="1.57" />
+        <dynamics damping="${d}" friction="0.1" />
     </joint>
     <joint name="LHipPitch" type="revolute">
@@ -710,6 +734,6 @@
         <child link="l_upper_leg" />
         <axis xyz="0 -1 0" />
-        <limit effort="${tofa*8.4}" velocity="4.712388975" lower="-0.48869219055720003" upper="1.919862177189" />
-        <dynamics damping="${d}" friction="${f}" />
+        <limit effort="7.57" velocity="8.22" lower="-0.48869219055720003" upper="1.919862177189" />
+        <dynamics damping="${d}" friction="0.1" />
     </joint>
     <joint name="LKnee" type="revolute">
@@ -718,6 +742,6 @@
         <child link="l_lower_leg" />
         <axis xyz="0 -1 0" />
-        <limit effort="${tofa*8.4}" velocity="4.712388975" lower="-2.74016693" upper="0" />
-        <dynamics damping="${d}" friction="${f}" />
+        <limit effort="7.57" velocity="8.22" lower="-2.74016693" upper="0" />
+        <dynamics damping="${d}" friction="0.1" />
     </joint>
     <joint name="LAnklePitch" type="revolute">
@@ -726,6 +750,6 @@
         <child link="l_ankle" />
         <axis xyz="0 1 0" />
-        <limit effort="${tofa*8.4}" velocity="4.712388975" lower="-1.6406094968706" upper="1.2391837689129" />
-        <dynamics damping="${d}" friction="${f}" />
+        <limit effort="7.57" velocity="8.22" lower="-1.6406094968706" upper="1.2391837689129" />
+        <dynamics damping="${d}" friction="0.1" />
     </joint>
     <joint name="LAnkleRoll" type="revolute">
@@ -734,6 +758,6 @@
         <child link="l_foot" />
         <axis xyz="-1 0 0" />
-        <limit effort="${tofa*6.0}" velocity="6.597344565" lower="-1.4660765716716" upper="1.4660765716716" />
-        <dynamics damping="${d}" friction="${f}" />
+        <limit effort="7.57" velocity="8.22" lower="-1.4660765716716" upper="1.4660765716716" />
+        <dynamics damping="${d}" friction="0.1" />
     </joint>
     <joint name="left_foot_to_sole" type="fixed">
@@ -764,6 +788,6 @@
         <child link="r_shoulder" />
         <axis xyz="0 -1 0" />
-        <limit effort="${tofa*6.0}" velocity="6.597344565" lower="-3.1415926535820002" upper="3.1415926535820002" />
-        <dynamics damping="${d}" friction="${f}" />
+        <limit effort="5.43" velocity="10.33" lower="-3.1415926535820002" upper="3.1415926535820002" />
+        <dynamics damping="${d}" friction="0.09" />
     </joint>
     <joint name="RShoulderRoll" type="revolute">
@@ -772,6 +796,6 @@
         <child link="r_upper_arm" />
         <axis xyz="-1 0 0" />
-        <limit effort="${tofa*2.5}" velocity="5.648668" lower="-0.7853981633955001" upper="2.3561944901865" />
-        <dynamics damping="${d}" friction="${f}" />
+        <limit effort="5.43" velocity="10.33" lower="-0.7853981633955001" upper="2.3561944901865" />
+        <dynamics damping="${d}" friction="0.09" />
     </joint>
     <joint name="RElbow" type="revolute">
@@ -780,6 +804,6 @@
         <child link="r_lower_arm" />
         <axis xyz="0 1 0" />
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
File: wolfgang_description/urdf/wolfgang_logitech.urdf.xacro (robot description, xacro)
@@ -627,4 +627,5 @@
     </gazebo>
     <link name="head">
+        <!-- TODO: measure weight for basler camera -->
         <inertial>
             <!--<origin xyz="0.004 0 0.096" rpy="0 0 0" />-->

Commit message: urdf basler: add missing value

File: wolfgang_description/urdf/wolfgang_basler.urdf.xacro (robot description, xacro)
@@ -858,5 +858,5 @@
     </joint>
     <joint name="head_to_camera" type="fixed">
-        <origin xyz="-0.00443 0.11475" rpy="0 0 0" />
+        <origin xyz="-0.00443 0 0.11475" rpy="0 0 0" />
         <parent link="head" />
         <child link="camera" />

Commit message: wolfgang_description: correct location of imu

File: wolfgang_description/urdf/wolfgang_basler.urdf.xacro (robot description, xacro)
@@ -781,5 +781,5 @@
         <parent link="torso" />
         <child link="imu_frame" />
-        <origin rpy="0.0 0 0" xyz="-0.045 0.025 0.023" />
+        <origin rpy="0.0 0 0" xyz="-0.050 0.023 0.018" />
     </joint>
     <joint name="RShoulderPitch" type="revolute">

File: wolfgang_description/urdf/wolfgang_logitech.urdf.xacro (robot description, xacro)
@@ -782,5 +782,5 @@
         <parent link="torso" />
         <child link="imu_frame" />
-        <origin rpy="0.0 0 0" xyz="-0.045 0.025 0.023" />
+        <origin rpy="0.0 0 0" xyz="-0.050 0.023 0.018" />
     </joint>
     <joint name="RShoulderPitch" type="revolute">
