Commit message: description: fix frame rotations

File: wolfgang_description/urdf/robot.urdf (robot description, URDF)
Before this commit: robot onshape, 36 links, 35 joints
Links:
- removed link right_hip_left_ankle_3
- added link camera_optical_frame, mass 1e-9
- added link left_hip_right_ankle_2, mass 0.319807; collision mesh filename=package://wolfgang_description/urdf/motor_connector.stl; collision mesh filename=package://wolfgang_description/urdf/motor_connector.stl
- link upper_leg_left_1: geometry collision mesh filename=package://wolfgang_description/urdf/knee_connector.stl; collision mesh filename=package://wolfgang_description/urdf/knee_connector.stl
Joints:
- added joint camera_optical_frame_frame: type fixed, parent head_1, child camera_optical_frame, origin xyz=0.0432 0.08 -0.0235 rpy=3.14159 -1.5708 0, axis 0 0 0
- joint HeadPan: origin xyz=1.19176e-17 0.0075 0.1465 rpy=3.14159 -0 -1.5708 -> xyz=-2.18523e-16 -0.0095 0.2345 rpy=3.14159 -1.14905e-16 1.5708
- joint HeadTilt: origin xyz=0.036 0.0235 -0.024 rpy=-1.5708 6.50218e-17 -3.25641e-16 -> xyz=0.036 0.0235 -0.024 rpy=-1.5708 9.39807e-16 -1.02779e-15
- joint LAnklePitch: child right_hip_left_ankle_3 -> right_hip_left_ankle_2; origin xyz=7.35523e-16 -0.0505 -0.17 rpy=-1.5708 -3.26396e-14 -3.14159 -> xyz=1.52656e-15 -0.0505 -0.17 rpy=-1.5708 7.6817e-16 3.14159
- joint LAnkleRoll: origin xyz=0.0691 -4.996e-16 -0.026 rpy=1.5708 -1.5708 0 -> xyz=0.0691 -5.55112e-17 -0.026 rpy=1.5708 -1.5708 0; parent right_hip_left_ankle_3 -> right_hip_left_ankle_2
- joint LElbow: origin xyz=-0.024 -0.144 -0.0235 rpy=-1.5708 7.60608e-16 1.5708 -> xyz=-0.024 -0.144 -0.0235 rpy=-1.5708 2.44249e-15 1.5708
- joint LHipPitch: axis 0 -1 0 -> -7.95491e-17 3.00167e-16 1; origin xyz=-0.026 0 -0.0691 rpy=-1.5708 1.5708 0 -> xyz=0.026 6.93889e-18 -0.0691 rpy=3.52442e-16 -1.5708 0; parent right_hip_left_ankle_2 -> left_hip_right_ankle_2
- joint LHipRoll: child right_hip_left_ankle_2 -> left_hip_right_ankle_2; origin xyz=-0.046 0.0414 -6.93889e-18 rpy=-3.14159 1.5708 0 -> xyz=-0.046 0.0414 -1.38778e-17 rpy=3.14159 1.5708 0
- joint LHipYaw: origin xyz=0.055 -0.002 -0.088 rpy=-1.5708 -0 -1.5708 -> xyz=-0.055 -2.29027e-16 -1.49295e-16 rpy=-1.5708 7.32452e-17 1.5708
- joint LKnee: origin xyz=-0.00435596 -0.002 -0.168793 rpy=3.42495e-16 -0.261799 -2.96624e-16 -> xyz=0.00435596 -0.168793 0.049 rpy=1.5708 1.05156e-16 2.87979
- joint LShoulderPitch: origin xyz=0.0765 -0.0005 0.1155 rpy=-3.14159 -1.80411e-16 1.5708 -> xyz=-0.0765 -0.0015 0.2035 rpy=3.14159 -0 -1.5708
- joint LShoulderRoll: origin xyz=-0.01695 0.042 5.55112e-17 rpy=-1.5708 -1.80221e-15 1.5708 -> xyz=-0.01695 0.042 2.77556e-17 rpy=-1.5708 -1.56545e-16 1.5708
- joint RAnklePitch: origin xyz=-2.01228e-16 0.0505 -0.17 rpy=-1.5708 2.8301e-15 -1.07331e-15 -> xyz=9.08995e-16 0.0505 -0.17 rpy=-1.5708 -5.70527e-16 -4.13194e-16
- joint RAnkleRoll: origin xyz=-0.0691 1.11022e-16 -0.026 rpy=1.5708 1.5708 0 -> xyz=-0.0691 -4.44089e-16 -0.026 rpy=1.5708 1.5708 0
- joint RElbow: origin xyz=0.024 -0.144 -0.0235 rpy=-1.5708 4.92144e-16 -1.5708 -> xyz=0.024 -0.144 -0.0235 rpy=-1.5708 1.73247e-15 -1.5708
- joint RHipPitch: origin xyz=-0.0265 8.32667e-17 -0.0691 rpy=-1.5708 1.5708 0 -> xyz=-0.0265 0 -0.0691 rpy=-1.5708 1.5708 0
- joint RHipRoll: origin xyz=-0.046 0.0414 -1.249e-16 rpy=-3.14159 1.5708 0 -> xyz=-0.046 0.0414 -1.38778e-17 rpy=-3.14159 1.5708 0
- joint RHipYaw: origin xyz=-0.055 -0.002 -0.088 rpy=-1.5708 6.12565e-17 -1.5708 -> xyz=0.055 -9.99201e-19 -9.54098e-18 rpy=-1.5708 1.09301e-26 1.5708
- joint RKnee: origin xyz=-0.00392295 -0.051 -0.169043 rpy=-9.05543e-17 -0.261799 1.15126e-16 -> xyz=-0.00392295 -0.051 -0.169043 rpy=2.60189e-15 -0.261799 -6.6404e-16
- joint RShoulderPitch: origin xyz=-0.0765 -0.0005 0.1155 rpy=3.72231e-24 1.72085e-15 1.5708 -> xyz=0.0765 -0.0015 0.2035 rpy=-5.36354e-17 1.72085e-15 -1.5708
- joint RShoulderRoll: origin xyz=-0.01695 0.042 2.77556e-17 rpy=1.5708 -1.16018e-14 -1.5708 -> xyz=-0.01695 0.042 0 rpy=1.5708 -1.50668e-15 -1.5708
- joint camera_frame: origin xyz=0.0437 0.0795 -0.0235 rpy=-3.24697e-15 9.53238e-16 1.80216e-15 -> xyz=0.0437 0.0795 -0.0235 rpy=-1.5708 -8.59213e-16 1.88738e-15
- joint imu_frame_frame: origin xyz=-0.0478024 0.0352504 0.1365 rpy=-1.11022e-16 -1.5708 0 -> xyz=0.0478024 -0.0367504 0.224 rpy=-2.37905e-17 9.04859e-17 1.5708
- joint l_cleat_l_back_frame: origin xyz=-0.06 -0.007 -0.05025 rpy=-1.5708 5.02934e-16 1.5708 -> xyz=-0.0605 -0.007 -0.04975 rpy=-4.85867e-15 -8.48619e-15 1.5708
- joint l_cleat_l_front_frame: origin xyz=-0.06 0.177 -0.05025 rpy=-1.5708 -9.63558e-15 1.5708 -> xyz=-0.0605 0.177 -0.04975 rpy=-2.40691e-16 1.48781e-15 1.5708
- joint l_cleat_r_back_frame: origin xyz=0.03 -0.007 -0.05025 rpy=-1.5708 -6.86763e-15 1.5708 -> xyz=0.0295 -0.007 -0.04975 rpy=-1.27389e-15 6.99799e-16 1.5708
- joint l_cleat_r_front_frame: origin xyz=0.03 0.177 -0.05025 rpy=-1.5708 -9.63558e-15 1.5708 -> xyz=0.0295 0.177 -0.04975 rpy=-2.40691e-16 1.48781e-15 1.5708
- joint l_sole_frame: origin xyz=-0.0152261 0.0902683 -0.039 rpy=-1.5708 -1.5708 0 -> xyz=-0.0152261 0.0907683 -0.0529 rpy=-2.97297e-17 -2.35463e-15 1.5708
- joint l_wrist_frame: origin xyz=1.73472e-17 -0.228682 -0.024 rpy=1.38778e-15 1.5708 0 -> xyz=8.32667e-17 -0.225182 -0.0235 rpy=-1.5708 1.45366e-16 -1.5708
- joint r_cleat_l_back_frame: origin xyz=-0.029996 -0.00745064 -0.05075 rpy=-1.5708 -6.1574e-15 1.5708 -> xyz=-0.030496 -0.00745064 -0.05025 rpy=9.51939e-16 -4.37921e-15 1.5708
- joint r_cleat_l_front_frame: origin xyz=-0.03 0.177 -0.05075 rpy=-1.5708 -3.29269e-15 1.5708 -> xyz=-0.0305 0.177 -0.05025 rpy=4.65062e-17 1.10045e-14 1.5708
- joint r_cleat_r_back_frame: origin xyz=0.06 -0.007 -0.05075 rpy=-1.5708 3.66536e-15 1.5708 -> xyz=0.0595 -0.007 -0.05025 rpy=7.70805e-16 -3.07597e-15 1.5708
- joint r_cleat_r_front_frame: origin xyz=0.06 0.177 -0.05075 rpy=-1.5708 -2.09851e-15 1.5708 -> xyz=0.0595 0.177 -0.05025 rpy=2.69391e-16 -5.00011e-15 1.5708
- joint r_sole_frame: origin xyz=0.0152261 0.0902683 -0.039 rpy=-1.5708 -1.5708 0 -> xyz=0.0152261 0.0907683 -0.0529 rpy=5.35395e-16 1.07005e-14 1.5708
- joint r_wrist_frame: origin xyz=7.28584e-17 -0.225682 -0.023 rpy=8.8601e-16 -1.5708 0 -> xyz=1.249e-16 -0.226182 -0.0235 rpy=1.5708 1.43787e-15 -1.5708

Commit message: description: fixes on urdf

File: wolfgang_description/urdf/robot.urdf (robot description, URDF)
Before this commit: robot onshape, 37 links, 36 joints
Joints:
- joint LKnee: limit lower=0 upper=2.96706 effort=10 velocity=10 -> lower=-2.96706 upper=0 effort=10 velocity=10

Commit message: description: fixed urdf

File: wolfgang_description/urdf/robot.urdf (robot description, URDF)
Before this commit: robot wolfgang, 37 links, 36 joints
Joints:
- joint HeadPan: origin xyz=-2.18523e-16 -0.0095 0.2345 rpy=3.14159 -1.14905e-16 1.5708 -> xyz=-0.0095 2.82644e-16 0.2345 rpy=-3.14159 3.41087e-16 -4.44089e-16
- joint HeadTilt: origin xyz=0.036 0.0235 -0.024 rpy=-1.5708 9.39807e-16 -1.02779e-15 -> xyz=0.036 0.0235 -0.024 rpy=-1.5708 3.17216e-15 -5.33479e-15
- joint LAnklePitch: origin xyz=1.52656e-15 -0.0505 -0.17 rpy=-1.5708 7.6817e-16 3.14159 -> xyz=3.5319e-15 -0.0505 -0.17 rpy=-1.5708 -8.72457e-16 3.14159
- joint LAnkleRoll: origin xyz=0.0691 -5.55112e-17 -0.026 rpy=1.5708 -1.5708 0 -> xyz=0.0691 2.22045e-16 -0.026 rpy=1.5708 -1.5708 0
- joint LElbow: origin xyz=-0.024 -0.144 -0.0235 rpy=-1.5708 2.44249e-15 1.5708 -> xyz=-0.024 -0.144 -0.0235 rpy=-1.5708 1.11022e-14 1.5708
- joint LHipPitch: origin xyz=0.026 6.93889e-18 -0.0691 rpy=3.52442e-16 -1.5708 0 -> xyz=0.026 6.93889e-18 -0.0691 rpy=2.67116e-16 -1.5708 0
- joint LHipRoll: origin xyz=-0.046 0.0414 -1.38778e-17 rpy=3.14159 1.5708 0 -> xyz=-0.046 0.0414 -7.97973e-16 rpy=3.14159 1.5708 0
- joint LHipYaw: origin xyz=-0.055 -2.29027e-16 -1.49295e-16 rpy=-1.5708 7.32452e-17 1.5708 -> xyz=-2.28983e-16 0.055 2.71051e-18 rpy=-1.5708 -0 0
- joint LKnee: origin xyz=0.00435596 -0.168793 0.049 rpy=1.5708 1.05156e-16 2.87979 -> xyz=0.00435596 -0.168793 0.049 rpy=1.5708 -1.75248e-15 2.87979
- joint LShoulderPitch: origin xyz=-0.0765 -0.0015 0.2035 rpy=3.14159 -0 -1.5708 -> xyz=-0.0015 0.0765 0.2035 rpy=3.14159 7.77156e-16 3.14159
- joint LShoulderRoll: origin xyz=-0.01695 0.042 2.77556e-17 rpy=-1.5708 -1.56545e-16 1.5708 -> xyz=-0.01695 0.042 8.32667e-17 rpy=-1.5708 8.42077e-17 1.5708
- joint RAnklePitch: origin xyz=9.08995e-16 0.0505 -0.17 rpy=-1.5708 -5.70527e-16 -4.13194e-16 -> xyz=2.69229e-15 0.0505 -0.17 rpy=-1.5708 -1.93533e-15 -2.52888e-15
- joint RAnkleRoll: origin xyz=-0.0691 -4.44089e-16 -0.026 rpy=1.5708 1.5708 0 -> xyz=-0.0691 5.55112e-17 -0.026 rpy=1.5708 1.5708 0
- joint RElbow: origin xyz=0.024 -0.144 -0.0235 rpy=-1.5708 1.73247e-15 -1.5708 -> xyz=0.024 -0.144 -0.0235 rpy=-1.5708 1.27676e-15 -1.5708
- joint RHipPitch: origin xyz=-0.0265 0 -0.0691 rpy=-1.5708 1.5708 0 -> xyz=-0.0265 -2.77556e-17 -0.0691 rpy=-1.5708 1.5708 0
- joint RHipRoll: origin xyz=-0.046 0.0414 -1.38778e-17 rpy=-3.14159 1.5708 0 -> xyz=-0.046 0.0414 5.34295e-16 rpy=-3.14159 1.5708 0
- joint RHipYaw: origin xyz=0.055 -9.99201e-19 -9.54098e-18 rpy=-1.5708 1.09301e-26 1.5708 -> xyz=-1.38778e-17 -0.055 -9.75782e-19 rpy=-1.5708 -0 0
- joint RKnee: origin xyz=-0.00392295 -0.051 -0.169043 rpy=2.60189e-15 -0.261799 -6.6404e-16 -> xyz=-0.00392295 -0.051 -0.169043 rpy=1.50246e-15 -0.261799 -1.61204e-15
- joint RShoulderPitch: origin xyz=0.0765 -0.0015 0.2035 rpy=-5.36354e-17 1.72085e-15 -1.5708 -> xyz=-0.0015 -0.0765 0.2035 rpy=-4.34612e-17 1.66533e-15 -3.14159
- joint RShoulderRoll: origin xyz=-0.01695 0.042 0 rpy=1.5708 -1.50668e-15 -1.5708 -> xyz=-0.01695 0.042 0 rpy=1.5708 8.32338e-16 -1.5708
- joint camera_frame: origin xyz=0.0437 0.0795 -0.0235 rpy=-1.5708 -8.59213e-16 1.88738e-15 -> xyz=0.0437 0.0795 -0.0235 rpy=-1.5708 -1.45465e-14 -3.33067e-16
- joint imu_frame_frame: origin xyz=0.0478024 -0.0367504 0.224 rpy=-2.37905e-17 9.04859e-17 1.5708 -> xyz=-0.0367504 -0.0478024 0.224 rpy=5.31321e-16 -3.12873e-17 4.65401e-17
- joint l_cleat_l_back_frame: origin xyz=-0.0605 -0.007 -0.04975 rpy=-4.85867e-15 -8.48619e-15 1.5708 -> xyz=-0.0605 -0.007 -0.04975 rpy=-2.04856e-14 -2.56773e-14 1.5708
- joint l_cleat_l_front_frame: origin xyz=-0.0605 0.177 -0.04975 rpy=-2.40691e-16 1.48781e-15 1.5708 -> xyz=-0.0605 0.177 -0.04975 rpy=-6.55214e-15 4.2513e-15 1.5708
- joint l_cleat_r_back_frame: origin xyz=0.0295 -0.007 -0.04975 rpy=-1.27389e-15 6.99799e-16 1.5708 -> xyz=0.0295 -0.007 -0.04975 rpy=-3.99384e-16 1.98982e-15 1.5708
- joint l_cleat_r_front_frame: origin xyz=0.0295 0.177 -0.04975 rpy=-2.40691e-16 1.48781e-15 1.5708 -> xyz=0.0295 0.177 -0.04975 rpy=-6.55214e-15 4.2513e-15 1.5708
- joint l_sole_frame: origin xyz=-0.0152261 0.0907683 -0.0529 rpy=-2.97297e-17 -2.35463e-15 1.5708 -> xyz=-0.0152261 0.0907683 -0.0529 rpy=-5.77818e-15 -7.01261e-15 1.5708
- joint l_wrist_frame: origin xyz=8.32667e-17 -0.225182 -0.0235 rpy=-1.5708 1.45366e-16 -1.5708 -> xyz=2.91434e-16 -0.225182 -0.0235 rpy=-1.5708 6.97876e-16 -1.5708
- joint r_cleat_l_back_frame: origin xyz=-0.030496 -0.00745064 -0.05025 rpy=9.51939e-16 -4.37921e-15 1.5708 -> xyz=-0.030496 -0.00745064 -0.05025 rpy=3.02062e-16 1.14651e-15 1.5708
- joint r_cleat_l_front_frame: origin xyz=-0.0305 0.177 -0.05025 rpy=4.65062e-17 1.10045e-14 1.5708 -> xyz=-0.0305 0.177 -0.05025 rpy=-1.09592e-15 3.40328e-16 1.5708
- joint r_cleat_r_back_frame: origin xyz=0.0595 -0.007 -0.05025 rpy=7.70805e-16 -3.07597e-15 1.5708 -> xyz=0.0595 -0.007 -0.05025 rpy=7.71897e-16 -3.20424e-15 1.5708
- joint r_cleat_r_front_frame: origin xyz=0.0595 0.177 -0.05025 rpy=2.69391e-16 -5.00011e-15 1.5708 -> xyz=0.0595 0.177 -0.05025 rpy=-1.69008e-16 -4.62076e-16 1.5708
- joint r_sole_frame: origin xyz=0.0152261 0.0907683 -0.0529 rpy=5.35395e-16 1.07005e-14 1.5708 -> xyz=0.0152261 0.0907683 -0.0529 rpy=3.33669e-15 3.2321e-14 1.5708
- joint r_wrist_frame: origin xyz=1.249e-16 -0.226182 -0.0235 rpy=1.5708 1.43787e-15 -1.5708 -> xyz=3.1225e-16 -0.226182 -0.0235 rpy=1.5708 7.31053e-15 -1.5708

Commit message: description: fix joint rotations

File: wolfgang_description/urdf/robot.urdf (robot description, URDF)
Before this commit: robot wolfgang, 37 links, 36 joints
Joints:
- joint LAnklePitch: axis 0 0 1 -> -0 -0 -1
- joint LAnkleRoll: axis 0 1 0 -> -0 -1 -0
- joint LHipPitch: axis -7.95491e-17 3.00167e-16 1 -> 7.95491e-17 -3.00167e-16 -1
- joint LHipRoll: axis 0 0 1 -> -0 -0 -1
- joint RAnklePitch: axis 0 0 1 -> -0 -0 -1
- joint RHipPitch: axis 0 -1 0 -> -0 1 -0
- joint RHipRoll: axis 0 0 1 -> -0 -0 -1

Commit message: description: add foot pressure sensors for gazebo, multiple fixes

File: wolfgang_description/urdf/robot.urdf (robot description, URDF)
Before this commit: robot wolfgang, 37 links, 36 joints
Links:
- removed link body_1
- removed link foot_left_1
- removed link foot_right_1
- removed link head_1
- removed link upper_leg_left_1
- removed link upper_leg_right_1
- added link head, mass 0.318645; collision mesh filename=package://wolfgang_description/urdf/basler_ace_gige_c-mount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; collision mesh filename=package://wolfgang_description/urdf/camera_lower_basler_wol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
- added link l_foot, mass 0.275133; collision mesh filename=package://wolfgang_description/urdf/ankle.stl; collision mesh filename=package://wolfgang_description/urdf/foot_cover.stl
- added link l_knee, mass 0.220799; collision mesh filename=package://wolfgang_description/urdf/knee_connector.stl; collision mesh filename=package://wolfgang_description/urdf/knee_connector.stl
- added link llb, mass 0.00165976; collision mesh filename=package://wolfgang_description/urdf/flex_stollen.stl; visual mesh filename=package://wolfgang_description/urdf/flex_stollen.stl
- added link llf, mass 0.00165976; collision mesh filename=package://wolfgang_description/urdf/flex_stollen.stl; visual mesh filename=package://wolfgang_description/urdf/flex_stollen.stl
- added link lrb, mass 0.00165976; collision mesh filename=package://wolfgang_description/urdf/flex_stollen.stl; visual mesh filename=package://wolfgang_description/urdf/flex_stollen.stl
- added link lrf, mass 0.00165976; collision mesh filename=package://wolfgang_description/urdf/flex_stollen.stl; visual mesh filename=package://wolfgang_description/urdf/flex_stollen.stl
- added link r_foot, mass 0.275133; collision mesh filename=package://wolfgang_description/urdf/ankle.stl; collision mesh filename=package://wolfgang_description/urdf/foot_cover.stl
- added link r_knee, mass 0.220799; collision mesh filename=package://wolfgang_description/urdf/knee_connector.stl; collision mesh filename=package://wolfgang_description/urdf/knee_connector.stl
- added link rlb, mass 0.00165976; collision mesh filename=package://wolfgang_description/urdf/flex_stollen.stl; visual mesh filename=package://wolfgang_description/urdf/flex_stollen.stl
- added link rlf, mass 0.00165976; collision mesh filename=package://wolfgang_description/urdf/flex_stollen.stl; visual mesh filename=package://wolfgang_description/urdf/flex_stollen.stl
- added link rrb, mass 0.00165976; collision mesh filename=package://wolfgang_description/urdf/flex_stollen.stl; visual mesh filename=package://wolfgang_description/urdf/flex_stollen.stl
- added link rrf, mass 0.00165976; collision mesh filename=package://wolfgang_description/urdf/flex_stollen.stl; visual mesh filename=package://wolfgang_description/urdf/flex_stollen.stl
- added link torso, mass 1.79116; collision mesh filename=package://wolfgang_description/urdf/baseplate_odroid_xu4_co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; collision mesh filename=package://wolfgang_description/urdf/battery_dummy.stl
Joints:
- added joint LLB: type fixed, parent l_foot, child llb, origin xyz=-0.06 -0.007 -0.03375 rpy=5.84053e-15 -4.62286e-15 -1.5708, axis 0 1.22465e-16 1, limit effort=0 velocity=0
- added joint LLF: type fixed, parent l_foot, child llf, origin xyz=-0.06 0.177 -0.03375 rpy=6.38353e-15 -4.80263e-15 -1.5708, axis 0 1.22465e-16 1, limit effort=0 velocity=0
- added joint LRB: type fixed, parent l_foot, child lrb, origin xyz=0.03 -0.007 -0.03375 rpy=-1.44208e-14 -1.69534e-14 -1.5708, axis 0 1.22465e-16 1, limit effort=0 velocity=0
- added joint LRF: type fixed, parent l_foot, child lrf, origin xyz=0.03 0.177 -0.03375 rpy=6.38353e-15 -4.80263e-15 -1.5708, axis 0 -1.22465e-16 -1, limit effort=0 velocity=0
- added joint RLB: type fixed, parent r_foot, child rlb, origin xyz=-0.029996 -0.00745064 -0.03425 rpy=-2.20568e-16 -1.47012e-15 -1.5708, axis 0 1.22465e-16 1, limit effort=0 velocity=0
- added joint RLF: type fixed, parent r_foot, child rlf, origin xyz=-0.03 0.177 -0.03425 rpy=-1.06437e-15 1.53365e-15 -1.5708, axis 0 1.22465e-16 1, limit effort=0 velocity=0
- added joint RRB: type fixed, parent r_foot, child rrb, origin xyz=0.06 -0.007 -0.03425 rpy=-1.81005e-15 5.43887e-14 -1.5708, axis 0 1.22465e-16 1, limit effort=0 velocity=0
- added joint RRF: type fixed, parent r_foot, child rrf, origin xyz=0.06 0.177 -0.03425 rpy=-8.29268e-17 1.38118e-15 -1.5708, axis 0 1.22465e-16 1, limit effort=0 velocity=0
- joint HeadPan: limit lower=-2.0944 upper=2.0944 effort=6 velocity=6 -> lower=-2.0944 upper=2.0944 effort=5.43 velocity=10.33; parent body_1 -> torso
- joint HeadTilt: child head_1 -> head; limit lower=0 upper=1.5708 effort=6 velocity=6 -> lower=0 upper=1.5708 effort=5.43 velocity=10.33
- joint LAnklePitch: limit lower=-1.22173 upper=1.5708 effort=9 velocity=9 -> lower=-1.22173 upper=1.5708 effort=7.57 velocity=8.22
- joint LAnkleRoll: child foot_left_1 -> l_foot; limit lower=-1.0472 upper=1.0472 effort=9 velocity=9 -> lower=-1.0472 upper=1.0472 effort=7.57 velocity=8.22
- joint LElbow: limit lower=-1.5708 upper=1.0472 effort=6 velocity=6 -> lower=-1.5708 upper=1.0472 effort=5.43 velocity=10.33
- joint LHipPitch: child upper_leg_left_1 -> l_knee; limit lower=-1.5708 upper=1.5708 effort=9 velocity=9 -> lower=-1.5708 upper=1.5708 effort=7.57 velocity=8.22
- joint LHipRoll: limit lower=-1.5708 upper=1.5708 effort=9 velocity=9 -> lower=-1.5708 upper=1.5708 effort=7.57 velocity=8.22
- joint LHipYaw: limit lower=-1.5708 upper=1.5708 effort=9 velocity=9 -> lower=-1.5708 upper=1.5708 effort=7.57 velocity=8.22; parent body_1 -> torso
- joint LKnee: parent upper_leg_left_1 -> l_knee
- joint LShoulderPitch: limit lower=-3.14159 upper=3.14159 effort=6 velocity=6 -> lower=-3.14159 upper=3.14159 effort=5.43 velocity=10.33; parent body_1 -> torso
- joint LShoulderRoll: limit lower=0 upper=3.14159 effort=6 velocity=6 -> lower=0 upper=3.14159 effort=5.43 velocity=10.33
- joint RAnklePitch: limit lower=-1.22173 upper=1.5708 effort=9 velocity=9 -> lower=-1.22173 upper=1.5708 effort=7.57 velocity=8.22
- joint RAnkleRoll: child foot_right_1 -> r_foot; limit lower=-1.0472 upper=1.0472 effort=9 velocity=9 -> lower=-1.0472 upper=1.0472 effort=7.57 velocity=8.22
- joint RElbow: limit lower=-1.0472 upper=1.5708 effort=6 velocity=6 -> lower=-1.0472 upper=1.5708 effort=5.43 velocity=10.33
- joint RHipPitch: child upper_leg_right_1 -> r_knee; limit lower=-1.5708 upper=1.5708 effort=9 velocity=9 -> lower=-1.5708 upper=1.5708 effort=7.57 velocity=8.22
- joint RHipRoll: limit lower=-1.5708 upper=1.5708 effort=9 velocity=9 -> lower=-1.5708 upper=1.5708 effort=7.57 velocity=8.22
- joint RHipYaw: limit lower=-1.5708 upper=1.5708 effort=9 velocity=9 -> lower=-1.5708 upper=1.5708 effort=7.57 velocity=8.22; parent body_1 -> torso
- joint RKnee: parent upper_leg_right_1 -> r_knee
- joint RShoulderPitch: limit lower=-3.14159 upper=3.14159 effort=6 velocity=6 -> lower=-3.14159 upper=3.14159 effort=5.43 velocity=10.33; parent body_1 -> torso
- joint RShoulderRoll: limit lower=-3.14159 upper=0 effort=6 velocity=6 -> lower=-3.14159 upper=0 effort=5.43 velocity=10.33
- joint base_link_to_base: child body_1 -> torso
- joint camera_frame: parent head_1 -> head
- joint camera_optical_frame_frame: parent head_1 -> head
- joint imu_frame_frame: parent body_1 -> torso
- joint l_cleat_l_back_frame: origin xyz=-0.0605 -0.007 -0.04975 rpy=-2.04856e-14 -2.56773e-14 1.5708 -> xyz=5.55112e-17 -0.0005 -0.016 rpy=1.97551e-16 -1.05004e-19 3.14159; parent foot_left_1 -> llb
- joint l_cleat_l_front_frame: origin xyz=-0.0605 0.177 -0.04975 rpy=-6.55214e-15 4.2513e-15 1.5708 -> xyz=8.32667e-17 -0.0005 -0.016 rpy=3.01686e-16 1.58286e-16 -3.14159; parent foot_left_1 -> llf
- joint l_cleat_r_back_frame: origin xyz=0.0295 -0.007 -0.04975 rpy=-3.99384e-16 1.98982e-15 1.5708 -> xyz=4.16334e-17 -0.0005 -0.016 rpy=2.92719e-16 -1.39845e-17 -3.14159; parent foot_left_1 -> lrb
- joint l_cleat_r_front_frame: origin xyz=0.0295 0.177 -0.04975 rpy=-6.55214e-15 4.2513e-15 1.5708 -> xyz=2.77556e-17 -0.0005 -0.016 rpy=3.30992e-16 -5.1163e-16 3.14159; parent foot_left_1 -> lrf
- joint l_sole_frame: parent foot_left_1 -> l_foot
- joint r_cleat_l_back_frame: origin xyz=-0.030496 -0.00745064 -0.05025 rpy=3.02062e-16 1.14651e-15 1.5708 -> xyz=-1.38778e-17 -0.0005 -0.016 rpy=8.14947e-17 -2.98734e-16 -3.14159; parent foot_right_1 -> rlb
- joint r_cleat_l_front_frame: origin xyz=-0.0305 0.177 -0.05025 rpy=-1.09592e-15 3.40328e-16 1.5708 -> xyz=-4.16334e-17 -0.0005 -0.016 rpy=2.82194e-16 1.83866e-15 3.14159; parent foot_right_1 -> rlf
- joint r_cleat_r_back_frame: origin xyz=0.0595 -0.007 -0.05025 rpy=7.71897e-16 -3.20424e-15 1.5708 -> xyz=-6.93889e-17 -0.0005 -0.016 rpy=2.94118e-16 4.11997e-17 -3.14159; parent foot_right_1 -> rrb
- joint r_cleat_r_front_frame: origin xyz=0.0595 0.177 -0.05025 rpy=-1.69008e-16 -4.62076e-16 1.5708 -> xyz=-2.80331e-15 -0.0005 -0.016 rpy=2.75421e-16 9.25503e-16 3.14159; parent foot_right_1 -> rrf
- joint r_sole_frame: parent foot_right_1 -> r_foot
