Commit message: simplify model for more performance. improve dynamic model

File: wolfgang_description/urdf/robot.urdf (robot description, URDF)
Before this commit: robot wolfgang, 45 links, 44 joints
Links:
- link head: geometry collision mesh filename=package://wolfgang_description/urdf/basler_ace_gige_c-mount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; collision mesh filename=package://wolfgang_description/urdf/camera_lower_basler_wol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
- link hip_u_connector_1: geometry collision mesh filename=package://wolfgang_description/urdf/hip_u_connector.stl; visual mesh filename=package://wolfgang_description/urdf/hip_u_connector_1.stl
- link hip_u_connector_2: geometry collision mesh filename=package://wolfgang_description/urdf/hip_u_connector.stl; visual mesh filename=package://wolfgang_description/urdf/hip_u_connector_2.stl
- link l_foot: geometry collision mesh filename=package://wolfgang_description/urdf/ankle.stl; collision mesh filename=package://wolfgang_description/urdf/foot_cover.stl
- link l_knee: geometry collision mesh filename=package://wolfgang_description/urdf/knee_connector.stl; collision mesh filename=package://wolfgang_description/urdf/knee_connector.stl
- link left_hip_right_ankle_1: geometry collision mesh filename=package://wolfgang_description/urdf/motor_connector.stl; collision mesh filename=package://wolfgang_description/urdf/motor_connector.stl
- link left_hip_right_ankle_2: geometry collision mesh filename=package://wolfgang_description/urdf/motor_connector.stl; collision mesh filename=package://wolfgang_description/urdf/motor_connector.stl
- link llb: geometry collision mesh filename=package://wolfgang_description/urdf/flex_stollen.stl; visual mesh filename=package://wolfgang_description/urdf/llb.stl
- link llf: geometry collision mesh filename=package://wolfgang_description/urdf/flex_stollen.stl; visual mesh filename=package://wolfgang_description/urdf/llf.stl
- link lower_arm_left_1: geometry collision mesh filename=package://wolfgang_description/urdf/hand.stl; collision mesh filename=package://wolfgang_description/urdf/lower_arm.stl
- link lower_arm_right_1: geometry collision mesh filename=package://wolfgang_description/urdf/hand.stl; collision mesh filename=package://wolfgang_description/urdf/lower_arm.stl
- link lower_leg_left_1: geometry collision mesh filename=package://wolfgang_description/urdf/knee_spacer.stl; collision mesh filename=package://wolfgang_description/urdf/knee_spacer.stl
- link lower_leg_right_1: geometry collision mesh filename=package://wolfgang_description/urdf/knee_spacer.stl; collision mesh filename=package://wolfgang_description/urdf/knee_spacer.stl
- link lrb: geometry collision mesh filename=package://wolfgang_description/urdf/flex_stollen.stl; visual mesh filename=package://wolfgang_description/urdf/lrb.stl
- link lrf: geometry collision mesh filename=package://wolfgang_description/urdf/flex_stollen.stl; visual mesh filename=package://wolfgang_description/urdf/lrf.stl
- link neck_1: geometry collision mesh filename=package://wolfgang_description/urdf/connector_shoulder.stl; collision mesh filename=package://wolfgang_description/urdf/mx-64-body.stl
- link r_foot: geometry collision mesh filename=package://wolfgang_description/urdf/ankle.stl; collision mesh filename=package://wolfgang_description/urdf/foot_cover.stl
- link r_knee: geometry collision mesh filename=package://wolfgang_description/urdf/knee_connector.stl; collision mesh filename=package://wolfgang_description/urdf/knee_connector.stl
- link right_hip_left_ankle_1: geometry collision mesh filename=package://wolfgang_description/urdf/motor_connector.stl; collision mesh filename=package://wolfgang_description/urdf/motor_connector.stl
- link right_hip_left_ankle_2: geometry collision mesh filename=package://wolfgang_description/urdf/motor_connector.stl; collision mesh filename=package://wolfgang_description/urdf/motor_connector.stl
- link rlb: geometry collision mesh filename=package://wolfgang_description/urdf/flex_stollen.stl; visual mesh filename=package://wolfgang_description/urdf/rlb.stl
- link rlf: geometry collision mesh filename=package://wolfgang_description/urdf/flex_stollen.stl; visual mesh filename=package://wolfgang_description/urdf/rlf.stl
- link rrb: geometry collision mesh filename=package://wolfgang_description/urdf/flex_stollen.stl; visual mesh filename=package://wolfgang_description/urdf/rrb.stl
- link rrf: geometry collision mesh filename=package://wolfgang_description/urdf/flex_stollen.stl; visual mesh filename=package://wolfgang_description/urdf/rrf.stl
- link shoulder_left_1: geometry collision mesh filename=package://wolfgang_description/urdf/sea_connector.stl; collision mesh filename=package://wolfgang_description/urdf/sea_ninjaflex.stl
- link shoulder_right_1: geometry collision mesh filename=package://wolfgang_description/urdf/sea_connector.stl; collision mesh filename=package://wolfgang_description/urdf/sea_ninjaflex.stl
- link torso: mass 1.79116 -> 2.03749; geometry collision mesh filename=package://wolfgang_description/urdf/baseplate_odroid_xu4_co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; collision mesh filename=package://wolfgang_description/urdf/battery_dummy.stl
- link upper_arm_1: geometry collision mesh filename=package://wolfgang_description/urdf/connector_shoulder.stl; collision mesh filename=package://wolfgang_description/urdf/connector_shoulder.stl
- link upper_arm_2: geometry collision mesh filename=package://wolfgang_description/urdf/connector_shoulder.stl; collision mesh filename=package://wolfgang_description/urdf/connector_shoulder.stl

Commit message: fix base link ineratia to zero, to prevent problems with pybullet

File: wolfgang_description/urdf/robot.urdf (robot description, URDF)
Before this commit: robot wolfgang, 45 links, 44 joints
Links:
- link base_link: mass None -> 0.0001

Commit message: corrected some link names

File: wolfgang_description/urdf/robot.urdf (robot description, URDF)
Before this commit: robot wolfgang, 45 links, 44 joints
Links:
- removed link hip_u_connector_1
- removed link hip_u_connector_2
- removed link l_knee
- removed link left_hip_right_ankle_1
- removed link left_hip_right_ankle_2
- removed link lower_arm_left_1
- removed link lower_arm_right_1
- removed link lower_leg_left_1
- removed link lower_leg_right_1
- removed link neck_1
- removed link r_knee
- removed link right_hip_left_ankle_1
- removed link right_hip_left_ankle_2
- removed link shoulder_left_1
- removed link shoulder_right_1
- removed link upper_arm_1
- removed link upper_arm_2
- added link l_ankle, mass 0.319807; collision mesh filename=package://wolfgang_description/urdf/motor_connector.stl; collision mesh filename=package://wolfgang_description/urdf/motor_connector.stl
- added link l_hip_1, mass 0.0689735; collision mesh filename=package://wolfgang_description/urdf/hip_u_connector.stl; visual mesh filename=package://wolfgang_description/urdf/l_hip_1.stl
- added link l_hip_2, mass 0.319807; collision mesh filename=package://wolfgang_description/urdf/motor_connector.stl; collision mesh filename=package://wolfgang_description/urdf/motor_connector.stl
- added link l_lower_arm, mass 0.207774; collision mesh filename=package://wolfgang_description/urdf/hand.stl; collision mesh filename=package://wolfgang_description/urdf/lower_arm.stl
- added link l_lower_leg, mass 0.0842512; collision mesh filename=package://wolfgang_description/urdf/knee_spacer.stl; collision mesh filename=package://wolfgang_description/urdf/knee_spacer.stl
- added link l_shoulder, mass 0.041445; collision mesh filename=package://wolfgang_description/urdf/sea_connector.stl; collision mesh filename=package://wolfgang_description/urdf/sea_ninjaflex.stl
- added link l_upper_arm, mass 0.206164; collision mesh filename=package://wolfgang_description/urdf/connector_shoulder.stl; collision mesh filename=package://wolfgang_description/urdf/connector_shoulder.stl
- added link l_upper_leg, mass 0.220799; collision mesh filename=package://wolfgang_description/urdf/knee_connector.stl; collision mesh filename=package://wolfgang_description/urdf/knee_connector.stl
- added link neck, mass 0.148233; collision mesh filename=package://wolfgang_description/urdf/connector_shoulder.stl; collision mesh filename=package://wolfgang_description/urdf/mx-64-body.stl
- added link r_ankle, mass 0.319807; collision mesh filename=package://wolfgang_description/urdf/motor_connector.stl; collision mesh filename=package://wolfgang_description/urdf/motor_connector.stl
- added link r_hip_1, mass 0.0689735; collision mesh filename=package://wolfgang_description/urdf/hip_u_connector.stl; visual mesh filename=package://wolfgang_description/urdf/r_hip_1.stl
- added link r_hip_2, mass 0.319807; collision mesh filename=package://wolfgang_description/urdf/motor_connector.stl; collision mesh filename=package://wolfgang_description/urdf/motor_connector.stl
- added link r_lower_arm, mass 0.207774; collision mesh filename=package://wolfgang_description/urdf/hand.stl; collision mesh filename=package://wolfgang_description/urdf/lower_arm.stl
- added link r_lower_leg, mass 0.0842452; collision mesh filename=package://wolfgang_description/urdf/knee_spacer.stl; collision mesh filename=package://wolfgang_description/urdf/knee_spacer.stl
- added link r_shoulder, mass 0.041445; collision mesh filename=package://wolfgang_description/urdf/sea_connector.stl; collision mesh filename=package://wolfgang_description/urdf/sea_ninjaflex.stl
- added link r_upper_arm, mass 0.206164; collision mesh filename=package://wolfgang_description/urdf/connector_shoulder.stl; collision mesh filename=package://wolfgang_description/urdf/connector_shoulder.stl
- added link r_upper_leg, mass 0.220799; collision mesh filename=package://wolfgang_description/urdf/knee_connector.stl; collision mesh filename=package://wolfgang_description/urdf/knee_connector.stl
Joints:
- joint HeadPan: child neck_1 -> neck
- joint HeadTilt: parent neck_1 -> neck
- joint LAnklePitch: child right_hip_left_ankle_2 -> l_ankle; parent lower_leg_left_1 -> l_lower_leg
- joint LAnkleRoll: parent right_hip_left_ankle_2 -> l_ankle
- joint LElbow: child lower_arm_left_1 -> l_lower_arm; parent upper_arm_2 -> l_upper_arm
- joint LHipPitch: child l_knee -> l_upper_leg; parent left_hip_right_ankle_2 -> l_hip_2
- joint LHipRoll: child left_hip_right_ankle_2 -> l_hip_2; parent hip_u_connector_2 -> l_hip_1
- joint LHipYaw: child hip_u_connector_2 -> l_hip_1
- joint LKnee: child lower_leg_left_1 -> l_lower_leg; parent l_knee -> l_upper_leg
- joint LShoulderPitch: child shoulder_left_1 -> l_shoulder
- joint LShoulderRoll: child upper_arm_2 -> l_upper_arm; parent shoulder_left_1 -> l_shoulder
- joint RAnklePitch: child left_hip_right_ankle_1 -> r_ankle; parent lower_leg_right_1 -> r_lower_leg
- joint RAnkleRoll: parent left_hip_right_ankle_1 -> r_ankle
- joint RElbow: child lower_arm_right_1 -> r_lower_arm; parent upper_arm_1 -> r_upper_arm
- joint RHipPitch: child r_knee -> r_upper_leg; parent right_hip_left_ankle_1 -> r_hip_2
- joint RHipRoll: child right_hip_left_ankle_1 -> r_hip_2; parent hip_u_connector_1 -> r_hip_1
- joint RHipYaw: child hip_u_connector_1 -> r_hip_1
- joint RKnee: child lower_leg_right_1 -> r_lower_leg; parent r_knee -> r_upper_leg
- joint RShoulderPitch: child shoulder_right_1 -> r_shoulder
- joint RShoulderRoll: child upper_arm_1 -> r_upper_arm; parent shoulder_right_1 -> r_shoulder
- joint l_wrist_frame: parent lower_arm_left_1 -> l_lower_arm
- joint r_wrist_frame: parent lower_arm_right_1 -> r_lower_arm

Commit message: update model

File: wolfgang_description/urdf/robot.urdf (robot description, URDF)
Before this commit: robot wolfgang, 45 links, 44 joints
Links:
- link head: geometry collision mesh filename=package://wolfgang_description/urdf/head.stl; visual mesh filename=package://wolfgang_description/urdf/head.stl
- link l_ankle: geometry collision mesh filename=package://wolfgang_description/urdf/l_ankle.stl; visual mesh filename=package://wolfgang_description/urdf/l_ankle.stl
- link l_foot: geometry collision mesh filename=package://wolfgang_description/urdf/l_foot.stl; visual mesh filename=package://wolfgang_description/urdf/l_foot.stl
- link l_hip_1: geometry collision mesh filename=package://wolfgang_description/urdf/l_hip_1.stl; visual mesh filename=package://wolfgang_description/urdf/l_hip_1.stl
- link l_hip_2: geometry collision mesh filename=package://wolfgang_description/urdf/l_hip_2.stl; visual mesh filename=package://wolfgang_description/urdf/l_hip_2.stl
- link l_lower_arm: geometry collision mesh filename=package://wolfgang_description/urdf/l_lower_arm.stl; visual mesh filename=package://wolfgang_description/urdf/l_lower_arm.stl
- link l_lower_leg: geometry collision mesh filename=package://wolfgang_description/urdf/l_lower_leg.stl; visual mesh filename=package://wolfgang_description/urdf/l_lower_leg.stl
- link l_shoulder: geometry collision mesh filename=package://wolfgang_description/urdf/l_shoulder.stl; visual mesh filename=package://wolfgang_description/urdf/l_shoulder.stl
- link l_upper_arm: geometry collision mesh filename=package://wolfgang_description/urdf/l_upper_arm.stl; visual mesh filename=package://wolfgang_description/urdf/l_upper_arm.stl
- link l_upper_leg: geometry collision mesh filename=package://wolfgang_description/urdf/l_upper_leg.stl; visual mesh filename=package://wolfgang_description/urdf/l_upper_leg.stl
- link llb: geometry collision mesh filename=package://wolfgang_description/urdf/llb.stl; visual mesh filename=package://wolfgang_description/urdf/llb.stl
- link llf: geometry collision mesh filename=package://wolfgang_description/urdf/llf.stl; visual mesh filename=package://wolfgang_description/urdf/llf.stl
- link lrb: geometry collision mesh filename=package://wolfgang_description/urdf/lrb.stl; visual mesh filename=package://wolfgang_description/urdf/lrb.stl
- link lrf: geometry collision mesh filename=package://wolfgang_description/urdf/lrf.stl; visual mesh filename=package://wolfgang_description/urdf/lrf.stl
- link neck: geometry collision mesh filename=package://wolfgang_description/urdf/neck.stl; visual mesh filename=package://wolfgang_description/urdf/neck.stl
- link r_ankle: geometry collision mesh filename=package://wolfgang_description/urdf/r_ankle.stl; visual mesh filename=package://wolfgang_description/urdf/r_ankle.stl
- link r_foot: geometry collision mesh filename=package://wolfgang_description/urdf/r_foot.stl; visual mesh filename=package://wolfgang_description/urdf/r_foot.stl
- link r_hip_1: geometry collision mesh filename=package://wolfgang_description/urdf/r_hip_1.stl; visual mesh filename=package://wolfgang_description/urdf/r_hip_1.stl
- link r_hip_2: geometry collision mesh filename=package://wolfgang_description/urdf/r_hip_2.stl; visual mesh filename=package://wolfgang_description/urdf/r_hip_2.stl
- link r_lower_arm: geometry collision mesh filename=package://wolfgang_description/urdf/r_lower_arm.stl; visual mesh filename=package://wolfgang_description/urdf/r_lower_arm.stl
- link r_lower_leg: geometry collision mesh filename=package://wolfgang_description/urdf/r_lower_leg.stl; visual mesh filename=package://wolfgang_description/urdf/r_lower_leg.stl
- link r_shoulder: geometry collision mesh filename=package://wolfgang_description/urdf/r_shoulder.stl; visual mesh filename=package://wolfgang_description/urdf/r_shoulder.stl
- link r_upper_arm: geometry collision mesh filename=package://wolfgang_description/urdf/r_upper_arm.stl; visual mesh filename=package://wolfgang_description/urdf/r_upper_arm.stl
- link r_upper_leg: geometry collision mesh filename=package://wolfgang_description/urdf/r_upper_leg.stl; visual mesh filename=package://wolfgang_description/urdf/r_upper_leg.stl
- link rlb: geometry collision mesh filename=package://wolfgang_description/urdf/rlb.stl; visual mesh filename=package://wolfgang_description/urdf/rlb.stl
- link rlf: geometry collision mesh filename=package://wolfgang_description/urdf/rlf.stl; visual mesh filename=package://wolfgang_description/urdf/rlf.stl
- link rrb: geometry collision mesh filename=package://wolfgang_description/urdf/rrb.stl; visual mesh filename=package://wolfgang_description/urdf/rrb.stl
- link rrf: geometry collision mesh filename=package://wolfgang_description/urdf/rrf.stl; visual mesh filename=package://wolfgang_description/urdf/rrf.stl
- link torso: geometry collision mesh filename=package://wolfgang_description/urdf/torso.stl; visual mesh filename=package://wolfgang_description/urdf/torso.stl

Commit message: description: updated wolfgang urdf

File: wolfgang_description/urdf/robot.urdf (robot description, URDF)
Before this commit: robot wolfgang, 45 links, 44 joints
Links:
- added link imu_frame_2, mass 1e-9
- link head: mass 0.318645 -> 0.301358
- link l_foot: mass 0.275133 -> 0.267778
- link l_lower_leg: mass 0.0842512 -> 0.112624
- link l_upper_arm: mass 0.206164 -> 0.228498
- link l_upper_leg: mass 0.220799 -> 0.242311
- link r_foot: mass 0.275133 -> 0.267778
- link r_lower_leg: mass 0.0842452 -> 0.112618
- link r_upper_arm: mass 0.206164 -> 0.228498
- link r_upper_leg: mass 0.220799 -> 0.242311
- link torso: mass 2.03749 -> 2.03744
Joints:
- added joint imu_frame_2_frame: type fixed, parent head, child imu_frame_2, origin xyz=-0.02545 0.0535 -0.0235 rpy=-1.5708 -3.88578e-16 3.33067e-16, axis 0 0 0
- joint HeadTilt: limit lower=0 upper=1.5708 effort=5.43 velocity=10.33 -> lower=-0.523599 upper=1.5708 effort=5.43 velocity=10.33
- joint LAnklePitch: origin xyz=3.5319e-15 -0.0505 -0.17 rpy=-1.5708 -8.72457e-16 3.14159 -> xyz=1.11022e-16 -0.0505 -0.17 rpy=-1.5708 -1.45847e-15 3.14159
- joint LAnkleRoll: origin xyz=0.0691 2.22045e-16 -0.026 rpy=1.5708 -1.5708 0 -> xyz=0.0691 1.66533e-16 -0.026 rpy=1.5708 -1.5708 0
- joint LHipRoll: origin xyz=-0.046 0.0414 -7.97973e-16 rpy=3.14159 1.5708 0 -> xyz=-0.046 0.0414 6.93889e-18 rpy=3.14159 1.5708 0
- joint LHipYaw: origin xyz=-2.28983e-16 0.055 2.71051e-18 rpy=-1.5708 -0 0 -> xyz=1.82493e-15 0.055 -4.22839e-18 rpy=-1.5708 -0 0
- joint LKnee: origin xyz=0.00435596 -0.168793 0.049 rpy=1.5708 -1.75248e-15 2.87979 -> xyz=0.00435596 -0.168793 0.049 rpy=1.5708 -4.90478e-17 2.87979
- joint LLB: origin xyz=-0.06 -0.007 -0.03375 rpy=5.84053e-15 -4.62286e-15 -1.5708 -> xyz=-0.06 -0.007 -0.034 rpy=1.75801e-15 -5.02709e-15 -1.5708
- joint LLF: origin xyz=-0.06 0.177 -0.03375 rpy=6.38353e-15 -4.80263e-15 -1.5708 -> xyz=-0.06 0.177 -0.034 rpy=2.68959e-15 -5.26048e-15 -1.5708
- joint LRB: origin xyz=0.03 -0.007 -0.03375 rpy=-1.44208e-14 -1.69534e-14 -1.5708 -> xyz=0.03 -0.007 -0.034 rpy=-1.44208e-14 -1.69268e-14 -1.5708
- joint LRF: origin xyz=0.03 0.177 -0.03375 rpy=6.38353e-15 -4.80263e-15 -1.5708 -> xyz=0.03 0.177 -0.034 rpy=2.68959e-15 -5.26048e-15 -1.5708
- joint LShoulderPitch: axis 0 -1 0 -> -0 1 -0
- joint RAnklePitch: limit lower=-1.22173 upper=1.5708 effort=7.57 velocity=8.22 -> lower=-1.5708 upper=1.22173 effort=7.57 velocity=8.22; origin xyz=2.69229e-15 0.0505 -0.17 rpy=-1.5708 -1.93533e-15 -2.52888e-15 -> xyz=4.23273e-16 0.0505 -0.17 rpy=-1.5708 -7.47915e-15 1.91582e-15
- joint RAnkleRoll: origin xyz=-0.0691 5.55112e-17 -0.026 rpy=1.5708 1.5708 0 -> xyz=-0.0691 0 -0.026 rpy=1.5708 1.5708 0
- joint RHipRoll: origin xyz=-0.046 0.0414 5.34295e-16 rpy=-3.14159 1.5708 0 -> xyz=-0.046 0.0414 6.93889e-18 rpy=-3.14159 1.5708 0
- joint RHipYaw: origin xyz=-1.38778e-17 -0.055 -9.75782e-19 rpy=-1.5708 -0 0 -> xyz=-1.33227e-15 -0.055 -7.91468e-18 rpy=-1.5708 -0 0
- joint RKnee: origin xyz=-0.00392295 -0.051 -0.169043 rpy=1.50246e-15 -0.261799 -1.61204e-15 -> xyz=-0.00392295 -0.051 -0.169043 rpy=1.05132e-15 -0.261799 -2.52921e-15
- joint RLB: origin xyz=-0.029996 -0.00745064 -0.03425 rpy=-2.20568e-16 -1.47012e-15 -1.5708 -> xyz=-0.03 -0.007 -0.034 rpy=-2.20568e-16 -1.44743e-15 -1.5708
- joint RLF: origin xyz=-0.03 0.177 -0.03425 rpy=-1.06437e-15 1.53365e-15 -1.5708 -> xyz=-0.03 0.177 -0.034 rpy=-1.06437e-15 1.50083e-15 -1.5708
- joint RRB: origin xyz=0.06 -0.007 -0.03425 rpy=-1.81005e-15 5.43887e-14 -1.5708 -> xyz=0.06 -0.007 -0.034 rpy=-1.81005e-15 5.43559e-14 -1.5708
- joint RRF: origin xyz=0.06 0.177 -0.03425 rpy=-8.29268e-17 1.38118e-15 -1.5708 -> xyz=0.06 0.177 -0.034 rpy=-8.29268e-17 1.40387e-15 -1.5708
- joint RShoulderPitch: axis 0 -1 0 -> -0 1 -0
- joint imu_frame_frame: origin xyz=-0.0367504 -0.0478024 0.224 rpy=5.31321e-16 -3.12873e-17 4.65401e-17 -> xyz=-0.0369597 -0.0475181 0.224 rpy=5.31321e-16 -3.12873e-17 4.65401e-17
- joint l_cleat_l_back_frame: origin xyz=5.55112e-17 -0.0005 -0.016 rpy=1.97551e-16 -1.05004e-19 3.14159 -> xyz=1.38778e-17 -0.0005 -0.016 rpy=1.67348e-16 -4.15297e-16 3.14159
- joint l_cleat_l_front_frame: origin xyz=8.32667e-17 -0.0005 -0.016 rpy=3.01686e-16 1.58286e-16 -3.14159 -> xyz=0 -0.0005 -0.016 rpy=3.06162e-16 -4.4319e-17 -3.14159
- joint l_cleat_r_back_frame: origin xyz=4.16334e-17 -0.0005 -0.016 rpy=2.92719e-16 -1.39845e-17 -3.14159 -> xyz=0 -0.0005 -0.016 rpy=2.92719e-16 -4.05989e-17 -3.14159
- joint l_cleat_r_front_frame: origin xyz=2.77556e-17 -0.0005 -0.016 rpy=3.30992e-16 -5.1163e-16 3.14159 -> xyz=0 -0.0005 -0.016 rpy=3.00788e-16 -1.03785e-15 -3.14159
- joint l_sole_frame: origin xyz=-0.0152261 0.0907683 -0.0529 rpy=-5.77818e-15 -7.01261e-15 1.5708 -> xyz=-0.0152219 0.0907683 -0.0529 rpy=-5.77818e-15 -6.98371e-15 1.5708
- joint r_cleat_l_back_frame: origin xyz=-1.38778e-17 -0.0005 -0.016 rpy=8.14947e-17 -2.98734e-16 -3.14159 -> xyz=0 -0.0005 -0.016 rpy=8.14947e-17 -3.2143e-16 -3.14159
- joint r_cleat_l_front_frame: origin xyz=-4.16334e-17 -0.0005 -0.016 rpy=2.82194e-16 1.83866e-15 3.14159 -> xyz=-1.38778e-17 -0.0005 -0.016 rpy=3.37705e-16 1.87148e-15 3.14159
- joint r_cleat_r_back_frame: origin xyz=-6.93889e-17 -0.0005 -0.016 rpy=2.94118e-16 4.11997e-17 -3.14159 -> xyz=1.38778e-17 -0.0005 -0.016 rpy=2.94118e-16 7.40154e-17 3.14159
- joint r_cleat_r_front_frame: origin xyz=-2.80331e-15 -0.0005 -0.016 rpy=2.75421e-16 9.25503e-16 3.14159 -> xyz=-1.38778e-17 -0.0005 -0.016 rpy=2.75421e-16 9.31542e-16 3.14159
- joint r_sole_frame: origin xyz=0.0152261 0.0907683 -0.0529 rpy=3.33669e-15 3.2321e-14 1.5708 -> xyz=0.0152219 0.0907683 -0.0529 rpy=3.33669e-15 3.22983e-14 1.5708
