Commit message: update stls

File: wolfgang_description/urdf/robot.urdf (robot description, URDF)
Before this commit: robot wolfgang, 46 links, 45 joints
Links:
- link head: geometry collision mesh filename=package://wolfgang_description/urdf/basler_ace_gige_c-mount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; collision mesh filename=package://wolfgang_description/urdf/camera_lower_basler_wol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
- link l_ankle: geometry collision mesh filename=package://wolfgang_description/urdf/motor_connector.stl; collision mesh filename=package://wolfgang_description/urdf/motor_connector.stl
- link l_foot: mass 0.267778 -> 0.267613; geometry collision mesh filename=package://wolfgang_description/urdf/ankle.stl; collision mesh filename=package://wolfgang_description/urdf/foot_cover.stl
- link l_hip_1: geometry collision mesh filename=package://wolfgang_description/urdf/hip_u_connector.stl; visual mesh filename=package://wolfgang_description/urdf/l_hip_1.stl
- link l_hip_2: geometry collision mesh filename=package://wolfgang_description/urdf/motor_connector.stl; collision mesh filename=package://wolfgang_description/urdf/motor_connector.stl
- link l_lower_arm: geometry collision mesh filename=package://wolfgang_description/urdf/hand.stl; collision mesh filename=package://wolfgang_description/urdf/lower_arm.stl
- link l_lower_leg: geometry collision mesh filename=package://wolfgang_description/urdf/knee_spacer.stl; collision mesh filename=package://wolfgang_description/urdf/knee_spacer.stl
- link l_shoulder: geometry collision mesh filename=package://wolfgang_description/urdf/sea_connector.stl; collision mesh filename=package://wolfgang_description/urdf/sea_ninjaflex.stl
- link l_upper_arm: geometry collision mesh filename=package://wolfgang_description/urdf/connector_shoulder.stl; collision mesh filename=package://wolfgang_description/urdf/connector_shoulder.stl
- link l_upper_leg: geometry collision mesh filename=package://wolfgang_description/urdf/knee_connector.stl; collision mesh filename=package://wolfgang_description/urdf/knee_connector.stl
- link llb: geometry collision mesh filename=package://wolfgang_description/urdf/flex_stollen.stl; visual mesh filename=package://wolfgang_description/urdf/llb.stl
- link llf: geometry collision mesh filename=package://wolfgang_description/urdf/flex_stollen.stl; visual mesh filename=package://wolfgang_description/urdf/llf.stl
- link lrb: geometry collision mesh filename=package://wolfgang_description/urdf/flex_stollen.stl; visual mesh filename=package://wolfgang_description/urdf/lrb.stl
- link lrf: geometry collision mesh filename=package://wolfgang_description/urdf/flex_stollen.stl; visual mesh filename=package://wolfgang_description/urdf/lrf.stl
- link neck: geometry collision mesh filename=package://wolfgang_description/urdf/connector_shoulder.stl; collision mesh filename=package://wolfgang_description/urdf/mx-64-body.stl
- link r_ankle: geometry collision mesh filename=package://wolfgang_description/urdf/motor_connector.stl; collision mesh filename=package://wolfgang_description/urdf/motor_connector.stl
- link r_foot: mass 0.267778 -> 0.267613; geometry collision mesh filename=package://wolfgang_description/urdf/ankle.stl; collision mesh filename=package://wolfgang_description/urdf/foot_cover.stl
- link r_hip_1: geometry collision mesh filename=package://wolfgang_description/urdf/hip_u_connector.stl; visual mesh filename=package://wolfgang_description/urdf/r_hip_1.stl
- link r_hip_2: geometry collision mesh filename=package://wolfgang_description/urdf/motor_connector.stl; collision mesh filename=package://wolfgang_description/urdf/motor_connector.stl
- link r_lower_arm: geometry collision mesh filename=package://wolfgang_description/urdf/hand.stl; collision mesh filename=package://wolfgang_description/urdf/lower_arm.stl
- link r_lower_leg: geometry collision mesh filename=package://wolfgang_description/urdf/knee_spacer.stl; collision mesh filename=package://wolfgang_description/urdf/knee_spacer.stl
- link r_shoulder: geometry collision mesh filename=package://wolfgang_description/urdf/sea_connector.stl; collision mesh filename=package://wolfgang_description/urdf/sea_ninjaflex.stl
- link r_upper_arm: geometry collision mesh filename=package://wolfgang_description/urdf/connector_shoulder.stl; collision mesh filename=package://wolfgang_description/urdf/connector_shoulder.stl
- link r_upper_leg: geometry collision mesh filename=package://wolfgang_description/urdf/knee_connector.stl; collision mesh filename=package://wolfgang_description/urdf/knee_connector.stl
- link rlb: geometry collision mesh filename=package://wolfgang_description/urdf/flex_stollen.stl; visual mesh filename=package://wolfgang_description/urdf/rlb.stl
- link rlf: geometry collision mesh filename=package://wolfgang_description/urdf/flex_stollen.stl; visual mesh filename=package://wolfgang_description/urdf/rlf.stl
- link rrb: geometry collision mesh filename=package://wolfgang_description/urdf/flex_stollen.stl; visual mesh filename=package://wolfgang_description/urdf/rrb.stl
- link rrf: geometry collision mesh filename=package://wolfgang_description/urdf/flex_stollen.stl; visual mesh filename=package://wolfgang_description/urdf/rrf.stl
- link torso: mass 2.03744 -> 2.21811; geometry collision mesh filename=package://wolfgang_description/urdf/baseplate_odroid_xu4_co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; collision mesh filename=package://wolfgang_description/urdf/battery.stl
Joints:
- joint LKnee: axis 0 -1 0 -> -0 1 -0; limit lower=-2.96706 upper=0 effort=10 velocity=10 -> lower=0 upper=2.96706 effort=10 velocity=10
- joint LShoulderRoll: axis 0 0 1 -> -0 -0 -1
- joint RKnee: axis 0 1 0 -> -0 -1 -0; limit lower=0 upper=2.96706 effort=10 velocity=10 -> lower=-2.96706 upper=0 effort=10 velocity=10
- joint RShoulderRoll: axis 0 0 1 -> -0 -0 -1
- joint imu_frame_frame: origin xyz=-0.0369597 -0.0475181 0.224 rpy=5.31321e-16 -3.12873e-17 4.65401e-17 -> xyz=-0.0369749 -0.0474614 0.224 rpy=5.31321e-16 -3.12873e-17 4.65401e-17
- joint l_sole_frame: origin xyz=-0.0152219 0.0907683 -0.0529 rpy=-5.77818e-15 -6.98371e-15 1.5708 -> xyz=-0.015201 0.0908434 -0.0529 rpy=-5.77818e-15 -6.98371e-15 1.5708
- joint r_sole_frame: origin xyz=0.0152219 0.0907683 -0.0529 rpy=3.33669e-15 3.22983e-14 1.5708 -> xyz=0.015201 0.0908434 -0.0529 rpy=3.33669e-15 3.22983e-14 1.5708

Commit message: corrected shoulder roll joint

File: wolfgang_description/urdf/robot.urdf (robot description, URDF)
Before this commit: robot wolfgang, 46 links, 45 joints
Joints:
- joint LShoulderRoll: limit lower=0 upper=3.14159 effort=5.43 velocity=10.33 -> lower=-3.14159 upper=0 effort=5.43 velocity=10.33
- joint RShoulderRoll: limit lower=-3.14159 upper=0 effort=5.43 velocity=10.33 -> lower=0 upper=3.14159 effort=5.43 velocity=10.33

Commit message: description: fix joint directions

File: wolfgang_description/urdf/robot.urdf (robot description, URDF)
Before this commit: robot wolfgang, 46 links, 45 joints
Links:
- link torso: mass 2.21811 -> 2.2039
Joints:
- joint HeadPan: axis 0 0 1 -> -0 -0 -1
- joint HeadTilt: axis 0 0 -1 -> -0 -0 1
- joint LElbow: origin xyz=-0.024 -0.144 -0.0235 rpy=-1.5708 1.11022e-14 1.5708 -> xyz=-0.024 -0.144 -0.0235 rpy=-1.5708 3.08909e-14 1.5708
- joint LHipYaw: axis 0 -1 0 -> -0 1 -0
- joint LShoulderPitch: origin xyz=-0.0015 0.0765 0.2035 rpy=3.14159 7.77156e-16 3.14159 -> xyz=-0.0015 0.0765 0.2035 rpy=-3.14159 1.66533e-16 3.14159
- joint LShoulderRoll: origin xyz=-0.01695 0.042 8.32667e-17 rpy=-1.5708 8.42077e-17 1.5708 -> xyz=-0.01695 0.042 -2.77556e-17 rpy=-1.5708 -5.19331e-15 1.5708
- joint RAnklePitch: origin xyz=4.23273e-16 0.0505 -0.17 rpy=-1.5708 -7.47915e-15 1.91582e-15 -> xyz=4.44089e-16 0.0505 -0.17 rpy=-1.5708 -7.47915e-15 1.91582e-15
- joint RAnkleRoll: origin xyz=-0.0691 0 -0.026 rpy=1.5708 1.5708 0 -> xyz=-0.0691 3.83027e-15 -0.026 rpy=1.5708 1.5708 0
- joint RHipPitch: origin xyz=-0.0265 -2.77556e-17 -0.0691 rpy=-1.5708 1.5708 0 -> xyz=-0.0265 -9.71445e-17 -0.0691 rpy=-1.5708 1.5708 0
- joint RHipYaw: axis 0 -1 0 -> -0 1 -0; origin xyz=-1.33227e-15 -0.055 -7.91468e-18 rpy=-1.5708 -0 0 -> xyz=7.99361e-15 -0.055 4.68375e-17 rpy=-1.5708 -0 0
- joint l_wrist_frame: origin xyz=2.91434e-16 -0.225182 -0.0235 rpy=-1.5708 6.97876e-16 -1.5708 -> xyz=-7.63278e-17 -0.225182 -0.0235 rpy=-1.5708 1.69653e-16 -1.5708

Commit message: description: fix joint limits

File: wolfgang_description/urdf/robot.urdf (robot description, URDF)
Before this commit: robot wolfgang, 46 links, 45 joints
Joints:
- joint HeadTilt: limit lower=-0.523599 upper=1.5708 effort=5.43 velocity=10.33 -> lower=-1.5708 upper=0.523599 effort=5.43 velocity=10.33
- joint LHipPitch: limit lower=-1.5708 upper=1.5708 effort=7.57 velocity=8.22 -> lower=-1.5708 upper=0.0139626 effort=7.57 velocity=8.22
- joint RAnklePitch: origin xyz=4.44089e-16 0.0505 -0.17 rpy=-1.5708 -7.47915e-15 1.91582e-15 -> xyz=-2.08167e-17 0.0505 -0.17 rpy=-1.5708 0.0364674 1.18307e-15
- joint RAnkleRoll: origin xyz=-0.0691 3.83027e-15 -0.026 rpy=1.5708 1.5708 0 -> xyz=-0.0691 -5.55112e-17 -0.026 rpy=5.46411e-15 1.54833 -1.5708
- joint RHipPitch: limit lower=-1.5708 upper=1.5708 effort=7.57 velocity=8.22 -> lower=-0.0139626 upper=1.5708 effort=7.57 velocity=8.22
- joint RLB: origin xyz=-0.03 -0.007 -0.034 rpy=-2.20568e-16 -1.44743e-15 -1.5708 -> xyz=-0.03 -0.007 -0.034 rpy=-2.98953e-16 -2.63023e-16 -1.5708
- joint RLF: origin xyz=-0.03 0.177 -0.034 rpy=-1.06437e-15 1.50083e-15 -1.5708 -> xyz=-0.03 0.177 -0.034 rpy=-1.37255e-15 5.10716e-16 -1.5708
- joint RRB: origin xyz=0.06 -0.007 -0.034 rpy=-1.81005e-15 5.43559e-14 -1.5708 -> xyz=0.06 -0.007 -0.034 rpy=-1.82057e-15 5.38982e-15 -1.5708
- joint RRF: origin xyz=0.06 0.177 -0.034 rpy=-8.29268e-17 1.40387e-15 -1.5708 -> xyz=0.06 0.177 -0.034 rpy=1.04023e-15 -2.05167e-15 -1.5708
- joint r_cleat_l_back_frame: origin xyz=0 -0.0005 -0.016 rpy=8.14947e-17 -3.2143e-16 -3.14159 -> xyz=1.38778e-17 -0.0005 -0.016 rpy=-1.16828e-15 -4.65794e-17 -3.14159
- joint r_cleat_l_front_frame: origin xyz=-1.38778e-17 -0.0005 -0.016 rpy=3.37705e-16 1.87148e-15 3.14159 -> xyz=0 -0.0005 -0.016 rpy=2.41328e-16 2.75668e-16 -3.14159
- joint r_cleat_r_back_frame: origin xyz=1.38778e-17 -0.0005 -0.016 rpy=2.94118e-16 7.40154e-17 3.14159 -> xyz=1.38778e-17 -0.0005 -0.016 rpy=3.36899e-17 -1.41669e-15 3.14159
- joint r_cleat_r_front_frame: origin xyz=-1.38778e-17 -0.0005 -0.016 rpy=2.75421e-16 9.31542e-16 3.14159 -> xyz=5.55112e-17 -0.0005 -0.016 rpy=6.426e-16 8.18562e-16 -3.14159
- joint r_sole_frame: origin xyz=0.015201 0.0908434 -0.0529 rpy=3.33669e-15 3.22983e-14 1.5708 -> xyz=0.015201 0.0908434 -0.0529 rpy=-4.18784e-16 2.31919e-15 1.5708

Commit message: fix urdf and moveit issues

File: wolfgang_description/urdf/robot.urdf (robot description, URDF)
Before this commit: robot wolfgang, 46 links, 45 joints
Links:
- link torso: mass 2.2039 -> 2.2036
Joints:
- joint LHipPitch: limit lower=-1.5708 upper=0.0139626 effort=7.57 velocity=8.22 -> lower=-0.785398 upper=1.5708 effort=7.57 velocity=8.22
- joint RHipPitch: limit lower=-0.0139626 upper=1.5708 effort=7.57 velocity=8.22 -> lower=-1.5708 upper=0.785398 effort=7.57 velocity=8.22

Commit message: Fix old urdf head joints

File: wolfgang_description/urdf/robot.urdf (robot description, URDF)
Before this commit: robot wolfgang, 45 links, 44 joints
Joints:
- joint HeadPan: axis 0 0 1 -> 0 0 -1
- joint HeadTilt: axis 0 0 -1 -> 0 0 1; limit lower=0 upper=1.5708 effort=5.43 velocity=10.33 -> lower=-1.5708 upper=0 effort=5.43 velocity=10.33

Commit message: description: fixed toes

File: wolfgang_description/urdf/robot.urdf (robot description, URDF)
Before this commit: robot wolfgang, 46 links, 45 joints
Links:
- added link l_toe, mass 1e-9
- added link r_toe, mass 1e-9
- link l_foot: mass 0.267613 -> 0.26824
- link r_foot: mass 0.267613 -> 0.26824
- link torso: mass 2.2036 -> 2.0839; geometry collision mesh filename=package://wolfgang_description/urdf/baseplate_odroid_xu4_co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; collision mesh filename=package://wolfgang_description/urdf/battery.stl
Joints:
- added joint l_toe_frame: type fixed, parent l_foot, child l_toe, origin xyz=-0.015 0.1845 -0.03775 rpy=-5.77818e-15 -6.88971e-15 1.5708, axis 0 0 0
- added joint r_toe_frame: type fixed, parent r_foot, child r_toe, origin xyz=0.015 0.1845 -0.03775 rpy=-1.35689e-15 2.56061e-15 1.5708, axis 0 0 0
- joint l_sole_frame: origin xyz=-0.015201 0.0908434 -0.0529 rpy=-5.77818e-15 -6.98371e-15 1.5708 -> xyz=-0.0152219 0.0907683 -0.0529 rpy=-5.77818e-15 -6.98371e-15 1.5708
- joint r_sole_frame: origin xyz=0.015201 0.0908434 -0.0529 rpy=-4.18784e-16 2.31919e-15 1.5708 -> xyz=0.0152219 0.0907683 -0.0529 rpy=-4.18784e-16 2.31919e-15 1.5708

Commit message: urdf: fix spring collision model

File: wolfgang_description/urdf/robot.urdf (robot description, URDF)
Before this commit: robot wolfgang, 48 links, 47 joints
Links:
- link head: geometry collision mesh filename=package://wolfgang_description/urdf/head.stl; visual mesh filename=package://wolfgang_description/urdf/head.stl
- link l_ankle: geometry collision mesh filename=package://wolfgang_description/urdf/l_ankle.stl; visual mesh filename=package://wolfgang_description/urdf/l_ankle.stl
- link l_foot: geometry collision mesh filename=package://wolfgang_description/urdf/l_foot.stl; visual mesh filename=package://wolfgang_description/urdf/l_foot.stl
- link l_hip_1: geometry collision mesh filename=package://wolfgang_description/urdf/l_hip_1.stl; visual mesh filename=package://wolfgang_description/urdf/l_hip_1.stl
- link l_hip_2: geometry collision mesh filename=package://wolfgang_description/urdf/l_hip_2.stl; visual mesh filename=package://wolfgang_description/urdf/l_hip_2.stl
- link l_lower_arm: geometry collision mesh filename=package://wolfgang_description/urdf/l_lower_arm.stl; visual mesh filename=package://wolfgang_description/urdf/l_lower_arm.stl
- link l_lower_leg: mass 0.112624 -> 0.0880635; geometry collision mesh filename=package://wolfgang_description/urdf/l_lower_leg.stl; visual mesh filename=package://wolfgang_description/urdf/l_lower_leg.stl
- link l_shoulder: geometry collision mesh filename=package://wolfgang_description/urdf/l_shoulder.stl; visual mesh filename=package://wolfgang_description/urdf/l_shoulder.stl
- link l_upper_arm: geometry collision mesh filename=package://wolfgang_description/urdf/l_upper_arm.stl; visual mesh filename=package://wolfgang_description/urdf/l_upper_arm.stl
- link l_upper_leg: geometry collision mesh filename=package://wolfgang_description/urdf/l_upper_leg.stl; visual mesh filename=package://wolfgang_description/urdf/l_upper_leg.stl
- link llb: geometry collision mesh filename=package://wolfgang_description/urdf/llb.stl; visual mesh filename=package://wolfgang_description/urdf/llb.stl
- link llf: geometry collision mesh filename=package://wolfgang_description/urdf/llf.stl; visual mesh filename=package://wolfgang_description/urdf/llf.stl
- link lrb: geometry collision mesh filename=package://wolfgang_description/urdf/lrb.stl; visual mesh filename=package://wolfgang_description/urdf/lrb.stl
- link lrf: geometry collision mesh filename=package://wolfgang_description/urdf/lrf.stl; visual mesh filename=package://wolfgang_description/urdf/lrf.stl
- link neck: geometry collision mesh filename=package://wolfgang_description/urdf/neck.stl; visual mesh filename=package://wolfgang_description/urdf/neck.stl
- link r_ankle: geometry collision mesh filename=package://wolfgang_description/urdf/r_ankle.stl; visual mesh filename=package://wolfgang_description/urdf/r_ankle.stl
- link r_foot: geometry collision mesh filename=package://wolfgang_description/urdf/r_foot.stl; visual mesh filename=package://wolfgang_description/urdf/r_foot.stl
- link r_hip_1: geometry collision mesh filename=package://wolfgang_description/urdf/r_hip_1.stl; visual mesh filename=package://wolfgang_description/urdf/r_hip_1.stl
- link r_hip_2: geometry collision mesh filename=package://wolfgang_description/urdf/r_hip_2.stl; visual mesh filename=package://wolfgang_description/urdf/r_hip_2.stl
- link r_lower_arm: geometry collision mesh filename=package://wolfgang_description/urdf/r_lower_arm.stl; visual mesh filename=package://wolfgang_description/urdf/r_lower_arm.stl
- link r_lower_leg: mass 0.112618 -> 0.0880635; geometry collision mesh filename=package://wolfgang_description/urdf/r_lower_leg.stl; visual mesh filename=package://wolfgang_description/urdf/r_lower_leg.stl
- link r_shoulder: geometry collision mesh filename=package://wolfgang_description/urdf/r_shoulder.stl; visual mesh filename=package://wolfgang_description/urdf/r_shoulder.stl
- link r_upper_arm: geometry collision mesh filename=package://wolfgang_description/urdf/r_upper_arm.stl; visual mesh filename=package://wolfgang_description/urdf/r_upper_arm.stl
- link r_upper_leg: geometry collision mesh filename=package://wolfgang_description/urdf/r_upper_leg.stl; visual mesh filename=package://wolfgang_description/urdf/r_upper_leg.stl
- link rlb: geometry collision mesh filename=package://wolfgang_description/urdf/rlb.stl; visual mesh filename=package://wolfgang_description/urdf/rlb.stl
- link rlf: geometry collision mesh filename=package://wolfgang_description/urdf/rlf.stl; visual mesh filename=package://wolfgang_description/urdf/rlf.stl
- link rrb: geometry collision mesh filename=package://wolfgang_description/urdf/rrb.stl; visual mesh filename=package://wolfgang_description/urdf/rrb.stl
- link rrf: geometry collision mesh filename=package://wolfgang_description/urdf/rrf.stl; visual mesh filename=package://wolfgang_description/urdf/rrf.stl
- link torso: geometry collision mesh filename=package://wolfgang_description/urdf/torso.stl; visual mesh filename=package://wolfgang_description/urdf/torso.stl
