Commit message: collision model replacement by boxes

File: wolfgang_description/urdf/robot.urdf (robot description, URDF)
Before this commit: robot wolfgang, 48 links, 47 joints
Links:
- link camera: mass 1e-9 -> 1e-09
- link camera_optical_frame: mass 1e-9 -> 1e-09
- link head: geometry collision box size=0.007101020310074093 0.05434203334722684 0.12845531548037442; collision box size=0.007101021707057951 0.05434203334722684 0.12845531548037442
- link imu_frame: mass 1e-9 -> 1e-09
- link imu_frame_2: mass 1e-9 -> 1e-09
- link l_ankle: geometry collision box size=0.005599999800334461 0.029999999329447746 0.030999999493360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; collision box size=0.006000000052154064 0.011599999852478506 0.028000000864267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
- link l_cleat_l_back: mass 1e-9 -> 1e-09
- link l_cleat_l_front: mass 1e-9 -> 1e-09
- link l_cleat_r_back: mass 1e-9 -> 1e-09
- link l_cleat_r_front: mass 1e-9 -> 1e-09
- link l_foot: geometry collision box size=0.0015999999595806113 0.05999999865889549 0.0599999986588955; collision box size=0.004000000189989805 0.008000000379979616 0.039999999105930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
- link l_hip_1: geometry collision box size=0.05000000167638064 0.053174532949924476 0.10000000149011612; visual mesh filename=package://wolfgang_description/urdf/hip_u_connector.stl
- link l_hip_2: geometry collision box size=0.005599999800334461 0.029999999329447746 0.030999999493360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; collision box size=0.006000000052154064 0.011599999852478506 0.028000000864267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
- link l_lower_arm: geometry collision box size=0.012 0.002 0.029; collision box size=0.012 0.002 0.029
- link l_lower_leg: geometry collision box size=0.0015000011771917456 0.03580509314602309 0.035946585881522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; collision box size=0.0015000011771917456 0.03580509314602309 0.035946585881522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
- link l_shoulder: geometry collision box size=0.03400000184774399 0.045000001788139336 0.06390000134706497; collision cylinder length=0.005 radius=0.025
- link l_sole: mass 1e-9 -> 1e-09
- link l_toe: mass 1e-9 -> 1e-09
- link l_upper_arm: geometry collision box size=0.0022499999322462853 0.03999999910593033 0.169780876487493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; collision box size=0.0022499999322462853 0.03999999910593033 0.169780876487493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
- link l_upper_leg: geometry collision box size=0.0020000000949949087 0.05184974683212369 0.1715841731155343; collision box size=0.0020000000949949087 0.05184974683212369 0.1715841731155343
- link l_wrist: mass 1e-9 -> 1e-09
- link neck: geometry collision box size=0.009300000034272672 0.035999998450279236 0.039999999105930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; collision box size=0.04019999876618385 0.04609999991953372 0.06109999865293502
- link r_ankle: geometry collision box size=0.005599999800334461 0.029999999329447746 0.030999999493360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; collision box size=0.006000000052154064 0.011599999852478506 0.028000000864267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
- link r_cleat_l_back: mass 1e-9 -> 1e-09
- link r_cleat_l_front: mass 1e-9 -> 1e-09
- link r_cleat_r_back: mass 1e-9 -> 1e-09
- link r_cleat_r_front: mass 1e-9 -> 1e-09
- link r_foot: geometry collision box size=0.0015999999595806113 0.05999999865889549 0.0599999986588955; collision box size=0.004000000189989805 0.008000000379979616 0.039999999105930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
- link r_hip_1: geometry collision box size=0.05000000167638064 0.053174532949924476 0.10000000149011612; visual mesh filename=package://wolfgang_description/urdf/hip_u_connector.stl
- link r_hip_2: geometry collision box size=0.005599999800334461 0.029999999329447746 0.030999999493360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; collision box size=0.006000000052154064 0.011599999852478506 0.028000000864267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
- link r_lower_arm: geometry collision box size=0.012 0.002 0.029; collision box size=0.012 0.002 0.029
- link r_lower_leg: geometry collision box size=0.0015000011771917456 0.03580509314602309 0.035946585881522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; collision box size=0.0015000011771917456 0.03580509314602309 0.035946585881522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
- link r_shoulder: geometry collision box size=0.03400000184774399 0.045000001788139336 0.06390000134706497; collision cylinder length=0.005 radius=0.025
- link r_sole: mass 1e-9 -> 1e-09
- link r_toe: mass 1e-9 -> 1e-09
- link r_upper_arm: geometry collision box size=0.0022499999322462853 0.03999999910593033 0.169780876487493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; collision box size=0.0022499999322462853 0.03999999910593033 0.169780876487493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
- link r_upper_leg: geometry collision box size=0.0020000000949949087 0.05184974683212369 0.1715841731155343; collision box size=0.0020000000949949087 0.05184974683212369 0.1715841731155343
- link r_wrist: mass 1e-9 -> 1e-09
- link torso: geometry collision box size=0.0020000000949949148 0.06599999964237213 0.131999999284744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; collision box size=0.002000000327825547 0.018999999389052395 0.083999998867511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
Joints:
- joint HeadPan: axis -0 -0 -1 -> -0.0 -0.0 -1.0
- joint HeadTilt: axis -0 -0 1 -> -0.0 -0.0 1.0
- joint LAnklePitch: axis -0 -0 -1 -> -0.0 -0.0 -1.0
- joint LAnkleRoll: axis -0 -1 -0 -> -0.0 -1.0 -0.0; origin xyz=0.0691 1.66533e-16 -0.026 rpy=1.5708 -1.5708 0 -> xyz=0.0691 1.66533e-16 -0.026 rpy=1.5708 -1.5708 0.0
- joint LElbow: axis 0 0 1 -> 0.0 0.0 1.0
- joint LHipPitch: axis 7.95491e-17 -3.00167e-16 -1 -> 7.95491e-17 -3.00167e-16 -1.0; origin xyz=0.026 6.93889e-18 -0.0691 rpy=2.67116e-16 -1.5708 0 -> xyz=0.026 6.93889e-18 -0.0691 rpy=2.67116e-16 -1.5708 0.0
- joint LHipRoll: axis -0 -0 -1 -> -0.0 -0.0 -1.0; origin xyz=-0.046 0.0414 6.93889e-18 rpy=3.14159 1.5708 0 -> xyz=-0.046 0.0414 6.93889e-18 rpy=3.14159 1.5708 0.0
- joint LHipYaw: axis -0 1 -0 -> -0.0 1.0 -0.0; origin xyz=1.82493e-15 0.055 -4.22839e-18 rpy=-1.5708 -0 0 -> xyz=1.82493e-15 0.055 -4.22839e-18 rpy=-1.5708 -0.0 0.0
- joint LKnee: axis -0 1 -0 -> -0.0 1.0 -0.0; limit lower=0 upper=2.96706 effort=10 velocity=10 -> lower=0.0 upper=2.96706 effort=10.0 velocity=10.0
- joint LLB: axis 0 1.22465e-16 1 -> 0.0 1.22465e-16 1.0; limit effort=0 velocity=0 -> lower=0 upper=0 effort=0.0 velocity=0.0
- joint LLF: axis 0 1.22465e-16 1 -> 0.0 1.22465e-16 1.0; limit effort=0 velocity=0 -> lower=0 upper=0 effort=0.0 velocity=0.0
- joint LRB: axis 0 1.22465e-16 1 -> 0.0 1.22465e-16 1.0; limit effort=0 velocity=0 -> lower=0 upper=0 effort=0.0 velocity=0.0
- joint LRF: axis 0 -1.22465e-16 -1 -> 0.0 -1.22465e-16 -1.0; limit effort=0 velocity=0 -> lower=0 upper=0 effort=0.0 velocity=0.0
- joint LShoulderPitch: axis -0 1 -0 -> -0.0 1.0 -0.0
- joint LShoulderRoll: axis -0 -0 -1 -> -0.0 -0.0 -1.0; limit lower=-3.14159 upper=0 effort=5.43 velocity=10.33 -> lower=-3.14159 upper=0.0 effort=5.43 velocity=10.33
- joint RAnklePitch: axis -0 -0 -1 -> -0.0 -0.0 -1.0
- joint RAnkleRoll: axis 0 -1 0 -> 0.0 -1.0 0.0
- joint RElbow: axis 0 0 1 -> 0.0 0.0 1.0
- joint RHipPitch: axis -0 1 -0 -> -0.0 1.0 -0.0; origin xyz=-0.0265 -9.71445e-17 -0.0691 rpy=-1.5708 1.5708 0 -> xyz=-0.0265 -9.71445e-17 -0.0691 rpy=-1.5708 1.5708 0.0
- joint RHipRoll: axis -0 -0 -1 -> -0.0 -0.0 -1.0; origin xyz=-0.046 0.0414 6.93889e-18 rpy=-3.14159 1.5708 0 -> xyz=-0.046 0.0414 6.93889e-18 rpy=-3.14159 1.5708 0.0
- joint RHipYaw: axis -0 1 -0 -> -0.0 1.0 -0.0; origin xyz=7.99361e-15 -0.055 4.68375e-17 rpy=-1.5708 -0 0 -> xyz=7.99361e-15 -0.055 4.68375e-17 rpy=-1.5708 -0.0 0.0
- joint RKnee: axis -0 -1 -0 -> -0.0 -1.0 -0.0; limit lower=-2.96706 upper=0 effort=10 velocity=10 -> lower=-2.96706 upper=0.0 effort=10.0 velocity=10.0
- joint RLB: axis 0 1.22465e-16 1 -> 0.0 1.22465e-16 1.0; limit effort=0 velocity=0 -> lower=0 upper=0 effort=0.0 velocity=0.0
- joint RLF: axis 0 1.22465e-16 1 -> 0.0 1.22465e-16 1.0; limit effort=0 velocity=0 -> lower=0 upper=0 effort=0.0 velocity=0.0
- joint RRB: axis 0 1.22465e-16 1 -> 0.0 1.22465e-16 1.0; limit effort=0 velocity=0 -> lower=0 upper=0 effort=0.0 velocity=0.0
- joint RRF: axis 0 1.22465e-16 1 -> 0.0 1.22465e-16 1.0; limit effort=0 velocity=0 -> lower=0 upper=0 effort=0.0 velocity=0.0
- joint RShoulderPitch: axis -0 1 -0 -> -0.0 1.0 -0.0
- joint RShoulderRoll: axis -0 -0 -1 -> -0.0 -0.0 -1.0; limit lower=0 upper=3.14159 effort=5.43 velocity=10.33 -> lower=0.0 upper=3.14159 effort=5.43 velocity=10.33; origin xyz=-0.01695 0.042 0 rpy=1.5708 8.32338e-16 -1.5708 -> xyz=-0.01695 0.042 0.0 rpy=1.5708 8.32338e-16 -1.5708
- joint base_link_to_base: origin xyz=0 0 0 rpy=0.0 0 0 -> xyz=0.0 0.0 0.0 rpy=0.0 0.0 0.0
- joint camera_frame: axis 0 0 0 -> 0.0 0.0 0.0
- joint camera_optical_frame_frame: axis 0 0 0 -> 0.0 0.0 0.0; origin xyz=0.0432 0.08 -0.0235 rpy=3.14159 -1.5708 0 -> xyz=0.0432 0.08 -0.0235 rpy=3.14159 -1.5708 0.0
- joint imu_frame_2_frame: axis 0 0 0 -> 0.0 0.0 0.0
- joint imu_frame_frame: axis 0 0 0 -> 0.0 0.0 0.0
- joint l_cleat_l_back_frame: axis 0 0 0 -> 0.0 0.0 0.0
- joint l_cleat_l_front_frame: axis 0 0 0 -> 0.0 0.0 0.0; origin xyz=0 -0.0005 -0.016 rpy=3.06162e-16 -4.4319e-17 -3.14159 -> xyz=0.0 -0.0005 -0.016 rpy=3.06162e-16 -4.4319e-17 -3.14159
- joint l_cleat_r_back_frame: axis 0 0 0 -> 0.0 0.0 0.0; origin xyz=0 -0.0005 -0.016 rpy=2.92719e-16 -4.05989e-17 -3.14159 -> xyz=0.0 -0.0005 -0.016 rpy=2.92719e-16 -4.05989e-17 -3.14159
- joint l_cleat_r_front_frame: axis 0 0 0 -> 0.0 0.0 0.0; origin xyz=0 -0.0005 -0.016 rpy=3.00788e-16 -1.03785e-15 -3.14159 -> xyz=0.0 -0.0005 -0.016 rpy=3.00788e-16 -1.03785e-15 -3.14159
- joint l_sole_frame: axis 0 0 0 -> 0.0 0.0 0.0
- joint l_toe_frame: axis 0 0 0 -> 0.0 0.0 0.0
- joint l_wrist_frame: axis 0 0 0 -> 0.0 0.0 0.0
- joint r_cleat_l_back_frame: axis 0 0 0 -> 0.0 0.0 0.0
- joint r_cleat_l_front_frame: axis 0 0 0 -> 0.0 0.0 0.0; origin xyz=0 -0.0005 -0.016 rpy=2.41328e-16 2.75668e-16 -3.14159 -> xyz=0.0 -0.0005 -0.016 rpy=2.41328e-16 2.75668e-16 -3.14159
- joint r_cleat_r_back_frame: axis 0 0 0 -> 0.0 0.0 0.0
- joint r_cleat_r_front_frame: axis 0 0 0 -> 0.0 0.0 0.0
- joint r_sole_frame: axis 0 0 0 -> 0.0 0.0 0.0
- joint r_toe_frame: axis 0 0 0 -> 0.0 0.0 0.0
- joint r_wrist_frame: axis 0 0 0 -> 0.0 0.0 0.0

Commit message: urdf and proto adjustments

File: wolfgang_description/urdf/robot.urdf (robot description, URDF)
Before this commit: robot wolfgang, 48 links, 47 joints
Joints:
- joint HeadTilt: limit lower=-1.5708 upper=0.523599 effort=5.43 velocity=10.33 -> lower=-1.5708 upper=1.0472 effort=5.43 velocity=10.33
- joint LHipPitch: limit lower=-0.785398 upper=1.5708 effort=7.57 velocity=8.22 -> lower=-1.91986 upper=2.0944 effort=7.57 velocity=8.22
- joint RHipPitch: limit lower=-1.5708 upper=0.785398 effort=7.57 velocity=8.22 -> lower=-2.0944 upper=1.91986 effort=7.57 velocity=8.22

Commit message: reduce SEA size to avoid collisions

File: wolfgang_description/urdf/robot.urdf (robot description, URDF)
Before this commit: robot wolfgang, 48 links, 47 joints
Links:
- link head: geometry collision box size=0.007101020310074093 0.05434203334722684 0.12845531548037442; collision box size=0.007101021707057951 0.05434203334722684 0.12845531548037442

Commit message: new export with correct motor bounding boxes and joint limits in ankles

File: wolfgang_description/urdf/robot.urdf (robot description, URDF)
Before this commit: robot wolfgang, 48 links, 47 joints
Links:
- link head: geometry collision box size=0.007101020310074093 0.05434203334722684 0.12845531548037442; collision box size=0.007101021707057951 0.05434203334722684 0.12845531548037442
- link l_ankle: geometry collision box size=0.005599999800334461 0.029999999329447746 0.030999999493360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; collision box size=0.006000000052154064 0.011599999852478506 0.028000000864267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
- link l_hip_2: geometry collision box size=0.005599999800334461 0.029999999329447746 0.030999999493360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; collision box size=0.006000000052154064 0.011599999852478506 0.028000000864267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
- link l_lower_arm: geometry collision box size=0.012 0.002 0.029; collision box size=0.012 0.002 0.029
- link l_upper_arm: geometry collision box size=0.0022499999322462853 0.03999999910593033 0.169780876487493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; collision box size=0.0022499999322462853 0.03999999910593033 0.169780876487493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
- link neck: geometry collision box size=0.009300000034272672 0.035999998450279236 0.039999999105930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; collision box size=0.0402 0.041 0.0611
- link r_ankle: geometry collision box size=0.005599999800334461 0.029999999329447746 0.030999999493360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; collision box size=0.006000000052154064 0.011599999852478506 0.028000000864267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
- link r_hip_2: geometry collision box size=0.005599999800334461 0.029999999329447746 0.030999999493360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; collision box size=0.006000000052154064 0.011599999852478506 0.028000000864267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
- link r_lower_arm: geometry collision box size=0.012 0.002 0.029; collision box size=0.012 0.002 0.029
- link r_upper_arm: geometry collision box size=0.0022499999322462853 0.03999999910593033 0.169780876487493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; collision box size=0.0022499999322462853 0.03999999910593033 0.169780876487493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
- link torso: geometry collision box size=0.0020000000949949148 0.06599999964237213 0.131999999284744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; collision box size=0.002000000327825547 0.018999999389052395 0.083999998867511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
Joints:
- joint LAnklePitch: limit lower=-1.22173 upper=1.5708 effort=7.57 velocity=8.22 -> lower=-1.22173 upper=1.74533 effort=7.57 velocity=8.22
- joint RAnklePitch: limit lower=-1.5708 upper=1.22173 effort=7.57 velocity=8.22 -> lower=-1.74533 upper=1.22173 effort=7.57 velocity=8.22; origin xyz=-2.08167e-17 0.0505 -0.17 rpy=-1.5708 0.0364674 1.18307e-15 -> xyz=4.16334e-16 0.0505 -0.17 rpy=-1.5708 4.23642e-15 1.2925e-15
- joint RAnkleRoll: origin xyz=-0.0691 -5.55112e-17 -0.026 rpy=5.46411e-15 1.54833 -1.5708 -> xyz=-0.0691 -1.11022e-16 -0.026 rpy=-1.46564e-14 1.54833 -1.5708
- joint RLB: origin xyz=-0.03 -0.007 -0.034 rpy=-2.98953e-16 -2.63023e-16 -1.5708 -> xyz=-0.03 -0.007 -0.034 rpy=-2.99252e-16 -3.15564e-16 -1.5708
- joint RLF: origin xyz=-0.03 0.177 -0.034 rpy=-1.37255e-15 5.10716e-16 -1.5708 -> xyz=-0.03 0.177 -0.034 rpy=-1.37387e-15 4.73288e-16 -1.5708
- joint RRB: origin xyz=0.06 -0.007 -0.034 rpy=-1.82057e-15 5.38982e-15 -1.5708 -> xyz=0.06 -0.007 -0.034 rpy=-1.81929e-15 5.34084e-15 -1.5708
- joint RRF: origin xyz=0.06 0.177 -0.034 rpy=1.04023e-15 -2.05167e-15 -1.5708 -> xyz=0.06 0.177 -0.034 rpy=1.04209e-15 -2.09028e-15 -1.5708
- joint r_cleat_l_back_frame: origin xyz=1.38778e-17 -0.0005 -0.016 rpy=-1.16828e-15 -4.65794e-17 -3.14159 -> xyz=0.0 -0.0005 -0.016 rpy=-1.17224e-15 -1.58433e-17 -3.14159
- joint r_cleat_l_front_frame: origin xyz=0.0 -0.0005 -0.016 rpy=2.41328e-16 2.75668e-16 -3.14159 -> xyz=-1.38778e-17 -0.0005 -0.016 rpy=2.44346e-16 2.736e-16 -3.14159
- joint r_cleat_r_back_frame: origin xyz=1.38778e-17 -0.0005 -0.016 rpy=3.36899e-17 -1.41669e-15 3.14159 -> xyz=-1.38778e-17 -0.0005 -0.016 rpy=3.0848e-17 -1.36062e-15 3.14159
- joint r_cleat_r_front_frame: origin xyz=5.55112e-17 -0.0005 -0.016 rpy=6.426e-16 8.18562e-16 -3.14159 -> xyz=-6.93889e-17 -0.0005 -0.016 rpy=6.44157e-16 8.47782e-16 -3.14159
- joint r_sole_frame: origin xyz=0.0152219 0.0907683 -0.0529 rpy=-4.18784e-16 2.31919e-15 1.5708 -> xyz=0.0152219 0.0907683 -0.0529 rpy=-4.1858e-16 2.36866e-15 1.5708
- joint r_toe_frame: origin xyz=0.015 0.1845 -0.03775 rpy=-1.35689e-15 2.56061e-15 1.5708 -> xyz=0.015 0.1845 -0.03775 rpy=-1.35775e-15 2.56512e-15 1.5708
