Commit message: scad fix and urdf

File: wolfgang_description/urdf/robot.urdf (robot description, URDF)
Before this commit: robot wolfgang, 48 links, 47 joints
Links:
- link camera: mass 1e-09 -> 1e-9
- link camera_optical_frame: mass 1e-09 -> 1e-9
- link head: geometry collision box size=0.006 0.072 0.03; collision box size=0.006 0.072 0.03
- link imu_frame: mass 1e-09 -> 1e-9
- link imu_frame_2: mass 1e-09 -> 1e-9
- link l_ankle: geometry collision box size=0.028 0.0035 0.0059; collision box size=0.028 0.0035 0.0059
- link l_cleat_l_back: mass 1e-09 -> 1e-9
- link l_cleat_l_front: mass 1e-09 -> 1e-9
- link l_cleat_r_back: mass 1e-09 -> 1e-9
- link l_cleat_r_front: mass 1e-09 -> 1e-9
- link l_foot: geometry collision box size=0.008 0.04 0.004; collision box size=0.008 0.04 0.004
- link l_hip_1: geometry collision box size=0.036 0.004 0.053; collision box size=0.036 0.004 0.053
- link l_hip_2: geometry collision box size=0.028 0.0035 0.0059; collision box size=0.028 0.0035 0.0059
- link l_lower_leg: geometry collision box size=0.014 0.0091 0.031; collision box size=0.034 0.002 0.16
- link l_shoulder: geometry collision box size=0.0015 0.045 0.028; collision box size=0.0015 0.045 0.028
- link l_sole: mass 1e-09 -> 1e-9
- link l_toe: mass 1e-09 -> 1e-9
- link l_upper_arm: geometry collision box size=0.036 0.04 0.0093; collision box size=0.036 0.04 0.0093
- link l_upper_leg: geometry collision box size=0.01 0.002 0.01; collision box size=0.01 0.002 0.01
- link l_wrist: mass 1e-09 -> 1e-9
- link neck: geometry collision box size=0.036 0.04 0.0093; collision box size=0.0402 0.041 0.0611
- link r_ankle: geometry collision box size=0.028 0.0035 0.0059; collision box size=0.028 0.0035 0.0059
- link r_cleat_l_back: mass 1e-09 -> 1e-9
- link r_cleat_l_front: mass 1e-09 -> 1e-9
- link r_cleat_r_back: mass 1e-09 -> 1e-9
- link r_cleat_r_front: mass 1e-09 -> 1e-9
- link r_foot: geometry collision box size=0.008 0.04 0.004; collision box size=0.008 0.04 0.004
- link r_hip_1: geometry collision box size=0.036 0.004 0.053; collision box size=0.036 0.004 0.053
- link r_hip_2: geometry collision box size=0.028 0.0035 0.0059; collision box size=0.028 0.0035 0.0059
- link r_lower_leg: geometry collision box size=0.014 0.0091 0.031; collision box size=0.034 0.002 0.16
- link r_shoulder: geometry collision box size=0.0015 0.045 0.028; collision box size=0.0015 0.045 0.028
- link r_sole: mass 1e-09 -> 1e-9
- link r_toe: mass 1e-09 -> 1e-9
- link r_upper_arm: geometry collision box size=0.036 0.04 0.0093; collision box size=0.036 0.04 0.0093
- link r_upper_leg: geometry collision box size=0.01 0.002 0.01; collision box size=0.01 0.002 0.01
- link r_wrist: mass 1e-09 -> 1e-9
- link torso: geometry collision box size=0.019 0.0468795 0.005; collision box size=0.019 0.0468795 0.005
Joints:
- joint HeadPan: axis -0.0 -0.0 -1.0 -> -0 -0 -1; limit lower=-2.0944 upper=2.0944 effort=5.43 velocity=10.33 -> lower=-2.0944 upper=2.0944 effort=5.475 velocity=8.17
- joint HeadTilt: axis -0.0 -0.0 1.0 -> -0 -0 1; limit lower=-1.5708 upper=1.0472 effort=5.43 velocity=10.33 -> lower=-1.5708 upper=1.0472 effort=5.475 velocity=8.17
- joint LAnklePitch: axis -0.0 -0.0 -1.0 -> -0 -0 -1; limit lower=-1.22173 upper=1.74533 effort=7.57 velocity=8.22 -> lower=-1.22173 upper=1.74533 effort=7.5 velocity=5.76
- joint LAnkleRoll: axis -0.0 -1.0 -0.0 -> -0 -1 -0; limit lower=-1.0472 upper=1.0472 effort=7.57 velocity=8.22 -> lower=-1.0472 upper=1.0472 effort=7.5 velocity=5.76; origin xyz=0.0691 1.66533e-16 -0.026 rpy=1.5708 -1.5708 0.0 -> xyz=0.0691 1.66533e-16 -0.026 rpy=1.5708 -1.5708 0
- joint LElbow: axis 0.0 0.0 1.0 -> 0 0 1; limit lower=-1.5708 upper=1.0472 effort=5.43 velocity=10.33 -> lower=-1.5708 upper=1.0472 effort=5.475 velocity=8.17
- joint LHipPitch: axis 7.95491e-17 -3.00167e-16 -1.0 -> 7.95491e-17 -3.00167e-16 -1; limit lower=-1.91986 upper=2.0944 effort=7.57 velocity=8.22 -> lower=-1.91986 upper=2.0944 effort=7.5 velocity=5.76; origin xyz=0.026 6.93889e-18 -0.0691 rpy=2.67116e-16 -1.5708 0.0 -> xyz=0.026 6.93889e-18 -0.0691 rpy=2.67116e-16 -1.5708 0
- joint LHipRoll: axis -0.0 -0.0 -1.0 -> -0 -0 -1; limit lower=-1.5708 upper=1.5708 effort=7.57 velocity=8.22 -> lower=-1.5708 upper=1.5708 effort=7.5 velocity=5.76; origin xyz=-0.046 0.0414 6.93889e-18 rpy=3.14159 1.5708 0.0 -> xyz=-0.046 0.0414 6.93889e-18 rpy=3.14159 1.5708 0
- joint LHipYaw: axis -0.0 1.0 -0.0 -> -0 1 -0; limit lower=-1.5708 upper=1.5708 effort=7.57 velocity=8.22 -> lower=-1.5708 upper=1.5708 effort=7.5 velocity=5.76; origin xyz=1.82493e-15 0.055 -4.22839e-18 rpy=-1.5708 -0.0 0.0 -> xyz=1.82493e-15 0.055 -4.22839e-18 rpy=-1.5708 -0 0
- joint LKnee: axis -0.0 1.0 -0.0 -> -0 1 -0; limit lower=0.0 upper=2.96706 effort=10.0 velocity=10.0 -> lower=0 upper=2.96706 effort=8.775 velocity=4.82
- joint LLB: axis 0.0 1.22465e-16 1.0 -> 0 1.22465e-16 1; limit lower=0 upper=0 effort=0.0 velocity=0.0 -> effort=0 velocity=0
- joint LLF: axis 0.0 1.22465e-16 1.0 -> 0 1.22465e-16 1; limit lower=0 upper=0 effort=0.0 velocity=0.0 -> effort=0 velocity=0
- joint LRB: axis 0.0 1.22465e-16 1.0 -> 0 1.22465e-16 1; limit lower=0 upper=0 effort=0.0 velocity=0.0 -> effort=0 velocity=0
- joint LRF: axis 0.0 -1.22465e-16 -1.0 -> 0 -1.22465e-16 -1; limit lower=0 upper=0 effort=0.0 velocity=0.0 -> effort=0 velocity=0
- joint LShoulderPitch: axis -0.0 1.0 -0.0 -> -0 1 -0; limit lower=-3.14159 upper=3.14159 effort=5.43 velocity=10.33 -> lower=-3.14159 upper=3.14159 effort=5.475 velocity=8.17
- joint LShoulderRoll: axis -0.0 -0.0 -1.0 -> -0 -0 -1; limit lower=-3.14159 upper=0.0 effort=5.43 velocity=10.33 -> lower=-3.14159 upper=0 effort=5.475 velocity=8.17
- joint RAnklePitch: axis -0.0 -0.0 -1.0 -> -0 -0 -1; limit lower=-1.74533 upper=1.22173 effort=7.57 velocity=8.22 -> lower=-1.74533 upper=1.22173 effort=7.5 velocity=5.76
- joint RAnkleRoll: axis 0.0 -1.0 0.0 -> 0 -1 0; limit lower=-1.0472 upper=1.0472 effort=7.57 velocity=8.22 -> lower=-1.0472 upper=1.0472 effort=7.5 velocity=5.76
- joint RElbow: axis 0.0 0.0 1.0 -> 0 0 1; limit lower=-1.0472 upper=1.5708 effort=5.43 velocity=10.33 -> lower=-1.0472 upper=1.5708 effort=5.475 velocity=8.17
- joint RHipPitch: axis -0.0 1.0 -0.0 -> -0 1 -0; limit lower=-2.0944 upper=1.91986 effort=7.57 velocity=8.22 -> lower=-2.0944 upper=1.91986 effort=7.5 velocity=5.76; origin xyz=-0.0265 -9.71445e-17 -0.0691 rpy=-1.5708 1.5708 0.0 -> xyz=-0.0265 -9.71445e-17 -0.0691 rpy=-1.5708 1.5708 0
- joint RHipRoll: axis -0.0 -0.0 -1.0 -> -0 -0 -1; limit lower=-1.5708 upper=1.5708 effort=7.57 velocity=8.22 -> lower=-1.5708 upper=1.5708 effort=7.5 velocity=5.76; origin xyz=-0.046 0.0414 6.93889e-18 rpy=-3.14159 1.5708 0.0 -> xyz=-0.046 0.0414 6.93889e-18 rpy=-3.14159 1.5708 0
- joint RHipYaw: axis -0.0 1.0 -0.0 -> -0 1 -0; limit lower=-1.5708 upper=1.5708 effort=7.57 velocity=8.22 -> lower=-1.5708 upper=1.5708 effort=7.5 velocity=5.76; origin xyz=7.99361e-15 -0.055 4.68375e-17 rpy=-1.5708 -0.0 0.0 -> xyz=7.99361e-15 -0.055 4.68375e-17 rpy=-1.5708 -0 0
- joint RKnee: axis -0.0 -1.0 -0.0 -> -0 -1 -0; limit lower=-2.96706 upper=0.0 effort=10.0 velocity=10.0 -> lower=-2.96706 upper=0 effort=8.775 velocity=4.82
- joint RLB: axis 0.0 1.22465e-16 1.0 -> 0 1.22465e-16 1; limit lower=0 upper=0 effort=0.0 velocity=0.0 -> effort=0 velocity=0
- joint RLF: axis 0.0 1.22465e-16 1.0 -> 0 1.22465e-16 1; limit lower=0 upper=0 effort=0.0 velocity=0.0 -> effort=0 velocity=0
- joint RRB: axis 0.0 1.22465e-16 1.0 -> 0 1.22465e-16 1; limit lower=0 upper=0 effort=0.0 velocity=0.0 -> effort=0 velocity=0
- joint RRF: axis 0.0 1.22465e-16 1.0 -> 0 1.22465e-16 1; limit lower=0 upper=0 effort=0.0 velocity=0.0 -> effort=0 velocity=0
- joint RShoulderPitch: axis -0.0 1.0 -0.0 -> -0 1 -0; limit lower=-3.14159 upper=3.14159 effort=5.43 velocity=10.33 -> lower=-3.14159 upper=3.14159 effort=5.475 velocity=8.17
- joint RShoulderRoll: axis -0.0 -0.0 -1.0 -> -0 -0 -1; limit lower=0.0 upper=3.14159 effort=5.43 velocity=10.33 -> lower=0 upper=3.14159 effort=5.475 velocity=8.17; origin xyz=-0.01695 0.042 0.0 rpy=1.5708 8.32338e-16 -1.5708 -> xyz=-0.01695 0.042 0 rpy=1.5708 8.32338e-16 -1.5708
- joint base_link_to_base: origin xyz=0.0 0.0 0.0 rpy=0.0 0.0 0.0 -> xyz=0 0 0 rpy=0.0 0 0
- joint camera_frame: axis 0.0 0.0 0.0 -> 0 0 0
- joint camera_optical_frame_frame: axis 0.0 0.0 0.0 -> 0 0 0; origin xyz=0.0432 0.08 -0.0235 rpy=3.14159 -1.5708 0.0 -> xyz=0.0432 0.08 -0.0235 rpy=3.14159 -1.5708 0
- joint imu_frame_2_frame: axis 0.0 0.0 0.0 -> 0 0 0
- joint imu_frame_frame: axis 0.0 0.0 0.0 -> 0 0 0
- joint l_cleat_l_back_frame: axis 0.0 0.0 0.0 -> 0 0 0
- joint l_cleat_l_front_frame: axis 0.0 0.0 0.0 -> 0 0 0; origin xyz=0.0 -0.0005 -0.016 rpy=3.06162e-16 -4.4319e-17 -3.14159 -> xyz=0 -0.0005 -0.016 rpy=3.06162e-16 -4.4319e-17 -3.14159
- joint l_cleat_r_back_frame: axis 0.0 0.0 0.0 -> 0 0 0; origin xyz=0.0 -0.0005 -0.016 rpy=2.92719e-16 -4.05989e-17 -3.14159 -> xyz=0 -0.0005 -0.016 rpy=2.92719e-16 -4.05989e-17 -3.14159
- joint l_cleat_r_front_frame: axis 0.0 0.0 0.0 -> 0 0 0; origin xyz=0.0 -0.0005 -0.016 rpy=3.00788e-16 -1.03785e-15 -3.14159 -> xyz=0 -0.0005 -0.016 rpy=3.00788e-16 -1.03785e-15 -3.14159
- joint l_sole_frame: axis 0.0 0.0 0.0 -> 0 0 0
- joint l_toe_frame: axis 0.0 0.0 0.0 -> 0 0 0
- joint l_wrist_frame: axis 0.0 0.0 0.0 -> 0 0 0
- joint r_cleat_l_back_frame: axis 0.0 0.0 0.0 -> 0 0 0; origin xyz=0.0 -0.0005 -0.016 rpy=-1.17224e-15 -1.58433e-17 -3.14159 -> xyz=0 -0.0005 -0.016 rpy=-1.17224e-15 -1.58433e-17 -3.14159
- joint r_cleat_l_front_frame: axis 0.0 0.0 0.0 -> 0 0 0
- joint r_cleat_r_back_frame: axis 0.0 0.0 0.0 -> 0 0 0
- joint r_cleat_r_front_frame: axis 0.0 0.0 0.0 -> 0 0 0
- joint r_sole_frame: axis 0.0 0.0 0.0 -> 0 0 0
- joint r_toe_frame: axis 0.0 0.0 0.0 -> 0 0 0
- joint r_wrist_frame: axis 0.0 0.0 0.0 -> 0 0 0

Commit message: more robot.urdf reformatting

File: wolfgang_description/urdf/robot.urdf (robot description, URDF)
Before this commit: robot wolfgang, 48 links, 47 joints
Links:
- link camera: mass 1e-9 -> 1e-09
- link camera_optical_frame: mass 1e-9 -> 1e-09
- link imu_frame: mass 1e-9 -> 1e-09
- link imu_frame_2: mass 1e-9 -> 1e-09
- link l_cleat_l_back: mass 1e-9 -> 1e-09
- link l_cleat_l_front: mass 1e-9 -> 1e-09
- link l_cleat_r_back: mass 1e-9 -> 1e-09
- link l_cleat_r_front: mass 1e-9 -> 1e-09
- link l_sole: mass 1e-9 -> 1e-09
- link l_toe: mass 1e-9 -> 1e-09
- link l_wrist: mass 1e-9 -> 1e-09
- link r_cleat_l_back: mass 1e-9 -> 1e-09
- link r_cleat_l_front: mass 1e-9 -> 1e-09
- link r_cleat_r_back: mass 1e-9 -> 1e-09
- link r_cleat_r_front: mass 1e-9 -> 1e-09
- link r_sole: mass 1e-9 -> 1e-09
- link r_toe: mass 1e-9 -> 1e-09
- link r_wrist: mass 1e-9 -> 1e-09
Joints:
- joint HeadPan: axis -0 -0 -1 -> -0.0 -0.0 -1.0
- joint HeadTilt: axis -0 -0 1 -> -0.0 -0.0 1.0
- joint LAnklePitch: axis -0 -0 -1 -> -0.0 -0.0 -1.0
- joint LAnkleRoll: axis -0 -1 -0 -> -0.0 -1.0 -0.0; origin xyz=0.0691 1.66533e-16 -0.026 rpy=1.5708 -1.5708 0 -> xyz=0.0691 1.66533e-16 -0.026 rpy=1.5708 -1.5708 0.0
- joint LElbow: axis 0 0 1 -> 0.0 0.0 1.0
- joint LHipPitch: axis 7.95491e-17 -3.00167e-16 -1 -> 7.95491e-17 -3.00167e-16 -1.0; origin xyz=0.026 6.93889e-18 -0.0691 rpy=2.67116e-16 -1.5708 0 -> xyz=0.026 6.93889e-18 -0.0691 rpy=2.67116e-16 -1.5708 0.0
- joint LHipRoll: axis -0 -0 -1 -> -0.0 -0.0 -1.0; origin xyz=-0.046 0.0414 6.93889e-18 rpy=3.14159 1.5708 0 -> xyz=-0.046 0.0414 6.93889e-18 rpy=3.14159 1.5708 0.0
- joint LHipYaw: axis -0 1 -0 -> -0.0 1.0 -0.0; origin xyz=1.82493e-15 0.055 -4.22839e-18 rpy=-1.5708 -0 0 -> xyz=1.82493e-15 0.055 -4.22839e-18 rpy=-1.5708 -0.0 0.0
- joint LKnee: axis -0 1 -0 -> -0.0 1.0 -0.0; limit lower=0 upper=2.96706 effort=8.775 velocity=4.82 -> lower=0.0 upper=2.96706 effort=8.775 velocity=4.82
- joint LLB: axis 0 1.22465e-16 1 -> 0.0 1.22465e-16 1.0; limit effort=0 velocity=0 -> lower=0 upper=0 effort=0.0 velocity=0.0
- joint LLF: axis 0 1.22465e-16 1 -> 0.0 1.22465e-16 1.0; limit effort=0 velocity=0 -> lower=0 upper=0 effort=0.0 velocity=0.0
- joint LRB: axis 0 1.22465e-16 1 -> 0.0 1.22465e-16 1.0; limit effort=0 velocity=0 -> lower=0 upper=0 effort=0.0 velocity=0.0
- joint LRF: axis 0 -1.22465e-16 -1 -> 0.0 -1.22465e-16 -1.0; limit effort=0 velocity=0 -> lower=0 upper=0 effort=0.0 velocity=0.0
- joint LShoulderPitch: axis -0 1 -0 -> -0.0 1.0 -0.0
- joint LShoulderRoll: axis -0 -0 -1 -> -0.0 -0.0 -1.0; limit lower=-3.14159 upper=0 effort=5.475 velocity=8.17 -> lower=-3.14159 upper=0.0 effort=5.475 velocity=8.17
- joint RAnklePitch: axis -0 -0 -1 -> -0.0 -0.0 -1.0
- joint RAnkleRoll: axis 0 -1 0 -> 0.0 -1.0 0.0
- joint RElbow: axis 0 0 1 -> 0.0 0.0 1.0
- joint RHipPitch: axis -0 1 -0 -> -0.0 1.0 -0.0; origin xyz=-0.0265 -9.71445e-17 -0.0691 rpy=-1.5708 1.5708 0 -> xyz=-0.0265 -9.71445e-17 -0.0691 rpy=-1.5708 1.5708 0.0
- joint RHipRoll: axis -0 -0 -1 -> -0.0 -0.0 -1.0; origin xyz=-0.046 0.0414 6.93889e-18 rpy=-3.14159 1.5708 0 -> xyz=-0.046 0.0414 6.93889e-18 rpy=-3.14159 1.5708 0.0
- joint RHipYaw: axis -0 1 -0 -> -0.0 1.0 -0.0; origin xyz=7.99361e-15 -0.055 4.68375e-17 rpy=-1.5708 -0 0 -> xyz=7.99361e-15 -0.055 4.68375e-17 rpy=-1.5708 -0.0 0.0
- joint RKnee: axis -0 -1 -0 -> -0.0 -1.0 -0.0; limit lower=-2.96706 upper=0 effort=8.775 velocity=4.82 -> lower=-2.96706 upper=0.0 effort=8.775 velocity=4.82
- joint RLB: axis 0 1.22465e-16 1 -> 0.0 1.22465e-16 1.0; limit effort=0 velocity=0 -> lower=0 upper=0 effort=0.0 velocity=0.0
- joint RLF: axis 0 1.22465e-16 1 -> 0.0 1.22465e-16 1.0; limit effort=0 velocity=0 -> lower=0 upper=0 effort=0.0 velocity=0.0
- joint RRB: axis 0 1.22465e-16 1 -> 0.0 1.22465e-16 1.0; limit effort=0 velocity=0 -> lower=0 upper=0 effort=0.0 velocity=0.0
- joint RRF: axis 0 1.22465e-16 1 -> 0.0 1.22465e-16 1.0; limit effort=0 velocity=0 -> lower=0 upper=0 effort=0.0 velocity=0.0
- joint RShoulderPitch: axis -0 1 -0 -> -0.0 1.0 -0.0
- joint RShoulderRoll: axis -0 -0 -1 -> -0.0 -0.0 -1.0; limit lower=0 upper=3.14159 effort=5.475 velocity=8.17 -> lower=0.0 upper=3.14159 effort=5.475 velocity=8.17; origin xyz=-0.01695 0.042 0 rpy=1.5708 8.32338e-16 -1.5708 -> xyz=-0.01695 0.042 0.0 rpy=1.5708 8.32338e-16 -1.5708
- joint base_link_to_base: origin xyz=0 0 0 rpy=0.0 0 0 -> xyz=0.0 0.0 0.0 rpy=0.0 0.0 0.0
- joint camera_frame: axis 0 0 0 -> 0.0 0.0 0.0
- joint camera_optical_frame_frame: axis 0 0 0 -> 0.0 0.0 0.0; origin xyz=0.0432 0.08 -0.0235 rpy=3.14159 -1.5708 0 -> xyz=0.0432 0.08 -0.0235 rpy=3.14159 -1.5708 0.0
- joint imu_frame_2_frame: axis 0 0 0 -> 0.0 0.0 0.0
- joint imu_frame_frame: axis 0 0 0 -> 0.0 0.0 0.0
- joint l_cleat_l_back_frame: axis 0 0 0 -> 0.0 0.0 0.0
- joint l_cleat_l_front_frame: axis 0 0 0 -> 0.0 0.0 0.0; origin xyz=0 -0.0005 -0.016 rpy=3.06162e-16 -4.4319e-17 -3.14159 -> xyz=0.0 -0.0005 -0.016 rpy=3.06162e-16 -4.4319e-17 -3.14159
- joint l_cleat_r_back_frame: axis 0 0 0 -> 0.0 0.0 0.0; origin xyz=0 -0.0005 -0.016 rpy=2.92719e-16 -4.05989e-17 -3.14159 -> xyz=0.0 -0.0005 -0.016 rpy=2.92719e-16 -4.05989e-17 -3.14159
- joint l_cleat_r_front_frame: axis 0 0 0 -> 0.0 0.0 0.0; origin xyz=0 -0.0005 -0.016 rpy=3.00788e-16 -1.03785e-15 -3.14159 -> xyz=0.0 -0.0005 -0.016 rpy=3.00788e-16 -1.03785e-15 -3.14159
- joint l_sole_frame: axis 0 0 0 -> 0.0 0.0 0.0
- joint l_toe_frame: axis 0 0 0 -> 0.0 0.0 0.0
- joint l_wrist_frame: axis 0 0 0 -> 0.0 0.0 0.0
- joint r_cleat_l_back_frame: axis 0 0 0 -> 0.0 0.0 0.0; origin xyz=0 -0.0005 -0.016 rpy=-1.17224e-15 -1.58433e-17 -3.14159 -> xyz=0.0 -0.0005 -0.016 rpy=-1.17224e-15 -1.58433e-17 -3.14159
- joint r_cleat_l_front_frame: axis 0 0 0 -> 0.0 0.0 0.0
- joint r_cleat_r_back_frame: axis 0 0 0 -> 0.0 0.0 0.0
- joint r_cleat_r_front_frame: axis 0 0 0 -> 0.0 0.0 0.0
- joint r_sole_frame: axis 0 0 0 -> 0.0 0.0 0.0
- joint r_toe_frame: axis 0 0 0 -> 0.0 0.0 0.0
- joint r_wrist_frame: axis 0 0 0 -> 0.0 0.0 0.0

Commit message: ankle and hip_u_connector model

File: wolfgang_description/urdf/robot.urdf (robot description, URDF)
Before this commit: robot wolfgang, 48 links, 47 joints
Links:
- link l_foot: geometry collision box size=0.008 0.04 0.004; collision box size=0.008 0.04 0.004
- link l_hip_1: geometry collision box size=0.0260229 0.004 0.053; collision box size=0.0260229 0.004 0.053
- link r_foot: geometry collision box size=0.008 0.04 0.004; collision box size=0.008 0.04 0.004
- link r_hip_1: geometry collision box size=0.0260229 0.004 0.053; collision box size=0.0260229 0.004 0.053

Commit message: change knee velocities to values from proto

File: wolfgang_description/urdf/robot.urdf (robot description, URDF)
Before this commit: robot wolfgang, 48 links, 47 joints
Joints:
- joint LKnee: limit lower=0.0 upper=2.96706 effort=8.775 velocity=4.82 -> lower=0.0 upper=2.96706 effort=8.775 velocity=3.87
- joint RKnee: limit lower=-2.96706 upper=0.0 effort=8.775 velocity=4.82 -> lower=-2.96706 upper=0.0 effort=8.775 velocity=3.87

Commit message: change cleat height to 14mm

File: wolfgang_description/urdf/robot.urdf (robot description, URDF)
Before this commit: robot wolfgang, 48 links, 47 joints
Joints:
- joint l_cleat_l_back_frame: origin xyz=1.38778e-17 -0.0005 -0.016 rpy=1.67348e-16 -4.15297e-16 3.14159 -> xyz=1.38778e-17 -0.0005 -0.014 rpy=1.67348e-16 -4.15297e-16 3.14159
- joint l_cleat_l_front_frame: origin xyz=0.0 -0.0005 -0.016 rpy=3.06162e-16 -4.4319e-17 -3.14159 -> xyz=0.0 -0.0005 -0.014 rpy=3.06162e-16 -4.4319e-17 -3.14159
- joint l_cleat_r_back_frame: origin xyz=0.0 -0.0005 -0.016 rpy=2.92719e-16 -4.05989e-17 -3.14159 -> xyz=0.0 -0.0005 -0.014 rpy=2.92719e-16 -4.05989e-17 -3.14159
- joint l_cleat_r_front_frame: origin xyz=0.0 -0.0005 -0.016 rpy=3.00788e-16 -1.03785e-15 -3.14159 -> xyz=0.0 -0.0005 -0.014 rpy=3.00788e-16 -1.03785e-15 -3.14159
- joint r_cleat_l_back_frame: origin xyz=0.0 -0.0005 -0.016 rpy=-1.17224e-15 -1.58433e-17 -3.14159 -> xyz=0.0 -0.0005 -0.014 rpy=-1.17224e-15 -1.58433e-17 -3.14159
- joint r_cleat_l_front_frame: origin xyz=-1.38778e-17 -0.0005 -0.016 rpy=2.44346e-16 2.736e-16 -3.14159 -> xyz=-1.38778e-17 -0.0005 -0.014 rpy=2.44346e-16 2.736e-16 -3.14159
- joint r_cleat_r_back_frame: origin xyz=-1.38778e-17 -0.0005 -0.016 rpy=3.0848e-17 -1.36062e-15 3.14159 -> xyz=-1.38778e-17 -0.0005 -0.014 rpy=3.0848e-17 -1.36062e-15 3.14159
- joint r_cleat_r_front_frame: origin xyz=-6.93889e-17 -0.0005 -0.016 rpy=6.44157e-16 8.47782e-16 -3.14159 -> xyz=-6.93889e-17 -0.0005 -0.014 rpy=6.44157e-16 8.47782e-16 -3.14159

Commit message: fix head position to correct limits

File: wolfgang_description/urdf/robot.urdf (robot description, URDF)
Before this commit: robot wolfgang, 48 links, 47 joints
Joints:
- joint HeadPan: limit lower=-2.0944 upper=2.0944 effort=5.475 velocity=8.17 -> lower=-2.36 upper=2.36 effort=5.475 velocity=8.17
- joint HeadTilt: limit lower=-1.5708 upper=1.0472 effort=5.475 velocity=8.17 -> lower=-1.57 upper=1.0472 effort=5.475 velocity=8.17

Commit message: fix

File: wolfgang_description/urdf/robot.urdf (robot description, URDF)
Before this commit: robot wolfgang, 48 links, 47 joints
Joints:
- joint HeadPan: limit lower=-2.36 upper=2.36 effort=5.475 velocity=8.17 -> lower=-2.35619 upper=2.35619 effort=5.475 velocity=8.17
- joint HeadTilt: limit lower=-1.57 upper=1.0472 effort=5.475 velocity=8.17 -> lower=-1.5708 upper=1.0472 effort=5.475 velocity=8.17

Commit message: urdf: change servo values to be same as in proto

File: wolfgang_description/urdf/robot.urdf (robot description, URDF)
Before this commit: robot wolfgang, 48 links, 47 joints
Joints:
- joint HeadPan: limit lower=-2.35619 upper=2.35619 effort=5.475 velocity=8.17 -> lower=-2.35619 upper=2.35619 effort=7.3 velocity=8.17
- joint HeadTilt: limit lower=-1.5708 upper=1.0472 effort=5.475 velocity=8.17 -> lower=-1.5708 upper=1.0472 effort=7.3 velocity=8.17
- joint LAnklePitch: limit lower=-1.22173 upper=1.74533 effort=7.5 velocity=5.76 -> lower=-1.22173 upper=1.74533 effort=10 velocity=5.76
- joint LAnkleRoll: limit lower=-1.0472 upper=1.0472 effort=7.5 velocity=5.76 -> lower=-1.0472 upper=1.0472 effort=10 velocity=5.76
- joint LElbow: limit lower=-1.5708 upper=1.0472 effort=5.475 velocity=8.17 -> lower=-1.5708 upper=1.0472 effort=7.3 velocity=8.17
- joint LHipPitch: limit lower=-1.91986 upper=2.0944 effort=7.5 velocity=5.76 -> lower=-1.91986 upper=2.0944 effort=10 velocity=5.76
- joint LHipRoll: limit lower=-1.5708 upper=1.5708 effort=7.5 velocity=5.76 -> lower=-1.5708 upper=1.5708 effort=10 velocity=5.76
- joint LHipYaw: limit lower=-1.5708 upper=1.5708 effort=7.5 velocity=5.76 -> lower=-1.5708 upper=1.5708 effort=10 velocity=5.76
- joint LKnee: limit lower=0.0 upper=2.96706 effort=8.775 velocity=3.87 -> lower=0.0 upper=2.96706 effort=12.9 velocity=3.87
- joint LShoulderPitch: limit lower=-3.14159 upper=3.14159 effort=5.475 velocity=8.17 -> lower=-3.14159 upper=3.14159 effort=7.3 velocity=8.17
- joint LShoulderRoll: limit lower=-3.14159 upper=0.0 effort=5.475 velocity=8.17 -> lower=-3.14159 upper=0.0 effort=7.3 velocity=8.17
- joint RAnklePitch: limit lower=-1.74533 upper=1.22173 effort=7.5 velocity=5.76 -> lower=-1.74533 upper=1.22173 effort=10 velocity=5.76
- joint RAnkleRoll: limit lower=-1.0472 upper=1.0472 effort=7.5 velocity=5.76 -> lower=-1.0472 upper=1.0472 effort=10 velocity=5.76
- joint RElbow: limit lower=-1.0472 upper=1.5708 effort=5.475 velocity=8.17 -> lower=-1.0472 upper=1.5708 effort=7.3 velocity=8.17
- joint RHipPitch: limit lower=-2.0944 upper=1.91986 effort=7.5 velocity=5.76 -> lower=-2.0944 upper=1.91986 effort=10 velocity=5.76
- joint RHipRoll: limit lower=-1.5708 upper=1.5708 effort=7.5 velocity=5.76 -> lower=-1.5708 upper=1.5708 effort=10 velocity=5.76
- joint RHipYaw: limit lower=-1.5708 upper=1.5708 effort=7.5 velocity=5.76 -> lower=-1.5708 upper=1.5708 effort=10 velocity=5.76
- joint RKnee: limit lower=-2.96706 upper=0.0 effort=8.775 velocity=3.87 -> lower=-2.96706 upper=0.0 effort=12.9 velocity=3.87
- joint RShoulderPitch: limit lower=-3.14159 upper=3.14159 effort=5.475 velocity=8.17 -> lower=-3.14159 upper=3.14159 effort=7.3 velocity=8.17
- joint RShoulderRoll: limit lower=0.0 upper=3.14159 effort=5.475 velocity=8.17 -> lower=0.0 upper=3.14159 effort=7.3 velocity=8.17

Commit message: last remaining files and delete parts in urdf

File: wolfgang_description/urdf/robot.urdf (robot description, URDF)
Before this commit: robot wolfgang, 47 links, 46 joints
Links:
- link l_foot: geometry collision box size=0.008 0.04 0.004; collision box size=0.008 0.04 0.004
- link l_upper_leg: geometry collision box size=0.01 0.002 0.01; collision box size=0.01 0.002 0.01
- link r_foot: geometry collision box size=0.008 0.04 0.004; collision box size=0.008 0.04 0.004
- link r_upper_leg: geometry collision box size=0.01 0.002 0.01; collision box size=0.01 0.002 0.01
- link torso: geometry collision box size=0.019 0.0468795 0.005; collision box size=0.019 0.0468795 0.005

Commit message: rm batttery cage holder from visual model

File: wolfgang_description/urdf/robot.urdf (robot description, URDF)
Before this commit: robot wolfgang, 47 links, 46 joints
Links:
- link torso: geometry collision box size=0.019 0.0468795 0.005; collision box size=0.019 0.0468795 0.005
