Commit message: command out joint constraints

File: bitbots_wolfgang/wolfgang_description/urdf/robot.urdf (robot description, URDF)
Before this commit: robot wolfgang, 48 links, 47 joints
Joints:
- joint LAnklePitch: limit lower=-1.22173 upper=1.74533 effort=10 velocity=5.76 -> lower=-10 upper=10 effort=10 velocity=5.76
- joint LAnkleRoll: limit lower=-1.0472 upper=1.0472 effort=10 velocity=5.76 -> lower=-10 upper=10 effort=10 velocity=5.76
- joint LHipPitch: limit lower=-1.91986 upper=2.0944 effort=10 velocity=5.76 -> lower=-10 upper=10 effort=10 velocity=5.76
- joint LHipRoll: limit lower=-1.5708 upper=1.5708 effort=10 velocity=5.76 -> lower=-10 upper=10 effort=10 velocity=5.76
- joint LHipYaw: limit lower=-1.5708 upper=1.5708 effort=10 velocity=5.76 -> lower=-10 upper=10 effort=10 velocity=5.76
- joint LKnee: limit lower=0.0 upper=2.96706 effort=12.9 velocity=3.87 -> lower=-10 upper=10 effort=12.9 velocity=3.87

Commit message: Smooth dynup and working side standup

File: bitbots_wolfgang/wolfgang_description/urdf/robot.urdf (robot description, URDF)
Before this commit: robot wolfgang, 48 links, 47 joints
Joints:
- joint LAnklePitch: limit lower=-10 upper=10 effort=10 velocity=5.76 -> lower=-1.42 upper=0.37 effort=10 velocity=5.76
- joint LAnkleRoll: limit lower=-10 upper=10 effort=10 velocity=5.76 -> lower=-1.58 upper=0.63 effort=10 velocity=5.76
- joint LHipPitch: limit lower=-10 upper=10 effort=10 velocity=5.76 -> lower=-0.9 upper=2.246 effort=10 velocity=5.76
- joint LHipRoll: limit lower=-10 upper=10 effort=10 velocity=5.76 -> lower=-0.871 upper=1.769 effort=10 velocity=5.76
- joint LHipYaw: limit lower=-10 upper=10 effort=10 velocity=5.76 -> lower=-1.5708 upper=1.5708 effort=10 velocity=5.76
- joint LKnee: limit lower=-10 upper=10 effort=12.9 velocity=3.87 -> lower=0 upper=2.88 effort=12.9 velocity=3.87
- joint RAnklePitch: limit lower=-1.74533 upper=1.22173 effort=10 velocity=5.76 -> lower=-0.37 upper=1.42 effort=10 velocity=5.76
- joint RAnkleRoll: limit lower=-1.0472 upper=1.0472 effort=10 velocity=5.76 -> lower=-0.63 upper=1.58 effort=10 velocity=5.76
- joint RHipPitch: limit lower=-2.0944 upper=1.91986 effort=10 velocity=5.76 -> lower=-2.246 upper=0.9 effort=10 velocity=5.76
- joint RHipRoll: limit lower=-1.5708 upper=1.5708 effort=10 velocity=5.76 -> lower=-1.769 upper=0.871 effort=10 velocity=5.76
- joint RKnee: limit lower=-2.96706 upper=0.0 effort=12.9 velocity=3.87 -> lower=-2.88 upper=0.0 effort=12.9 velocity=3.87

Commit message: wolfgang_description: update joint limits

File: bitbots_wolfgang/wolfgang_description/urdf/robot.urdf (robot description, URDF)
Before this commit: robot wolfgang, 48 links, 47 joints
Joints:
- joint HeadTilt: limit lower=-1.5708 upper=1.0472 effort=7.3 velocity=8.17 -> lower=-1.923 upper=1.24 effort=7.3 velocity=8.17
- joint LAnkleRoll: limit lower=-1.58 upper=0.63 effort=10 velocity=5.76 -> lower=-1.58 upper=1.4 effort=10 velocity=5.76
- joint LElbow: limit lower=-1.5708 upper=1.0472 effort=7.3 velocity=8.17 -> lower=-1.5708 upper=0.78 effort=7.3 velocity=8.17
- joint LHipPitch: limit lower=-0.9 upper=2.246 effort=10 velocity=5.76 -> lower=-0.87 upper=2.77 effort=10 velocity=5.76
- joint LHipRoll: limit lower=-0.871 upper=1.769 effort=10 velocity=5.76 -> lower=-1.6 upper=1.9 effort=10 velocity=5.76
- joint LKnee: limit lower=0 upper=2.88 effort=12.9 velocity=3.87 -> lower=-0.2 upper=2.8 effort=12.9 velocity=3.87
- joint LShoulderRoll: limit lower=-3.14159 upper=0.0 effort=7.3 velocity=8.17 -> lower=-3.1416 upper=0.12 effort=7.3 velocity=8.17
- joint RAnkleRoll: limit lower=-0.63 upper=1.58 effort=10 velocity=5.76 -> lower=-1.4 upper=1.58 effort=10 velocity=5.76
- joint RElbow: limit lower=-1.0472 upper=1.5708 effort=7.3 velocity=8.17 -> lower=-0.78 upper=1.5708 effort=7.3 velocity=8.17
- joint RHipPitch: limit lower=-2.246 upper=0.9 effort=10 velocity=5.76 -> lower=-2.77 upper=0.87 effort=10 velocity=5.76
- joint RHipRoll: limit lower=-1.769 upper=0.871 effort=10 velocity=5.76 -> lower=-1.9 upper=1.6 effort=10 velocity=5.76
- joint RKnee: limit lower=-2.88 upper=0.0 effort=12.9 velocity=3.87 -> lower=-2.8 upper=0.2 effort=12.9 velocity=3.87
- joint RShoulderRoll: limit lower=0.0 upper=3.14159 effort=7.3 velocity=8.17 -> lower=-0.12 upper=3.1416 effort=7.3 velocity=8.17

Commit message: Update HipPitch limits with new upper leg spacers

File: bitbots_wolfgang/wolfgang_description/urdf/robot.urdf (robot description, URDF)
Before this commit: robot wolfgang, 48 links, 47 joints
Joints:
- joint LHipPitch: limit lower=-0.87 upper=2.77 effort=10 velocity=5.76 -> lower=-0.79 upper=2.77 effort=10 velocity=5.76
- joint RHipPitch: limit lower=-2.77 upper=0.87 effort=10 velocity=5.76 -> lower=-2.77 upper=0.79 effort=10 velocity=5.76

Commit message: experimental 5 cm foot pitch rigging offset

File: bitbots_wolfgang/wolfgang_description/urdf/robot.urdf (robot description, URDF)
Before this commit: robot wolfgang, 48 links, 47 joints
Joints:
- joint l_sole_frame: origin xyz=-0.0152219 0.0907683 -0.0529 rpy=-5.77818e-15 -6.98371e-15 1.5708 -> xyz=-0.0152219 0.1407683 -0.0529 rpy=-5.77818e-15 -6.98371e-15 1.5708
- joint r_sole_frame: origin xyz=0.0152219 0.0907683 -0.0529 rpy=-4.1858e-16 2.36866e-15 1.5708 -> xyz=0.0152219 0.1407683 -0.0529 rpy=-4.1858e-16 2.36866e-15 1.5708

Commit message: moved IK to absolute front of toe, for reference

File: bitbots_wolfgang/wolfgang_description/urdf/robot.urdf (robot description, URDF)
Before this commit: robot wolfgang, 48 links, 47 joints
Joints:
- joint l_sole_frame: origin xyz=-0.0152219 0.1407683 -0.0529 rpy=-5.77818e-15 -6.98371e-15 1.5708 -> xyz=-0.0152219 0.175 -0.039 rpy=-5.77818e-15 -6.98371e-15 1.5708
- joint r_sole_frame: origin xyz=0.0152219 0.1407683 -0.0529 rpy=-4.1858e-16 2.36866e-15 1.5708 -> xyz=0.0152219 0.175 -0.039 rpy=-4.1858e-16 2.36866e-15 1.5708

Commit message: study 2: IK endpoint at correct toe joint position

File: bitbots_wolfgang/wolfgang_description/urdf/robot.urdf (robot description, URDF)
Before this commit: robot wolfgang, 48 links, 47 joints
Joints:
- joint l_sole_frame: origin xyz=-0.0152219 0.175 -0.039 rpy=-5.77818e-15 -6.98371e-15 1.5708 -> xyz=-0.0152219 0.121 -0.039 rpy=-5.77818e-15 -6.98371e-15 1.5708
- joint r_sole_frame: origin xyz=0.0152219 0.175 -0.039 rpy=-4.1858e-16 2.36866e-15 1.5708 -> xyz=0.0152219 0.121 -0.039 rpy=-4.1858e-16 2.36866e-15 1.5708
