Commit message: sry wolfgang

File: bitbots_robot/wolfgang_description/urdf/robot.urdf (robot description, URDF)
Before this commit: robot wolfgang, 48 links, 47 joints
Joints:
- joint LShoulderRoll: limit lower=-3.1416 upper=0.12 effort=7.3 velocity=8.17 -> lower=-3.1416 upper=0.33 effort=7.3 velocity=8.17
- joint RShoulderRoll: limit lower=-0.12 upper=3.1416 effort=7.3 velocity=8.17 -> lower=-0.33 upper=3.1416 effort=7.3 velocity=8.17
