Commit message: client to control x02 via websocket

File: bitbots_robot/x02_description/urdf/robot.urdf (robot description, URDF)
Before this commit: robot x2, 27 links, 26 joints
Links:
- removed link world
- added link imu_frame_uncalibrated
Joints:
- removed joint pelvis_link
- added joint imu_frame_uncalibrated_joint: type fixed, parent base_link, child imu_frame_uncalibrated, origin xyz=0.0 0 0.0 rpy=0 0 0
- joint L_shoulder_yaw: axis 0 0 1 -> (none); limit lower=-2.618 upper=2.618 effort=45 velocity=30 -> (none)
- joint R_shoulder_yaw: axis 0 0 -1 -> (none); limit lower=-2.618 upper=2.618 effort=45 velocity=30 -> (none)
- joint logo: axis 0 0 0 -> (none)
- joint torso: axis 0 0 0 -> (none); child base_link -> waist_yaw_link; origin xyz=0 0 0.03675 rpy=0 0 0 -> xyz=0 0 -0.03675 rpy=0 0 0; parent waist_yaw_link -> base_link
- joint waist_yaw: axis 0 0 1 -> (none); child waist_yaw_link -> pelvis_link; limit lower=-1.047 upper=1.047 effort=83.5 velocity=43 -> (none); origin xyz=0 0 0.08375 rpy=0 0 0 -> xyz=0 0 -0.08375 rpy=0 0 0; parent pelvis_link -> waist_yaw_link

Commit message: changes for running demo behavior

File: bitbots_robot/x02_description/urdf/robot.urdf (robot description, URDF)
Before this commit: robot x2, 27 links, 26 joints
Links:
- added link camera_frame_uncalibrated
- added link camera_optical_frame_uncalibrated
Joints:
- added joint camera_frame_uncalibrated_joint: type fixed, parent base_link, child camera_frame_uncalibrated, origin xyz=0.085 0.0 0.43 rpy=0 1.035398163 0
- added joint camera_optical_frame_uncalibrated_joint: type fixed, parent camera_frame_uncalibrated, child camera_optical_frame_uncalibrated, origin xyz=0.0 0.0 0.0 rpy=-1.570796327 0 -1.570796327
