Commit message: fix camera pose for different x02 head

File: src/bitbots_robot/x02_description/urdf/robot.urdf (robot description, URDF)
Before this commit: robot x2, 29 links, 28 joints
Joints:
- joint camera_frame_uncalibrated_joint: origin xyz=0.085 0.0 0.43 rpy=0 1.035398163 0 -> xyz=0.085 0.0 0.58 rpy=0 0.25 0
