Commit message: Fix r ankle roll angle
Signed-off-by: Florian Vahl <florian@flova.de>

File: src/bitbots_robot/wolfgang_description/urdf/robot.urdf (robot description, URDF)
Before this commit: robot wolfgang, 48 links, 47 joints
Joints:
- joint RAnkleRoll: origin xyz=-0.0691 -1.11022e-16 -0.026 rpy=-1.46564e-14 1.54833 -1.5708 -> xyz=-0.0691 -1.11022e-16 -0.026 rpy=-1.46564e-14 1.5708 -1.5708
