Commit message: path names for meshes changed

File: src/bitbots_robot/x02_description/x02.urdf (robot description, URDF)
Before this commit: robot x2, 25 links, 24 joints
Links:
- link L_ankle_pitch_link: geometry collision sphere radius=0.005; collision sphere radius=0.005
- link L_elbow_pitch_link: geometry collision mesh filename=package://x02_description/urdf/meshes/L_elbow_pitch_link.STL; visual mesh filename=package://x02_description/urdf/meshes/L_elbow_pitch_link.STL
- link L_hip_pitch_link: geometry collision mesh filename=package://x02_description/urdf/package://x02_description/ur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; visual mesh filename=package://x02_description/urdf/package://x02_description/ur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
- link L_hip_roll_link: geometry collision mesh filename=package://x02_description/urdf/package://x02_description/ur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; visual mesh filename=package://x02_description/urdf/package://x02_description/ur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
- link L_hip_yaw_link: geometry collision mesh filename=package://x02_description/urdf/package://x02_description/ur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; visual mesh filename=package://x02_description/urdf/package://x02_description/ur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
- link L_knee_pitch_link: geometry collision mesh filename=package://x02_description/urdf/package://x02_description/ur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; visual mesh filename=package://x02_description/urdf/package://x02_description/ur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
- link L_shoulder_pitch_link: geometry collision mesh filename=package://x02_description/urdf/meshes/L_shoulder_pitch_link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; visual mesh filename=package://x02_description/urdf/meshes/L_shoulder_pitch_link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
- link L_shoulder_roll_link: geometry collision mesh filename=package://x02_description/urdf/meshes/L_shoulder_roll_link.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; visual mesh filename=package://x02_description/urdf/meshes/L_shoulder_roll_link.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
- link L_shoulder_yaw_link: geometry collision mesh filename=package://x02_description/urdf/meshes/L_shoulder_yaw_link.S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; visual mesh filename=package://x02_description/urdf/meshes/L_shoulder_yaw_link.S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
- link R_ankle_pitch_link: geometry collision sphere radius=0.005; collision sphere radius=0.005
- link R_elbow_pitch_link: geometry collision mesh filename=package://x02_description/urdf/meshes/R_elbow_pitch_link.STL; visual mesh filename=package://x02_description/urdf/meshes/R_elbow_pitch_link.STL
- link R_hip_pitch_link: geometry collision mesh filename=package://x02_description/urdf/package://x02_description/ur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; visual mesh filename=package://x02_description/urdf/package://x02_description/ur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
- link R_hip_roll_link: geometry collision mesh filename=package://x02_description/urdf/package://x02_description/ur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; visual mesh filename=package://x02_description/urdf/package://x02_description/ur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
- link R_hip_yaw_link: geometry collision mesh filename=package://x02_description/urdf/package://x02_description/ur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; visual mesh filename=package://x02_description/urdf/package://x02_description/ur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
- link R_knee_pitch_link: geometry collision mesh filename=package://x02_description/urdf/package://x02_description/ur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; visual mesh filename=package://x02_description/urdf/package://x02_description/ur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
- link R_shoulder_pitch_link: geometry collision mesh filename=package://x02_description/urdf/meshes/R_shoulder_pitch_link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; visual mesh filename=package://x02_description/urdf/meshes/R_shoulder_pitch_link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
- link R_shoulder_roll_link: geometry collision mesh filename=package://x02_description/urdf/meshes/R_shoulder_roll_link.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; visual mesh filename=package://x02_description/urdf/meshes/R_shoulder_roll_link.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
- link R_shoulder_yaw_link: geometry collision mesh filename=package://x02_description/urdf/meshes/R_shoulder_yaw_link.S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; visual mesh filename=package://x02_description/urdf/meshes/R_shoulder_yaw_link.S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
- link base_link: geometry collision mesh filename=package://x02_description/urdf/package://x02_description/ur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; visual mesh filename=package://x02_description/urdf/package://x02_description/ur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
- link head_link: geometry collision mesh filename=package://x02_description/urdf/meshes/head_link.STL; visual mesh filename=package://x02_description/urdf/meshes/head_link.STL
- link logo_link: geometry collision mesh filename=package://x02_description/urdf/meshes/logo_link.STL; visual mesh filename=package://x02_description/urdf/meshes/logo_link.STL
- link pelvis_link: geometry collision mesh filename=package://x02_description/urdf/package://x02_description/ur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; visual mesh filename=package://x02_description/urdf/package://x02_description/ur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

Commit message: effort values for hip changed

File: src/bitbots_robot/x02_description/x02.urdf (robot description, URDF)
Before this commit: robot x2, 25 links, 24 joints
Joints:
- joint LHipPitch: limit lower=-0.5236 upper=2.13 effort=72 velocity=9.163 -> lower=-0.5236 upper=2.13 effort=45 velocity=9.163
- joint LHipRoll: limit lower=-0.2618 upper=0.524 effort=50 velocity=10.471975511965978 -> lower=-0.2618 upper=0.524 effort=45 velocity=10.471975511965978
- joint LHipYaw: limit lower=-0.55 upper=0.55 effort=50 velocity=10.472 -> lower=-0.55 upper=0.55 effort=30 velocity=10.472
- joint RHipPitch: limit lower=-0.5236 upper=2.13 effort=72 velocity=9.163 -> lower=-0.5236 upper=2.13 effort=45 velocity=9.163
- joint RHipRoll: limit lower=-0.2618 upper=0.524 effort=50 velocity=10.472 -> lower=-0.2618 upper=0.524 effort=45 velocity=10.472
- joint RHipYaw: limit lower=-0.55 upper=0.55 effort=50 velocity=10.472 -> lower=-0.55 upper=0.55 effort=30 velocity=10.472

Commit message: urdf update

File: src/bitbots_robot/x02_description/x02.urdf (robot description, URDF)
Before this commit: robot x2, 25 links, 24 joints
Links:
- link L_ankle_pitch_link: geometry collision sphere radius=0.005; collision sphere radius=0.005
- link L_hip_pitch_link: geometry collision mesh filename=package://x02_description/urdf/meshes/L_hip_pitch_link.STL; visual mesh filename=package://x02_description/urdf/meshes/L_hip_pitch_link.STL
- link L_hip_roll_link: geometry collision mesh filename=package://x02_description/urdf/meshes/L_hip_roll_link.STL; visual mesh filename=package://x02_description/urdf/meshes/L_hip_roll_link.STL
- link L_hip_yaw_link: geometry collision mesh filename=package://x02_description/urdf/meshes/L_hip_yaw_link.STL; visual mesh filename=package://x02_description/urdf/meshes/L_hip_yaw_link.STL
- link L_knee_pitch_link: geometry collision mesh filename=package://x02_description/urdf/meshes/L_knee_pitch_link.STL; visual mesh filename=package://x02_description/urdf/meshes/L_knee_pitch_link.STL
- link R_ankle_pitch_link: geometry collision sphere radius=0.005; collision sphere radius=0.005
- link R_hip_pitch_link: geometry collision mesh filename=package://x02_description/urdf/meshes/R_hip_pitch_link.STL; visual mesh filename=package://x02_description/urdf/meshes/R_hip_pitch_link.STL
- link R_hip_roll_link: geometry collision mesh filename=package://x02_description/urdf/meshes/R_hip_roll_link.STL; visual mesh filename=package://x02_description/urdf/meshes/R_hip_roll_link.STL
- link R_hip_yaw_link: geometry collision mesh filename=package://x02_description/urdf/meshes/R_hip_yaw_link.STL; visual mesh filename=package://x02_description/urdf/meshes/R_hip_yaw_link.STL
- link R_knee_pitch_link: geometry collision mesh filename=package://x02_description/urdf/meshes/R_knee_pitch_link.STL; visual mesh filename=package://x02_description/urdf/meshes/R_knee_pitch_link.STL
- link base_link: geometry collision mesh filename=package://x02_description/urdf/meshes/torso_link.STL; visual mesh filename=package://x02_description/urdf/meshes/torso_link.STL
- link pelvis_link: geometry collision mesh filename=package://x02_description/urdf/meshes/pelvis_link.STL; visual mesh filename=package://x02_description/urdf/meshes/pelvis_link.STL
Joints:
- joint LAnklePitch: limit lower=-1 upper=1 effort=30 velocity=10 -> lower=-1.14 upper=1.128 effort=30 velocity=10
- joint LElbow: limit lower=-1.57 upper=0.9 effort=24 velocity=37 -> lower=-0.25 upper=2.35 effort=24 velocity=37; origin xyz=0.01 0 -0.173 rpy=0 -1.57 0 -> xyz=0.01 0 -0.173 rpy=0 -0.25 0
- joint LHipPitch: limit lower=-0.5236 upper=2.13 effort=45 velocity=9.163 -> lower=-0.45 upper=2.076 effort=72 velocity=9.163
- joint LHipRoll: limit lower=-0.2618 upper=0.524 effort=45 velocity=10.471975511965978 -> lower=-0.35 upper=0.524 effort=50 velocity=10.471975511965978
- joint LHipYaw: limit lower=-0.55 upper=0.55 effort=30 velocity=10.472 -> lower=-0.55 upper=0.55 effort=50 velocity=10.472
- joint LKnee: limit lower=-2.3 upper=0 effort=60 velocity=7.3304 -> lower=-2.216 upper=0.016 effort=60 velocity=7.3304
- joint LShoulderPitch: limit lower=-1.57 upper=3.14 effort=24 velocity=37 -> lower=-2.66 upper=2.88 effort=24 velocity=37; origin xyz=-0.01 0.14477 0.31534 rpy=0.17453 0 0 -> xyz=-0.01 0.14477 0.31534 rpy=0.17453 0.12 0
- joint LShoulderRoll: limit lower=0 upper=3.141 effort=24 velocity=37 -> lower=-0.15 upper=3.54 effort=24 velocity=37
- joint LShoulderYaw: limit lower=-2.1 upper=2.1 effort=24 velocity=37 -> lower=-2.1 upper=2.25 effort=24 velocity=37
- joint RAnklePitch: limit lower=-1 upper=1 effort=30 velocity=10 -> lower=-1.14 upper=1.128 effort=30 velocity=10
- joint RElbow: limit lower=-1.57 upper=0.9 effort=24 velocity=37 -> lower=-0.25 upper=2.35 effort=24 velocity=37; origin xyz=0.010039 0 -0.173 rpy=0 -1.57 0 -> xyz=0.010039 0 -0.173 rpy=0 -0.25 0
- joint RHipPitch: limit lower=-0.5236 upper=2.13 effort=45 velocity=9.163 -> lower=-0.45 upper=2.076 effort=72 velocity=9.163
- joint RHipRoll: limit lower=-0.2618 upper=0.524 effort=45 velocity=10.472 -> lower=-0.35 upper=0.524 effort=50 velocity=10.472
- joint RHipYaw: limit lower=-0.55 upper=0.55 effort=30 velocity=10.472 -> lower=-0.55 upper=0.55 effort=50 velocity=10.472
- joint RKnee: limit lower=-2.3 upper=0 effort=60 velocity=7.3304 -> lower=-2.216 upper=0.016 effort=60 velocity=7.3304
- joint RShoulderPitch: limit lower=-1.57 upper=3.14 effort=24 velocity=37 -> lower=-2.66 upper=2.88 effort=24 velocity=37; origin xyz=-0.01 -0.14477 0.31534 rpy=-0.17453 0 0 -> xyz=-0.01 -0.14477 0.31534 rpy=-0.17453 0.12 0
- joint RShoulderRoll: limit lower=0 upper=3.141 effort=24 velocity=37 -> lower=-0.15 upper=3.54 effort=24 velocity=37
- joint RShoulderYaw: limit lower=-2.1 upper=2.1 effort=24 velocity=37 -> lower=-2.1 upper=2.25 effort=24 velocity=37
- joint torso: type revolute -> fixed
