Commit message: piplus updated urdf

File: src/bitbots_robot/piplus_description/urdf/pi_plus_22dof.urdf.xacro (robot description, xacro)
@@ -1,1290 +1,821 @@
-<?xml version="1.0" encoding="utf-8"?>
- <robot name="pi_plus_24dof">
-   <link name="base_link">
-     <inertial>
-       <origin xyz="0.0005802 0.0000447 0.0564524" rpy="0 0 0" />
-       <mass value="2.7616497"/>
-       <inertia ixx="0.0216372" ixy="0.0000104" ixz="0.0000694" iyy="0.0185642" iyz="-0.0000113" izz="0.0075903" />
-     </inertial>
-     <visual>
-       <origin xyz="0 0 0" rpy="0 0 0" />
-       <geometry>
-         <mesh filename="package://piplus_description/urdf/meshes/base_link.STL" />
-       </geometry>
-       <material name="">
-         <color rgba="0.75294 0.75294 0.75294 1" />
-       </material>
-     </visual>
-     <collision>
-       <origin xyz="0 0.0 0.07" rpy="0 0 0" />
-       <geometry>
-         <box size="0.154 0.09 0.14"/> <!-- 单位：米，格式为"长 宽 高" -->
-       </geometry>
-     </collision>
-     <collision>
-       <origin xyz="0 0.0 0.16" rpy="0 0 0" />
-       <geometry>
-         <!--mesh filename="package://piplus_description/urdf/meshes/base_link.STL" />-->
-         <box size="0.035 0.035 0.074"/> <!-- 单位：米，格式为"长 宽 高" -->
-       </geometry>
-     </collision>
-     <collision>
-       <origin xyz="-0.007 0.0 0.142" rpy="0 0 0" />
-       <geometry>
-         <box size="0.176 0.092 0.006"/> <!-- 单位：米，格式为"长 宽 高" -->
-       </geometry>
-     </collision>
-     <collision>
-       <origin xyz="0.000 0.0 0.003" rpy="0 0 0" />
-       <geometry>
-         <box size="0.162 0.092 0.006"/> <!-- 单位：米，格式为"长 宽 高" -->
-       </geometry>
-     </collision>
-     <collision>
-       <origin xyz="0 -0.075 0.118" rpy="0 0 0" />
-       <geometry>
-         <box size="0.045 0.055 0.045"/> <!-- 单位：米，格式为"长 宽 高" -->
-       </geometry>
-     </collision>
-     <collision>
-       <origin xyz="0 0.075 0.118" rpy="0 0 0" />
-       <geometry>
-         <box size="0.045 0.055 0.045"/> <!-- 单位：米，格式为"长 宽 高" -->
-       </geometry>
-     </collision>
-     <collision>
-       <origin xyz="0 0.0 -0.035" rpy="0 0 0" />
-       <geometry>
-         <box size="0.06 0.09 0.07"/> <!-- 单位：米，格式为"长 宽 高" -->
-       </geometry>
-     </collision>
-   </link>
-   <link name="l_hip_pitch_link">
-     <inertial>
-       <origin xyz="0.0013686 0.0306252 0.0005611" rpy="0 0 0" />
-       <mass value="0.3985763" />
-       <inertia ixx=" 0.0001039" ixy=" -0.0000021" ixz="0.0000001" iyy=" 0.0000971" iyz=" -0.0000008" izz="0.0001242" />
-     </inertial>
-     <visual>
-       <origin xyz="0 0 0" rpy="0 0 0" />
-       <geometry>
-         <mesh filename="package://piplus_description/urdf/meshes/l_hip_pitch_link.STL" />
-       </geometry>
-       <material name="">
-         <color rgba="0.752941176470588 0.752941176470588 0.752941176470588 1" />
-       </material>
-     </visual>
-     <collision>
-       <origin xyz="0 0.0 0" rpy="0 0 0" />
-       <geometry>
-         <mesh filename="package://piplus_description/urdf/meshes/l_hip_pitch_link.STL" />
-         <!--box size="0.06 0.04 0.05"/>--> <!-- 单位：米，格式为"长 宽 高" -->
-       </geometry>
-     </collision>
-   </link>
-   <joint name="l_hip_pitch_joint" type="revolute">
-     <origin xyz="0 0.0475 -0.04379" rpy="0 0 0" />
-     <parent link="base_link" />
-     <child link="l_hip_pitch_link" />
-     <axis xyz="0 1 0" />
-     <limit lower="-1.45" upper="1.45" effort="20" velocity="5.45" />
-     <dynamics damping="0.08" friction="0.0"/> <!-- 即使很小的阻尼也能极大改善稳定性 -->
-   </joint>
-   <link name="l_hip_roll_link">
-     <inertial>
-       <origin xyz="0.0009844 0.0001364 -0.0612495" rpy="0 0 0" />
-       <mass value="0.4857183" />
-       <inertia ixx="0.0004833" ixy="-0.0000004" ixz="-0.0000210" iyy="0.0005742" iyz="0.0000008" izz="0.0002219" />
-     </inertial>
-     <visual>
-       <origin xyz="0 0 0" rpy="0 0 0" />
-       <geometry>
-         <mesh filename="package://piplus_description/urdf/meshes/l_hip_roll_link.STL" />
-       </geometry>
-       <material name="">
-         <color rgba="0.752941176470588 0.752941176470588 0.752941176470588 1" />
-       </material>
-     </visual>
-     <collision>
-       <origin xyz="0 0 0" rpy="0 0 0" />
-       <geometry>
-         <mesh filename="package://piplus_description/urdf/meshes/l_hip_roll_link.STL" />
-       </geometry>
-     </collision>
-   </link>
-   <joint name="l_hip_roll_joint" type="revolute">
-     <origin xyz="0 0.034 0.00028984" rpy="0 0 0" />
-     <parent link="l_hip_pitch_link" />
-     <child link="l_hip_roll_link" />
-     <axis xyz="1 0 0" />
-     <limit lower="-0.31" upper="1.2" effort="20" velocity="5.45" />
-     <dynamics damping="0.08" friction="0.0"/> <!-- 即使很小的阻尼也能极大改善稳定性 -->
-   </joint>
-   <link name="l_thigh_link">
-     <inertial>
-       <origin xyz="0.0000000 -0.0009550 -0.0239847" rpy="0 0 0" />
-       <mass value="0.1093797" />
-       <inertia ixx=" 0.0001198" ixy=" 0.0000000" ixz=" 0.0000000" iyy=" 0.0000574" iyz="-0.0000043" izz="0.0000901" />
-     </inertial>
-     <visual>
-       <origin xyz="0 0 0" rpy="0 0 0" />
-       <geometry>
-         <mesh filename="package://piplus_description/urdf/meshes/l_thigh_link.STL" />
-       </geometry>
-       <material name="">
-         <color rgba="0.752941176470588 0.752941176470588 0.752941176470588 1" />
-       </material>
-     </visual>
-     <collision>
-       <origin xyz="0 0 0" rpy="0 0 0" />
-       <geometry>
-         <mesh filename="package://piplus_description/urdf/meshes/l_thigh_link.STL" />
-       </geometry>
-     </collision>
-   </link>
-   <joint name="l_thigh_joint" type="revolute">
-     <origin xyz="-0.00025 0 -0.0974" rpy="0 0 0" />
-     <parent link="l_hip_roll_link" />
-     <child link="l_thigh_link" />
-     <axis xyz="0 0 1" />
-     <limit lower="-1.2" upper="0.6" effort="20" velocity="5.45" />
-     <dynamics damping="0.08" friction="0.0"/> <!-- 即使很小的阻尼也能极大改善稳定性 -->
-   </joint>
-   <link name="l_calf_link">
-     <inertial>
-       <origin xyz="-0.0000136 0.0027624 -0.0700557" rpy="0 0 0" />
-       <mass value="0.8028699" />
-       <inertia ixx=" 0.0037268" ixy="0.0000000" ixz="-0.0000149" iyy="0.0037147" iyz="-0.0000011" izz="0.0001840" />
-     </inertial>
-     <visual>
-       <origin xyz="0 0 0" rpy="0 0 0" />
-       <geometry>
-         <mesh filename="package://piplus_description/urdf/meshes/l_calf_link.STL" />
-       </geometry>
-       <material name="">
-         <color rgba="0.752941176470588 0.752941176470588 0.752941176470588 1" />
-       </material>
-     </visual>
-     <!-- <collision>
-       <origin xyz="0 0 0" rpy="0 0 0" />
-       <geometry>
-         <mesh filename="package://piplus_description/urdf/meshes/l_calf_link_1.STL" />
-       </geometry>
-     </collision> -->
-     <collision>
-       <origin xyz="0 0 0" rpy="0 0 0" />
-       <geometry>
-         <mesh filename="package://piplus_description/urdf/meshes/l_calf_link_2.STL" />
-       </geometry>
-     </collision>
-     <!-- <collision>
-       <origin xyz="0 0 0" rpy="0 0 0" />
-       <geometry>
-         <mesh filename="package://piplus_description/urdf/meshes/l_calf_link_3.STL" />
-       </geometry>
-     </collision> -->
-     <!-- <collision>
-       <origin xyz="0 0 0" rpy="0 0 0" />
-       <geometry>
-         <mesh filename="package://piplus_description/urdf/meshes/l_calf_link_4.STL" />
-       </geometry>
-     </collision> -->
-     <collision>
-       <origin xyz="0 0 0" rpy="0 0 0" />
-       <geometry>
-         <mesh filename="package://piplus_description/urdf/meshes/l_calf_link_5.STL" />
-       </geometry>
-     </collision>
-     <collision>
-       <origin xyz="0 0 0" rpy="0 0 0" />
-       <geometry>
-         <mesh filename="package://piplus_description/urdf/meshes/l_calf_link_6.STL" />
-       </geometry>
-     </collision>
-     <!-- <collision>
-       <origin xyz="0 0 0" rpy="0 0 0" />
-       <geometry>
-         <mesh filename="package://piplus_description/urdf/meshes/l_calf_link_7.STL" />
-       </geometry>
-     </collision> -->
-     <!--collision>
-       <origin xyz="0 0 -0.0030" rpy="0 0 0" />
-       <geometry>
-         <box size="0.05 0.05 0.056"/>
-       </geometry>
-     </collision>-->
-     <collision>
-       <origin xyz="0 0 -0.055" rpy="0 0 0" />
-       <geometry>
-         <box size="0.01 0.02 0.055"/>
-       </geometry>
-     </collision>
-     <!--collision>
-       <origin xyz="0 0 -0.138" rpy="0 0 0" />
-       <geometry>
-         <box size="0.046 0.046 0.045"/>
-       </geometry>
-     </collision>-->
-   </link>
-   <joint name="l_calf_joint" type="revolute">
-     <origin xyz="0 0 -0.0453" rpy="0 0 0" />
-     <parent link="l_thigh_link" />
-     <child link="l_calf_link" />
-     <axis xyz="0 1 0" />
-     <limit lower="-0.05" upper="2.4" effort="20" velocity="5.45" />
-     <dynamics damping="0.08" friction="0.0"/> <!-- 即使很小的阻尼也能极大改善稳定性 -->
-   </joint>
-   <link name="l_ankle_pitch_link">
-     <inertial>
-       <origin xyz="0.0065537 -0.0021861 0.0000145" rpy="0 0 0" />
-       <mass value="0.1655827" />
-       <inertia ixx="0.0001202" ixy="-0.0000024" ixz="-0.0000001" iyy=" 0.0001846" iyz="0.0000000" izz="0.0002720" />
-     </inertial>
-     <visual>
-       <origin xyz="0 0 0" rpy="0 0 0" />
-       <geometry>
-         <mesh filename="package://piplus_description/urdf/meshes/l_ankle_pitch_link.STL" />
-       </geometry>
-       <material name="">
-         <color rgba="0.752941176470588 0.752941176470588 0.752941176470588 1" />
-       </material>
-     </visual>
-     <collision>
-       <origin xyz="0 0.03 0" rpy="0 0 0" />
-       <geometry>
-         <!--mesh filename="package://piplus_description/urdf/meshes/l_ankle_pitch_link.STL" /> -->
-         <box size="0.08 0.006 0.03"/> <!-- 单位：米，格式为"长 宽 高" -->
-       </geometry>
-     </collision>
-     <collision>
-       <origin xyz="0 -0.03 0" rpy="0 0 0" />
-       <geometry>
-         <box size="0.08 0.006 0.03"/> <!-- 单位：米，格式为"长 宽 高" -->
-       </geometry>
-     </collision>
-     <collision>
-       <origin xyz="-0.042 0.0 0" rpy="0 0 0" />
-       <geometry>
-         <box size="0.006 0.06 0.03"/> <!-- 单位：米，格式为"长 宽 高" -->
-       </geometry>
-     </collision>
-     <collision>
-       <origin xyz="0.042 0.0 0" rpy="0 0 0" />
-       <geometry>
-         <box size="0.006 0.06 0.03"/> <!-- 单位：米，格式为"长 宽 高" -->
-       </geometry>
-     </collision>
-   </link>
-   <joint name="l_ankle_pitch_joint" type="revolute">
-     <origin xyz="0 0 -0.14" rpy="0 0 0" />
-     <parent link="l_calf_link" />
-     <child link="l_ankle_pitch_link" />
-     <axis xyz="0 1 0" />
-     <limit lower="-0.5" upper="0.92" effort="20" velocity="5.45" />
-     <dynamics damping="0.08" friction="0.0"/> <!-- 即使很小的阻尼也能极大改善稳定性 -->
-   </joint>
-   <link name="l_ankle_roll_link">
-     <inertial>
-       <origin xyz="0.0026578 0.0001757 -0.0126664" rpy="0 0 0" />
-       <mass value="0.6223485" />
-       <inertia ixx="0.0004400" ixy="-0.0000023" ixz="-0.0002309" iyy="0.0014685" iyz="-0.0000008" izz="0.0012907" />
-     </inertial>
-     <visual>
-       <origin xyz="0 0 0" rpy="0 0 0" />
-       <geometry>
-         <mesh filename="package://piplus_description/urdf/meshes/l_ankle_roll_link.STL" />
-       </geometry>
-       <material name="">
-         <color rgba="0.752941176470588 0.752941176470588 0.752941176470588 1" />
-       </material>
-     </visual>
-     <!-- <collision>
-       <origin xyz="0 0 0" rpy="0 0 0" />
-       <geometry>
-         <mesh filename="package://piplus_description/urdf/meshes/l_ankle_roll_link_1.STL" />
-       </geometry>
-     </collision>
-     <collision>
-       <origin xyz="0 0 0" rpy="0 0 0" />
-       <geometry>
-         <mesh filename="package://piplus_description/urdf/meshes/l_ankle_roll_link_2.STL" />
-       </geometry>
-     </collision>
-     <collision>
-       <origin xyz="0 0 0" rpy="0 0 0" />
-       <geometry>
-         <mesh filename="package://piplus_description/urdf/meshes/l_ankle_roll_link_3.STL" />
-       </geometry>
-     </collision>
-     <collision>
-       <origin xyz="0 0 0" rpy="0 0 0" />
-       <geometry>
-         <mesh filename="package://piplus_description/urdf/meshes/l_ankle_roll_link_4.STL" />
-       </geometry>
-     </collision>
-     <collision>
-       <origin xyz="0 0 0" rpy="0 0 0" />
-       <geometry>
-         <mesh filename="package://piplus_description/urdf/meshes/l_ankle_roll_link_5.STL" />
-       </geometry>
-     </collision>
-     <collision>
-       <origin xyz="0 0 0" rpy="0 0 0" />
-       <geometry>
-         <mesh filename="package://piplus_description/urdf/meshes/l_ankle_roll_link_6.STL" />
-       </geometry>
-     </collision>
-     <collision>
-       <origin xyz="0 0 0" rpy="0 0 0" />
-       <geometry>
-         <mesh filename="package://piplus_description/urdf/meshes/l_ankle_roll_link_7.STL" />
-       </geometry>
-     </collision> -->
-     <collision>
-       <origin xyz="0 0 0" rpy="0 0 0" />
-       <geometry>
-         <mesh filename="package://piplus_description/urdf/meshes/ankle_roll_link_simplify.STL" />
-       </geometry>
-     </collision>
-     <!--collision>
-       <origin xyz="0.030 0 -0.01" rpy="0 0 0" />
-       <geometry>
-         <box size="0.05 0.06 0.06"/>
-       </geometry>
-     </collision>
-     <collision>
-       <origin xyz="-0.028 0 -0.04470" rpy="0 0 0" />
-       <geometry>
-         <box size="0.17 0.07 0.0105"/>
-       </geometry>
-     </collision>
-     <collision>
-       <origin xyz="-0.1 0 -0.013" rpy="0 0 0" />
-       <geometry>
-         <box size="0.006 0.03 0.056"/>
-       </geometry>
-     </collision>-->
-   </link>
-   <joint name="l_ankle_roll_joint" type="revolute">
-     <origin xyz="0.051 0 0" rpy="0 0 0" />
-     <parent link="l_ankle_pitch_link" />
-     <child link="l_ankle_roll_link" />
-     <axis xyz="1 0 0" />
-     <limit lower="-0.78" upper="0.78" effort="20" velocity="5.45" />
-     <dynamics damping="0.08" friction="0.0"/> <!-- 即使很小的阻尼也能极大改善稳定性 -->
-   </joint>
-   <link name="r_hip_pitch_link">
-     <inertial>
-       <origin xyz="0.0013698 -0.0311672 0.0005611" rpy="0 0 0" />
-       <mass value="0.3985763" />
-       <inertia ixx="0.0001052" ixy="0.0000018" ixz="0.0000001" iyy="0.0000971" iyz="-0.0000003" izz="0.0001256" />
-     </inertial>
-     <visual>
-       <origin xyz="0 0 0" rpy="0 0 0" />
-       <geometry>
-         <mesh filename="package://piplus_description/urdf/meshes/r_hip_pitch_link.STL" />
-       </geometry>
-       <material name="">
-         <color rgba="0.752941176470588 0.752941176470588 0.752941176470588 1" />
-       </material>
-     </visual>
-     <collision>
-       <origin xyz="0 0 0" rpy="0 0 0" />
-       <geometry>
-         <mesh filename="package://piplus_description/urdf/meshes/r_hip_pitch_link.STL" />
-         <!--box size="0.06 0.04 0.05"/>--> <!-- 单位：米，格式为"长 宽 高" -->
-       </geometry>
-     </collision>
-   </link>
-   <joint name="r_hip_pitch_joint" type="revolute">
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
Commit message: imu uncalibrated and camera optical uncalibrated frames

File: src/bitbots_robot/piplus_description/urdf/pi_plus_22dof.urdf.xacro (robot description, xacro)
@@ -54,9 +54,9 @@
     <dynamics damping="0.02" friction="0.0"/>
   </joint>
-  <link name="imu_frame"/>
+  <link name="imu_frame_uncalibrated"/>
   <joint name="imu_frame_joint" type="fixed">
     <origin xyz="0 0 0.1" rpy="0 0 0" />
     <parent link="torso_link" />
-    <child link="imu_frame" />
+    <child link="imu_frame_uncalibrated" />
   </joint>
   <link name="r_shoulder_pitch_link">
@@ -418,4 +418,16 @@
     <axis xyz="0 0 0" />
     <dynamics damping="0.02" friction="0.0"/>
+  </joint>
+  <link name="camera_optical_frame_uncalibrated" /> <!-- left camera -->
+  <joint name="camera_joint_uncalibrated" type="fixed">
+    <origin xyz="0.03 -0.039 0.0" rpy="-1.57 0 -1.57" />
+    <parent link="camera_link" />
+    <child link="camera_optical_frame_uncalibrated" />
+  </joint>
+  <link name="camera_optical_frame_right_uncalibrated" /> <!-- right camera -->
+  <joint name="camera_joint_right_uncalibrated" type="fixed">
+    <origin xyz="0.03 0.024 0.0" rpy="-1.57 0 -1.57" />
+    <parent link="camera_link" />
+    <child link="camera_optical_frame_right_uncalibrated" />
   </joint>
   <link name="r_hip_pitch_link">

Commit message: motor directions in urdf

File: src/bitbots_robot/piplus_description/urdf/pi_plus_22dof.urdf.xacro (robot description, xacro)
@@ -77,8 +77,8 @@
   </link>
   <joint name="r_shoulder_pitch_joint" type="revolute">
-    <origin xyz="0 -0.1084 0.117" rpy="0 0 0" />
+    <origin xyz="0 -0.1084 0.117" rpy="0 1.57079632679 0" />
     <parent link="torso_link" />
     <child link="r_shoulder_pitch_link" />
-    <axis xyz="0 1 0" />
+    <axis xyz="0 -1 0" />
     <limit lower="-4.18" upper="1.04" effort="10" velocity="15.91" />
     <dynamics damping="0.02" friction="0.0"/>
@@ -101,5 +101,5 @@
   </link>
   <joint name="r_shoulder_roll_joint" type="revolute">
-    <origin xyz="0 -0.038 0" rpy="0 0 0" />
+    <origin xyz="0 -0.038 0" rpy="-1.57079632679 0 0" />
     <parent link="r_shoulder_pitch_link" />
     <child link="r_shoulder_roll_link" />
@@ -134,5 +134,5 @@
     <parent link="r_shoulder_roll_link" />
     <child link="r_upper_arm_link" />
-    <axis xyz="0 0 1" />
+    <axis xyz="0 0 -1" />
     <limit lower="-2.16" upper="2.16" effort="10" velocity="15.91" />
     <dynamics damping="0.02" friction="0.0"/>
@@ -158,5 +158,5 @@
     <parent link="r_upper_arm_link" />
     <child link="r_elbow_link" />
-    <axis xyz="0 1 0" />
+    <axis xyz="0 -1 0" />
     <limit lower="-2" upper="2" effort="10" velocity="15.91" />
     <dynamics damping="0.02" friction="0.0"/>
@@ -215,5 +215,5 @@
   </link>
   <joint name="l_shoulder_pitch_joint" type="revolute">
-    <origin xyz="0 0.1084 0.11698" rpy="0 0 0" />
+    <origin xyz="0 0.1084 0.11698" rpy="0 1.57079632679 0" />
     <parent link="torso_link" />
     <child link="l_shoulder_pitch_link" />
@@ -239,5 +239,5 @@
   </link>
   <joint name="l_shoulder_roll_joint" type="revolute">
-    <origin xyz="0 0.038 0" rpy="0 0 0" />
+    <origin xyz="0 0.038 0" rpy="1.57079632679 0 0" />
     <parent link="l_shoulder_pitch_link" />
     <child link="l_shoulder_roll_link" />
@@ -272,5 +272,5 @@
     <parent link="l_shoulder_roll_link" />
     <child link="l_upper_arm_link" />
-    <axis xyz="0 0 1" />
+    <axis xyz="0 0 -1" />
     <limit lower="-2.16" upper="2.16" effort="10" velocity="15.91" />
     <dynamics damping="0.02" friction="0.0"/>
@@ -451,5 +451,5 @@
     <parent link="base_link" />
     <child link="r_hip_pitch_link" />
-    <axis xyz="0 1 0" />
+    <axis xyz="0 -1 0" />
     <limit lower="-1.76" upper="1.76" effort="20" velocity="5.45" />
     <dynamics damping="0.02" friction="0.0"/>
@@ -505,5 +505,5 @@
     <parent link="r_hip_roll_link" />
     <child link="r_thigh_link" />
-    <axis xyz="0 0 1" />
+    <axis xyz="0 0 -1" />
     <limit lower="-2.87" upper="2.87" effort="20" velocity="5.45" />
     <dynamics damping="0.02" friction="0.0"/>
@@ -572,5 +572,5 @@
     <parent link="r_calf_link" />
     <child link="r_ankle_pitch_link" />
-    <axis xyz="0 1 0" />
+    <axis xyz="0 -1 0" />
     <limit lower="-0.97" upper="0.92" effort="20" velocity="5.45" />
     <dynamics damping="0.02" friction="0.0"/>
@@ -705,5 +705,5 @@
     <parent link="l_hip_roll_link" />
     <child link="l_thigh_link" />
-    <axis xyz="0 0 1" />
+    <axis xyz="0 0 -1" />
     <limit lower="-2.87" upper="2.87" effort="20" velocity="5.45" />
     <dynamics damping="0.02" friction="0.0"/> <!-- 即使很小的阻尼也能极大改善稳定性 -->
@@ -742,5 +742,5 @@
     <parent link="l_thigh_link" />
     <child link="l_calf_link" />
-    <axis xyz="0 1 0" />
+    <axis xyz="0 -1 0" />
     <limit lower="-2.14" upper="2.35" effort="20" velocity="5.45" />
     <dynamics damping="0.02" friction="0.0"/>

Commit message: Add sole frames
Signed-off-by: Florian Vahl <florian@flova.de>

File: src/bitbots_robot/piplus_description/urdf/pi_plus_22dof.urdf.xacro (robot description, xacro)
@@ -631,4 +631,10 @@
     <dynamics damping="0.02" friction="0.0"/>
   </joint>
+    <joint name="r_sole_joint" type="fixed">
+    <origin xyz="-0.051 0 -0.05" rpy="0 0 0" />
+    <parent link="r_ankle_roll_link" />
+    <child link="r_sole" />
+  </joint>
+  <link name="r_sole"></link>
   <link name="l_hip_pitch_link">
     <inertial>
@@ -831,3 +837,9 @@
     <dynamics damping="0.02" friction="0.0"/>
   </joint>
+  <joint name="l_sole_joint" type="fixed">
+    <origin xyz="-0.051 0 -0.05" rpy="0 0 0" />
+    <parent link="l_ankle_roll_link" />
+    <child link="l_sole" />
+  </joint>
+  <link name="l_sole"></link>
 </robot>
