Commit message: joint limits in urdf

File: src/bitbots_robot/piplus_description/urdf/pi_plus_22dof.urdf.xacro (robot description, xacro)
@@ -81,5 +81,5 @@
     <child link="r_shoulder_pitch_link" />
     <axis xyz="0 -1 0" />
-    <limit lower="-4.18" upper="1.04" effort="10" velocity="15.91" />
+    <limit lower="-2.6" upper="2.6" effort="10" velocity="15.91" />
     <dynamics damping="0.02" friction="0.0"/>
   </joint>
@@ -105,5 +105,5 @@
     <child link="r_shoulder_roll_link" />
     <axis xyz="1 0 0" />
-    <limit lower="-3.34" upper="0.13" effort="10" velocity="15.91" />
+    <limit lower="-1.65" upper="1.46" effort="10" velocity="15.91" />
     <dynamics damping="0.02" friction="0.0"/>
   </joint>
@@ -135,5 +135,5 @@
     <child link="r_upper_arm_link" />
     <axis xyz="0 0 -1" />
-    <limit lower="-2.16" upper="2.16" effort="10" velocity="15.91" />
+    <limit lower="-2.6" upper="2.6" effort="10" velocity="15.91" />
     <dynamics damping="0.02" friction="0.0"/>
   </joint>
@@ -159,5 +159,5 @@
     <child link="r_elbow_link" />
     <axis xyz="0 -1 0" />
-    <limit lower="-2" upper="2" effort="10" velocity="15.91" />
+    <limit lower="-1.86" upper="2.1" effort="10" velocity="15.91" />
     <dynamics damping="0.02" friction="0.0"/>
   </joint>
@@ -219,5 +219,5 @@
     <child link="l_shoulder_pitch_link" />
     <axis xyz="0 1 0" />
-    <limit lower="-4.18" upper="1.04" effort="10" velocity="15.91" />
+    <limit lower="-2.6" upper="2.6" effort="10" velocity="15.91" />
     <dynamics damping="0.02" friction="0.0"/>
   </joint>
@@ -243,5 +243,5 @@
     <child link="l_shoulder_roll_link" />
     <axis xyz="1 0 0" />
-    <limit lower="-0.13" upper="3.34" effort="10" velocity="15.91" />
+    <limit lower="-1.46" upper="1.65" effort="10" velocity="15.91" />
     <dynamics damping="0.02" friction="0.0"/>
   </joint>
@@ -273,5 +273,5 @@
     <child link="l_upper_arm_link" />
     <axis xyz="0 0 -1" />
-    <limit lower="-2.16" upper="2.16" effort="10" velocity="15.91" />
+    <limit lower="-2.6" upper="2.6" effort="10" velocity="15.91" />
     <dynamics damping="0.02" friction="0.0"/>
   </joint>
@@ -297,5 +297,5 @@
     <child link="l_elbow_link" />
     <axis xyz="0 1 0" />
-    <limit lower="-2" upper="2" effort="10" velocity="15.91" />
+    <limit lower="-2.1" upper="1.86" effort="10" velocity="15.91" />
     <dynamics damping="0.02" friction="0.0"/>
   </joint>
@@ -452,5 +452,5 @@
     <child link="r_hip_pitch_link" />
     <axis xyz="0 -1 0" />
-    <limit lower="-1.76" upper="1.76" effort="20" velocity="5.45" />
+    <limit lower="-2.89" upper="2.89" effort="20" velocity="5.45" />
     <dynamics damping="0.02" friction="0.0"/>
   </joint>
@@ -476,5 +476,5 @@
     <child link="r_hip_roll_link" />
     <axis xyz="1 0 0" />
-    <limit lower="-2.46" upper="0.17" effort="20" velocity="5.45" />
+    <limit lower="-3.14" upper="0.2" effort="20" velocity="5.45" />
     <dynamics damping="0.02" friction="0.0"/>
   </joint>
@@ -506,5 +506,5 @@
     <child link="r_thigh_link" />
     <axis xyz="0 0 -1" />
-    <limit lower="-2.87" upper="2.87" effort="20" velocity="5.45" />
+    <limit lower="-2.82" upper="2.49" effort="20" velocity="5.45" />
     <dynamics damping="0.02" friction="0.0"/>
   </joint>
@@ -543,5 +543,5 @@
     <child link="r_calf_link" />
     <axis xyz="0 1 0" />
-    <limit lower="-2.14" upper="2.35" effort="20" velocity="5.45" />
+    <limit lower="-2.14" upper="2.26" effort="20" velocity="5.45" />
     <dynamics damping="0.02" friction="0.0"/>
   </joint>
@@ -573,5 +573,5 @@
     <child link="r_ankle_pitch_link" />
     <axis xyz="0 -1 0" />
-    <limit lower="-0.97" upper="0.92" effort="20" velocity="5.45" />
+    <limit lower="-1" upper="0.87" effort="20" velocity="5.45" />
     <dynamics damping="0.02" friction="0.0"/>
   </joint>
@@ -658,5 +658,5 @@
     <child link="l_hip_pitch_link" />
     <axis xyz="0 1 0" />
-    <limit lower="-1.76" upper="1.76" effort="20" velocity="5.45" />
+    <limit lower="-2.89" upper="2.89" effort="20" velocity="5.45" />
     <dynamics damping="0.02" friction="0.0"/>
   </joint>
@@ -682,5 +682,5 @@
     <child link="l_hip_roll_link" />
     <axis xyz="1 0 0" />
-    <limit lower="-0.17" upper="2.46" effort="20" velocity="5.45" />
+    <limit lower="-0.2" upper="3.14" effort="20" velocity="5.45" />
     <dynamics damping="0.02" friction="0.0"/>
   </joint>
@@ -712,5 +712,5 @@
     <child link="l_thigh_link" />
     <axis xyz="0 0 -1" />
-    <limit lower="-2.87" upper="2.87" effort="20" velocity="5.45" />
+    <limit lower="-2.82" upper="2.49" effort="20" velocity="5.45" />
     <dynamics damping="0.02" friction="0.0"/> <!-- 即使很小的阻尼也能极大改善稳定性 -->
   </joint>
@@ -749,5 +749,5 @@
     <child link="l_calf_link" />
     <axis xyz="0 -1 0" />
-    <limit lower="-2.14" upper="2.35" effort="20" velocity="5.45" />
+    <limit lower="-2.26" upper="2.14" effort="20" velocity="5.45" />
     <dynamics damping="0.02" friction="0.0"/>
   </joint>
@@ -779,5 +779,5 @@
     <child link="l_ankle_pitch_link" />
     <axis xyz="0 1 0" />
-    <limit lower="-0.97" upper="0.92" effort="20" velocity="5.45" />
+    <limit lower="-0.87" upper="1" effort="20" velocity="5.45" />
     <dynamics damping="0.02" friction="0.0"/>
   </joint>

Commit message: urdf file with updated values and safe joint limits

File: src/bitbots_robot/piplus_description/urdf/pi_plus_22dof.urdf.xacro (robot description, xacro)
@@ -81,5 +81,5 @@
     <child link="r_shoulder_pitch_link" />
     <axis xyz="0 -1 0" />
-    <limit lower="-2.6" upper="2.6" effort="10" velocity="15.91" />
+    <limit lower="-2.55" upper="2.55" effort="10" velocity="15.91" />
     <dynamics damping="0.02" friction="0.0"/>
   </joint>
@@ -105,5 +105,5 @@
     <child link="r_shoulder_roll_link" />
     <axis xyz="1 0 0" />
-    <limit lower="-1.65" upper="1.46" effort="10" velocity="15.91" />
+    <limit lower="-1.65" upper="1.4" effort="10" velocity="15.91" />
     <dynamics damping="0.02" friction="0.0"/>
   </joint>
@@ -135,5 +135,5 @@
     <child link="r_upper_arm_link" />
     <axis xyz="0 0 -1" />
-    <limit lower="-2.6" upper="2.6" effort="10" velocity="15.91" />
+    <limit lower="-2.55" upper="2.55" effort="10" velocity="15.91" />
     <dynamics damping="0.02" friction="0.0"/>
   </joint>
@@ -159,5 +159,5 @@
     <child link="r_elbow_link" />
     <axis xyz="0 -1 0" />
-    <limit lower="-1.86" upper="2.1" effort="10" velocity="15.91" />
+    <limit lower="-1.8" upper="2.04" effort="10" velocity="15.91" />
     <dynamics damping="0.02" friction="0.0"/>
   </joint>
@@ -219,5 +219,5 @@
     <child link="l_shoulder_pitch_link" />
     <axis xyz="0 1 0" />
-    <limit lower="-2.6" upper="2.6" effort="10" velocity="15.91" />
+    <limit lower="-2.55" upper="2.55" effort="10" velocity="15.91" />
     <dynamics damping="0.02" friction="0.0"/>
   </joint>
@@ -243,5 +243,5 @@
     <child link="l_shoulder_roll_link" />
     <axis xyz="1 0 0" />
-    <limit lower="-1.46" upper="1.65" effort="10" velocity="15.91" />
+    <limit lower="-1.4" upper="1.65" effort="10" velocity="15.91" />
     <dynamics damping="0.02" friction="0.0"/>
   </joint>
@@ -273,5 +273,5 @@
     <child link="l_upper_arm_link" />
     <axis xyz="0 0 -1" />
-    <limit lower="-2.6" upper="2.6" effort="10" velocity="15.91" />
+    <limit lower="-2.55" upper="2.55" effort="10" velocity="15.91" />
     <dynamics damping="0.02" friction="0.0"/>
   </joint>
@@ -297,5 +297,5 @@
     <child link="l_elbow_link" />
     <axis xyz="0 1 0" />
-    <limit lower="-2.1" upper="1.86" effort="10" velocity="15.91" />
+    <limit lower="-2.04" upper="1.8" effort="10" velocity="15.91" />
     <dynamics damping="0.02" friction="0.0"/>
   </joint>
@@ -452,5 +452,5 @@
     <child link="r_hip_pitch_link" />
     <axis xyz="0 -1 0" />
-    <limit lower="-2.89" upper="2.89" effort="20" velocity="5.45" />
+    <limit lower="-2.84" upper="2.84" effort="20" velocity="5.45" />
     <dynamics damping="0.02" friction="0.0"/>
   </joint>
@@ -476,5 +476,5 @@
     <child link="r_hip_roll_link" />
     <axis xyz="1 0 0" />
-    <limit lower="-3.14" upper="0.2" effort="20" velocity="5.45" />
+    <limit lower="-3.1" upper="0.15" effort="20" velocity="5.45" />
     <dynamics damping="0.02" friction="0.0"/>
   </joint>
@@ -506,5 +506,5 @@
     <child link="r_thigh_link" />
     <axis xyz="0 0 -1" />
-    <limit lower="-2.82" upper="2.49" effort="20" velocity="5.45" />
+    <limit lower="-2.77" upper="2.45" effort="20" velocity="5.45" />
     <dynamics damping="0.02" friction="0.0"/>
   </joint>
@@ -543,5 +543,5 @@
     <child link="r_calf_link" />
     <axis xyz="0 1 0" />
-    <limit lower="-2.14" upper="2.26" effort="20" velocity="5.45" />
+    <limit lower="-1.97" upper="2.21" effort="20" velocity="5.45" />
     <dynamics damping="0.02" friction="0.0"/>
   </joint>
@@ -573,5 +573,5 @@
     <child link="r_ankle_pitch_link" />
     <axis xyz="0 -1 0" />
-    <limit lower="-1" upper="0.87" effort="20" velocity="5.45" />
+    <limit lower="0.95" upper="0.85" effort="20" velocity="5.45" />
     <dynamics damping="0.02" friction="0.0"/>
   </joint>
@@ -628,5 +628,5 @@
     <child link="r_ankle_roll_link" />
     <axis xyz="1 0 0" />
-    <limit lower="-0.78" upper="0.78" effort="20" velocity="5.45" />
+    <limit lower="-0.72" upper="0.72" effort="20" velocity="5.45" />
     <dynamics damping="0.02" friction="0.0"/>
   </joint>
@@ -658,5 +658,5 @@
     <child link="l_hip_pitch_link" />
     <axis xyz="0 1 0" />
-    <limit lower="-2.89" upper="2.89" effort="20" velocity="5.45" />
+    <limit lower="-2.84" upper="2.84" effort="20" velocity="5.45" />
     <dynamics damping="0.02" friction="0.0"/>
   </joint>
@@ -682,5 +682,5 @@
     <child link="l_hip_roll_link" />
     <axis xyz="1 0 0" />
-    <limit lower="-0.2" upper="3.14" effort="20" velocity="5.45" />
+    <limit lower="-0.15" upper="3.1" effort="20" velocity="5.45" />
     <dynamics damping="0.02" friction="0.0"/>
   </joint>
@@ -712,5 +712,5 @@
     <child link="l_thigh_link" />
     <axis xyz="0 0 -1" />
-    <limit lower="-2.82" upper="2.49" effort="20" velocity="5.45" />
+    <limit lower="-2.77" upper="2.45" effort="20" velocity="5.45" />
     <dynamics damping="0.02" friction="0.0"/> <!-- 即使很小的阻尼也能极大改善稳定性 -->
   </joint>
@@ -749,5 +749,5 @@
     <child link="l_calf_link" />
     <axis xyz="0 -1 0" />
-    <limit lower="-2.26" upper="2.14" effort="20" velocity="5.45" />
+    <limit lower="-2.21" upper="1.97" effort="20" velocity="5.45" />
     <dynamics damping="0.02" friction="0.0"/>
   </joint>
@@ -779,5 +779,5 @@
     <child link="l_ankle_pitch_link" />
     <axis xyz="0 1 0" />
-    <limit lower="-0.87" upper="1" effort="20" velocity="5.45" />
+    <limit lower="-0.85" upper="0.95" effort="20" velocity="5.45" />
     <dynamics damping="0.02" friction="0.0"/>
   </joint>
@@ -834,5 +834,5 @@
     <child link="l_ankle_roll_link" />
     <axis xyz="1 0 0" />
-    <limit lower="-0.78" upper="0.78" effort="20" velocity="5.45" />
+    <limit lower="-0.72" upper="0.72" effort="20" velocity="5.45" />
     <dynamics damping="0.02" friction="0.0"/>
   </joint>

Commit message: Fix: Swap camera frames to specify left and right optical frames in URDF and launch files

File: src/bitbots_robot/piplus_description/urdf/pi_plus_22dof.urdf.xacro (robot description, xacro)
@@ -419,15 +419,15 @@
     <dynamics damping="0.02" friction="0.0"/>
   </joint>
-  <link name="camera_optical_frame_uncalibrated" /> <!-- left camera -->
-  <joint name="camera_joint_uncalibrated" type="fixed">
+  <link name="camera_optical_frame_right_uncalibrated" />
+  <joint name="camera_joint_right_uncalibrated" type="fixed">
     <origin xyz="0.03 -0.039 0.0" rpy="-1.57 0 -1.57" />
     <parent link="camera_link" />
-    <child link="camera_optical_frame_uncalibrated" />
-  </joint>
-  <link name="camera_optical_frame_right_uncalibrated" /> <!-- right camera -->
-  <joint name="camera_joint_right_uncalibrated" type="fixed">
+    <child link="camera_optical_frame_right_uncalibrated" />
+  </joint>
+  <link name="camera_optical_frame_left_uncalibrated" />
+  <joint name="camera_joint_left_uncalibrated" type="fixed">
     <origin xyz="0.03 0.024 0.0" rpy="-1.57 0 -1.57" />
     <parent link="camera_link" />
-    <child link="camera_optical_frame_right_uncalibrated" />
+    <child link="camera_optical_frame_left_uncalibrated" />
   </joint>
   <link name="r_hip_pitch_link">
