Commit message: rotate camera in urdf and mjcf

File: src/bitbots_robot/piplus_description/urdf/pi_plus_22dof.urdf.xacro (robot description, xacro)
@@ -421,5 +421,5 @@
   <link name="camera_optical_frame_right_uncalibrated" />
   <joint name="camera_joint_right_uncalibrated" type="fixed">
-    <origin xyz="0.03 -0.039 0.0" rpy="-1.57 0 -1.57" />
+    <origin xyz="0.03 -0.039 0.0" rpy="-2.093 -0.0 -1.57" />
     <parent link="camera_link" />
     <child link="camera_optical_frame_right_uncalibrated" />
@@ -427,5 +427,5 @@
   <link name="camera_optical_frame_left_uncalibrated" />
   <joint name="camera_joint_left_uncalibrated" type="fixed">
-    <origin xyz="0.03 0.024 0.0" rpy="-1.57 0 -1.57" />
+    <origin xyz="0.03 0.024 0.0" rpy="-2.093 -0.0 -1.57" />
     <parent link="camera_link" />
     <child link="camera_optical_frame_left_uncalibrated" />
